Commit message: Update moveit_config

File: moveit_config/aist_moveit_config/config/gazebo_aist_base_scene.urdf (robot description, URDF)
Before this commit: robot aist_base_scene, 202 links, 201 joints
Links:
- added link a_bot_usb_repeater_base_link
- added link a_bot_usb_repeater_body, mass 1.0; collision box size=0.033 0.055 0.014; visual box size=0.033 0.055 0.014
- added link a_bot_usb_repeater_front_leg, mass 1.0; collision cylinder length=0.01 radius=0.003; visual cylinder length=0.01 radius=0.003
- added link a_bot_usb_repeater_left_leg, mass 1.0; collision cylinder length=0.01 radius=0.003; visual cylinder length=0.01 radius=0.003
- added link a_bot_usb_repeater_plate, mass 1.0; collision cylinder length=0.004 radius=0.0375; visual cylinder length=0.004 radius=0.0375
- added link a_bot_usb_repeater_right_leg, mass 1.0; collision cylinder length=0.01 radius=0.003; visual cylinder length=0.01 radius=0.003
- added link b_bot_usb_repeater_base_link
- added link b_bot_usb_repeater_body, mass 1.0; collision box size=0.033 0.055 0.014; visual box size=0.033 0.055 0.014
- added link b_bot_usb_repeater_front_leg, mass 1.0; collision cylinder length=0.01 radius=0.003; visual cylinder length=0.01 radius=0.003
- added link b_bot_usb_repeater_left_leg, mass 1.0; collision cylinder length=0.01 radius=0.003; visual cylinder length=0.01 radius=0.003
- added link b_bot_usb_repeater_plate, mass 1.0; collision cylinder length=0.004 radius=0.0375; visual cylinder length=0.004 radius=0.0375
- added link b_bot_usb_repeater_right_leg, mass 1.0; collision cylinder length=0.01 radius=0.003; visual cylinder length=0.01 radius=0.003
Joints:
- added joint a_bot_usb_repeater_base_link: type fixed, parent a_bot_wrist_2_link, child a_bot_usb_repeater_base_link, origin xyz=0.000 -0.051 0.000 rpy=1.5707963267948966 -1.5707963267948966 0
- added joint a_bot_usb_repeater_body: type fixed, parent a_bot_usb_repeater_plate, child a_bot_usb_repeater_body, origin xyz=0 0 0.011 rpy=0 0 0
- added joint a_bot_usb_repeater_front_leg: type fixed, parent a_bot_usb_repeater_base_link, child a_bot_usb_repeater_front_leg, origin xyz=0.031 0 0 rpy=0 0 0
- added joint a_bot_usb_repeater_left_leg: type fixed, parent a_bot_usb_repeater_base_link, child a_bot_usb_repeater_left_leg, origin xyz=-0.0155 0.026846 0 rpy=0 0 0
- added joint a_bot_usb_repeater_plate: type fixed, parent a_bot_usb_repeater_base_link, child a_bot_usb_repeater_plate, origin xyz=0 0 0.01 rpy=0 0 0
- added joint a_bot_usb_repeater_right_leg: type fixed, parent a_bot_usb_repeater_base_link, child a_bot_usb_repeater_right_leg, origin xyz=-0.0155 -0.026846 0 rpy=0 0 0
- added joint b_bot_usb_repeater_base_link: type fixed, parent b_bot_wrist_2_link, child b_bot_usb_repeater_base_link, origin xyz=0.000 -0.051 0.000 rpy=1.5707963267948966 -1.5707963267948966 0
- added joint b_bot_usb_repeater_body: type fixed, parent b_bot_usb_repeater_plate, child b_bot_usb_repeater_body, origin xyz=0 0 0.011 rpy=0 0 0
- added joint b_bot_usb_repeater_front_leg: type fixed, parent b_bot_usb_repeater_base_link, child b_bot_usb_repeater_front_leg, origin xyz=0.031 0 0 rpy=0 0 0
- added joint b_bot_usb_repeater_left_leg: type fixed, parent b_bot_usb_repeater_base_link, child b_bot_usb_repeater_left_leg, origin xyz=-0.0155 0.026846 0 rpy=0 0 0
- added joint b_bot_usb_repeater_plate: type fixed, parent b_bot_usb_repeater_base_link, child b_bot_usb_repeater_plate, origin xyz=0 0 0.01 rpy=0 0 0
- added joint b_bot_usb_repeater_right_leg: type fixed, parent b_bot_usb_repeater_base_link, child b_bot_usb_repeater_right_leg, origin xyz=-0.0155 -0.026846 0 rpy=0 0 0
- joint a_bot_camera_joint: origin xyz=0.026      0.0      0.0595 rpy=0.0      0.3491      0.0 -> xyz=0.08046421018432694      -0.013512509598350497      0.09167488147585981 rpy=0.005347150648361527      0.38666681358877475      0.0005141030065124729
- joint a_motioncam_link_joint: origin xyz=0.5264331391465542 -0.10089186963870693 0.6628505002312947 rpy=0.08450640838509203 1.0689731022296014 -3.047472137518003 -> xyz=0.5276042818292748 -0.07468461065230031 0.6581105757417809 rpy=-0.03928732754619564 1.0628695458424167 3.104012489951837
- joint b_bot_camera_joint: origin xyz=0.026      0.0      0.0595 rpy=0.0      0.3491      0.0 -> xyz=0.03583950688939626      -0.01906877964474716      0.08153437390863827 rpy=0.025965299312343315      0.39909087634186097      0.03917642821862998
- joint virtual_screen_joint: origin xyz=0 0 0.81 rpy=0 0 0 -> xyz=0 0 0.8180000000000001 rpy=0 0 0
- joint workspace_live_camera_joint: origin xyz=0.43314679324975547 -0.10556504271980752 0.7460823474831381 rpy=-2.6534537924083277 0.05764023800141899 1.623811236576318 -> xyz=0.4370288783995411 -0.071661759880621 0.745049041752134 rpy=-2.664930711433391 -0.012207193910574477 1.602272823676792

Commit message: Retrieve workbench to kitting scene

File: moveit_config/aist_moveit_config/config/gazebo_aist_base_scene.urdf (robot description, URDF)
Before this commit: robot aist_base_scene, 214 links, 213 joints
Links:
- added link base_fixture_base_link, mass 0.86387; collision box size=0.049 0.058 0.026; visual mesh filename=package://aist_fastening_tools/meshes/visual/MGPM12-20Z_bod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 scale=0.001 0.001 0.001
- added link base_fixture_piston, mass 0.03804; collision box size=0.007 0.056 0.022; visual mesh filename=package://aist_fastening_tools/meshes/visual/MGPM12-20Z_pis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 scale=0.001 0.001 0.001
- added link base_fixture_piston_head
- added link base_fixture_tip_link
- added link screw_feeder_m3_base_link, mass 1.0; collision box size=0.126 0.126 0.147; visual box size=0.126 0.126 0.147
- added link screw_feeder_m3_front_side, mass 1.0; collision box size=0.056 0.126 0.079; visual box size=0.056 0.126 0.079
- added link screw_feeder_m3_gap, mass 1.0; collision box size=0.056 0.02 0.002; visual box size=0.056 0.02 0.002
- added link screw_feeder_m3_inlet_link
- added link screw_feeder_m3_outlet_link
- added link screw_feeder_m4_base_link, mass 1.0; collision box size=0.126 0.126 0.147; visual box size=0.126 0.126 0.147
- added link screw_feeder_m4_front_side, mass 1.0; collision box size=0.056 0.126 0.079; visual box size=0.056 0.126 0.079
- added link screw_feeder_m4_gap, mass 1.0; collision box size=0.056 0.02 0.002; visual box size=0.056 0.02 0.002
- added link screw_feeder_m4_inlet_link
- added link screw_feeder_m4_outlet_link
- added link workbench_back_bar, mass 1.0; collision box size=0.48 0.02 0.02; visual box size=0.48 0.02 0.02
- added link workbench_base_link, mass 1.0; collision box size=0.48 0.02 0.02; visual box size=0.48 0.02 0.02
- added link workbench_center_bar, mass 1.0; collision box size=0.02 0.28 0.02; visual box size=0.02 0.28 0.02
- added link workbench_front_border, mass 1.0; collision box size=0.08 0.016 0.003; visual box size=0.08 0.016 0.003
- added link workbench_holder_link
- added link workbench_right_bar, mass 1.0; collision box size=0.02 0.28 0.02; visual box size=0.02 0.28 0.02
- added link workbench_right_border, mass 1.0; collision box size=0.016 0.064 0.003; visual box size=0.016 0.064 0.003
- added link workbench_table_base_link, mass 1.0; collision box size=0.02 0.02 0.125; visual box size=0.02 0.02 0.125
- added link workbench_table_leg1, mass 1.0; collision box size=0.02 0.02 0.125; visual box size=0.02 0.02 0.125
- added link workbench_table_leg2, mass 1.0; collision box size=0.02 0.02 0.125; visual box size=0.02 0.02 0.125
- added link workbench_table_leg3, mass 1.0; collision box size=0.02 0.02 0.125; visual box size=0.02 0.02 0.125
- added link workbench_table_top, mass 1.0; collision box size=0.21 0.32 0.005; visual box size=0.21 0.32 0.005
- added link workbench_table_top_center
- added link workbench_table_top_origin
Joints:
- added joint base_fixture_base_joint: type fixed, parent workbench_table_top_origin, child base_fixture_base_link, origin xyz=0.05729961772434791 0.24786931916155724 0 rpy=0 0 -1.0304423903774522
- added joint base_fixture_piston_head_joint: type fixed, parent base_fixture_piston, child base_fixture_piston_head, origin xyz=0.013      0.0      0.013 rpy=0.0      0.0      0.0
- added joint base_fixture_piston_joint: type prismatic, parent base_fixture_base_link, child base_fixture_piston, axis 1 0 0, limit lower=0 upper=0.02 effort=130 velocity=0.15
- added joint base_fixture_tip_link_joint: type fixed, parent base_fixture_base_link, child base_fixture_tip_link, origin xyz=0.033      0.0      0.013 rpy=0.0      0.0      0.0
- added joint screw_feeder_m3_base_link: type fixed, parent workbench_base_link, child screw_feeder_m3_base_link, origin xyz=0.01 0.03 0 rpy=0 0 0
- added joint screw_feeder_m3_front_side: type fixed, parent screw_feeder_m3_base_link, child screw_feeder_m3_front_side, origin xyz=0.126 0 0 rpy=0 0 0
- added joint screw_feeder_m3_gap: type fixed, parent screw_feeder_m3_front_side, child screw_feeder_m3_gap, origin xyz=0 0.053 0.079 rpy=0 0 0
- added joint screw_feeder_m3_inlet_joint: type fixed, parent screw_feeder_m3_base_link, child screw_feeder_m3_inlet_link, origin xyz=0.072 0.032 0.147 rpy=0 0 0
- added joint screw_feeder_m3_outlet_joint: type fixed, parent screw_feeder_m3_gap, child screw_feeder_m3_outlet_link, origin xyz=0.046 0.01 0.002 rpy=0 0 0
- added joint screw_feeder_m4_base_link: type fixed, parent screw_feeder_m3_base_link, child screw_feeder_m4_base_link, origin xyz=0 0.126 0 rpy=0 0 0
- added joint screw_feeder_m4_front_side: type fixed, parent screw_feeder_m4_base_link, child screw_feeder_m4_front_side, origin xyz=0.126 0 0 rpy=0 0 0
- added joint screw_feeder_m4_gap: type fixed, parent screw_feeder_m4_front_side, child screw_feeder_m4_gap, origin xyz=0 0.053 0.079 rpy=0 0 0
- added joint screw_feeder_m4_inlet_joint: type fixed, parent screw_feeder_m4_base_link, child screw_feeder_m4_inlet_link, origin xyz=0.072 0.032 0.147 rpy=0 0 0
- added joint screw_feeder_m4_outlet_joint: type fixed, parent screw_feeder_m4_gap, child screw_feeder_m4_outlet_link, origin xyz=0.046 0.01 0.002 rpy=0 0 0
- added joint workbench_back_bar: type fixed, parent workbench_base_link, child workbench_back_bar, origin xyz=0 0.3 0 rpy=0 0 0
- added joint workbench_base_link: type fixed, parent cage_workspace_bar, child workbench_base_link, origin xyz=0.04    0.63    0.01 rpy=0 0 0
- added joint workbench_center_bar: type fixed, parent workbench_base_link, child workbench_center_bar, origin xyz=0.27 0.02 0 rpy=0 0 0
- added joint workbench_front_border: type fixed, parent workbench_table_top_origin, child workbench_front_border, origin xyz=0.13 0 0 rpy=0 0 0
- added joint workbench_holder_link_joint: type fixed, parent workbench_table_top_origin, child workbench_holder_link, origin xyz=0.194 0.016 0 rpy=0 0 1.5707963267948966
- added joint workbench_right_bar: type fixed, parent workbench_base_link, child workbench_right_bar, origin xyz=0.45999999999999996 0.02 0 rpy=0 0 0
- added joint workbench_right_border: type fixed, parent workbench_table_top_origin, child workbench_right_border, origin xyz=0.194 0.016 0 rpy=0 0 0
- added joint workbench_table_base_link: type fixed, parent workbench_base_link, child workbench_table_base_link, origin xyz=0.27 0  0.02 rpy=0 0 0
- added joint workbench_table_leg1: type fixed, parent workbench_table_base_link, child workbench_table_leg1, origin xyz=0.19 0 0 rpy=0 0 0
- added joint workbench_table_leg2: type fixed, parent workbench_table_base_link, child workbench_table_leg2, origin xyz=0 0.3 0 rpy=0 0 0
- added joint workbench_table_leg3: type fixed, parent workbench_table_base_link, child workbench_table_leg3, origin xyz=0.19      0.3      0 rpy=0 0 0
- added joint workbench_table_top: type fixed, parent workbench_table_base_link, child workbench_table_top, origin xyz=0 0 0.125 rpy=0 0 0
- added joint workbench_table_top_center_joint: type fixed, parent workbench_table_top_origin, child workbench_table_top_center, origin xyz=0.105 0.16 0 rpy=0 0 0
- added joint workbench_table_top_origin_joint: type fixed, parent workbench_table_top, child workbench_table_top_origin, origin xyz=0 0 0.005 rpy=0 0 0
- joint a_motioncam_link_joint: origin xyz=0.5276042818292748 -0.07468461065230031 0.6581105757417809 rpy=-0.03928732754619564 1.0628695458424167 3.104012489951837 -> xyz=0.5265706741269142 -0.07428942604572367 0.6593245247844437 rpy=-0.037302689521065885 1.0630553725803307 3.106909218955615
