Commit message: Improve screw feeder model

File: aist_description/objects/urdf/screw_feeder.urdf.xacro (robot description, xacro)
@@ -2,14 +2,17 @@
 <robot xmlns:xacro="http://www.ros.org/wiki/xacro" name="screw_feeder">
   <xacro:macro name="screw_feeder" params="prefix parent *origin">
-    <xacro:property name="length"	value=".126"/>
-    <xacro:property name="gap_width"	value=".020"/>
-    <xacro:property name="gap_depth"	value=".002"/>
-    <xacro:property name="gap_height"	value=".081"/>
+    <xacro:property name="length"		value=".126"/>
+    <xacro:property name="front_width"		value=".056"/>
+    <xacro:property name="front_height"		value=".081"/>
+    <xacro:property name="front_left_length"	value=".055"/>
+    <xacro:property name="front_right_length"	value=".040"/>
+    <xacro:property name="back_width"		value=".126"/>
+    <xacro:property name="back_height"		value=".147"/>
+    <xacro:property name="gap_width"	value="${length - front_left_length
+						- front_right_length}"/>
+    <xacro:property name="gap_height"	value=".072"/>
+    <xacro:property name="gap_depth"	value="${front_height - gap_height}"/>
     <xacro:property name="gap_x"	value=".046"/>
     <xacro:property name="gap_y"	value="${length/2}"/>
-    <xacro:property name="front_width"	value=".056"/>
-    <xacro:property name="front_height"	value="${gap_height - gap_depth}"/>
-    <xacro:property name="back_width"	value=".126"/>
-    <xacro:property name="back_height"	value=".147"/>
     <xacro:include filename="$(find aist_description
 			     )/objects/urdf/aist_box.urdf.xacro" />
@@ -21,22 +24,30 @@
       <xacro:insert_block name="origin"/>
     </xacro:aist_box>
-    <!-- Front side -->
-    <xacro:aist_box name="${prefix}front_side" parent="${prefix}base_link"
-		    width="${front_width}" length="${length}"
+    <!-- Front left side -->
+    <xacro:aist_box name="${prefix}front_left_side" parent="${prefix}base_link"
+		    width="${front_width}" length="${front_left_length}"
 		    height="${front_height}"
 		    rgba="0.2 0.2 0.2 1.0" color_name="black">
       <origin xyz="${back_width} 0 0" rpy="0 0 0"/>
     </xacro:aist_box>
+    <!-- Front right side -->
+    <xacro:aist_box name="${prefix}front_right_side" parent="${prefix}base_link"
+		    width="${front_width}" length="${front_right_length}"
+		    height="${front_height}"
+		    rgba="0.2 0.2 0.2 1.0" color_name="black">
+      <origin xyz="${back_width} ${front_left_length + gap_width} 0"
+	      rpy="0 0 0"/>
+    </xacro:aist_box>
     <!-- Gap -->
-    <xacro:aist_box name="${prefix}gap" parent="${prefix}front_side"
+    <xacro:aist_box name="${prefix}gap" parent="${prefix}front_left_side"
 		    width="${front_width}" length="${gap_width}"
-		    height="${gap_depth}"
+		    height="${gap_height}"
 		    rgba="0.6 0.6 0.6 1.0" color_name="grey">
-      <origin xyz="0 ${gap_y - gap_width/2} ${front_height}" rpy="0 0 0"/>
+      <origin xyz="0 ${front_left_length} 0" rpy="0 0 0"/>
     </xacro:aist_box>
     <joint name="${prefix}outlet_joint" type="fixed">
       <parent link="${prefix}gap"/>
       <child  link="${prefix}outlet_link"/>
-      <origin xyz="${gap_x} ${gap_width/2} ${gap_depth}"
+      <origin xyz="${gap_x} ${gap_y - front_left_length} ${gap_height}"
 	      rpy="0 0 0"/>
     </joint>

Commit message: Refine screw feeder model

File: aist_description/objects/urdf/screw_feeder.urdf.xacro (robot description, xacro)
@@ -11,6 +11,6 @@
     <xacro:property name="gap_width"	value="${length - front_left_length
 						- front_right_length}"/>
-    <xacro:property name="gap_height"	value=".072"/>
-    <xacro:property name="gap_depth"	value="${front_height - gap_height}"/>
+    <xacro:property name="gap_depth"	value=".012"/>
+    <xacro:property name="gap_height"	value="${front_height - gap_depth}"/>
     <xacro:property name="gap_x"	value=".046"/>
     <xacro:property name="gap_y"	value="${length/2}"/>

File: aist_description/scenes/urdf/assembly.urdf.xacro (robot description, xacro)
@@ -7,5 +7,5 @@
   <xacro:property name="workbench_bar_width"	 value="0.480"/>
   <xacro:property name="workbench_y"		 value="0.630"/>
-  <xacro:property name="screw_feeder_width"	 value="0.126"/>
+  <xacro:property name="screw_feeder_width"	 value="0.1268"/>
   <xacro:property name="screw_feeder_y"		 value="0.034"/>
   <xacro:property name="screw_feeder_x"		 value="0.014"/>

Commit message: Adjust model for picking screws

File: aist_description/objects/urdf/screw_feeder.urdf.xacro (robot description, xacro)
@@ -11,5 +11,5 @@
     <xacro:property name="gap_width"	value="${length - front_left_length
 						- front_right_length}"/>
-    <xacro:property name="gap_depth"	value=".012"/>
+    <xacro:property name="gap_depth"	value=".013"/>
     <xacro:property name="gap_height"	value="${front_height - gap_depth}"/>
     <xacro:property name="gap_x"	value=".046"/>
