Commit message: WIP: trying conveni picking

File: aist_description/objects/urdf/tray.urdf.xacro (robot description, xacro)
@@ -6,10 +6,10 @@
     <xacro:property name="tray_thickness"	value="0.005" />
     <xacro:property name="item_radius"		value="0.04" />
-    <link name="${prefix}tray"/>
-    <joint name="${prefix}tray_joint" type="floating">
-      <parent link="${parent}" />
-      <child  link="${prefix}tray" />
-      <xacro:insert_block name="origin"/>
-    </joint>
+    <!-- <link name="${prefix}tray"/> -->
+    <!-- <joint name="${prefix}tray_joint" type="floating"> -->
+    <!--   <parent link="${parent}" /> -->
+    <!--   <child  link="${prefix}tray" /> -->
+    <!--   <xacro:insert_block name="origin"/> -->
+    <!-- </joint> -->
     <xacro:aist_box name="${prefix}tray_bottom"
 		    width="${width}"
@@ -17,5 +17,5 @@
 		    height="${tray_thickness}"
 		    parent="${parent}">
-      <origin xyz="${-width/2} ${-tray_thickness/2} 0" rpy="0 0 0"/>
+      <xacro:insert_block name="origin"/>
     </xacro:aist_box>
     <xacro:aist_box name="${prefix}tray_wall0"
@@ -48,43 +48,49 @@
 	      rpy="0 0 0"/>
     </xacro:aist_box>
-    <link name="b_item_on_${prefix}tray"/>
-    <joint name="b_item_on_${prefix}tray_joint" type="fixed">
+    <link name="${prefix}tray_bottom_center"/>
+    <joint name="${prefix}tray_bottom_center_joint" type="fixed">
       <parent link ="${prefix}tray_bottom"/>
-      <child  link="b_item_on_${prefix}tray"/>
-      <origin xyz="${width/2}
-		   ${length/2}
-		   ${tray_thickness + item_radius}"
-    	      rpy="0 0 ${pi/2}"/>
+      <child  link="${prefix}tray_bottom_center"/>
+      <origin xyz="${width/2} ${length/2} ${tray_thickness}" rpy="0 0 0"/>
     </joint>
-    <link name="a_item_on_${prefix}tray"/>
-    <joint name="a_item_on_${prefix}tray_joint" type="fixed">
-      <parent link ="b_item_on_${prefix}tray"/>
-      <child  link="a_item_on_${prefix}tray"/>
-      <origin xyz="0 ${width/3 + tray_thickness/2} 0" rpy="0 0 0"/>
-    </joint>
-    <link name="c_item_on_${prefix}tray"/>
-    <joint name="c_item_on_${prefix}tray_joint" type="fixed">
-      <parent link ="b_item_on_${prefix}tray"/>
-      <child  link="c_item_on_${prefix}tray"/>
-      <origin xyz="0 ${-width/3 - tray_thickness/2} 0" rpy="0 0 0"/>
-    </joint>
-    <link name="d_item_on_${prefix}tray"/>
-    <joint name="d_item_on_${prefix}tray_joint" type="fixed">
-      <parent link ="a_item_on_${prefix}tray"/>
-      <child  link="d_item_on_${prefix}tray"/>
-      <origin xyz="0 0 0" rpy="0 0 0"/>
-    </joint>
-    <link name="e_item_on_${prefix}tray"/>
-    <joint name="e_item_on_${prefix}tray_joint" type="fixed">
-      <parent link ="b_item_on_${prefix}tray"/>
-      <child  link="e_item_on_${prefix}tray"/>
-      <origin xyz="0 0 0" rpy="0 0 0"/>
-    </joint>
-    <link name="f_item_on_${prefix}tray"/>
-    <joint name="f_item_on_${prefix}tray_joint" type="fixed">
-      <parent link ="c_item_on_${prefix}tray"/>
-      <child  link="f_item_on_${prefix}tray"/>
-      <origin xyz="0 0 0" rpy="0 0 0"/>
-    </joint>
+    <!-- <link name="b_item_on_${prefix}tray"/> -->
+    <!-- <joint name="b_item_on_${prefix}tray_joint" type="fixed"> -->
+    <!--   <parent link ="${prefix}tray_bottom"/> -->
+    <!--   <child  link="b_item_on_${prefix}tray"/> -->
+    <!--   <origin xyz="${width/2} -->
+    <!-- 		   ${length/2} -->
+    <!-- 		   ${tray_thickness + item_radius}" -->
+    <!-- 	      rpy="0 0 ${pi/2}"/> -->
+    <!-- </joint> -->
+    <!-- <link name="a_item_on_${prefix}tray"/> -->
+    <!-- <joint name="a_item_on_${prefix}tray_joint" type="fixed"> -->
+    <!--   <parent link ="b_item_on_${prefix}tray"/> -->
+    <!--   <child  link="a_item_on_${prefix}tray"/> -->
+    <!--   <origin xyz="0 ${width/3 + tray_thickness/2} 0" rpy="0 0 0"/> -->
+    <!-- </joint> -->
+    <!-- <link name="c_item_on_${prefix}tray"/> -->
+    <!-- <joint name="c_item_on_${prefix}tray_joint" type="fixed"> -->
+    <!--   <parent link ="b_item_on_${prefix}tray"/> -->
+    <!--   <child  link="c_item_on_${prefix}tray"/> -->
+    <!--   <origin xyz="0 ${-width/3 - tray_thickness/2} 0" rpy="0 0 0"/> -->
+    <!-- </joint> -->
+    <!-- <link name="d_item_on_${prefix}tray"/> -->
+    <!-- <joint name="d_item_on_${prefix}tray_joint" type="fixed"> -->
+    <!--   <parent link ="a_item_on_${prefix}tray"/> -->
+    <!--   <child  link="d_item_on_${prefix}tray"/> -->
+    <!--   <origin xyz="0 0 0" rpy="0 0 0"/> -->
+    <!-- </joint> -->
+    <!-- <link name="e_item_on_${prefix}tray"/> -->
+    <!-- <joint name="e_item_on_${prefix}tray_joint" type="fixed"> -->
+    <!--   <parent link ="b_item_on_${prefix}tray"/> -->
+    <!--   <child  link="e_item_on_${prefix}tray"/> -->
+    <!--   <origin xyz="0 0 0" rpy="0 0 0"/> -->
+    <!-- </joint> -->
+    <!-- <link name="f_item_on_${prefix}tray"/> -->
+    <!-- <joint name="f_item_on_${prefix}tray_joint" type="fixed"> -->
+    <!--   <parent link ="c_item_on_${prefix}tray"/> -->
+    <!--   <child  link="f_item_on_${prefix}tray"/> -->
+    <!--   <origin xyz="0 0 0" rpy="0 0 0"/> -->
+    <!-- </joint> -->
   </xacro:macro>
 </robot>

File: aist_description/scenes/urdf/g_bot_base_scene.urdf.xacro (robot description, xacro)
@@ -3,16 +3,21 @@
   <!-- This is the main file defining our robot arrangement and physical environment. -->
   <xacro:arg name="scene" default=""/>
-  <xacro:property name="g_bot_x"   value="0.050"/>
-  <xacro:property name="g_bot_y"   value="-0.900"/>
-  <xacro:property name="g_bot_z"   value="0.698"/>
-  <xacro:property name="cabinet_w" value="0.900"/>
-  <xacro:property name="cabinet_l" value="0.400"/>
-  <xacro:property name="cabinet_b" value="0.100"/>
-  <xacro:property name="shelf1_h"  value="0.600"/>
-  <xacro:property name="shelf2_h"  value="0.940"/>
-  <xacro:property name="back_h"    value="1.500"/>
-  <xacro:property name="wall_t"    value="0.012"/>
-  <xacro:property name="mounter_w" value="0.200"/>
-  <xacro:property name="mounter_l" value="0.200"/>
+  <xacro:property name="g_bot_x"	value="0.050"/>
+  <xacro:property name="g_bot_y"	value="-0.900"/>
+  <xacro:property name="g_bot_z"	value="0.698"/>
+  <xacro:property name="cabinet_w"	value="0.900"/>
+  <xacro:property name="cabinet_l"	value="0.400"/>
+  <xacro:property name="cabinet_b"	value="0.100"/>
+  <xacro:property name="shelf1_h"	value="0.600"/>
+  <xacro:property name="shelf2_h"	value="0.940"/>
+  <xacro:property name="back_h"		value="1.500"/>
+  <xacro:property name="wall_t"		value="0.012"/>
+  <xacro:property name="mounter_w"	value="0.200"/>
+  <xacro:property name="mounter_l"	value="0.200"/>
+  <xacro:property name="box_w"		value="0.465"/>
+  <xacro:property name="box_l"		value="0.340"/>
+  <xacro:property name="box_h"		value="0.245"/>
+  <xacro:property name="box_bottom_t"	value="0.010"/>
+  <xacro:property name="box_side_t"	value="0.020"/>
   <link name="ground"/>
   <!-- Main workspace -->
@@ -91,4 +96,12 @@
     	    rpy="${origin[3]} ${origin[4]} ${origin[5]}"/>
   </xacro:sensor_d435>
+  <!-- Box -->
+  <xacro:include filename="$(find aist_description
+			   )/objects/urdf/tray.urdf.xacro"/>
+  <xacro:tray prefix=""
+  	      width="${box_w}" length="${box_l}" height="${box_h}"
+	      parent="mounter_table_base_link">
+    <origin xyz="-0.330 0 0.4" rpy="0 0 ${pi/2}"/>
+  </xacro:tray>
   <!-- I would like to remove the "world" link definition, but apparently it is necessary for Gazebo -->
   <link name="world"/>
