Commit message: Correct inertia matrices

File: aist_description/objects/urdf/aist_box.urdf.xacro (robot description, xacro)
@@ -3,6 +3,8 @@
   <xacro:macro name="aist_box"
 	       params="name width length height parent
-		       rgba:='0.7 0.7 0.7 1' color_name:=aist_color
+		       rgba:='0.7 0.7 0.7 1' color_name:=aist_color mass:=1.0
 		       *origin">
+    <xacro:include filename="$(find aist_description
+			     )/objects/urdf/primitive_inertia.urdf.xacro"/>
     <link name="${name}">
       <!-- w is in x, l is in y, h is in z -->
@@ -24,7 +26,7 @@
       <!-- This is required for Gazebo. -->
       <inertial>
-        <mass value="1.0"/>
-        <!-- <origin xyz="${width/2} ${length} ${height/2}" rpy="0 0 0"/> -->
-        <inertia ixx="0.0" ixy="0.0" ixz="0.0" iyy="0.0" iyz="0.0" izz="0.0"/>
+	<origin xyz="${width/2} ${length} ${height/2}" rpy="0 0 0"/>
+	<xacro:box_inertia width="${width}" length="${length}"
+			   height="${height}" mass="${mass}"/>
       </inertial>
     </link>

File: aist_description/objects/urdf/usb_repeater.urdf.xacro (robot description, xacro)
@@ -2,14 +2,19 @@
 <robot xmlns:xacro="http://wiki.ros.org/xacro" name="usb_repeater">
   <xacro:macro name="usb_repeater" params="prefix parent *origin">
+    <xacro:include filename="$(find aist_description
+			     )/objects/urdf/primitive_inertia.urdf.xacro"/>
     <xacro:property name="arrangement_radius"	value="0.031"/>
     <xacro:property name="leg_radius"		value="0.003"/>
     <xacro:property name="leg_height"		value="0.010"/>
+    <xacro:property name="leg_mass"		value="0.005"/>
     <xacro:property name="plate_radius"		value="0.0375"/>
     <xacro:property name="plate_thickness"	value="0.004"/>
+    <xacro:property name="plate_mass"		value="0.030"/>
     <xacro:property name="repeater_width"	value="0.033"/>
     <xacro:property name="repeater_length"	value="0.055"/>
     <xacro:property name="repeater_height"	value="0.014"/>
+    <xacro:property name="repeater_mass"	value="0.050"/>
     <xacro:macro name="my_cylinder"
-		 params="name parent radius thickness *origin">
+		 params="name parent radius thickness mass *origin">
       <link name="${name}">
 	<visual>
@@ -29,6 +34,7 @@
 	</collision>
 	<inertial>
-          <mass value="1.0"/>
-          <inertia ixx="0.0" ixy="0.0" ixz="0.0" iyy="0.0" iyz="0.0" izz="0.0"/>
+          <origin xyz="0 0 ${thickness/2}" rpy="0 0 0"/>
+          <xacro:cylinder_inertia radius="${radius}" height="${thickness}"
+				  mass="${mass}"/>
 	</inertial>
       </link>
@@ -48,24 +54,24 @@
       <xacro:insert_block name="origin"/>
     </joint>
-    <xacro:my_cylinder name="${prefix}front_leg"
-		 radius="${leg_radius}" thickness="${leg_height}"
-		 parent="${prefix}base_link">
+    <xacro:my_cylinder name="${prefix}front_leg" parent="${prefix}base_link"
+		       radius="${leg_radius}" thickness="${leg_height}"
+		       mass="${leg_mass}">
       <origin xyz="${arrangement_radius} 0 0" rpy="0 0 0"/>
     </xacro:my_cylinder>
-    <xacro:my_cylinder name="${prefix}left_leg"
-		 radius="${leg_radius}" thickness="${leg_height}"
-		 parent="${prefix}base_link">
+    <xacro:my_cylinder name="${prefix}left_leg" parent="${prefix}base_link"
+		       radius="${leg_radius}" thickness="${leg_height}"
+		       mass="${leg_mass}">
       <origin xyz="${-0.5*arrangement_radius} ${0.866*arrangement_radius} 0"
 	      rpy="0 0 0"/>
     </xacro:my_cylinder>
-    <xacro:my_cylinder name="${prefix}right_leg"
-		 radius="${leg_radius}" thickness="${leg_height}"
-		 parent="${prefix}base_link">
+    <xacro:my_cylinder name="${prefix}right_leg" parent="${prefix}base_link"
+		       radius="${leg_radius}" thickness="${leg_height}"
+		       mass="${leg_mass}">
       <origin xyz="${-0.5*arrangement_radius} ${-0.866*arrangement_radius} 0"
 	      rpy="0 0 0"/>
     </xacro:my_cylinder>
-    <xacro:my_cylinder name="${prefix}plate"
-		 radius="${plate_radius}" thickness="${plate_thickness}"
-		 parent="${prefix}base_link">
+    <xacro:my_cylinder name="${prefix}plate" parent="${prefix}base_link"
+		       radius="${plate_radius}" thickness="${plate_thickness}"
+		       mass="${plate_mass}">
       <origin xyz="0 0 ${leg_height}" rpy="0 0 0"/>
     </xacro:my_cylinder>
@@ -85,6 +91,8 @@
       </collision>
       <inertial>
-        <mass value="1.0"/>
-        <inertia ixx="0.0" ixy="0.0" ixz="0.0" iyy="0.0" iyz="0.0" izz="0.0"/>
+        <xacro:box_inertia width="${repeater_width}"
+			   length="${repeater_length}"
+			   height="${repeater_height}"
+			   mass="${repeater_mass}"/>
       </inertial>
     </link>

File: aist_description/scenes/urdf/a_bot_base_scene.urdf.xacro (robot description, xacro)
@@ -1,5 +1,17 @@
 <?xml version="1.0"?>
 <robot xmlns:xacro="http://wiki.ros.org/xacro" name="a_bot_base_scene" >
-  <xacro:arg name="scene"		default=""/>
+  <xacro:arg name="scene"	default=""/>
+  <xacro:arg name="sim"		default="false"/>
+  <!-- ur_robot_driver -->
+  <xacro:property name="a_bot_ip"	value="10.66.171.40"/>
+  <xacro:property name="script_filename"
+		  value="$(find ur_client_library
+			 )/resources/external_control.urscript"/>
+  <xacro:property name="output_recipe_filename"
+		  value="$(find ur_robot_driver
+			 )/resources/rtde_output_recipe.txt"/>
+  <xacro:property name="input_recipe_filename"
+		  value="$(find ur_robot_driver
+			 )/resources/rtde_input_recipe.txt"/>
   <xacro:arg name="hw_interface"	default="PositionJointInterface"/>
 					<!-- or "VelocityJointInterface" -->
@@ -87,23 +99,26 @@
   </xacro:suction_tool_holder>
   <!-- robot arms -->
-  <xacro:include filename="$(find ur_gazebo)/urdf/ur_macro.xacro"/>
-  <xacro:ur_robot_gazebo
-      prefix="a_bot_"
-      joint_limits_parameters_file="$(find ur_description
-				    )/config/ur5e/joint_limits.yaml"
-      physical_parameters_file="$(find ur_description
-				)/config/ur5e/physical_parameters.yaml"
-      visual_parameters_file="$(find ur_description
-			      )/config/ur5e/visual_parameters.yaml"
-      kinematics_parameters_file="$(find aist_bringup
-				  )/config/a_bot_calibration.yaml"
-      transmission_hw_interface="hardware_interface/$(arg hw_interface)"
+  <xacro:include
+      filename="$(find aist_description
+		)/devices/urdf/ur_robot_with_ros2_control.urdf.xacro"/>
+  <xacro:ur_robot_with_ros2_control
+      name="a_bot"
+      sim="$(arg sim)"
+      ur_type="ur5e"
+      tf_prefix="a_bot_"
+      parent="a_bot_table_top_center"
       safety_limits="true"
-      safety_pos_margin="0.3"/>
-  <joint name="a_bot_base_link_joint" type="fixed">
-    <parent link="a_bot_table_top_center"/>
-    <child  link="a_bot_base_link"/>
+      safety_pos_margin="0.15"
+      script_filename="${script_filename}"
+      input_recipe_filename="${input_recipe_filename}"
+      output_recipe_filename="${output_recipe_filename}"
+      robot_ip="${a_bot_ip}"
+      reverse_port="50001"
+      script_sender_port="50002"
+      reverse_ip="0.0.0.0"
+      script_command_port="50004"
+      trajectory_port="50003">
     <origin xyz="0 0 0 " rpy="0 0 0"/>
-  </joint>
+  </xacro:ur_robot_with_ros2_control>
   <!-- Set gazebo plugin for FT-sensors -->
   <xacro:include filename="$(find aist_description
@@ -135,10 +150,10 @@
     <origin xyz="0.000 -0.051 0.000" rpy="${pi/2} ${-pi/2} 0"/>
   </xacro:usb_repeater>
-  <!-- RealSense cameras -->
+  <!-- <!-\- RealSense cameras -\-> -->
   <xacro:include filename="$(find aist_description
-  			   )/devices/urdf/sr305_on_2f140.urdf.xacro" />
+			   )/devices/urdf/sr305_on_2f140.urdf.xacro" />
   <xacro:sr305_on_2f140 prefix="a_bot_"
-  			parent="a_bot_gripper_base_link"
-  			use_nominal_extrinsics="true"/>
+			parent="a_bot_gripper_base_link"
+			use_nominal_extrinsics="true"/>
   <!-- I would like to remove the "world" link definition, but apparently it is necessary for Gazebo -->
   <link name="world"/>

File: aist_description/scenes/urdf/aist_base_scene.urdf.xacro (robot description, xacro)
@@ -1,5 +1,19 @@
 <?xml version="1.0"?>
 <robot xmlns:xacro="http://wiki.ros.org/xacro" name="aist_base_scene" >
-  <xacro:arg name="scene" default=""/>
+  <xacro:arg name="scene"	default=""/>
+  <xacro:arg name="sim"		default="false"/>
+  <!-- ur_robot_driver -->
+  <xacro:property name="a_bot_ip"	value="10.66.171.40"/>
+  <xacro:property name="b_bot_ip"	value="10.66.171.41"/>
+  <xacro:property name="script_filename"
+		  value="$(find ur_client_library
+			 )/resources/external_control.urscript"/>
+  <xacro:property name="output_recipe_filename"
+		  value="$(find ur_robot_driver
+			 )/resources/rtde_output_recipe.txt"/>
+  <xacro:property name="input_recipe_filename"
+		  value="$(find ur_robot_driver
+			 )/resources/rtde_input_recipe.txt"/>
+  <!-- location of robot arms -->
   <xacro:property name="a_bot_x"	value="0"/>
   <xacro:property name="a_bot_y"	value="-0.4875"/>
@@ -96,37 +110,45 @@
   </xacro:suction_tool_holder>
   <!-- robot arms -->
-  <xacro:include filename="$(find ur_description)/urdf/ur_macro.xacro"/>
-  <xacro:ur_robot
+  <xacro:include
+      filename="$(find aist_description
+		)/devices/urdf/ur_robot_with_ros2_control.urdf.xacro"/>
+  <xacro:ur_robot_with_ros2_control
+      sim="$(arg sim)"
+      ur_type="ur5e"
       name="a_bot"
       tf_prefix="a_bot_"
       parent="a_bot_table_top_center"
-      joint_limits_parameters_file="$(find ur_description
-				    )/config/ur5e/joint_limits.yaml"
-      physical_parameters_file="$(find ur_description
-				)/config/ur5e/physical_parameters.yaml"
-      visual_parameters_file="$(find ur_description
-			      )/config/ur5e/visual_parameters.yaml"
-      kinematics_parameters_file="$(find aist_description
-				  )/scenes/calib/a_bot.yaml"
       safety_limits="true"
-      safety_pos_margin="0.15">
+      safety_pos_margin="0.15"
+      script_filename="${script_filename}"
+      input_recipe_filename="${input_recipe_filename}"
+      output_recipe_filename="${output_recipe_filename}"
+      robot_ip="${a_bot_ip}"
+      reverse_port="50001"
+      script_sender_port="50002"
+      reverse_ip="0.0.0.0"
+      script_command_port="50004"
+      trajectory_port="50003">
     <origin xyz="0 0 0 " rpy="0 0 0"/>
-  </xacro:ur_robot>
-  <xacro:ur_robot
+  </xacro:ur_robot_with_ros2_control>
+  <xacro:ur_robot_with_ros2_control
+      sim="$(arg sim)"
+      ur_type="ur5e"
       name="b_bot"
       tf_prefix="b_bot_"
       parent="b_bot_table_top_center"
-      joint_limits_parameters_file="$(find ur_description
-				    )/config/ur5e/joint_limits.yaml"
-      physical_parameters_file="$(find ur_description
-				)/config/ur5e/physical_parameters.yaml"
-      visual_parameters_file="$(find ur_description
-			      )/config/ur5e/visual_parameters.yaml"
-      kinematics_parameters_file="$(find aist_description
-				  )/scenes/calib/b_bot.yaml"
       safety_limits="true"
-      safety_pos_margin="0.15">
+      safety_pos_margin="0.15"
+      script_filename=""
+      input_recipe_filename=""
+      output_recipe_filename=""
+      robot_ip="${b_bot_ip}"
+      reverse_port="50005"
+      script_sender_port="50006"
+      reverse_ip="0.0.0.0"
+      script_command_port="50008"
+      trajectory_port="50007">
     <origin xyz="0 0 0" rpy="0 0 ${b_bot_theta}"/>
-  </xacro:ur_robot>
+  </xacro:ur_robot_with_ros2_control>
   <!-- Spawn and attach grippers -->
   <xacro:include filename="$(find aist_robotiq
@@ -176,14 +198,15 @@
   </xacro:motioncam_m_camera>
   <!-- Add RealSense cameras -->
-  <!-- <xacro:include filename="$(find aist_description -->
-  <!-- 			   )/devices/urdf/sr305_on_2f140.urdf.xacro" /> -->
-  <!-- <xacro:sr305_on_2f140 prefix="a_bot_" -->
-  <!-- 			parent="a_bot_gripper_base_link" -->
-  <!-- 			use_nominal_extrinsics="true"/> -->
-  <!-- <xacro:include filename="$(find aist_description -->
-  <!-- 			   )/devices/urdf/sr305_on_2f85.urdf.xacro" /> -->
-  <!-- <xacro:sr305_on_2f85 prefix="b_bot_" -->
-  <!-- 		       parent="b_bot_gripper_base_link" -->
-  <!-- 		       use_nominal_extrinsics="true"/> -->
+  <xacro:include filename="$(find aist_description
+			   )/devices/urdf/sr305_on_2f140.urdf.xacro" />
+  <xacro:sr305_on_2f140 prefix="a_bot_"
+			parent="a_bot_gripper_base_link"
+			use_nominal_extrinsics="true"/>
+  <xacro:include filename="$(find aist_description
+			   )/devices/urdf/sr305_on_2f85.urdf.xacro" />
+  <xacro:sr305_on_2f85 prefix="b_bot_"
+		       parent="b_bot_gripper_base_link"
+		       use_nominal_extrinsics="true"/>
+l
   <!-- Add live camera -->
   <xacro:load_calibration filename="$(find aist_description

File: aist_description/scenes/urdf/b_bot_base_scene.urdf.xacro (robot description, xacro)
@@ -1,5 +1,19 @@
 <?xml version="1.0"?>
 <robot xmlns:xacro="http://wiki.ros.org/xacro" name="b_bot_base_scene" >
-  <xacro:arg name="scene" default=""/>
+  <xacro:arg name="scene"	default=""/>
+  <xacro:arg name="sim"		default="false"/>
+  <!-- ur_robot_driver -->
+  <xacro:property name="b_bot_ip"	value="10.66.171.41"/>
+  <xacro:property name="script_filename"
+		  value="$(find ur_client_library
+			 )/resources/external_control.urscript"/>
+  <xacro:property name="output_recipe_filename"
+		  value="$(find ur_robot_driver
+			 )/resources/rtde_output_recipe.txt"/>
+  <xacro:property name="input_recipe_filename"
+		  value="$(find ur_robot_driver
+			 )/resources/rtde_input_recipe.txt"/>
+  <xacro:arg name="hw_interface"	default="PositionJointInterface"/>
+					<!-- or "VelocityJointInterface" -->
   <xacro:property name="b_bot_x"	value="0"/>
   <xacro:property name="b_bot_y"	value="0.4875"/>
@@ -80,23 +94,26 @@
   </xacro:suction_tool_holder>
   <!-- robot arms -->
-  <xacro:include filename="$(find ur_gazebo)/urdf/ur_macro.xacro"/>
-  <xacro:ur_robot_gazebo
-      prefix="b_bot_"
-      joint_limits_parameters_file="$(find ur_description
-				    )/config/ur5e/joint_limits.yaml"
-      physical_parameters_file="$(find ur_description
-				)/config/ur5e/physical_parameters.yaml"
-      visual_parameters_file="$(find ur_description
-			      )/config/ur5e/visual_parameters.yaml"
-      kinematics_parameters_file="$(find aist_bringup
-				  )/config/b_bot_calibration.yaml"
-      transmission_hw_interface="hardware_interface/PositionJointInterface"
+  <xacro:include
+      filename="$(find aist_description
+		)/devices/urdf/ur_robot_with_ros2_control.urdf.xacro"/>
+  <xacro:ur_robot_with_ros2_control
+      name="b_bot"
+      sim="$(arg sim)"
+      ur_type="ur5e"
+      tf_prefix="b_bot_"
+      parent="b_bot_table_top_center"
       safety_limits="true"
-      safety_pos_margin="0.3"/>
-  <joint name="b_bot_base_link_joint" type="fixed">
-    <parent link="b_bot_table_top_center"/>
-    <child  link="b_bot_base_link"/>
-    <origin xyz="0 0 0 " rpy="0 0 ${b_bot_theta}"/>
-  </joint>
+      safety_pos_margin="0.15"
+      script_filename=""
+      input_recipe_filename=""
+      output_recipe_filename=""
+      robot_ip="${b_bot_ip}"
+      reverse_port="50005"
+      script_sender_port="50006"
+      reverse_ip="0.0.0.0"
+      script_command_port="50008"
+      trajectory_port="50007">
+    <origin xyz="0 0 0" rpy="0 0 ${b_bot_theta}"/>
+  </xacro:ur_robot_with_ros2_control>
   <!-- Spawn and attach gripper -->
   <xacro:include filename="$(find aist_robotiq
@@ -132,9 +149,9 @@
   <!-- Add RealSense cameras -->
   <xacro:include filename="$(find aist_description
-  			   )/devices/urdf/sr305_on_2f85.urdf.xacro" />
+			   )/devices/urdf/sr305_on_2f85.urdf.xacro" />
   <xacro:sr305_on_2f85 prefix="b_bot_"
-  		       parent="b_bot_gripper_base_link"
-  		       use_nominal_extrinsics="true"/>
-  <!-- Add live camera -->
+		       parent="b_bot_gripper_base_link"
+		       use_nominal_extrinsics="true"/>
+  Add live camera
   <xacro:load_calibration filename="$(find aist_camera_calibration
 				    )/calib/live_camera.yaml"/>

File: aist_fastening_tools/urdf/base_fixture.urdf.xacro (robot description, xacro)
@@ -2,4 +2,6 @@
 <robot xmlns:xacro="http://ros.org/wiki/xacro">
   <xacro:macro name="base_fixture" params="prefix parent *origin">
+    <xacro:include filename="$(find aist_description
+			     )/objects/urdf/primitive_inertia.urdf.xacro"/>
     <xacro:macro name="load_properties" params="filename">
       <xacro:property name="properties"
@@ -37,7 +39,7 @@
 		     ${body_vorigin[1]}
 		     ${body_vorigin[2]}"
-		rpy="${body_vorigin[3]*pi/180.0}
-		     ${body_vorigin[4]*pi/180.0}
-		     ${body_vorigin[5]*pi/180.0}"/>
+		rpy="${radians(body_vorigin[3])}
+		     ${radians(body_vorigin[4])}
+		     ${radians(body_vorigin[5])}"/>
         <geometry>
           <mesh filename="${visual_meshes[0]['url']}"
@@ -53,7 +55,7 @@
 		     ${body_corigin[1]}
 		     ${body_corigin[2]}"
-		rpy="${body_corigin[3]*pi/180.0}
-		     ${body_corigin[4]*pi/180.0}
-		     ${body_corigin[5]*pi/180.0}"/>
+		rpy="${radians(body_corigin[3])}
+		     ${radians(body_corigin[4])}
+		     ${radians(body_corigin[5])}"/>
         <geometry>
 	  <box size="${body_cdims[0]} ${body_cdims[1]} ${body_cdims[2]}"/>
@@ -61,8 +63,14 @@
       </collision>
       <inertial>
-        <origin xyz="0 0 0" rpy="0 0 0"/>
-        <mass value="0.86387"/>
-        <inertia ixx="1017560E-9" ixy="0" ixz="2235E-9"
-		 iyy="1028041E-9" iyz="0" izz="489810E-9"/>
+	<origin xyz="${body_corigin[0]}
+		     ${body_corigin[1]}
+		     ${body_corigin[2]}"
+		rpy="${radians(body_corigin[3])}
+		     ${radians(body_corigin[4])}
+		     ${radians(body_corigin[5])}"/>
+        <xacro:box_inertia width="${body_cdims[0]}"
+			   length="${body_cdims[1]}"
+			   height="${body_cdims[2]}"
+			   mass="0.86387"/>
       </inertial>
     </link>
@@ -89,7 +97,7 @@
       		     ${piston_vorigin[1]}
       		     ${piston_vorigin[2]}"
-      		rpy="${piston_vorigin[3]*pi/180.0}
-      		     ${piston_vorigin[4]*pi/180.0}
-      		     ${piston_vorigin[5]*pi/180.0}"/>
+      		rpy="${radians(piston_vorigin[3])}
+      		     ${radians(piston_vorigin[4])}
+      		     ${radians(piston_vorigin[5])}"/>
         <geometry>
           <mesh filename="${visual_meshes[1]['url']}"
@@ -107,7 +115,7 @@
 		     ${piston_corigin[1]}
 		     ${piston_corigin[2]}"
-		rpy="${piston_corigin[3]*pi/180.0}
-		     ${piston_corigin[4]*pi/180.0}
-		     ${piston_corigin[5]*pi/180.0}"/>
+		rpy="${radians(piston_corigin[3])}
+		     ${radians(piston_corigin[4])}
+		     ${radians(piston_corigin[5])}"/>
         <geometry>
 	  <box size="${piston_cdims[0]}
@@ -117,8 +125,15 @@
       </collision>
       <inertial>
-        <origin xyz="0.02262 -0.00759 0.00738" rpy="0 0 0"/>
+	<origin xyz="${piston_corigin[0]}
+		     ${piston_corigin[1]}
+		     ${piston_corigin[2]}"
+		rpy="${radians(piston_corigin[3])}
+		     ${radians(piston_corigin[4])}
+		     ${radians(piston_corigin[5])}"/>
         <mass value="0.03804"/>
-        <inertia ixx="13567E-9" ixy="1849E-9" ixz="3622E-9"
-		 iyy="15784E-9" iyz="3616E-9" izz="7478E-9"/>
+        <xacro:box_inertia width="${piston_cdims[0]}"
+			   length="${piston_cdims[1]}"
+			   height="${piston_cdims[2]}"
+			   mass="0.03804"/>
       </inertial>
     </link>
@@ -132,7 +147,7 @@
 		   ${tip_link_origin[1]}
 		   ${tip_link_origin[2]}"
-	      rpy="${tip_link_origin[3]*pi/180.0}
-		   ${tip_link_origin[4]*pi/180.0}
-		   ${tip_link_origin[5]*pi/180.0}"/>
+	      rpy="${radians(tip_link_origin[3])}
+		   ${radians(tip_link_origin[4])}
+		   ${radians(tip_link_origin[5])}"/>
     </joint>
     <link name="${prefix}tip_link"/>
@@ -146,7 +161,7 @@
 		   ${piston_head_origin[1]}
 		   ${piston_head_origin[2]}"
-	      rpy="${piston_head_origin[3]*pi/180.0}
-		   ${piston_head_origin[4]*pi/180.0}
-		   ${piston_head_origin[5]*pi/180.0}"/>
+	      rpy="${radians(piston_head_origin[3])}
+		   ${radians(piston_head_origin[4])}
+		   ${radians(piston_head_origin[5])}"/>
     </joint>
     <link name="${prefix}piston_head"/>
