Commit message: Update base_fixture_head

File: aist_description/objects/urdf/base_fixture_head.urdf.xacro (robot description, xacro)
@@ -6,5 +6,5 @@
     <link name="${prefix}base_link">
       <visual>
-        <origin xyz="-0.007 -0.0331 -0.011" rpy="0 0 0"/>
+        <origin xyz="-0.007 -0.033 -0.011" rpy="0 0 0"/>
 	<geometry>
           <mesh filename="package://aist_description/objects/meshes/base_fixture_head.stl" scale="0.001 0.001 0.001"/>
@@ -16,5 +16,5 @@
       <collision>
       <!-- avoid collision -->
-        <origin xyz="-0.007 -0.0331 -0.011" rpy="0 0 0"/>
+        <origin xyz="-0.007 -0.033 -0.011" rpy="0 0 0"/>
 	<geometry>
 	  <mesh
@@ -34,5 +34,5 @@
       <parent link="${prefix}base_link"/>
       <child  link="${prefix}tip_link"/>
-      <origin xyz="0.007 0.0 -0.013" rpy="0 0 ${-33.2749*pi/180}"/>
+      <origin xyz="0.007 0.0 -0.013" rpy="0 0 ${-30.9639*pi/180}"/>
     </joint>
   </xacro:macro>

Commit message: Confirmed that handeye calibration works for a_motioncam, a_bot_camera and b_bot_camera

File: aist_description/objects/urdf/base_fixture_head.urdf.xacro (robot description, xacro)
@@ -19,5 +19,5 @@
 	<geometry>
 	  <mesh
-	      filename="package://aist_description/objects/meshes/base_fixture_head-collision.stl" scale="0.001 0.001 0.001"/>
+	      filename="package://aist_description/objects/meshes/collision/base_fixture_head.stl" scale="0.001 0.001 0.001"/>
 	</geometry>
       </collision>

File: aist_description/objects/urdf/sr305_mount_2f140.urdf.xacro (robot description, xacro)
@@ -2,11 +2,10 @@
 <!-- This macro adds a convenient TF frame at the tip of the closed gripper. -->
 <!-- The position of the TF frame has not been measured at all and needs to be calibrated. -->
-<robot name="sr305_on_2f85" xmlns:xacro="http://www.ros.org/wiki/xacro">
-  <xacro:macro name="sr305_on_2f85"
-	       params="prefix parent use_nominal_extrinsics:=false">
+<robot name="sr305_mount_2f140" xmlns:xacro="http://www.ros.org/wiki/xacro">
+  <xacro:macro name="sr305_mount_2f140" params="prefix parent">
     <xacro:include filename="$(find aist_description
 			     )/devices/urdf/_sr305.urdf.xacro"/>
     <xacro:property name="mesh_dir"
-		    value="package://aist_description/devices/meshes"/>
+		    value="package://aist_description/objects/meshes"/>
     <link name="${prefix}camera_mount">
       <inertial>
@@ -18,5 +17,5 @@
         <origin rpy="${pi} 0 ${pi/2}" xyz="0 0 0.0"/>
         <geometry>
-          <mesh filename="${mesh_dir}/sr305_mount_2f85.stl"
+          <mesh filename="${mesh_dir}/sr305_mount_2f140.stl"
 		scale=".001 .001 .001"/>
         </geometry>
@@ -28,5 +27,5 @@
         <origin rpy="${pi} 0 ${pi/2}" xyz="0 0 0.0"/>
         <geometry>
-          <mesh filename="${mesh_dir}/collision/sr305_mount_2f85.stl"
+          <mesh filename="${mesh_dir}/collision/sr305_mount_2f140.stl"
 		scale=".001 .001 .001"/>
         </geometry>
@@ -38,18 +37,10 @@
       <origin xyz="0.035 0.0 0.025" rpy="0 0 0"/>
     </joint>
-    <xacro:include filename="$(find aist_description
-			     )/scenes/urdf/load_calibration.urdf.xacro"/>
-    <xacro:load_calibration filename="$(find aist_description
-				      )/scenes/calib/${prefix}camera.yaml"
-			    propname="camera_origin"/>
-    <xacro:sensor_sr305 name="${prefix}camera" parent="${parent}"
-			use_nominal_extrinsics="${use_nominal_extrinsics}">
-      <origin xyz="${camera_origin[0]}
-		   ${camera_origin[1]}
-		   ${camera_origin[2]}"
-    	      rpy="${camera_origin[3]}
-		   ${camera_origin[4]}
-		   ${camera_origin[5]}"/>
-    </xacro:sensor_sr305>
+    <link name="${prefix}camera_mount_flange"/>
+    <joint name="${prefix}camera_mount_flange_joint" type="fixed">
+      <parent link="${prefix}camera_mount" />
+      <child  link="${prefix}camera_mount_flange" />
+      <origin xyz="0.0546 0.015 0.0645" rpy="0 ${20.0*pi/180.0} 0"/>
+    </joint>
   </xacro:macro>
 </robot>

File: aist_description/scenes/urdf/a_bot_base_scene.urdf.xacro (robot description, xacro)
@@ -160,20 +160,30 @@
   </xacro:usb_repeater>
   <!-- Add Motioncam-3D scanner -->
-  <xacro:include filename="$(find aist_description
-			   )/scenes/urdf/load_calibration.urdf.xacro"/>
-  <xacro:load_calibration filename="$(find aist_description
-				    )/scenes/calib/a_motioncam.yaml"/>
   <xacro:include filename="$(find aist_phoxi_camera
 			   )/urdf/motioncam_m_camera.urdf.xacro"/>
-  <xacro:motioncam_m_camera name="a_motioncam" parent="workspace_center">
-    <origin xyz="${origin[0]} ${origin[1]} ${origin[2]}"
-    	    rpy="${origin[3]} ${origin[4]} ${origin[5]}"/>
+  <xacro:motioncam_m_camera name="a_motioncam" parent="workspace_center"
+			    use_nominal_extrinsics="$(arg sim)">
+    <origin xyz="0.524 -0.074 0.657" rpy="-0.015 1.063 3.134"/>
   </xacro:motioncam_m_camera>
-  <!-- RealSense cameras -->
-  <xacro:include filename="$(find aist_description
-			   )/devices/urdf/sr305_on_2f140.urdf.xacro" />
-  <xacro:sr305_on_2f140 prefix="a_bot_"
-			parent="a_bot_gripper_base_link"
-			use_nominal_extrinsics="true"/>
+  <!-- Add RealSense camera mount and camera -->
+  <xacro:include filename="$(find aist_description
+			   )/objects/urdf/sr305_mount_2f140.urdf.xacro"/>
+  <xacro:sr305_mount_2f140 prefix="a_bot_"
+			   parent="a_bot_gripper_coupling_flange_link"/>
+  <xacro:include filename="$(find aist_description
+			   )/devices/urdf/_sr305.urdf.xacro"/>
+  <xacro:sensor_sr305 name="a_bot_camera" parent="a_bot_camera_mount_flange"
+		      use_nominal_extrinsics="$(arg sim)">
+    <origin xyz="0 0 0" rpy="0 0 0"/>
+  </xacro:sensor_sr305>
+  <!-- Add camera optical links from camera calibrations -->
+  <xacro:unless value="$(arg sim)">
+    <xacro:include filename="$(find aist_description
+			     )/scenes/urdf/load_link.urdf.xacro"/>
+    <xacro:load_link filename="$(find aist_description
+			       )/scenes/calib/a_motioncam.yaml"/>
+    <xacro:load_link filename="$(find aist_description
+			       )/scenes/calib/a_bot_camera.yaml"/>
+  </xacro:unless>
   <!-- I would like to remove the "world" link definition, but apparently it is necessary for Gazebo -->
   <link name="world"/>

File: aist_description/scenes/urdf/aist_base_scene.urdf.xacro (robot description, xacro)
@@ -1,5 +1,5 @@
 <?xml version="1.0"?>
 <robot xmlns:xacro="http://wiki.ros.org/xacro" name="aist_base_scene" >
-  <xacro:arg name="scene"	default="kitting"/>
+  <xacro:arg name="scene"	default=""/>
   <xacro:arg name="sim"		default="false"/>
   <xacro:arg name="transmission_hw_interface"
@@ -199,36 +199,42 @@
   </xacro:usb_repeater>
   <!-- Add Motioncam-3D scanner -->
-  <xacro:include filename="$(find aist_description
-			   )/scenes/urdf/load_calibration.urdf.xacro"/>
-  <xacro:load_calibration filename="$(find aist_description
-				    )/scenes/calib/a_motioncam.yaml"/>
   <xacro:include filename="$(find aist_phoxi_camera
 			   )/urdf/motioncam_m_camera.urdf.xacro"/>
   <xacro:motioncam_m_camera name="a_motioncam" parent="workspace_center"
-			    use_nominal_extrinsics="true">
-    <origin xyz="${origin[0]} ${origin[1]} ${origin[2]}"
-    	    rpy="${origin[3]} ${origin[4]} ${origin[5]}"/>
+			    use_nominal_extrinsics="$(arg sim)">
+    <origin xyz="0.524 -0.074 0.657" rpy="-0.015 1.063 3.134"/>
   </xacro:motioncam_m_camera>
-  <!-- Add RealSense cameras -->
-  <xacro:include filename="$(find aist_description
-			   )/devices/urdf/sr305_on_2f140.urdf.xacro" />
-  <xacro:sr305_on_2f140 prefix="a_bot_"
-			parent="a_bot_gripper_coupling_flange_link"
-			use_nominal_extrinsics="true"/>
-  <xacro:include filename="$(find aist_description
-			   )/devices/urdf/sr305_on_2f85.urdf.xacro" />
-  <xacro:sr305_on_2f85 prefix="b_bot_"
-		       parent="b_bot_gripper_coupling_flange_link"
-		       use_nominal_extrinsics="true"/>
-  <!-- Add live camera -->
-  <xacro:load_calibration filename="$(find aist_description
-				    )/scenes/calib/live_camera.yaml"/>
-  <link name="live_camera_optical_frame"/>
-  <joint name="live_camera_joint" type="fixed">
-    <parent link="workspace_center"/>
-    <child  link="live_camera_optical_frame"/>
-    <origin xyz="${origin[0]} ${origin[1]} ${origin[2]}"
-    	    rpy="${origin[3]} ${origin[4]} ${origin[5]}"/>
-  </joint>
+  <!-- Add RealSense camera mounts and cameras -->
+  <xacro:include filename="$(find aist_description
+			   )/objects/urdf/sr305_mount_2f140.urdf.xacro"/>
+  <xacro:sr305_mount_2f140 prefix="a_bot_"
+			   parent="a_bot_gripper_coupling_flange_link"/>
+  <xacro:include filename="$(find aist_description
+			   )/devices/urdf/_sr305.urdf.xacro"/>
+  <xacro:sensor_sr305 name="a_bot_camera" parent="a_bot_camera_mount_flange"
+		      use_nominal_extrinsics="$(arg sim)">
+    <origin xyz="0 0 0" rpy="0 0 0"/>
+  </xacro:sensor_sr305>
+  <xacro:include filename="$(find aist_description
+			   )/objects/urdf/sr305_mount_2f85.urdf.xacro"/>
+  <xacro:sr305_mount_2f85 prefix="b_bot_"
+			  parent="b_bot_gripper_coupling_flange_link"/>
+  <xacro:sensor_sr305 name="b_bot_camera" parent="b_bot_camera_mount_flange"
+		      use_nominal_extrinsics="$(arg sim)">
+    <origin xyz="0 0 0" rpy="0 0 0"/>
+  </xacro:sensor_sr305>
+  <!-- Add camera optical links from camera calibrations -->
+  <xacro:unless value="$(arg sim)">
+    <xacro:include filename="$(find aist_description
+			     )/scenes/urdf/load_link.urdf.xacro"/>
+    <xacro:load_link filename="$(find aist_description
+			       )/scenes/calib/a_motioncam.yaml"/>
+    <xacro:load_link filename="$(find aist_description
+			       )/scenes/calib/a_bot_camera.yaml"/>
+    <xacro:load_link filename="$(find aist_description
+			       )/scenes/calib/b_bot_camera.yaml"/>
+    <xacro:load_link filename="$(find aist_description
+			       )/scenes/calib/live_camera.yaml"/>
+  </xacro:unless>
   <!-- Add virtual screen -->
   <link name="virtual_screen"/>

File: aist_description/scenes/urdf/b_bot_base_scene.urdf.xacro (robot description, xacro)
@@ -148,30 +148,32 @@
   </xacro:usb_repeater>
   <!-- Add Motioncam-3D scanner -->
-  <xacro:include filename="$(find aist_description
-			   )/scenes/urdf/load_calibration.urdf.xacro"/>
-  <xacro:load_calibration filename="$(find aist_description
-				    )/scenes/calib/a_motioncam.yaml"/>
   <xacro:include filename="$(find aist_phoxi_camera
 			   )/urdf/motioncam_m_camera.urdf.xacro"/>
-  <xacro:motioncam_m_camera name="a_motioncam" parent="workspace_center">
-    <origin xyz="${origin[0]} ${origin[1]} ${origin[2]}"
-    	    rpy="${origin[3]} ${origin[4]} ${origin[5]}"/>
+  <xacro:motioncam_m_camera name="a_motioncam" parent="workspace_center"
+			    use_nominal_extrinsics="$(arg sim)">
+    <origin xyz="0.524 -0.074 0.657" rpy="-0.015 1.063 3.134"/>
   </xacro:motioncam_m_camera>
   <!-- Add RealSense cameras -->
   <xacro:include filename="$(find aist_description
-			   )/devices/urdf/sr305_on_2f85.urdf.xacro" />
-  <xacro:sr305_on_2f85 prefix="b_bot_"
-		       parent="b_bot_gripper_base_link"
-		       use_nominal_extrinsics="true"/>
-  <!-- Add live camera -->
-  <xacro:load_calibration filename="$(find aist_description
-				    )/scenes/calib/live_camera.yaml"/>
-  <link name="live_camera_optical_frame"/>
-  <joint name="live_camera_joint" type="fixed">
-    <parent link="workspace_center"/>
-    <child  link="live_camera_optical_frame"/>
-    <origin xyz="${origin[0]} ${origin[1]} ${origin[2]}"
-    	    rpy="${origin[3]} ${origin[4]} ${origin[5]}"/>
-  </joint>
+			   )/objects/urdf/sr305_mount_2f85.urdf.xacro"/>
+  <xacro:sr305_mount_2f85 prefix="b_bot_"
+			  parent="b_bot_gripper_coupling_flange_link"/>
+  <xacro:include filename="$(find aist_description
+			   )/devices/urdf/_sr305.urdf.xacro"/>
+  <xacro:sensor_sr305 name="b_bot_camera" parent="b_bot_camera_mount_flange"
+		      use_nominal_extrinsics="$(arg sim)">
+    <origin xyz="0 0 0" rpy="0 0 0"/>
+  </xacro:sensor_sr305>
+  <!-- Add camera optical links from camera calibrations -->
+  <xacro:unless value="$(arg sim)">
+    <xacro:include filename="$(find aist_description
+			     )/scenes/urdf/load_link.urdf.xacro"/>
+    <xacro:load_link filename="$(find aist_description
+			       )/scenes/calib/a_motioncam.yaml"/>
+    <xacro:load_link filename="$(find aist_description
+			       )/scenes/calib/b_bot_camera.yaml"/>
+    <xacro:load_link filename="$(find aist_description
+			       )/scenes/calib/live_camera.yaml"/>
+  </xacro:unless>
   <!-- Add virtual screen -->
   <link name="virtual_screen"/>
