Commit message: Adjust screw feeders' location

File: aist_description/scenes/urdf/assembly.urdf.xacro (robot description, xacro)
@@ -8,6 +8,6 @@
   <xacro:property name="workbench_y"		 value="0.630"/>
   <xacro:property name="screw_feeder_width"	 value="0.126"/>
-  <xacro:property name="screw_feeder_y"		 value="0.030"/>
-  <xacro:property name="screw_feeder_x"		 value="0.010"/>
+  <xacro:property name="screw_feeder_y"		 value="0.034"/>
+  <xacro:property name="screw_feeder_x"		 value="0.014"/>
   <xacro:include filename="$(find aist_description
 			   )/objects/urdf/workbench.urdf.xacro"/>

Commit message: Add tray_1 to assembly scene

File: aist_description/scenes/urdf/assembly.urdf.xacro (robot description, xacro)
@@ -32,3 +32,23 @@
     <origin xyz="0 ${screw_feeder_width} 0" rpy="0 0 0"/>
   </xacro:screw_feeder>
+  <!-- additional trays -->
+  <xacro:include filename="$(find aist_description
+			   )/wrc/urdf/kitting_trays.urdf.xacro" />
+  <xacro:kitting_tray trayname="tray_1" parent="workbench_base_link">
+    <origin xyz="${workbench_bar_width - tray_width} 0 0"
+	    rpy="0 0 ${-pi/2}"/>
+  </xacro:kitting_tray>
+  <!-- frames on tray_1 -->
+  <link name="tray_1_frame_1"/>
+  <joint name="tray1_frame_1_joint" type="fixed">
+    <parent link="tray_1"/>
+    <child  link="tray_1_frame_1"/>
+    <origin xyz="0.080 0.050 0.0075" rpy="0 0 ${-pi/2}"/>
+  </joint>
+  <link name="tray_1_frame_2"/>
+  <joint name="tray1_frame_2_joint" type="fixed">
+    <parent link="tray_1"/>
+    <child  link="tray_1_frame_2"/>
+    <origin xyz="0.150 0.050 0.0075" rpy="0 0 ${-pi/2}"/>
+  </joint>
 </robot>
