Commit message: Confirmed real g_bot works

File: aist_description/scenes/urdf/g_bot_base_scene.urdf.xacro (robot description, xacro)
@@ -3,12 +3,12 @@
   <!-- This is the main file defining our robot arrangement and physical environment. -->
   <xacro:arg name="scene" default=""/>
-  <xacro:property name="g_bot_x"   value="0"/>
-  <xacro:property name="g_bot_y"   value="-0.9"/>
-  <xacro:property name="g_bot_z"   value="0.700"/>
+  <xacro:property name="g_bot_x"   value="0.050"/>
+  <xacro:property name="g_bot_y"   value="-0.900"/>
+  <xacro:property name="g_bot_z"   value="0.698"/>
   <xacro:property name="cabinet_w" value="0.900"/>
   <xacro:property name="cabinet_l" value="0.400"/>
   <xacro:property name="cabinet_b" value="0.100"/>
   <xacro:property name="shelf1_h"  value="0.600"/>
-  <xacro:property name="shelf2_h"  value="0.790"/>
+  <xacro:property name="shelf2_h"  value="0.940"/>
   <xacro:property name="back_h"    value="1.500"/>
   <xacro:property name="wall_t"    value="0.012"/>
@@ -77,5 +77,5 @@
 			   )/devices/urdf/conveni_suction_gripper.urdf.xacro"/>
   <xacro:conveni_suction_gripper prefix="g_bot_gripper_" parent="g_bot_tool0">
-    <origin xyz="0 0 0" rpy="0 ${-pi/2} ${-pi/2}"/>
+    <origin xyz="0 0 0" rpy="0 ${-pi/2} ${pi/2}"/>
   </xacro:conveni_suction_gripper>
   <!-- Attach RealSense camera -->

File: moveit_config/g_bot_moveit_config/config/gazebo_g_bot_base_scene.urdf (robot description, URDF)
Before this commit: robot g_bot_base_scene, 45 links, 44 joints
Links:
- link mounter_table_base_link: geometry collision box size=0.05 0.05 0.6779999999999999; visual box size=0.05 0.05 0.6779999999999999
- link mounter_table_leg1: geometry collision box size=0.05 0.05 0.6779999999999999; visual box size=0.05 0.05 0.6779999999999999
- link mounter_table_leg2: geometry collision box size=0.05 0.05 0.6779999999999999; visual box size=0.05 0.05 0.6779999999999999
- link mounter_table_leg3: geometry collision box size=0.05 0.05 0.6779999999999999; visual box size=0.05 0.05 0.6779999999999999
Joints:
- joint cabinet_shelf2: origin xyz=0 0 0.778 rpy=0 0 0 -> xyz=0 0 0.9279999999999999 rpy=0 0 0
- joint g_bot_camera_joint: origin xyz=0.05 0.032 -0.047 rpy=3.14159 0.0 0.0 -> xyz=0.048 0.035 -0.048 rpy=3.141592 0 0
- joint g_bot_gripper_base_joint: origin xyz=0 0 0 rpy=0 -1.5707963267948966 -1.5707963267948966 -> xyz=0 0 0 rpy=0 -1.5707963267948966 1.5707963267948966
- joint ground_g_bot_joint: origin xyz=0 -0.9 0.7 rpy=0 0 0 -> xyz=0.05 -0.9 0.698 rpy=0 0 0
- joint ground_to_workspace: origin xyz=0 0 0.79 rpy=0 0 0 -> xyz=0 0 0.94 rpy=0 0 0
- joint mounter_table_base_link: origin xyz=-0.1 -1.0 0 rpy=0 0 0 -> xyz=-0.05 -1.0 0 rpy=0 0 0
- joint mounter_table_top: origin xyz=0 0 0.6799999999999999 rpy=0 0 0 -> xyz=0 0 0.6779999999999999 rpy=0 0 0

Commit message: Succeeded in perform ConveniPick action

File: aist_description/scenes/urdf/g_bot_base_scene.urdf.xacro (robot description, xacro)
@@ -78,9 +78,17 @@
     <origin xyz="${g_bot_x} ${g_bot_y} ${g_bot_z}" rpy="0 0 0"/>
   </joint>
+  <!-- Attach coupling -->
+  <xacro:include filename="$(find aist_robotiq
+			   )/urdf/robotiq_arg2f_coupling.urdf.xacro"/>
+  <xacro:robotiq_arg2f_coupling prefix="g_bot_gripper_coupling_"
+				parent="g_bot_tool0">
+    <origin xyz="0 0 0" rpy="0 ${-pi/2} ${pi/2}"/>
+  </xacro:robotiq_arg2f_coupling>
   <!-- Attach gripper -->
   <xacro:include filename="$(find aist_description
 			   )/devices/urdf/conveni_suction_gripper.urdf.xacro"/>
-  <xacro:conveni_suction_gripper prefix="g_bot_gripper_" parent="g_bot_tool0">
-    <origin xyz="0 0 0" rpy="0 ${-pi/2} ${pi/2}"/>
+  <xacro:conveni_suction_gripper prefix="g_bot_gripper_"
+				 parent="g_bot_gripper_coupling_flange_link">
+    <origin xyz="0 0 0" rpy="0 0 0"/>
   </xacro:conveni_suction_gripper>
   <!-- Attach RealSense camera -->
@@ -102,5 +110,5 @@
   	      width="${box_w}" length="${box_l}" height="${box_h}"
 	      parent="mounter_table_base_link">
-    <origin xyz="-0.330 0 0.4" rpy="0 0 ${pi/2}"/>
+    <origin xyz="-0.330 0 0" rpy="0 0 ${pi/2}"/>
   </xacro:tray>
   <!-- I would like to remove the "world" link definition, but apparently it is necessary for Gazebo -->

File: moveit_config/g_bot_moveit_config/config/gazebo_g_bot_base_scene.urdf (robot description, URDF)
Before this commit: robot g_bot_base_scene, 45 links, 44 joints
Links:
- added link g_bot_gripper_coupling_base_link, mass 0.22652; collision cylinder length=0.0111 radius=0.0375; visual mesh filename=package://aist_robotiq/meshes/visual/robotiq_arg2f_coupling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 scale=0.001 0.001 0.001
- added link g_bot_gripper_coupling_flange_link
- added link tray_bottom, mass 1.0; collision box size=0.465 0.34 0.005; visual box size=0.465 0.34 0.005
- added link tray_bottom_center
- added link tray_wall0, mass 1.0; collision box size=0.465 0.005 0.24; visual box size=0.465 0.005 0.24
- added link tray_wall1, mass 1.0; collision box size=0.005 0.33 0.24; visual box size=0.005 0.33 0.24
- added link tray_wall2, mass 1.0; collision box size=0.465 0.005 0.24; visual box size=0.465 0.005 0.24
- added link tray_wall3, mass 1.0; collision box size=0.005 0.33 0.24; visual box size=0.005 0.33 0.24
Joints:
- added joint g_bot_gripper_coupling_base_joint: type fixed, parent g_bot_tool0, child g_bot_gripper_coupling_base_link, origin xyz=0 0 0 rpy=0 -1.5707963267948966 1.5707963267948966
- added joint g_bot_gripper_coupling_flange_joint: type fixed, parent g_bot_gripper_coupling_base_link, child g_bot_gripper_coupling_flange_link, origin xyz=0.0111 0 0 rpy=0 0 0
- added joint tray_bottom: type fixed, parent mounter_table_base_link, child tray_bottom, origin xyz=-0.330 0 0 rpy=0 0 1.5707963267948966
- added joint tray_bottom_center_joint: type fixed, parent tray_bottom, child tray_bottom_center, origin xyz=0.2325 0.17 0.005 rpy=0 0 0
- added joint tray_wall0: type fixed, parent tray_bottom, child tray_wall0, origin xyz=0 0 0.005 rpy=0 0 0
- added joint tray_wall1: type fixed, parent tray_bottom, child tray_wall1, origin xyz=0 0.005 0.005 rpy=0 0 0
- added joint tray_wall2: type fixed, parent tray_bottom, child tray_wall2, origin xyz=0 0.335 0.005 rpy=0 0 0
- added joint tray_wall3: type fixed, parent tray_bottom, child tray_wall3, origin xyz=0.46 0.005 0.005 rpy=0 0 0
- joint g_bot_camera_joint: origin xyz=0.048 0.035 -0.048 rpy=3.141592 0 0 -> xyz=0.06024814741236267 0.027958310168559694 -0.05110849290213207 rpy=-3.1348546450858628 -0.0019238101643268973 -0.002535493397081582
- joint g_bot_elbow_joint: origin xyz=-0.425 0 0 rpy=0 0 0 -> xyz=-0.4251908452257245 0 0 rpy=3.139869694262028 -3.140398826093042 3.141590836422541
- joint g_bot_gripper_base_joint: origin xyz=0 0 0 rpy=0 -1.5707963267948966 1.5707963267948966 -> xyz=0 0 0 rpy=0 0 0; parent g_bot_tool0 -> g_bot_gripper_coupling_flange_link
- joint g_bot_shoulder_lift_joint: origin xyz=0 0 0 rpy=1.570796327 0 0 -> xyz=0.0001430786699741724 0 0 rpy=1.570971815456283 0 9.457243266515344e-07
- joint g_bot_shoulder_pan_joint: origin xyz=0 0 0.1625 rpy=0 0 0 -> xyz=0 0 0.1627961697284888 rpy=0 0 1.584854035507899e-08
- joint g_bot_wrist_1_joint: origin xyz=-0.3922 0 0.1333 rpy=0 0 0 -> xyz=-0.392263363687393 -0.001205219753418507 0.1337101152065678 rpy=0.009013432628028227 0.001425591184320421 -7.049255850808575e-06
- joint g_bot_wrist_2_joint: origin xyz=0 -0.0997 -2.044881182297852e-11 rpy=1.570796327 0 0 -> xyz=-0.0001199371355449129 -0.09960234639722144 0.0001395405546602166 rpy=1.569395351131029 0 2.256950157694887e-06
- joint g_bot_wrist_3_joint: origin xyz=0 0.0996 -2.042830148012698e-11 rpy=1.570796326589793 3.141592653589793 3.141592653589793 -> xyz=-2.659467120614162e-05 0.09975515497396804 -5.891598578624916e-07 rpy=1.570790420735626 3.141592653589793 -3.141592181860087
