Commit message: Add support for AIREC3

File: aist_description/scenes/urdf/a_bot_calibration.urdf.xacro (robot description, xacro)
@@ -5,5 +5,5 @@
   <xacro:ar_marker prefix="workspace_"
 		   parent="workspace_center"
-		   marker_id="17_26_32_256"
+		   marker_id="100_101_102_103"
 		   width="0.105" height="0.105" margin="0.007"
 		   thickness="0.001">

File: aist_description/scenes/urdf/calibration.urdf.xacro (robot description, xacro)
@@ -10,10 +10,4 @@
     <origin xyz="0.163 0.0 0.0215" rpy="0 0 ${pi/2}"/>
   </xacro:ar_marker>
-  <!-- <xacro:ar_marker prefix="workspace_" -->
-  <!-- 		   parent="workspace_center" -->
-  <!-- 		   marker_id="17_26_32_256" -->
-  <!-- 		   width="0.150" height="0.150" margin="0.005" -->
-  <!-- 		   thickness="0.001"> -->
-  <!--   <origin xyz="0.0 0.0 0.0005" rpy="0 0 0"/> -->
   <xacro:ar_marker prefix="workbench_"
 		   parent="workbench_table_top_origin"

File: aist_description/scenes/urdf/ceatec.urdf.xacro (robot description, xacro)
@@ -1,11 +1,168 @@
 <?xml version="1.0"?>
-<robot xmlns:xacro="http://wiki.ros.org/xacro" name="ceatec" >
-  <!-- Environment of "ceatec" scene (root = "world") -->
-  <xacro:include filename="$(find aist_description)/scenes/urdf/ceatec_environment.urdf.xacro"/>
-  <!-- Make "map" frame a child of "world" frame -->
-  <joint name="world_map_joint" type="fixed">
-    <parent link="world"/>
-    <child  link="map"/>
-    <origin xyz="0 0 0" rpy="0 0 0"/>
+<robot xmlns:xacro="http://wiki.ros.org/xacro" name="ceatec">
+  <xacro:property name="workspace_offset_x"	value="0.300"/>
+  <xacro:property name="workspace_offset_y"	value="0.500"/>
+  <xacro:property name="workspace_width"	value="3.000"/>
+  <xacro:property name="workspace_length"	value="2.000"/>
+  <xacro:property name="a_table_width"		value="0.530"/>
+  <xacro:property name="a_table_length"		value="0.315"/>
+  <xacro:property name="a_table_height"		value="0.540"/>
+  <xacro:property name="b_table_width"		value="0.700"/>
+  <xacro:property name="b_table_length"		value="0.350"/>
+  <xacro:property name="b_table_height"		value="0.600"/>
+  <xacro:property name="cabinet_width"		value="0.925"/>
+  <xacro:property name="cabinet_length"		value="0.420"/>
+  <xacro:property name="cabinet_base_height"	value="0.180"/>
+  <xacro:property name="cabinet_shelf1_height"	value="0.443"/>
+  <xacro:property name="cabinet_shelf2_height"	value="0.743"/>
+  <xacro:property name="cabinet_back_height"	value="1.711"/>
+  <xacro:property name="tray_width"		value="0.340"/>
+  <xacro:property name="tray_length"		value="0.250"/>
+  <xacro:property name="tray_height"		value="0.062"/>
+  <!-- Root frame -->
+  <link name="ground"/>
+  <!-- a_table -->
+  <xacro:include filename="$(find aist_description)/objects/urdf/table.urdf.xacro"/>
+  <xacro:table prefix="a_table_"
+	       width="${a_table_width}"
+	       length="${a_table_length}"
+	       height="${a_table_height}"
+	       parent="ground">
+    <origin xyz="${workspace_offset_x + workspace_width/2 - cabinet_length - 0.86}
+		 ${workspace_offset_y + 0.6 - (workspace_length/2 - cabinet_width/2)}
+		 0"
+	    rpy="0 0 ${-pi/6}"/>
+  </xacro:table>
+  <!-- Frame to place trays on a_table -->
+  <link name="a_tray_on_a_table" />
+  <joint name="a_tray_on_a_table_joint" type="fixed">
+    <parent link="a_table_top_center" />
+    <child  link="a_tray_on_a_table" />
+    <origin xyz="0 ${-tray_length/2} 0" rpy="0 0 0" />
   </joint>
+  <link name="b_tray_on_a_table" />
+  <joint name="b_tray_on_a_table_joint" type="fixed">
+    <parent link="a_table_top_center" />
+    <child  link="b_tray_on_a_table" />
+    <origin xyz="0 ${-tray_length/2} 0" rpy="0 0 0" />
+  </joint>
+  <link name="a_table_standpoint"/>
+  <joint name="a_table_standpoint_joint" type="fixed">
+    <parent link="a_table_base_link" />
+    <child  link="a_table_standpoint" />
+    <origin xyz="${a_table_width/2} -0.7 0" rpy="0 0 ${pi/2}" />
+  </joint>
+  <!-- b_table -->
+  <xacro:table prefix="b_table_"
+	       width="${b_table_width}"
+	       length="${b_table_length}"
+	       height="${b_table_height}"
+	       parent="ground">
+    <origin xyz="${workspace_offset_x - b_table_width/2-(1.0-0.2)}
+		 ${workspace_offset_y - b_table_length/2+(0.78-0.5)}
+		 0"
+	    rpy="0 0 0"/>
+  </xacro:table>
+  <!-- Frame to place trays on b_table -->
+  <link name="a_tray_on_b_table" />
+  <joint name="a_tray_on_b_table_joint" type="fixed">
+    <parent link="b_table_top_center" />
+    <child  link="a_tray_on_b_table" />
+    <origin xyz="${-tray_width/2 - 0.05} ${-tray_length/2} 0" rpy="0 0 0" />
+  </joint>
+  <link name="b_tray_on_b_table" />
+  <joint name="b_tray_on_b_table_joint" type="fixed">
+    <parent link="b_table_top_center" />
+    <child  link="b_tray_on_b_table" />
+    <origin xyz="0 ${-tray_length/2} 0" rpy="0 0 0" />
+  </joint>
+  <link name="b_table_standpoint"/>
+  <joint name="b_table_standpoint_joint" type="fixed">
+    <parent link="b_table_base_link" />
+    <child  link="b_table_standpoint" />
+    <origin xyz="${b_table_width/2} -0.7 0" rpy="0 0 ${pi/2}" />
+  </joint>
+  <!-- Cabinet -->
+  <xacro:include filename="$(find aist_description)/objects/urdf/cabinet.urdf.xacro"/>
+  <xacro:cabinet prefix="a_"
+		 width="${cabinet_width}"
+		 length="${cabinet_length}"
+		 base_height="${cabinet_base_height}"
+		 shelf1_height="${cabinet_shelf1_height}"
+		 shelf2_height="${cabinet_shelf2_height}"
+		 back_height="${cabinet_back_height}" parent="ground">
+    <origin xyz="${workspace_offset_x + workspace_width/2   - cabinet_length}
+		 ${workspace_offset_y - workspace_length/2 + cabinet_width}
+		 0"
+	    rpy="0 0 ${-pi/2}"/>
+  </xacro:cabinet>
+  <link name="a_cabinet_standpoint"/>
+  <joint name="a_cabinet_standpoint_joint" type="fixed">
+    <parent link="a_cabinet_base" />
+    <child  link="a_cabinet_standpoint" />
+    <origin xyz="${cabinet_width/2} -0.9 0" rpy="0 0 ${pi/2}" />
+  </joint>
+  <!-- Frames to place items on cabinet -->
+  <link name="a_item_in_cabinet"/>
+  <joint name="a_item_in_cabinet_joint" type="fixed">
+    <parent link="a_cabinet_shelf1_origin" />
+    <child  link="a_item_in_cabinet" />
+    <origin xyz="${cabinet_width/12} 0.1 0.08" rpy="${pi/2} ${-pi/2} 0"/>
+  </joint>
+  <link name="b_item_in_cabinet"/>
+  <joint name="b_item_in_cabinet_joint" type="fixed">
+    <parent link="a_item_in_cabinet" />
+    <child  link="b_item_in_cabinet" />
+    <origin xyz="0 ${-cabinet_width/6} 0" rpy="0 0 0" />
+  </joint>
+  <link name="c_item_in_cabinet"/>
+  <joint name="c_item_in_cabinet_joint" type="fixed">
+    <parent link="b_item_in_cabinet" />
+    <child  link="c_item_in_cabinet" />
+    <origin xyz="0 ${-cabinet_width/6} 0" rpy="0 0 0" />
+  </joint>
+  <link name="d_item_in_cabinet"/>
+  <joint name="d_item_in_cabinet_joint" type="fixed">
+    <parent link="c_item_in_cabinet" />
+    <child  link="d_item_in_cabinet" />
+    <origin xyz="0 ${-cabinet_width/6} 0" rpy="0 0 0" />
+  </joint>
+  <link name="e_item_in_cabinet"/>
+  <joint name="e_item_in_cabinet_joint" type="fixed">
+    <parent link="d_item_in_cabinet" />
+    <child  link="e_item_in_cabinet" />
+    <origin xyz="0 ${-cabinet_width/6} 0" rpy="0 0 0" />
+  </joint>
+  <link name="f_item_in_cabinet"/>
+  <joint name="f_item_in_cabinet_joint" type="fixed">
+    <parent link="e_item_in_cabinet" />
+    <child  link="f_item_in_cabinet" />
+    <origin xyz="0 ${-cabinet_width/6} 0" rpy="0 0 0" />
+  </joint>
+  <!-- AR markers -->
+  <xacro:include filename="$(find aist_aruco_ros)/urdf/ar_marker.urdf.xacro"/>
+  <xacro:ar_marker prefix="a_cabinet_" parent="a_cabinet_shelf1_origin"
+		   marker_id="17" width="0.07" height="0.07" margin="0.005" thickness="0.001">
+    <origin xyz="${cabinet_width - 0.040} 0.040 0.001" rpy="0 0 0"/>
+  </xacro:ar_marker>
+  <xacro:ar_marker prefix="a_table_" parent="a_table_top_origin"
+		   marker_id="26" width="0.07" height="0.07" margin="0.005" thickness="0.001">
+    <origin xyz="0.040 0.040 0.001" rpy="0 0 0"/>
+  </xacro:ar_marker>
+  <!-- Trays -->
+  <xacro:include filename="$(find aist_description)/objects/urdf/tray.urdf.xacro"/>
+  <xacro:tray prefix="a_"
+	      width="${tray_width}"
+	      length="${tray_length}"
+	      height="${tray_height}"
+	      parent="a_tray_on_a_table">
+    <origin xyz="${-tray_width/2} 0 0" rpy="0 0 0"/>
+  </xacro:tray>
+  <xacro:tray prefix="b_"
+	      width="${tray_width}"
+	      length="${tray_length}"
+	      height="${tray_height}"
+	      parent="b_tray_on_b_table">
+    <origin xyz="${-tray_width/2} 0 0" rpy="0 0 0"/>
+  </xacro:tray>
 </robot>

File: aist_description/scenes/urdf/ceatec_environment.urdf.xacro (robot description, xacro)
@@ -1,181 +1,11 @@
 <?xml version="1.0"?>
-<robot xmlns:xacro="http://wiki.ros.org/xacro"
-       name="ceatec_environment">
-  <xacro:property name="workspace_width"	value="3.000"/>
-  <xacro:property name="workspace_length"	value="2.000"/>
-  <xacro:property name="a_table_width"		value="0.530"/>
-  <xacro:property name="a_table_length"		value="0.315"/>
-  <xacro:property name="a_table_height"		value="0.540"/>
-  <xacro:property name="b_table_width"		value="0.700"/>
-  <xacro:property name="b_table_length"		value="0.350"/>
-  <xacro:property name="b_table_height"		value="0.600"/>
-  <xacro:property name="cabinet_width"		value="0.925"/>
-  <xacro:property name="cabinet_length"		value="0.420"/>
-  <xacro:property name="cabinet_base_height"	value="0.180"/>
-  <xacro:property name="cabinet_shelf1_height"	value="0.443"/>
-  <xacro:property name="cabinet_shelf2_height"	value="0.743"/>
-  <xacro:property name="cabinet_shelf3_height"	value="1.043"/>
-  <xacro:property name="cabinet_shelf4_height"	value="1.366"/>
-  <xacro:property name="cabinet_back_height"	value="1.711"/>
-  <xacro:property name="tray_width"		value="0.340"/>
-  <xacro:property name="tray_length"		value="0.250"/>
-  <xacro:property name="tray_height"		value="0.062"/>
+<robot xmlns:xacro="http://wiki.ros.org/xacro" name="ceatec_environment">
   <!-- Root frame -->
   <link name="world"/>
-  <!-- Main workspace -->
-  <link name="ground"/>
-  <joint name="world_ground_joint" type="fixed">
+  <joint name="ground_joint" type="fixed">
     <parent link="world"/>
     <child  link="ground"/>
-    <origin xyz="0.3 0.5 0" rpy="0 0 0"/>
   </joint>
-  <!-- a_table -->
-  <xacro:include filename="$(find aist_description)/objects/urdf/table.urdf.xacro"/>
-  <xacro:table prefix="a_table_"
-	       width="${a_table_width}"
-	       length="${a_table_length}"
-	       height="${a_table_height}"
-	       parent="ground">
-    <!-- <origin xyz="${workspace_width/2  - cabinet_length - a_table_width - 0.2}
-		 ${workspace_length/2 - a_table_length - 0.2}
-		 0" rpy="0 0 0"/> -->
-    <origin xyz="${workspace_width/2 - cabinet_length - 0.86}
-		 ${0.6 - (workspace_length/2 - cabinet_width/2)}
-		 0"
-	    rpy="0 0 ${-pi/6}"/>
-  </xacro:table>
-  <!-- Frame to place trays on a_table -->
-  <link name="a_tray_on_a_table" />
-  <joint name="a_tray_on_a_table_joint" type="fixed">
-    <parent link="a_table_top_origin_center" />
-    <child  link="a_tray_on_a_table" />
-    <origin xyz="0 ${-tray_length/2} 0" rpy="0 0 0" />
-  </joint>
-  <link name="b_tray_on_a_table" />
-  <joint name="b_tray_on_a_table_joint" type="fixed">
-    <parent link="a_table_top_origin_center" />
-    <child  link="b_tray_on_a_table" />
-    <origin xyz="0 ${-tray_length/2} 0" rpy="0 0 0" />
-  </joint>
-  <link name="a_table_standpoint"/>
-  <joint name="a_table_standpoint_joint" type="fixed">
-    <parent link="a_table_leg0" />
-    <child  link="a_table_standpoint" />
-    <origin xyz="${a_table_width/2} -0.7 0" rpy="0 0 ${pi/2}" />
-  </joint>
-  <!-- b_table -->
-  <xacro:table prefix="b_table_"
-	       width="${b_table_width}"
-	       length="${b_table_length}"
-	       height="${b_table_height}"
-	       parent="ground">
-    <origin xyz="${-b_table_width/2-(1.0-0.2)}
-		 ${-b_table_length/2+(0.78-0.5)}
-		 0"
-	    rpy="0 0 0"/>
-  </xacro:table>
-  <!-- Frame to place trays on b_table -->
-  <link name="a_tray_on_b_table" />
-  <joint name="a_tray_on_b_table_joint" type="fixed">
-    <parent link="b_table_top_origin_center" />
-    <child  link="a_tray_on_b_table" />
-    <origin xyz="${-tray_width/2 - 0.05} ${-tray_length/2} 0" rpy="0 0 0" />
-  </joint>
-  <link name="b_tray_on_b_table" />
-  <joint name="b_tray_on_b_table_joint" type="fixed">
-    <parent link="b_table_top_origin_center" />
-    <child  link="b_tray_on_b_table" />
-    <origin xyz="${tray_width/2 + 0.05} ${-tray_length/2} 0" rpy="0 0 0" />
-  </joint>
-  <link name="b_table_standpoint"/>
-  <joint name="b_table_standpoint_joint" type="fixed">
-    <parent link="b_table_leg0" />
-    <child  link="b_table_standpoint" />
-    <origin xyz="${b_table_width/2} -0.7 0" rpy="0 0 ${pi/2}" />
-  </joint>
-  <!-- Cabinet -->
-  <xacro:include filename="$(find aist_description)/objects/urdf/cabinet.urdf.xacro"/>
-  <xacro:cabinet prefix="a_"
-		 width="${cabinet_width}"
-		 length="${cabinet_length}"
-		 base_height="${cabinet_base_height}"
-		 shelf1_height="${cabinet_shelf1_height}"
-		 shelf2_height="${cabinet_shelf2_height}"
-		 shelf3_height="${cabinet_shelf3_height}"
-		 shelf4_height="${cabinet_shelf4_height}"
-		 back_height="${cabinet_back_height}" parent="ground">
-    <origin xyz="${workspace_width/2   - cabinet_length}
-		 ${-workspace_length/2 + cabinet_width}
-		 0"
-	    rpy="0 0 ${-pi/2}"/>
-  </xacro:cabinet>
-  <link name="a_cabinet_standpoint"/>
-  <joint name="a_cabinet_standpoint_joint" type="fixed">
-    <parent link="a_cabinet_base" />
-    <child  link="a_cabinet_standpoint" />
-    <origin xyz="${cabinet_width/2} -0.9 0" rpy="0 0 ${pi/2}" />
-  </joint>
-  <!-- Frames to place items on cabinet -->
-  <link name="a_item_in_cabinet"/>
-  <joint name="a_item_in_cabinet_joint" type="fixed">
-    <parent link="a_cabinet_shelf1_origin" />
-    <child  link="a_item_in_cabinet" />
-    <origin xyz="${cabinet_width/12} 0.1 0.08" rpy="${pi/2} ${-pi/2} 0"/>
-  </joint>
-  <link name="b_item_in_cabinet"/>
-  <joint name="b_item_in_cabinet_joint" type="fixed">
-    <parent link="a_item_in_cabinet" />
-    <child  link="b_item_in_cabinet" />
-    <origin xyz="0 ${-cabinet_width/6} 0" rpy="0 0 0" />
-  </joint>
-  <link name="c_item_in_cabinet"/>
-  <joint name="c_item_in_cabinet_joint" type="fixed">
-    <parent link="b_item_in_cabinet" />
-    <child  link="c_item_in_cabinet" />
-    <origin xyz="0 ${-cabinet_width/6} 0" rpy="0 0 0" />
-  </joint>
-  <link name="d_item_in_cabinet"/>
-  <joint name="d_item_in_cabinet_joint" type="fixed">
-    <parent link="c_item_in_cabinet" />
-    <child  link="d_item_in_cabinet" />
-    <origin xyz="0 ${-cabinet_width/6} 0" rpy="0 0 0" />
-  </joint>
-  <link name="e_item_in_cabinet"/>
-  <joint name="e_item_in_cabinet_joint" type="fixed">
-    <parent link="d_item_in_cabinet" />
-    <child  link="e_item_in_cabinet" />
-    <origin xyz="0 ${-cabinet_width/6} 0" rpy="0 0 0" />
-  </joint>
-  <link name="f_item_in_cabinet"/>
-  <joint name="f_item_in_cabinet_joint" type="fixed">
-    <parent link="e_item_in_cabinet" />
-    <child  link="f_item_in_cabinet" />
-    <origin xyz="0 ${-cabinet_width/6} 0" rpy="0 0 0" />
-  </joint>
-  <!-- AR markers -->
-  <xacro:include filename="$(find aist_description)/objects/urdf/ar_markers.urdf.xacro"/>
-  <xacro:ar_marker prefix="a_cabinet_" parent="a_cabinet_shelf1_origin"
-		   marker_id="17" size="0.1" margin="0.005" thickness="0.001">
-    <origin xyz="${cabinet_width - 0.055} 0.055 0.001" rpy="0 0 0"/>
-  </xacro:ar_marker>
-  <xacro:ar_marker prefix="a_table_" parent="a_table_top_origin"
-		   marker_id="26" size="0.1" margin="0.005" thickness="0.001">
-    <origin xyz="0.055 0.055 0.001" rpy="0 0 0"/>
-  </xacro:ar_marker>
-  <!-- Trays -->
-  <xacro:include filename="$(find aist_description)/objects/urdf/tray.urdf.xacro"/>
-  <xacro:tray prefix="a_"
-	      width="${tray_width}"
-	      length="${tray_length}"
-	      height="${tray_height}"
-	      parent="a_tray_on_a_table">
-    <origin xyz="${-tray_width/2} 0 0" rpy="0 0 0"/>
-  </xacro:tray>
-  <xacro:tray prefix="b_"
-	      width="${tray_width}"
-	      length="${tray_length}"
-	      height="${tray_height}"
-	      parent="b_tray_on_b_table">
-    <origin xyz="${-tray_width/2} 0 0" rpy="0 0 0"/>
-  </xacro:tray>
+  <xacro:include filename="$(find aist_description
+			   )/scenes/urdf/ceatec.urdf.xacro"/>
 </robot>

File: aist_description/scenes/urdf/fetch_base_scene.urdf.xacro (robot description, xacro)
@@ -3,13 +3,22 @@
   <xacro:arg name="scene" default=""/>
   <!-- Fetch robot (root = "base_link") -->
-  <xacro:include filename="$(find fetch_gazebo)/robots/fetch.gazebo.xacro"/>
+  <xacro:include filename="$(find fetch_gazebo
+			   )/robots/fetch.gazebo.xacro"/>
+  <!-- Root frame -->
+  <link name="world"/>
+  <!-- Make "map" frame a child of "world" frame -->
   <link  name="map"/>
+  <joint name="map_joint" type="fixed">
+    <parent link="world"/>
+    <child  link="map"/>
+    <origin xyz="0 0 0" rpy="0 0 0"/>
+  </joint>
   <link  name="odom"/>
-  <joint name="map_odom_joint" type="planar">
+  <joint name="odom_joint" type="planar">
     <parent link="map"/>
     <child  link="odom"/>
     <axis   xyz="0 0 1"/>
   </joint>
-  <joint name="odom_base_joint" type="planar">
+  <joint name="base_joint" type="planar">
     <parent link="odom"/>
     <child  link="base_link"/>
@@ -17,6 +26,9 @@
   </joint>
   <!-- Include indivisual scene file -->
-  <xacro:property name="scene_name" value="$(arg scene)"/>
-  <xacro:if value="${scene_name != ''}">
+  <xacro:if value="${'$(arg scene)' != ''}">
+    <joint name="ground_joint" type="fixed">
+      <parent link="world"/>
+      <child  link="ground"/>
+    </joint>
     <xacro:include filename="$(find aist_description)/scenes/urdf/$(arg
 			     scene).urdf.xacro"/>
