Commit message: Add Aurec3Routines and airec3_interactive.py

File: aist_description/scenes/urdf/airec3_base_scene.urdf.xacro (robot description, xacro)
@@ -5,8 +5,25 @@
 					 )/config/products/default.yaml"/>
   <xacro:arg name="sim"		default="true"/>
+  <xacro:arg name="create_srdf"	default="false"/>
   <!-- Torobo robot (root = "world") -->
   <xacro:include filename="$(find torobo_description
 			   )/urdf/load_robot.urdf.xacro"/>
-  <!-- Include indivisual scene file -->
+  <xacro:if value="${'$(arg create_srdf)'}">
+    <joint name="map_joint" type="floating">
+      <parent link="world"/>
+      <child  link="map"/>
+    </joint>
+    <link name="map"/>
+    <joint name="odom_joint" type="floating">
+      <parent link="map"/>
+      <child  link="odom"/>
+    </joint>
+    <link name="odom"/>
+    <joint name="base_footprint_joint2" type="floating">
+      <parent link="odom"/>
+      <child  link="base_footprint"/>
+    </joint>
+  </xacro:if>
+  <!-- Import indivisual scene (root = "ground") -->
   <xacro:if value="${'$(arg scene)' != ''}">
     <joint name="ground_joint" type="fixed">

File: aist_description/scenes/urdf/conveni.urdf.xacro (robot description, xacro)
@@ -27,7 +27,22 @@
   <xacro:include filename="$(find aist_aruco_ros)/urdf/ar_marker.urdf.xacro"/>
   <xacro:ar_marker prefix="a_cabinet_" parent="a_cabinet_shelf2_origin"
-		   marker_id="100_101_102_103" width="0.105" height="0.105"
-		   margin="0.007" thickness="0.001">
-    <origin xyz="${cabinet_width/2} 0.0595 0.001" rpy="0 0 0"/>
+		   marker_id="100_101_102_103" width="0.150" height="0.150"
+		   margin="0.005" thickness="0.001">
+    <origin xyz="${cabinet_width/2} 0.080 0.001" rpy="0 0 0"/>
   </xacro:ar_marker>
+  <!-- Stand points -->
+  <link name="left_standpoint"/>
+  <joint name="left_standpoint_joint" type="fixed">
+    <parent link="ground"/>
+    <child  link="left_standpoint"/>
+    <origin xyz="${cabinet_x - 0.7} ${cabinet_y + cabinet_width/2 + 0.4} 0"
+	    rpy="0 0 ${-pi/6}"/>
+  </joint>
+  <link name="right_standpoint"/>
+  <joint name="right_standpoint_joint" type="fixed">
+    <parent link="ground"/>
+    <child  link="right_standpoint"/>
+    <origin xyz="${cabinet_x - 0.7} ${cabinet_y - cabinet_width/2 - 0.4} 0"
+	    rpy="0 0 ${pi/6}"/>
+  </joint>
 </robot>

File: moveit_config/airec3_moveit_config/config/gazebo_airec3_base_scene.urdf (robot description, URDF)
Before this commit: robot airec3_base_scene, 240 links, 239 joints
Links:
- removed link a_cabinet_standpoint
- added link left_standpoint
- added link right_standpoint
- link a_cabinet_ar_marker: geometry collision box size=0.119 0.119 0.001; visual box size=0.119 0.119 0.001
Joints:
- removed joint a_cabinet_standpoint_joint
- added joint left_standpoint_joint: type fixed, parent ground, child left_standpoint, origin xyz=-0.19999999999999996 0.8625 0 rpy=0 0 -0.5235987755982988
- added joint right_standpoint_joint: type fixed, parent ground, child right_standpoint, origin xyz=-0.19999999999999996 -0.8625 0 rpy=0 0 0.5235987755982988
- joint a_cabinet_ar_marker_joint: origin xyz=0.885 0.040 0.001 rpy=0 0 0 -> xyz=0.4625 0.0595 0.001 rpy=0 0 0; parent a_cabinet_shelf1_origin -> a_cabinet_shelf2_origin
- joint a_cabinet_base: origin xyz=1.3800000000000001    0.42500000000000004    0 rpy=0 0 -1.5707963267948966 -> xyz=0.5 0.4625 0 rpy=0 0 -1.5707963267948966

Commit message: WIP

File: aist_description/scenes/urdf/airec3_base_scene.urdf.xacro (robot description, xacro)
@@ -1,30 +1,51 @@
 <?xml version="1.0"?>
-<robot xmlns:xacro="http://wiki.ros.org/xacro" name="airec3_base_scene" >
+<robot xmlns:xacro="http://wiki.ros.org/xacro" name="torobo" >
   <xacro:arg name="scene"	default=""/>
+  <!-- Torobo robot (root = "base_footprint") -->
   <xacro:arg name="path"	default="$(find torobo_description
 					 )/config/products/default.yaml"/>
   <xacro:arg name="sim"		default="true"/>
-  <xacro:arg name="create_srdf"	default="false"/>
-  <!-- Torobo robot (root = "world") -->
   <xacro:include filename="$(find torobo_description
 			   )/urdf/load_robot.urdf.xacro"/>
-  <xacro:if value="${'$(arg create_srdf)'}">
-    <joint name="map_joint" type="floating">
-      <parent link="world"/>
-      <child  link="map"/>
-    </joint>
-    <link name="map"/>
-    <joint name="odom_joint" type="floating">
-      <parent link="map"/>
-      <child  link="odom"/>
-    </joint>
-    <link name="odom"/>
-    <joint name="base_footprint_joint2" type="floating">
-      <parent link="odom"/>
-      <child  link="base_footprint"/>
-    </joint>
-  </xacro:if>
-  <!-- Import indivisual scene (root = "ground") -->
   <xacro:if value="${'$(arg scene)' != ''}">
+    <!-- <link name="world"/> -->
+    <!-- <joint name="map_joint" type="fixed"> -->
+    <!--   <parent link="world"/> -->
+    <!--   <child  link="map"/> -->
+    <!-- </joint> -->
+    <!-- <link name="map"/> -->
+    <!-- <joint name="odom_joint" type="planar"> -->
+    <!--   <parent link="map"/> -->
+    <!--   <child  link="odom"/> -->
+    <!-- </joint> -->
+    <!-- <link name="odom"/> -->
+    <!-- <joint name="base_footprint_joint" type="planar"> -->
+    <!--   <parent link="odom"/> -->
+    <!--   <child  link="base_footprint"/> -->
+    <!-- </joint> -->
+    <!-- <joint name="base_joint_trans_x" type="prismatic"> -->
+    <!--   <parent link="world"/> -->
+    <!--   <child  link="base_link_trans_x"/> -->
+    <!--   <axis xyz="1 0 0"/> -->
+    <!--   <limit lower="-1e+4" upper="1e+4" -->
+    <!-- 	     effort="600" velocity="10" acceleration="10" jerk="10"/> -->
+    <!-- </joint> -->
+    <!-- <link name="base_link_trans_x"/> -->
+    <!-- <joint name="base_joint_trans_y" type="prismatic"> -->
+    <!--   <parent link="base_link_trans_x"/> -->
+    <!--   <child  link="base_link_trans_y"/> -->
+    <!--   <axis xyz="0 1 0"/> -->
+    <!--   <limit lower="-1e+4" upper="1e+4" -->
+    <!-- 	     effort="600" velocity="10" acceleration="10" jerk="10"/> -->
+    <!-- </joint> -->
+    <!-- <link name="base_link_trans_y"/> -->
+    <!-- <joint name="base_joint_rot_yaw" type="continuous"> -->
+    <!--   <parent link="base_link_trans_y"/> -->
+    <!--   <child  link="base_link_rot_yaw"/> -->
+    <!--   <axis xyz="0 0 1"/> -->
+    <!--   <limit effort="600" velocity="10" acceleration="10" jerk="10"/> -->
+    <!-- </joint> -->
+    <!-- <link name="base_link_rot_yaw"/> -->
+    <!-- Import indivisual scene (root = "ground") -->
     <joint name="ground_joint" type="fixed">
       <parent link="world"/>

File: aist_description/scenes/urdf/conveni.urdf.xacro (robot description, xacro)
@@ -1,4 +1,4 @@
 <?xml version="1.0"?>
-<robot xmlns:xacro="http://wiki.ros.org/xacro" name="ceatec">
+<robot xmlns:xacro="http://wiki.ros.org/xacro" name="conveni">
   <xacro:property name="cabinet_x"		value="0.500"/>
   <xacro:property name="cabinet_y"		value="0.000"/>

Commit message: WIP: Add test launch files for airec3

File: aist_description/scenes/urdf/airec3_base_scene.urdf.xacro (robot description, xacro)
@@ -4,47 +4,51 @@
   <!-- Torobo robot (root = "base_footprint") -->
   <xacro:arg name="path"	default="$(find torobo_description
-					 )/config/products/default.yaml"/>
+					 )/config/products/aist.yaml"/>
   <xacro:arg name="sim"		default="true"/>
   <xacro:include filename="$(find torobo_description
 			   )/urdf/load_robot.urdf.xacro"/>
+  <!-- <link name="world"/> -->
+  <!-- <joint name="map_joint" type="floating"> -->
+  <!--   <parent link="world"/> -->
+  <!--   <child  link="map"/> -->
+  <!-- </joint> -->
+  <!-- <link name="map"/> -->
+  <!-- <joint name="odom_joint" type="planar"> -->
+  <!--   <parent link="map"/> -->
+  <!--   <child  link="odom"/> -->
+  <!-- </joint> -->
+  <!-- <link name="odom"/> -->
+  <!-- <joint name="base_footprint_joint" type="planar"> -->
+  <!--   <parent link="odom"/> -->
+  <!--   <child  link="base_footprint"/> -->
+  <!-- </joint> -->
+  <!-- <joint name="base_joint_trans_x" type="prismatic"> -->
+  <!--   <parent link="world"/> -->
+  <!--   <child  link="base_link_trans_x"/> -->
+  <!--   <axis xyz="1 0 0"/> -->
+  <!--   <limit lower="-1e+4" upper="1e+4" -->
+  <!-- 	   effort="600" velocity="10" acceleration="10" jerk="10"/> -->
+  <!-- </joint> -->
+  <!-- <link name="base_link_trans_x"/> -->
+  <!-- <joint name="base_joint_trans_y" type="prismatic"> -->
+  <!--   <parent link="base_link_trans_x"/> -->
+  <!--   <child  link="base_link_trans_y"/> -->
+  <!--   <axis xyz="0 1 0"/> -->
+  <!--   <limit lower="-1e+4" upper="1e+4" -->
+  <!-- 	   effort="600" velocity="10" acceleration="10" jerk="10"/> -->
+  <!-- </joint> -->
+  <!-- <link name="base_link_trans_y"/> -->
+  <!-- <joint name="base_joint_rot_yaw" type="continuous"> -->
+  <!--   <parent link="base_link_trans_y"/> -->
+  <!--   <child  link="base_link_rot_yaw"/> -->
+  <!--   <axis xyz="0 0 1"/> -->
+  <!--   <limit effort="600" velocity="10" acceleration="10" jerk="10"/> -->
+  <!-- </joint> -->
+  <!-- <link name="base_link_rot_yaw"/> -->
+  <!-- <joint name="base_footprint_joint" type="fixed"> -->
+  <!--   <parent link="base_link_rot_yaw"/> -->
+  <!--   <child  link="base_footprint"/> -->
+  <!-- </joint> -->
   <xacro:if value="${'$(arg scene)' != ''}">
-    <!-- <link name="world"/> -->
-    <!-- <joint name="map_joint" type="fixed"> -->
-    <!--   <parent link="world"/> -->
-    <!--   <child  link="map"/> -->
-    <!-- </joint> -->
-    <!-- <link name="map"/> -->
-    <!-- <joint name="odom_joint" type="planar"> -->
-    <!--   <parent link="map"/> -->
-    <!--   <child  link="odom"/> -->
-    <!-- </joint> -->
-    <!-- <link name="odom"/> -->
-    <!-- <joint name="base_footprint_joint" type="planar"> -->
-    <!--   <parent link="odom"/> -->
-    <!--   <child  link="base_footprint"/> -->
-    <!-- </joint> -->
-    <!-- <joint name="base_joint_trans_x" type="prismatic"> -->
-    <!--   <parent link="world"/> -->
-    <!--   <child  link="base_link_trans_x"/> -->
-    <!--   <axis xyz="1 0 0"/> -->
-    <!--   <limit lower="-1e+4" upper="1e+4" -->
-    <!-- 	     effort="600" velocity="10" acceleration="10" jerk="10"/> -->
-    <!-- </joint> -->
-    <!-- <link name="base_link_trans_x"/> -->
-    <!-- <joint name="base_joint_trans_y" type="prismatic"> -->
-    <!--   <parent link="base_link_trans_x"/> -->
-    <!--   <child  link="base_link_trans_y"/> -->
-    <!--   <axis xyz="0 1 0"/> -->
-    <!--   <limit lower="-1e+4" upper="1e+4" -->
-    <!-- 	     effort="600" velocity="10" acceleration="10" jerk="10"/> -->
-    <!-- </joint> -->
-    <!-- <link name="base_link_trans_y"/> -->
-    <!-- <joint name="base_joint_rot_yaw" type="continuous"> -->
-    <!--   <parent link="base_link_trans_y"/> -->
-    <!--   <child  link="base_link_rot_yaw"/> -->
-    <!--   <axis xyz="0 0 1"/> -->
-    <!--   <limit effort="600" velocity="10" acceleration="10" jerk="10"/> -->
-    <!-- </joint> -->
-    <!-- <link name="base_link_rot_yaw"/> -->
     <!-- Import indivisual scene (root = "ground") -->
     <joint name="ground_joint" type="fixed">

Commit message: Cleanup launch files for airec3

File: aist_description/scenes/urdf/airec3_base_scene.urdf.xacro (robot description, xacro)
@@ -9,22 +9,23 @@
 			   )/urdf/load_robot.urdf.xacro"/>
   <!-- <link name="world"/> -->
-  <!-- <joint name="map_joint" type="floating"> -->
-  <!--   <parent link="world"/> -->
-  <!--   <child  link="map"/> -->
-  <!-- </joint> -->
-  <!-- <link name="map"/> -->
-  <!-- <joint name="odom_joint" type="planar"> -->
+  <joint name="map_joint" type="fixed">
+    <parent link="world"/>
+    <child  link="map"/>
+  </joint>
+  <link name="map"/>
+  <!-- <joint name="odom_joint" type="floating"> -->
   <!--   <parent link="map"/> -->
   <!--   <child  link="odom"/> -->
   <!-- </joint> -->
   <!-- <link name="odom"/> -->
-  <!-- <joint name="base_footprint_joint" type="planar"> -->
+  <!-- <joint name="base_footprint_joint2" type="planar"> -->
   <!--   <parent link="odom"/> -->
   <!--   <child  link="base_footprint"/> -->
+  <!--   <axis   xyz="0 0 1"/> -->
   <!-- </joint> -->
   <!-- <joint name="base_joint_trans_x" type="prismatic"> -->
   <!--   <parent link="world"/> -->
   <!--   <child  link="base_link_trans_x"/> -->
-  <!--   <axis xyz="1 0 0"/> -->
+  <!--   <axis   xyz="1 0 0"/> -->
   <!--   <limit lower="-1e+4" upper="1e+4" -->
   <!-- 	   effort="600" velocity="10" acceleration="10" jerk="10"/> -->
@@ -34,5 +35,5 @@
   <!--   <parent link="base_link_trans_x"/> -->
   <!--   <child  link="base_link_trans_y"/> -->
-  <!--   <axis xyz="0 1 0"/> -->
+  <!--   <axis   xyz="0 1 0"/> -->
   <!--   <limit lower="-1e+4" upper="1e+4" -->
   <!-- 	   effort="600" velocity="10" acceleration="10" jerk="10"/> -->
@@ -42,5 +43,5 @@
   <!--   <parent link="base_link_trans_y"/> -->
   <!--   <child  link="base_link_rot_yaw"/> -->
-  <!--   <axis xyz="0 0 1"/> -->
+  <!--   <axis   xyz="0 0 1"/> -->
   <!--   <limit effort="600" velocity="10" acceleration="10" jerk="10"/> -->
   <!-- </joint> -->
@@ -50,6 +51,6 @@
   <!--   <child  link="base_footprint"/> -->
   <!-- </joint> -->
+  <!-- Import indivisual scene whose root is "ground" -->
   <xacro:if value="${'$(arg scene)' != ''}">
-    <!-- Import indivisual scene (root = "ground") -->
     <joint name="ground_joint" type="fixed">
       <parent link="world"/>
