Commit message: Add URDF model of USB repeater attached to arms

File: aist_description/scenes/urdf/a_bot_base_scene.urdf.xacro (robot description, xacro)
@@ -128,4 +128,11 @@
     <origin xyz="0 0 0" rpy="0 0 0"/>
   </xacro:robotiq_140_gripper>
+  <!-- Add USB repeater -->
+  <xacro:include filename="$(find aist_description
+			   )/objects/urdf/usb_repeater.urdf.xacro"/>
+  <xacro:usb_repeater prefix="a_bot_usb_repeater_"
+		      parent="a_bot_wrist_2_link">
+    <origin xyz="0.000 -0.051 0.000" rpy="${pi/2} ${-pi/2} 0"/>
+  </xacro:usb_repeater>
   <!-- RealSense cameras -->
   <xacro:include filename="$(find aist_description

File: aist_description/scenes/urdf/aist_base_scene.urdf.xacro (robot description, xacro)
@@ -142,5 +142,5 @@
   <!--   <origin xyz="0 0 0" rpy="${pi} 0 0"/> -->
   <!-- </xacro:ft300> -->
-  <!-- Spawn and attach gripper -->
+  <!-- Spawn and attach grippers -->
   <xacro:include filename="$(find aist_robotiq
 			   )/urdf/robotiq_arg2f_coupling.urdf.xacro"/>
@@ -165,21 +165,15 @@
     <origin xyz="0 0 0" rpy="0 0 0"/>
   </xacro:robotiq_85_gripper>
-  <!-- <xacro:include filename="$(find aist_description -->
-  <!-- 			   )/devices/urdf/single_suction_gripper.urdf.xacro"/> -->
-  <!-- <xacro:single_suction_gripper prefix="b_bot_gripper_" -->
-  <!-- 				parent="b_bot_ftsensor_flange_link"> -->
-  <!--   <origin xyz="0 0 0" rpy="0 ${0.3*pi/180} ${0.2*pi/180}"/> -->
-  <!-- </xacro:single_suction_gripper> -->
-  <!-- Add PhoXi 3D scanner -->
-  <!-- <xacro:include filename="$(find aist_description -->
-  <!-- 			   )/scenes/urdf/load_calibration.urdf.xacro"/> -->
-  <!-- <xacro:load_calibration filename="$(find aist_handeye_calibration -->
-  <!-- 				    )/calib/a_phoxi_m_camera.yaml"/> -->
-  <!-- <xacro:include filename="$(find aist_phoxi_camera -->
-  <!-- 			   )/urdf/phoxi_m_camera.urdf.xacro"/> -->
-  <!-- <xacro:phoxi_m_camera name="a_phoxi_m_camera" parent="workspace_center"> -->
-  <!--   <origin xyz="${origin[0]} ${origin[1]} ${origin[2]}" -->
-  <!--   	    rpy="${origin[3]} ${origin[4]} ${origin[5]}"/> -->
-  <!-- </xacro:phoxi_m_camera> -->
+  <!-- Add USB repeaters -->
+  <xacro:include filename="$(find aist_description
+			   )/objects/urdf/usb_repeater.urdf.xacro"/>
+  <xacro:usb_repeater prefix="a_bot_usb_repeater_"
+		      parent="a_bot_wrist_2_link">
+    <origin xyz="0.000 -0.051 0.000" rpy="${pi/2} ${-pi/2} 0"/>
+  </xacro:usb_repeater>
+  <xacro:usb_repeater prefix="b_bot_usb_repeater_"
+		      parent="b_bot_wrist_2_link">
+    <origin xyz="0.000 -0.051 0.000" rpy="${pi/2} ${-pi/2} 0"/>
+  </xacro:usb_repeater>
   <!-- Add Motioncam-3D scanner -->
   <xacro:include filename="$(find aist_description
@@ -193,5 +187,5 @@
     	    rpy="${origin[3]} ${origin[4]} ${origin[5]}"/>
   </xacro:motioncam_m_camera>
-  <!-- RealSense cameras -->
+  <!-- Add RealSense cameras -->
   <xacro:include filename="$(find aist_description
   			   )/devices/urdf/sr305_on_2f140.urdf.xacro" />
@@ -204,5 +198,5 @@
   		       parent="b_bot_gripper_base_link"
   		       use_nominal_extrinsics="true"/>
-  <!-- live camera -->
+  <!-- Add live camera -->
   <xacro:load_calibration filename="$(find aist_camera_calibration
 				    )/calib/live_camera.yaml"/>
@@ -214,5 +208,5 @@
     	    rpy="${origin[3]} ${origin[4]} ${origin[5]}"/>
   </joint>
-  <!-- virtual screen -->
+  <!-- Add virtual screen -->
   <link name="virtual_screen"/>
   <joint name="virtual_screen_joint" type="fixed">

Commit message: Always include assembly scene

File: aist_description/scenes/urdf/a_bot_base_scene.urdf.xacro (robot description, xacro)
@@ -148,5 +148,8 @@
     <origin xyz="0 0 0" rpy="0 0 0"/>
   </joint>
-  <!-- Include indivisual scene file -->
+  <!-- Import assembly scene -->
+  <xacro:include filename="$(find aist_description
+			   )/scenes/urdf/assembly.urdf.xacro"/>
+  <!-- Import indivisual scene -->
   <xacro:if value="${'$(arg scene)' != ''}">
     <xacro:include filename="$(find aist_description)/scenes/urdf/$(arg

File: aist_description/scenes/urdf/aist_base_scene.urdf.xacro (robot description, xacro)
@@ -222,5 +222,8 @@
     <origin xyz="0 0 0" rpy="0 0 0"/>
   </joint>
-  <!-- Include indivisual scene file -->
+  <!-- Import assembly scene -->
+  <xacro:include filename="$(find aist_description
+			   )/scenes/urdf/assembly.urdf.xacro"/>
+  <!-- Import indivisual scene -->
   <xacro:if value="${'$(arg scene)' != ''}">
     <xacro:include filename="$(find aist_description)/scenes/urdf/$(arg

File: aist_description/scenes/urdf/calibration.urdf.xacro (robot description, xacro)
@@ -1,7 +1,4 @@
 <?xml version="1.0"?>
 <robot xmlns:xacro="http://wiki.ros.org/xacro" name="calibration">
-  <!-- import assembly scene -->
-  <!-- <xacro:include filename="$(find aist_description -->
-  <!-- 			   )/scenes/urdf/assembly.urdf.xacro"/> -->
   <!-- Add AR markers -->
   <xacro:include filename="$(find aist_aruco_ros)/urdf/ar_marker.urdf.xacro"/>
@@ -20,10 +17,3 @@
     <origin xyz="0.0 0.0 0.0005" rpy="0 0 0"/>
   </xacro:ar_marker>
-  <!-- <xacro:ar_marker prefix="workspace_" -->
-  <!-- 		   parent="workspace_center" -->
-  <!-- 		   marker_id="6x4" -->
-  <!-- 		   width="0.246" height="0.162" margin="0.006" -->
-  <!-- 		   thickness="0.001"> -->
-  <!--   <origin xyz="0.0 0.0 0.0005" rpy="0 0 0"/> -->
-  <!-- </xacro:ar_marker> -->
 </robot>

File: aist_description/scenes/urdf/kitting.urdf.xacro (robot description, xacro)
@@ -1,7 +1,4 @@
 <?xml version="1.0"?>
 <robot xmlns:xacro="http://wiki.ros.org/xacro" name="kitting">
-  <!-- import assembly scene -->
-  <xacro:include filename="$(find aist_description
-  			   )/scenes/urdf/assembly.urdf.xacro"/>
   <xacro:property name="plate_w" value="0.42"/>
   <xacro:property name="plate_l" value="0.68"/>

Commit message: Separate tables into for workspace and for arms

File: aist_description/scenes/urdf/a_bot_base_scene.urdf.xacro (robot description, xacro)
@@ -6,6 +6,6 @@
   <xacro:property name="a_bot_x"	value="0"/>
   <xacro:property name="a_bot_y"	value="-0.4875"/>
-  <xacro:property name="bots_z"		value="0.770"/>
-  <xacro:property name="screen_z"	value="${bots_z + 0.0347}"/>
+  <xacro:property name="a_bot_z"	value="0.770"/>
+  <xacro:property name="table_h"	value="0.770"/>
   <!-- ground -->
   <link name="ground"/>
@@ -25,5 +25,5 @@
 	      width="${cage_w}" length="${cage_l}" height="${cage_h}"
 	      thickness="${cage_t}"
-	      workspace_height="${bots_z - cage_z}"
+	      workspace_height="${table_h - cage_z}"
 	      tool_bar_height="${tool_bar_h}"
 	      camera_bar_height="${camera_bar_h}"
@@ -36,9 +36,9 @@
   <!-- workspace -->
   <xacro:property name="table_w"	value="0.900"/>
-  <xacro:property name="table_l"	value="1.800"/>
+  <xacro:property name="table_l"	value="0.700"/>
   <xacro:include filename="$(find aist_description
 			   )/objects/urdf/table.urdf.xacro"/>
   <xacro:table prefix="workspace_table_"
-	       width="${table_w}" length="${table_l}" height="${bots_z}"
+	       width="${table_w}" length="${table_l}" height="${table_h}"
 	       parent="ground">
     <origin xyz="${-cage_w/2 + cage_offset_x + cage_t} ${-table_l/2} 0"
@@ -46,9 +46,17 @@
   </xacro:table>
   <link name="workspace_center"/>
-  <joint name="ground_to_workspace" type="fixed">
+  <joint name="workspace_joint" type="fixed">
     <parent link="ground"/>
     <child  link="workspace_center"/>
-    <origin xyz="0 0 ${bots_z}" rpy="0 0 0"/>
+    <origin xyz="0 0 ${table_h}" rpy="0 0 0"/>
   </joint>
+  <!-- tables for mounting robot arms -->
+  <xacro:property name="bot_table_size"	value="0.275"/>
+  <xacro:table prefix="a_bot_table_"
+	       width="${bot_table_size}" length="${bot_table_size}"
+	       height="${a_bot_z}" parent="ground">
+    <origin xyz="${a_bot_x - bot_table_size/2} ${a_bot_y - bot_table_size/2} 0"
+	    rpy="0 0 0"/>
+  </xacro:table>
   <!-- tool holders -->
   <xacro:property name="precision_tool_holder_y"	value="0.60"/>
@@ -93,26 +101,9 @@
       safety_limits="true"
       safety_pos_margin="0.3"/>
-  <joint name="ground_a_bot_joint" type="fixed">
-    <parent link="ground"/>
+  <joint name="a_bot_base_link_joint" type="fixed">
+    <parent link="a_bot_table_top_center"/>
     <child  link="a_bot_base_link"/>
-    <origin xyz="${a_bot_x} ${a_bot_y} ${bots_z}" rpy="0 0 0"/>
+    <origin xyz="0 0 0 " rpy="0 0 0"/>
   </joint>
-  <!-- Attach mounter for Zivid2+ camera -->
-  <!-- <xacro:include filename="$(find aist_description)/devices/urdf/zivid_coupling.urdf.xacro"/> -->
-  <!-- <xacro:zivid_coupling prefix="a_bot_zivid_coupling_" parent="a_bot_flange"> -->
-  <!--   <origin xyz="0 0 0" rpy="${pi} 0 0" /> -->
-  <!-- </xacro:zivid_coupling> -->
-  <!-- <!-\- Spawn and attach Zivid2+ camera -\-> -->
-  <!-- <xacro:include filename="$(find aist_description -->
-  <!-- 			   )/scenes/urdf/load_calibration.urdf.xacro"/> -->
-  <!-- <xacro:load_calibration filename="$(find aist_handeye_calibration -->
-  <!-- 				    )/calib/a_bot_zivid.yaml"/> -->
-  <!-- <xacro:include filename="$(find aist_description -->
-  <!-- 			   )/devices/urdf/zivid2plus.urdf.xacro"/> -->
-  <!-- <xacro:zivid2plus name="a_bot_zivid" -->
-  <!-- 		    parent="a_bot_zivid_coupling_flange_link"> -->
-  <!--   <origin xyz="${origin[0]} ${origin[1]} ${origin[2]}" -->
-  <!--   	    rpy="${origin[3]} ${origin[4]} ${origin[5]}"/> -->
-  <!-- </xacro:zivid2plus> -->
   <!-- Spawn and attach gripper -->
   <xacro:include filename="$(find aist_robotiq
@@ -143,5 +134,5 @@
   <!-- I would like to remove the "world" link definition, but apparently it is necessary for Gazebo -->
   <link name="world"/>
-  <joint name="world_ground_joint" type="fixed">
+  <joint name="ground_joint" type="fixed">
     <parent link="world"/>
     <child  link="ground"/>

File: aist_description/scenes/urdf/aist_base_scene.urdf.xacro (robot description, xacro)
@@ -39,5 +39,5 @@
   <!-- workspace -->
   <xacro:property name="table_w"	value="0.900"/>
-  <xacro:property name="table_l"	value="1.800"/>
+  <xacro:property name="table_l"	value="0.700"/>
   <xacro:include filename="$(find aist_description
 			   )/objects/urdf/table.urdf.xacro"/>
@@ -49,9 +49,23 @@
   </xacro:table>
   <link name="workspace_center"/>
-  <joint name="ground_to_workspace" type="fixed">
+  <joint name="workspace_joint" type="fixed">
     <parent link="ground"/>
     <child  link="workspace_center"/>
     <origin xyz="0 0 ${table_h}" rpy="0 0 0"/>
   </joint>
+  <!-- tables for mounting robot arms -->
+  <xacro:property name="bot_table_size"	value="0.275"/>
+  <xacro:table prefix="a_bot_table_"
+	       width="${bot_table_size}" length="${bot_table_size}"
+	       height="${a_bot_z}" parent="ground">
+    <origin xyz="${a_bot_x - bot_table_size/2} ${a_bot_y - bot_table_size/2} 0"
+	    rpy="0 0 0"/>
+  </xacro:table>
+  <xacro:table prefix="b_bot_table_"
+	       width="${bot_table_size}" length="${bot_table_size}"
+	       height="${b_bot_z}" parent="ground">
+    <origin xyz="${b_bot_x - bot_table_size/2} ${b_bot_y - bot_table_size/2} 0"
+	    rpy="0 0 0"/>
+  </xacro:table>
   <!-- tool holders -->
   <xacro:property name="precision_tool_holder_y"	value="0.60"/>
@@ -109,13 +123,13 @@
       safety_limits="true"
       safety_pos_margin="0.15"/>
-  <joint name="ground_a_bot_joint" type="fixed">
-    <parent link="ground"/>
+  <joint name="a_bot_base_link_joint" type="fixed">
+    <parent link="a_bot_table_top_center"/>
     <child  link="a_bot_base_link"/>
-    <origin xyz="${a_bot_x} ${a_bot_y} ${a_bot_z}" rpy="0 0 0"/>
-  </joint>
-  <joint name="ground_b_bot_joint" type="fixed">
-    <parent link="ground"/>
+    <origin xyz="0 0 0 " rpy="0 0 0"/>
+  </joint>
+  <joint name="b_bot_base_link_joint" type="fixed">
+    <parent link="b_bot_table_top_center"/>
     <child  link="b_bot_base_link"/>
-    <origin xyz="${b_bot_x} ${b_bot_y} ${b_bot_z}" rpy="0 0 ${b_bot_theta}"/>
+    <origin xyz="0 0 0" rpy="0 0 ${b_bot_theta}"/>
   </joint>
   <!-- Attach mounter for Zivid2+ camera -->
@@ -204,5 +218,5 @@
 				    )/calib/live_camera.yaml"/>
   <link name="live_camera_optical_frame"/>
-  <joint name="workspace_live_camera_joint" type="fixed">
+  <joint name="live_camera_joint" type="fixed">
     <parent link="workspace_center"/>
     <child  link="live_camera_optical_frame"/>
@@ -219,5 +233,5 @@
   <!-- I would like to remove the "world" link definition, but apparently it is necessary for Gazebo -->
   <link name="world"/>
-  <joint name="world_ground_joint" type="fixed">
+  <joint name="ground_joint" type="fixed">
     <parent link="world"/>
     <child  link="ground"/>

File: aist_description/scenes/urdf/b_bot_base_scene.urdf.xacro (robot description, xacro)
@@ -4,7 +4,8 @@
   <xacro:property name="b_bot_x"	value="0"/>
   <xacro:property name="b_bot_y"	value="0.4875"/>
+  <xacro:property name="b_bot_z"	value="0.770"/>
   <xacro:property name="b_bot_theta"	value="${pi}"/>
-  <xacro:property name="bots_z"		value="0.770"/>
-  <xacro:property name="screen_z"	value="${bots_z + 0.0347}"/>
+  <xacro:property name="table_h"	value="0.770"/>
+  <xacro:property name="screen_z"	value="0.048"/>
   <!-- ground -->
   <link name="ground"/>
@@ -24,5 +25,5 @@
 	      width="${cage_w}" length="${cage_l}" height="${cage_h}"
 	      thickness="${cage_t}"
-	      workspace_height="${bots_z - cage_z}"
+	      workspace_height="${table_h - cage_z}"
 	      tool_bar_height="${tool_bar_h}"
 	      camera_bar_height="${camera_bar_h}"
@@ -35,9 +36,9 @@
   <!-- workspace -->
   <xacro:property name="table_w"	value="0.900"/>
-  <xacro:property name="table_l"	value="1.800"/>
+  <xacro:property name="table_l"	value="0.700"/>
   <xacro:include filename="$(find aist_description
 			   )/objects/urdf/table.urdf.xacro"/>
   <xacro:table prefix="workspace_table_"
-	       width="${table_w}" length="${table_l}" height="${bots_z}"
+	       width="${table_w}" length="${table_l}" height="${table_h}"
 	       parent="ground">
     <origin xyz="${-cage_w/2 + cage_offset_x + cage_t} ${-table_l/2} 0"
@@ -45,9 +46,17 @@
   </xacro:table>
   <link name="workspace_center"/>
-  <joint name="ground_to_workspace" type="fixed">
+  <joint name="workspace_joint" type="fixed">
     <parent link="ground"/>
     <child  link="workspace_center"/>
-    <origin xyz="0 0 ${bots_z}" rpy="0 0 0"/>
+    <origin xyz="0 0 ${table_h}" rpy="0 0 0"/>
   </joint>
+  <!-- tables for mounting robot arms -->
+  <xacro:property name="bot_table_size"	value="0.275"/>
+  <xacro:table prefix="b_bot_table_"
+	       width="${bot_table_size}" length="${bot_table_size}"
+	       height="${b_bot_z}" parent="ground">
+    <origin xyz="${b_bot_x - bot_table_size/2} ${b_bot_y - bot_table_size/2} 0"
+	    rpy="0 0 0"/>
+  </xacro:table>
   <!-- tool holders -->
   <xacro:property name="screw_tool_m3_holder_y"	value="0.75"/>
@@ -85,8 +94,8 @@
       safety_limits="true"
       safety_pos_margin="0.3"/>
-  <joint name="ground_b_bot_joint" type="fixed">
-    <parent link="ground"/>
+  <joint name="b_bot_base_link_joint" type="fixed">
+    <parent link="b_bot_table_top_center"/>
     <child  link="b_bot_base_link"/>
-    <origin xyz="${b_bot_x} ${b_bot_y} ${bots_z}" rpy="0 0 ${b_bot_theta}"/>
+    <origin xyz="0 0 0 " rpy="0 0 ${b_bot_theta}"/>
   </joint>
   <!-- Spawn and attach force sensor -->
@@ -114,9 +123,9 @@
     	    rpy="${origin[3]} ${origin[4]} ${origin[5]}"/>
   </xacro:phoxi_m_camera>
-  <!-- live camera -->
+  <!-- Add live camera -->
   <xacro:load_calibration filename="$(find aist_camera_calibration
 				    )/calib/live_camera.yaml"/>
   <link name="live_camera_optical_frame"/>
-  <joint name="workspace_live_camera_joint" type="fixed">
+  <joint name="live_camera_joint" type="fixed">
     <parent link="workspace_center"/>
     <child  link="live_camera_optical_frame"/>
@@ -124,8 +133,8 @@
     	    rpy="${origin[3]} ${origin[4]} ${origin[5]}"/>
   </joint>
-  <!-- virtual screen -->
+  <!-- Add virtual screen -->
   <link name="virtual_screen"/>
   <joint name="virtual_screen_joint" type="fixed">
-    <parent link="ground"/>
+    <parent link="workspace_center"/>
     <child  link="virtual_screen"/>
     <origin xyz="0 0 ${screen_z}" rpy="0 0 0"/>
@@ -133,5 +142,5 @@
   <!-- I would like to remove the "world" link definition, but apparently it is necessary for Gazebo -->
   <link name="world"/>
-  <joint name="world_ground_joint" type="fixed">
+  <joint name="ground_joint" type="fixed">
     <parent link="world"/>
     <child  link="ground"/>
