Commit message: Separate tables into for workspace and for arms

File: moveit_config/aist_moveit_config/config/gazebo_aist_base_scene.urdf (robot description, URDF)
Before this commit: robot aist_base_scene, 242 links, 241 joints
Links:
- removed link bin_1_part_16
- removed link bin_1_part_16_bottom_back_left_corner
- removed link bin_1_part_16_bottom_back_right_corner
- removed link bin_1_part_16_bottom_front_left_corner
- removed link bin_1_part_16_bottom_front_right_corner
- removed link bin_1_part_16_top_back_left_corner
- removed link bin_1_part_16_top_back_right_corner
- removed link bin_1_part_16_top_front_left_corner
- removed link bin_1_part_16_top_front_right_corner
- removed link bin_1_part_17
- removed link bin_1_part_17_bottom_back_left_corner
- removed link bin_1_part_17_bottom_back_right_corner
- removed link bin_1_part_17_bottom_front_left_corner
- removed link bin_1_part_17_bottom_front_right_corner
- removed link bin_1_part_17_top_back_left_corner
- removed link bin_1_part_17_top_back_right_corner
- removed link bin_1_part_17_top_front_left_corner
- removed link bin_1_part_17_top_front_right_corner
- removed link bin_1_part_5
- removed link bin_1_part_5_bottom_back_left_corner
- removed link bin_1_part_5_bottom_back_right_corner
- removed link bin_1_part_5_bottom_front_left_corner
- removed link bin_1_part_5_bottom_front_right_corner
- removed link bin_1_part_5_top_back_left_corner
- removed link bin_1_part_5_top_back_right_corner
- removed link bin_1_part_5_top_front_left_corner
- removed link bin_1_part_5_top_front_right_corner
- removed link bin_2_part_4
- removed link bin_2_part_4_bottom_back_left_corner
- removed link bin_2_part_4_bottom_back_right_corner
- removed link bin_2_part_4_bottom_front_left_corner
- removed link bin_2_part_4_bottom_front_right_corner
- removed link bin_2_part_4_top_back_left_corner
- removed link bin_2_part_4_top_back_right_corner
- removed link bin_2_part_4_top_front_left_corner
- removed link bin_2_part_4_top_front_right_corner
- removed link bin_2_part_7
- removed link bin_2_part_7_bottom_back_left_corner
- removed link bin_2_part_7_bottom_back_right_corner
- removed link bin_2_part_7_bottom_front_left_corner
- removed link bin_2_part_7_bottom_front_right_corner
- removed link bin_2_part_7_top_back_left_corner
- removed link bin_2_part_7_top_back_right_corner
- removed link bin_2_part_7_top_front_left_corner
- removed link bin_2_part_7_top_front_right_corner
- removed link bin_2_part_8
- removed link bin_2_part_8_bottom_back_left_corner
- removed link bin_2_part_8_bottom_back_right_corner
- removed link bin_2_part_8_bottom_front_left_corner
- removed link bin_2_part_8_bottom_front_right_corner
- removed link bin_2_part_8_top_back_left_corner
- removed link bin_2_part_8_top_back_right_corner
- removed link bin_2_part_8_top_front_left_corner
- removed link bin_2_part_8_top_front_right_corner
- removed link plate
- removed link plate_lower_left_corner
- removed link screw_feeder_m3_front_side
- removed link screw_feeder_m4_front_side
- removed link tray_2
- removed link tray_2_divider2
- removed link tray_2_partition_1
- removed link tray_2_partition_1_pickup
- removed link tray_2_partition_2
- removed link tray_2_partition_2_pickup
- removed link tray_2_partition_3
- removed link tray_2_partition_3_pickup
- removed link tray_2_partition_4
- removed link tray_2_partition_4_pickup
- removed link tray_2_partition_5
- removed link tray_2_partition_5_pickup
- removed link tray_2_partition_6
- removed link tray_2_partition_6_pickup
- removed link tray_2_partition_7
- removed link tray_2_partition_7_pickup
- removed link tray_2_partition_8
- removed link tray_2_partition_8_pickup_1
- removed link tray_2_partition_8_pickup_2
- removed link tray_2_screw_holder
- removed link tray_2_screw_m3_1
- removed link tray_2_screw_m3_2
- removed link tray_2_screw_m3_3
- removed link tray_2_screw_m3_4
- removed link tray_2_screw_m3_5
- removed link tray_2_screw_m3_6
- removed link tray_2_screw_m4_1
- removed link tray_2_screw_m4_2
- removed link tray_2_screw_m4_3
- removed link tray_2_screw_m4_4
- removed link tray_2_screw_m4_5
- removed link tray_2_screw_m4_6
- removed link tray_2_screw_m4_7
- removed link tray_2_screw_m4_8
- removed link tray_2_screw_m4_9
- added link a_bot_table_base_link, mass 1.0; collision box size=0.05 0.05 0.75; visual box size=0.05 0.05 0.75
- added link a_bot_table_leg1, mass 1.0; collision box size=0.05 0.05 0.75; visual box size=0.05 0.05 0.75
- added link a_bot_table_leg2, mass 1.0; collision box size=0.05 0.05 0.75; visual box size=0.05 0.05 0.75
- added link a_bot_table_leg3, mass 1.0; collision box size=0.05 0.05 0.75; visual box size=0.05 0.05 0.75
- added link a_bot_table_top, mass 1.0; collision box size=0.275 0.275 0.02; visual box size=0.275 0.275 0.02
- added link a_bot_table_top_center
- added link a_bot_table_top_origin
- added link b_bot_table_base_link, mass 1.0; collision box size=0.05 0.05 0.75; visual box size=0.05 0.05 0.75
- added link b_bot_table_leg1, mass 1.0; collision box size=0.05 0.05 0.75; visual box size=0.05 0.05 0.75
- added link b_bot_table_leg2, mass 1.0; collision box size=0.05 0.05 0.75; visual box size=0.05 0.05 0.75
- added link b_bot_table_leg3, mass 1.0; collision box size=0.05 0.05 0.75; visual box size=0.05 0.05 0.75
- added link b_bot_table_top, mass 1.0; collision box size=0.275 0.275 0.02; visual box size=0.275 0.275 0.02
- added link b_bot_table_top_center
- added link b_bot_table_top_origin
- added link base_fixture_head_base_link, mass 0.1; collision mesh filename=package://aist_description/objects/meshes/base_fixture_head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 scale=0.001 0.001 0.001; visual mesh filename=package://aist_description/objects/meshes/base_fixture_head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 scale=0.001 0.001 0.001
- added link base_fixture_head_tip_link
- added link screw_feeder_m3_front_left_side, mass 1.0; collision box size=0.056 0.055 0.081; visual box size=0.056 0.055 0.081
- added link screw_feeder_m3_front_right_side, mass 1.0; collision box size=0.056 0.04 0.081; visual box size=0.056 0.04 0.081
- added link screw_feeder_m4_front_left_side, mass 1.0; collision box size=0.056 0.055 0.081; visual box size=0.056 0.055 0.081
- added link screw_feeder_m4_front_right_side, mass 1.0; collision box size=0.056 0.04 0.081; visual box size=0.056 0.04 0.081
- link screw_feeder_m3_gap: geometry collision box size=0.056 0.031000000000000007 0.069; visual box size=0.056 0.031000000000000007 0.069
- link screw_feeder_m4_gap: geometry collision box size=0.056 0.031000000000000007 0.069; visual box size=0.056 0.031000000000000007 0.069
- link workbench_front_border: geometry collision box size=0.082 0.018 0.005; visual box size=0.082 0.018 0.005
- link workbench_right_border: geometry collision box size=0.018 0.075 0.005; visual box size=0.018 0.075 0.005
- link workspace_table_top: geometry collision box size=0.9 0.7 0.02; visual box size=0.9 0.7 0.02
Joints:
- removed joint bin_1_part_16
- removed joint bin_1_part_16_bottom_back_left_corner_joint
- removed joint bin_1_part_16_bottom_back_right_corner_joint
- removed joint bin_1_part_16_bottom_front_left_corner_joint
- removed joint bin_1_part_16_bottom_front_right_corner_joint
- removed joint bin_1_part_16_top_back_left_corner_joint
- removed joint bin_1_part_16_top_back_right_corner_joint
- removed joint bin_1_part_16_top_front_left_corner_joint
- removed joint bin_1_part_16_top_front_right_corner_joint
- removed joint bin_1_part_17
- removed joint bin_1_part_17_bottom_back_left_corner_joint
- removed joint bin_1_part_17_bottom_back_right_corner_joint
- removed joint bin_1_part_17_bottom_front_left_corner_joint
- removed joint bin_1_part_17_bottom_front_right_corner_joint
- removed joint bin_1_part_17_top_back_left_corner_joint
- removed joint bin_1_part_17_top_back_right_corner_joint
- removed joint bin_1_part_17_top_front_left_corner_joint
- removed joint bin_1_part_17_top_front_right_corner_joint
- removed joint bin_1_part_5
- removed joint bin_1_part_5_bottom_back_left_corner_joint
- removed joint bin_1_part_5_bottom_back_right_corner_joint
- removed joint bin_1_part_5_bottom_front_left_corner_joint
- removed joint bin_1_part_5_bottom_front_right_corner_joint
- removed joint bin_1_part_5_top_back_left_corner_joint
- removed joint bin_1_part_5_top_back_right_corner_joint
- removed joint bin_1_part_5_top_front_left_corner_joint
- removed joint bin_1_part_5_top_front_right_corner_joint
- removed joint bin_2_part_4
- removed joint bin_2_part_4_bottom_back_left_corner_joint
- removed joint bin_2_part_4_bottom_back_right_corner_joint
- removed joint bin_2_part_4_bottom_front_left_corner_joint
- removed joint bin_2_part_4_bottom_front_right_corner_joint
- removed joint bin_2_part_4_top_back_left_corner_joint
- removed joint bin_2_part_4_top_back_right_corner_joint
- removed joint bin_2_part_4_top_front_left_corner_joint
- removed joint bin_2_part_4_top_front_right_corner_joint
- removed joint bin_2_part_7
- removed joint bin_2_part_7_bottom_back_left_corner_joint
- removed joint bin_2_part_7_bottom_back_right_corner_joint
- removed joint bin_2_part_7_bottom_front_left_corner_joint
- removed joint bin_2_part_7_bottom_front_right_corner_joint
- removed joint bin_2_part_7_top_back_left_corner_joint
- removed joint bin_2_part_7_top_back_right_corner_joint
- removed joint bin_2_part_7_top_front_left_corner_joint
- removed joint bin_2_part_7_top_front_right_corner_joint
- removed joint bin_2_part_8
- removed joint bin_2_part_8_bottom_back_left_corner_joint
- removed joint bin_2_part_8_bottom_back_right_corner_joint
- removed joint bin_2_part_8_bottom_front_left_corner_joint
- removed joint bin_2_part_8_bottom_front_right_corner_joint
- removed joint bin_2_part_8_top_back_left_corner_joint
- removed joint bin_2_part_8_top_back_right_corner_joint
- removed joint bin_2_part_8_top_front_left_corner_joint
- removed joint bin_2_part_8_top_front_right_corner_joint
- removed joint ground_a_bot_joint
- removed joint ground_b_bot_joint
- removed joint plate
- removed joint plate_corner_joint
- removed joint screw_feeder_m3_front_side
- removed joint screw_feeder_m4_front_side
- removed joint tray_2
- removed joint tray_2_divider2_joint
- removed joint tray_2_partition_1
- removed joint tray_2_partition_1_pickup
- removed joint tray_2_partition_2
- removed joint tray_2_partition_2_pickup
- removed joint tray_2_partition_3
- removed joint tray_2_partition_3_pickup
- removed joint tray_2_partition_4
- removed joint tray_2_partition_4_pickup
- removed joint tray_2_partition_5
- removed joint tray_2_partition_5_pickup
- removed joint tray_2_partition_6
- removed joint tray_2_partition_6_pickup
- removed joint tray_2_partition_7
- removed joint tray_2_partition_7_pickup
- removed joint tray_2_partition_8
- removed joint tray_2_partition_8_pickup_1
- removed joint tray_2_partition_8_pickup_2
- removed joint tray_2_screw_holder_joint
- removed joint tray_2_screw_m3_1
- removed joint tray_2_screw_m3_2
- removed joint tray_2_screw_m3_3
- removed joint tray_2_screw_m3_4
- removed joint tray_2_screw_m3_5
- removed joint tray_2_screw_m3_6
- removed joint tray_2_screw_m4_1
- removed joint tray_2_screw_m4_2
- removed joint tray_2_screw_m4_3
- removed joint tray_2_screw_m4_4
- removed joint tray_2_screw_m4_5
- removed joint tray_2_screw_m4_6
- removed joint tray_2_screw_m4_7
- removed joint tray_2_screw_m4_8
- removed joint tray_2_screw_m4_9
- added joint a_bot_base_link_joint: type fixed, parent a_bot_table_top_center, child a_bot_base_link, origin xyz=0 0 0  rpy=0 0 0
- added joint a_bot_table_base_link: type fixed, parent ground, child a_bot_table_base_link, origin xyz=-0.1375 -0.625 0 rpy=0 0 0
- added joint a_bot_table_leg1: type fixed, parent a_bot_table_base_link, child a_bot_table_leg1, origin xyz=0.22500000000000003 0 0 rpy=0 0 0
- added joint a_bot_table_leg2: type fixed, parent a_bot_table_base_link, child a_bot_table_leg2, origin xyz=0 0.22500000000000003 0 rpy=0 0 0
- added joint a_bot_table_leg3: type fixed, parent a_bot_table_base_link, child a_bot_table_leg3, origin xyz=0.22500000000000003      0.22500000000000003      0 rpy=0 0 0
- added joint a_bot_table_top: type fixed, parent a_bot_table_base_link, child a_bot_table_top, origin xyz=0 0 0.75 rpy=0 0 0
- added joint a_bot_table_top_center_joint: type fixed, parent a_bot_table_top_origin, child a_bot_table_top_center, origin xyz=0.1375 0.1375 0 rpy=0 0 0
- added joint a_bot_table_top_origin_joint: type fixed, parent a_bot_table_top, child a_bot_table_top_origin, origin xyz=0 0 0.02 rpy=0 0 0
- added joint b_bot_base_link_joint: type fixed, parent b_bot_table_top_center, child b_bot_base_link, origin xyz=0 0 0 rpy=0 0 3.141592653589793
- added joint b_bot_table_base_link: type fixed, parent ground, child b_bot_table_base_link, origin xyz=-0.1375 0.35 0 rpy=0 0 0
- added joint b_bot_table_leg1: type fixed, parent b_bot_table_base_link, child b_bot_table_leg1, origin xyz=0.22500000000000003 0 0 rpy=0 0 0
- added joint b_bot_table_leg2: type fixed, parent b_bot_table_base_link, child b_bot_table_leg2, origin xyz=0 0.22500000000000003 0 rpy=0 0 0
- added joint b_bot_table_leg3: type fixed, parent b_bot_table_base_link, child b_bot_table_leg3, origin xyz=0.22500000000000003      0.22500000000000003      0 rpy=0 0 0
- added joint b_bot_table_top: type fixed, parent b_bot_table_base_link, child b_bot_table_top, origin xyz=0 0 0.75 rpy=0 0 0
- added joint b_bot_table_top_center_joint: type fixed, parent b_bot_table_top_origin, child b_bot_table_top_center, origin xyz=0.1375 0.1375 0 rpy=0 0 0
- added joint b_bot_table_top_origin_joint: type fixed, parent b_bot_table_top, child b_bot_table_top_origin, origin xyz=0 0 0.02 rpy=0 0 0
- added joint base_fixture_head_base_joint: type fixed, parent base_fixture_piston_head, child base_fixture_head_base_link, origin xyz=0 0 0 rpy=0 0 0
- added joint base_fixture_head_tip_joint: type fixed, parent base_fixture_head_base_link, child base_fixture_head_tip_link, origin xyz=0.007 0.0 -0.013 rpy=0 0 -0.5404220042582721
- added joint screw_feeder_m3_front_left_side: type fixed, parent screw_feeder_m3_base_link, child screw_feeder_m3_front_left_side, origin xyz=0.126 0 0 rpy=0 0 0
- added joint screw_feeder_m3_front_right_side: type fixed, parent screw_feeder_m3_base_link, child screw_feeder_m3_front_right_side, origin xyz=0.126 0.08600000000000001 0 rpy=0 0 0
- added joint screw_feeder_m4_front_left_side: type fixed, parent screw_feeder_m4_base_link, child screw_feeder_m4_front_left_side, origin xyz=0.126 0 0 rpy=0 0 0
- added joint screw_feeder_m4_front_right_side: type fixed, parent screw_feeder_m4_base_link, child screw_feeder_m4_front_right_side, origin xyz=0.126 0.08600000000000001 0 rpy=0 0 0
- joint base_fixture_base_joint: origin xyz=0.05729961772434791 0.24786931916155724 0 rpy=0 0 -1.0304423903774522 -> xyz=0.05399264856003658 0.24801225239993904 0 rpy=0 0 -1.0303768265243125
- joint screw_feeder_m3_base_link: origin xyz=0.01 0.03 0 rpy=0 0 0 -> xyz=0.014 0.034 0 rpy=0 0 0
- joint screw_feeder_m3_gap: origin xyz=0 0.053 0.079 rpy=0 0 0 -> xyz=0 0.055 0 rpy=0 0 0; parent screw_feeder_m3_front_side -> screw_feeder_m3_front_left_side
- joint screw_feeder_m3_outlet_joint: origin xyz=0.046 0.01 0.002 rpy=0 0 0 -> xyz=0.046 0.008 0.069 rpy=0 0 0
- joint screw_feeder_m4_base_link: origin xyz=0 0.126 0 rpy=0 0 0 -> xyz=0 0.1268 0 rpy=0 0 0
- joint screw_feeder_m4_gap: origin xyz=0 0.053 0.079 rpy=0 0 0 -> xyz=0 0.055 0 rpy=0 0 0; parent screw_feeder_m4_front_side -> screw_feeder_m4_front_left_side
- joint screw_feeder_m4_outlet_joint: origin xyz=0.046 0.01 0.002 rpy=0 0 0 -> xyz=0.046 0.008 0.069 rpy=0 0 0
- joint virtual_screen_joint: origin xyz=0 0 0.8180000000000001 rpy=0 0 0 -> xyz=0 0 0.048 rpy=0 0 0; parent ground -> workspace_center
- joint workbench_front_border: origin xyz=0.13 0 0 rpy=0 0 0 -> xyz=0.128 0 0 rpy=0 0 0
- joint workbench_holder_link_joint: origin xyz=0.194 0.016 0 rpy=0 0 1.5707963267948966 -> xyz=0.192 0.018 0 rpy=0 0 1.5707963267948966
- joint workbench_right_border: origin xyz=0.194 0.016 0 rpy=0 0 0 -> xyz=0.192 0.018 0 rpy=0 0 0
- joint workspace_table_base_link: origin xyz=-0.5449999999999999 -0.9 0 rpy=0 0 0 -> xyz=-0.5449999999999999 -0.35 0 rpy=0 0 0
- joint workspace_table_leg2: origin xyz=0 1.75 0 rpy=0 0 0 -> xyz=0 0.6499999999999999 0 rpy=0 0 0
- joint workspace_table_leg3: origin xyz=0.85      1.75      0 rpy=0 0 0 -> xyz=0.85      0.6499999999999999      0 rpy=0 0 0
- joint workspace_table_top_center_joint: origin xyz=0.45 0.9 0 rpy=0 0 0 -> xyz=0.45 0.35 0 rpy=0 0 0

Commit message: Change table size

File: aist_description/scenes/urdf/a_bot_base_scene.urdf.xacro (robot description, xacro)
@@ -36,5 +36,5 @@
   <!-- workspace -->
   <xacro:property name="table_w"	value="0.900"/>
-  <xacro:property name="table_l"	value="0.700"/>
+  <xacro:property name="table_l"	value="0.750"/>
   <xacro:include filename="$(find aist_description
 			   )/objects/urdf/table.urdf.xacro"/>
@@ -52,5 +52,5 @@
   </joint>
   <!-- tables for mounting robot arms -->
-  <xacro:property name="bot_table_size"	value="0.275"/>
+  <xacro:property name="bot_table_size"	value="0.225"/>
   <xacro:table prefix="a_bot_table_"
 	       width="${bot_table_size}" length="${bot_table_size}"

File: aist_description/scenes/urdf/aist_base_scene.urdf.xacro (robot description, xacro)
@@ -39,5 +39,5 @@
   <!-- workspace -->
   <xacro:property name="table_w"	value="0.900"/>
-  <xacro:property name="table_l"	value="0.700"/>
+  <xacro:property name="table_l"	value="0.750"/>
   <xacro:include filename="$(find aist_description
 			   )/objects/urdf/table.urdf.xacro"/>
@@ -55,5 +55,5 @@
   </joint>
   <!-- tables for mounting robot arms -->
-  <xacro:property name="bot_table_size"	value="0.275"/>
+  <xacro:property name="bot_table_size"	value="0.225"/>
   <xacro:table prefix="a_bot_table_"
 	       width="${bot_table_size}" length="${bot_table_size}"

File: aist_description/scenes/urdf/b_bot_base_scene.urdf.xacro (robot description, xacro)
@@ -36,5 +36,5 @@
   <!-- workspace -->
   <xacro:property name="table_w"	value="0.900"/>
-  <xacro:property name="table_l"	value="0.700"/>
+  <xacro:property name="table_l"	value="0.750"/>
   <xacro:include filename="$(find aist_description
 			   )/objects/urdf/table.urdf.xacro"/>
@@ -52,5 +52,5 @@
   </joint>
   <!-- tables for mounting robot arms -->
-  <xacro:property name="bot_table_size"	value="0.275"/>
+  <xacro:property name="bot_table_size"	value="0.225"/>
   <xacro:table prefix="b_bot_table_"
 	       width="${bot_table_size}" length="${bot_table_size}"

Commit message: Add optional parameters to collision_object_manager

File: aist_description/scenes/urdf/a_bot_base_scene.urdf.xacro (robot description, xacro)
@@ -6,5 +6,5 @@
   <xacro:property name="a_bot_x"	value="0"/>
   <xacro:property name="a_bot_y"	value="-0.4875"/>
-  <xacro:property name="a_bot_z"	value="0.770"/>
+  <xacro:property name="a_bot_z"	value="0.766"/>
   <xacro:property name="table_h"	value="0.770"/>
   <!-- ground -->
