Commit message: Include tool0 link into moveit group chain

File: aist_description/scenes/urdf/a_bot_base_scene.urdf.xacro (robot description, xacro)
@@ -118,6 +118,6 @@
 			   )/urdf/robotiq_arg2f_coupling.urdf.xacro"/>
   <xacro:robotiq_arg2f_coupling prefix="a_bot_gripper_coupling_"
-				parent="a_bot_flange">
-    <origin xyz="0 0 0" rpy="${pi} 0 0"/>
+				parent="a_bot_tool0">
+    <origin xyz="0 0 0" rpy="0 ${-pi/2} ${pi/2}"/>
   </xacro:robotiq_arg2f_coupling>
   <xacro:include filename="$(find aist_robotiq

File: aist_description/scenes/urdf/aist_base_scene.urdf.xacro (robot description, xacro)
@@ -162,6 +162,6 @@
 			   )/urdf/robotiq_arg2f_coupling.urdf.xacro"/>
   <xacro:robotiq_arg2f_coupling prefix="a_bot_gripper_coupling_"
-				parent="a_bot_flange">
-    <origin xyz="0 0 0" rpy="${pi} 0 0"/>
+				parent="a_bot_tool0">
+    <origin xyz="0 0 0" rpy="0 ${-pi/2} ${pi/2}"/>
   </xacro:robotiq_arg2f_coupling>
   <xacro:include filename="$(find aist_robotiq
@@ -172,6 +172,6 @@
   </xacro:robotiq_140_gripper>
   <xacro:robotiq_arg2f_coupling prefix="b_bot_gripper_coupling_"
-				parent="b_bot_flange">
-    <origin xyz="0 0 0" rpy="${pi} 0 0"/>
+				parent="b_bot_tool0">
+    <origin xyz="0 0 0" rpy="0 ${-pi/2} ${pi/2}"/>
   </xacro:robotiq_arg2f_coupling>
   <xacro:include filename="$(find aist_robotiq

File: aist_description/scenes/urdf/b_bot_base_scene.urdf.xacro (robot description, xacro)
@@ -101,6 +101,6 @@
   <!-- Spawn and attach force sensor -->
   <xacro:include filename="$(find aist_robotiq)/urdf/ft300.urdf.xacro"/>
-  <xacro:ft300 prefix="b_bot_ftsensor_" parent="b_bot_flange">
-    <origin xyz="0 0 0" rpy="${pi} 0 0"/>
+  <xacro:ft300 prefix="b_bot_ftsensor_" parent="b_bot_tool0">
+    <origin xyz="0 0 0" rpy="0 ${-pi/2} ${pi/2}"/>
   </xacro:ft300>
   <!-- Spawn and attach gripper -->

File: aist_description/scenes/urdf/dur5e_base_scene.urdf.xacro (robot description, xacro)
@@ -63,6 +63,6 @@
 			   )/urdf/robotiq_arg2f_coupling.urdf.xacro"/>
   <xacro:robotiq_arg2f_coupling prefix="c_bot_gripper_coupling_"
-				parent="c_bot_flange">
-    <origin xyz="0 0 0" rpy="${pi} 0 0"/>
+				parent="c_bot_tool0">
+    <origin xyz="0 0 0" rpy="0 ${-pi/2} ${pi/2}"/>
   </xacro:robotiq_arg2f_coupling>
   <xacro:include filename="$(find aist_robotiq
@@ -86,6 +86,6 @@
   <!-- </xacro:robotiq_85_gripper_with_tip_link> -->
   <xacro:robotiq_arg2f_coupling prefix="d_bot_gripper_coupling_"
-				parent="d_bot_falnge">
-    <origin xyz="0 0 0" rpy="${pi} 0 0"/>
+				parent="d_bot_tool0">
+    <origin xyz="0 0 0" rpy="0 ${-pi/2} ${pi/2}"/>
   </xacro:robotiq_arg2f_coupling>
   <xacro:include filename="$(find aist_robotiq

File: aist_description/scenes/urdf/f_bot_base_scene.urdf.xacro (robot description, xacro)
@@ -54,6 +54,6 @@
   <!-- Attach force sensor -->
   <xacro:include filename="$(find aist_robotiq)/urdf/ft300.urdf.xacro"/>
-  <xacro:ft300 prefix="f_bot_ftsensor_" parent="f_bot_flange">
-    <origin xyz="0 0 0" rpy="${pi} 0 0"/>
+  <xacro:ft300 prefix="f_bot_ftsensor_" parent="f_bot_tool0">
+    <origin xyz="0 0 0" rpy="0 ${-pi/2} ${pi/2}"/>
   </xacro:ft300>
   <!-- Attach gripper -->

File: aist_description/scenes/urdf/fvision_base_scene.urdf.xacro (robot description, xacro)
@@ -48,6 +48,6 @@
 			   )/urdf/robotiq_dual_bracket.urdf.xacro"/>
   <xacro:robotiq_dual_bracket prefix="d_bot_dual_bracket_"
-			      parent="d_bot_flange">
-    <origin xyz="0 0 0" rpy="${pi} 0 0"/>
+			      parent="d_bot_tool0">
+    <origin xyz="0 0 0" rpy="0 ${-pi/2} ${pi/2}"/>
   </xacro:robotiq_dual_bracket>
   <xacro:include filename="$(find aist_robotiq

File: aist_description/scenes/urdf/g_bot_base_scene.urdf.xacro (robot description, xacro)
@@ -77,6 +77,6 @@
 			   )/urdf/robotiq_arg2f_coupling.urdf.xacro"/>
   <xacro:robotiq_arg2f_coupling prefix="g_bot_gripper_coupling_"
-				parent="g_bot_flange">
-    <origin xyz="0 0 0" rpy="${pi} 0 0"/>
+				parent="g_bot_tool0">
+    <origin xyz="0 0 0" rpy="0 ${-pi/2} ${pi/2}"/>
   </xacro:robotiq_arg2f_coupling>
   <xacro:include filename="$(find aist_robotiq

File: aist_description/scenes/urdf/mocap_base_scene.urdf.xacro (robot description, xacro)
@@ -45,6 +45,6 @@
 			   )/urdf/robotiq_arg2f_coupling.urdf.xacro"/>
   <xacro:robotiq_arg2f_coupling prefix="c_bot_gripper_coupling_"
-				parent="c_bot_flange">
-    <origin xyz="0 0 0" rpy="${pi} 0 0"/>
+				parent="c_bot_tool0">
+    <origin xyz="0 0 0" rpy="0 ${-pi/2} ${pi/2}"/>
   </xacro:robotiq_arg2f_coupling>
   <xacro:include filename="$(find aist_robotiq

Commit message: Add short finger option to robotiq_140

File: aist_description/scenes/urdf/a_bot_base_scene.urdf.xacro (robot description, xacro)
@@ -124,5 +124,6 @@
 			   )/urdf/robotiq_140_gripper.urdf.xacro"/>
   <xacro:robotiq_140_gripper prefix="a_bot_gripper_"
-			     parent="a_bot_gripper_coupling_flange_link">
+			     parent="a_bot_gripper_coupling_flange_link"
+			     short_finger="true">
     <origin xyz="0 0 0" rpy="0 0 0"/>
   </xacro:robotiq_140_gripper>

File: aist_description/scenes/urdf/aist_base_scene.urdf.xacro (robot description, xacro)
@@ -168,5 +168,6 @@
 			   )/urdf/robotiq_140_gripper.urdf.xacro"/>
   <xacro:robotiq_140_gripper prefix="a_bot_gripper_"
-			     parent="a_bot_gripper_coupling_flange_link">
+			     parent="a_bot_gripper_coupling_flange_link"
+			     short_finger="true">
     <origin xyz="0 0 0" rpy="0 0 0"/>
   </xacro:robotiq_140_gripper>

File: aist_robotiq/urdf/robotiq_140_gripper.urdf.xacro (robot description, xacro)
@@ -171,4 +171,26 @@
     </gazebo>
   </xacro:macro>
+  <xacro:macro name="short_inner_finger_pad" params="prefix fingerprefix">
+    <link name="${prefix}${fingerprefix}_inner_finger_pad">
+      <visual>
+        <origin xyz="0 -0.00275 0" rpy="0 0 0"/>
+        <geometry>
+          <box size="0.027 0.0375 0.0075"/>
+        </geometry>
+        <material name="">
+          <color rgba="0.9 0.9 0.9 1"/>
+        </material>
+      </visual>
+      <collision>
+        <origin xyz="0 -0.00275 0" rpy="0 0 0"/>
+        <geometry>
+          <box size="0.027 0.0375 0.0075"/>
+        </geometry>
+        <material name="">
+          <color rgba="0.9 0.0 0.0 1"/>
+        </material>
+      </collision>
+    </link>
+  </xacro:macro>
   <xacro:macro name="outer_finger_joint" params="prefix fingerprefix">
     <joint name="${prefix}${fingerprefix}_outer_finger_joint" type="fixed">
@@ -234,5 +256,6 @@
   </xacro:macro>
   <!-- Initialization of all joints and links -->
-  <xacro:macro name="robotiq_140_gripper" params="prefix parent *origin">
+  <xacro:macro name="robotiq_140_gripper"
+	       params="prefix parent short_finger:=false *origin">
     <joint name="${prefix}base_joint" type="fixed">
       <parent link="${parent}"/>
@@ -249,10 +272,17 @@
       <parent link="${prefix}base_link"/>
       <child link="${prefix}tip_link"/>
-      <origin rpy="0.0 ${-pi/2} 0.0" xyz=".2328 0.0 0.0"/>
+      <xacro:if value="${short_finger}">
+	<origin rpy="0.0 ${-pi/2} 0.0" xyz=".2168 0.0 0.0"/>
+      </xacro:if>
+      <xacro:unless value="${short_finger}">
+	<origin rpy="0.0 ${-pi/2} 0.0" xyz=".2328 0.0 0.0"/>
+      </xacro:unless>
     </joint>
     <link name="${prefix}tip_link"/>
     <xacro:robotiq_arg2f_base_link prefix="${prefix}"/>
-    <xacro:finger_links prefix="${prefix}" fingerprefix="left" stroke="140"/>
-    <xacro:finger_links prefix="${prefix}" fingerprefix="right" stroke="140"/>
+    <xacro:finger_links prefix="${prefix}" fingerprefix="left"
+			stroke="140" short_finger="${short_finger}"/>
+    <xacro:finger_links prefix="${prefix}" fingerprefix="right"
+			stroke="140" short_finger="${short_finger}"/>
     <xacro:finger_joint prefix="${prefix}"/>
     <xacro:right_outer_knuckle_joint prefix="${prefix}"/>

File: aist_robotiq/urdf/robotiq_arg2f.xacro (robot description, xacro)
@@ -34,9 +34,19 @@
     <xacro:inner_finger_pad_joint prefix="${prefix}" fingerprefix="${fingerprefix}"/>
   </xacro:macro>
-  <xacro:macro name="finger_links" params="prefix fingerprefix stroke">
+  <xacro:macro name="finger_links" params="prefix fingerprefix stroke
+					   short_finger:=false">
     <xacro:outer_knuckle prefix="${prefix}" fingerprefix="${fingerprefix}" stroke="${stroke}"/>
     <xacro:outer_finger prefix="${prefix}" fingerprefix="${fingerprefix}" stroke="${stroke}"/>
-    <xacro:inner_finger prefix="${prefix}" fingerprefix="${fingerprefix}" stroke="${stroke}"/>
-    <xacro:inner_finger_pad prefix="${prefix}" fingerprefix="${fingerprefix}"/>
+    <xacro:inner_finger prefix="${prefix}"
+			fingerprefix="${fingerprefix}"
+			stroke="${stroke}"/>
+    <xacro:if value="${short_finger}">
+      <xacro:short_inner_finger_pad prefix="${prefix}"
+				    fingerprefix="${fingerprefix}"/>
+    </xacro:if>
+    <xacro:unless value="${short_finger}">
+      <xacro:inner_finger_pad prefix="${prefix}"
+			      fingerprefix="${fingerprefix}"/>
+    </xacro:unless>
     <xacro:inner_knuckle prefix="${prefix}" fingerprefix="${fingerprefix}" stroke="${stroke}"/>
   </xacro:macro>
