Commit message: Improve API and add functions for fix/release base

File: aist_description/scenes/urdf/aist_base_scene.urdf.xacro (robot description, xacro)
@@ -4,9 +4,11 @@
   <xacro:property name="a_bot_x"	value="0"/>
   <xacro:property name="a_bot_y"	value="-0.4875"/>
+  <xacro:property name="a_bot_z"	value="0.770"/>
   <xacro:property name="b_bot_x"	value="0"/>
   <xacro:property name="b_bot_y"	value="0.4875"/>
+  <xacro:property name="b_bot_z"	value="0.770"/>
   <xacro:property name="b_bot_theta"	value="${pi}"/>
-  <xacro:property name="bots_z"		value="0.770"/>
-  <xacro:property name="screen_z"	value="${bots_z + 0.048}"/>
+  <xacro:property name="table_h"	value="0.770"/>
+  <xacro:property name="screen_z"	value="0.048"/>
   <!-- ground -->
   <link name="ground"/>
@@ -26,5 +28,5 @@
 	      width="${cage_w}" length="${cage_l}" height="${cage_h}"
 	      thickness="${cage_t}"
-	      workspace_height="${bots_z - cage_z}"
+	      workspace_height="${table_h - cage_z}"
 	      tool_bar_height="${tool_bar_h}"
 	      camera_bar_height="${camera_bar_h}"
@@ -41,5 +43,5 @@
 			   )/objects/urdf/table.urdf.xacro"/>
   <xacro:table prefix="workspace_table_"
-	       width="${table_w}" length="${table_l}" height="${bots_z}"
+	       width="${table_w}" length="${table_l}" height="${table_h}"
 	       parent="ground">
     <origin xyz="${-cage_w/2 + cage_offset_x + cage_t} ${-table_l/2} 0"
@@ -50,5 +52,5 @@
     <parent link="ground"/>
     <child  link="workspace_center"/>
-    <origin xyz="0 0 ${bots_z}" rpy="0 0 0"/>
+    <origin xyz="0 0 ${table_h}" rpy="0 0 0"/>
   </joint>
   <!-- tool holders -->
@@ -110,10 +112,10 @@
     <parent link="ground"/>
     <child  link="a_bot_base_link"/>
-    <origin xyz="${a_bot_x} ${a_bot_y} ${bots_z}" rpy="0 0 0"/>
+    <origin xyz="${a_bot_x} ${a_bot_y} ${a_bot_z}" rpy="0 0 0"/>
   </joint>
   <joint name="ground_b_bot_joint" type="fixed">
     <parent link="ground"/>
     <child  link="b_bot_base_link"/>
-    <origin xyz="${b_bot_x} ${b_bot_y} ${bots_z}" rpy="0 0 ${b_bot_theta}"/>
+    <origin xyz="${b_bot_x} ${b_bot_y} ${b_bot_z}" rpy="0 0 ${b_bot_theta}"/>
   </joint>
   <!-- Attach mounter for Zivid2+ camera -->
@@ -211,5 +213,5 @@
   <link name="virtual_screen"/>
   <joint name="virtual_screen_joint" type="fixed">
-    <parent link="ground"/>
+    <parent link="workspace_center"/>
     <child  link="virtual_screen"/>
     <origin xyz="0 0 ${screen_z}" rpy="0 0 0"/>

Commit message: Calibrate poses of a_bot and b_bot

File: aist_description/scenes/urdf/aist_base_scene.urdf.xacro (robot description, xacro)
@@ -4,8 +4,8 @@
   <xacro:property name="a_bot_x"	value="0"/>
   <xacro:property name="a_bot_y"	value="-0.4875"/>
-  <xacro:property name="a_bot_z"	value="0.770"/>
-  <xacro:property name="b_bot_x"	value="0"/>
+  <xacro:property name="a_bot_z"	value="0.766"/>
+  <xacro:property name="b_bot_x"	value="-0.002"/>
   <xacro:property name="b_bot_y"	value="0.4875"/>
-  <xacro:property name="b_bot_z"	value="0.770"/>
+  <xacro:property name="b_bot_z"	value="0.769"/>
   <xacro:property name="b_bot_theta"	value="${pi}"/>
   <xacro:property name="table_h"	value="0.770"/>

File: aist_description/scenes/urdf/kitting.urdf.xacro (robot description, xacro)
@@ -11,5 +11,5 @@
 		  height="${plate_h}"
 		  parent="workspace_center">
-    <origin xyz="-0.062 ${-plate_l/2} 0" rpy="0 0 0"/>
+    <origin xyz="-0.065 ${-plate_l/2} 0" rpy="0 0 0"/>
   </xacro:aist_box>
   <link name="plate_lower_left_corner"/>

Commit message: Calibrate b_bot again

File: aist_description/scenes/urdf/aist_base_scene.urdf.xacro (robot description, xacro)
@@ -5,7 +5,7 @@
   <xacro:property name="a_bot_y"	value="-0.4875"/>
   <xacro:property name="a_bot_z"	value="0.766"/>
-  <xacro:property name="b_bot_x"	value="-0.002"/>
-  <xacro:property name="b_bot_y"	value="0.4875"/>
-  <xacro:property name="b_bot_z"	value="0.769"/>
+  <xacro:property name="b_bot_x"	value="-0.003"/>
+  <xacro:property name="b_bot_y"	value="0.4876"/>
+  <xacro:property name="b_bot_z"	value="0.768"/>
   <xacro:property name="b_bot_theta"	value="${pi}"/>
   <xacro:property name="table_h"	value="0.770"/>
@@ -93,5 +93,5 @@
   <xacro:suction_tool_holder prefix="suction_tool_holder_"
 			   parent="cage_tool_bar">
-    <origin xyz="0 ${suction_tool_holder_y} ${cage_t}" rpy="0 0 0"/>
+    <origin xyz="-0.003 ${suction_tool_holder_y} ${cage_t}" rpy="0 0 0"/>
   </xacro:suction_tool_holder>
   <!-- robot arms -->

Commit message: Confirmed that multuple robots succesfully spawned in gz simulation

File: aist_description/scenes/urdf/aist_base_scene.urdf.xacro (robot description, xacro)
@@ -15,4 +15,11 @@
 		  value="$(find ur_robot_driver
 			 )/resources/rtde_input_recipe.txt"/>
+  <xacro:property name="initial_positions"
+		  value="${dict(shoulder_pan_joint=1.5708,
+			        shoulder_lift_joint=-2.1,
+				elbow_joint=1.4,
+				wrist_1_joint=-0.85,
+				wrist_2_joint=-1.5708,
+				wrist_3_joint=0.0)}"/>
   <!-- location of robot arms -->
   <xacro:property name="a_bot_x"	value="0"/>
@@ -115,6 +122,6 @@
   <xacro:ur_robot_with_ros2_control
       sim="$(arg sim)"
+      name="a_bot"
       ur_type="ur5e"
-      name="a_bot"
       parent="a_bot_table_top_center"
       safety_limits="true"
@@ -123,4 +130,5 @@
       input_recipe_filename="${input_recipe_filename}"
       output_recipe_filename="${output_recipe_filename}"
+      initial_positions="${initial_positions}"
       robot_ip="${a_bot_ip}"
       reverse_port="50001"
@@ -133,6 +141,6 @@
   <xacro:ur_robot_with_ros2_control
       sim="$(arg sim)"
+      name="b_bot"
       ur_type="ur5e"
-      name="b_bot"
       parent="b_bot_table_top_center"
       safety_limits="true"
@@ -141,4 +149,5 @@
       input_recipe_filename=""
       output_recipe_filename=""
+      initial_positions="${initial_positions}"
       robot_ip="${b_bot_ip}"
       reverse_port="50005"
