Commit message: Update b_bot config

File: aist_description/scenes/urdf/b_bot_base_scene.urdf.xacro (robot description, xacro)
@@ -84,9 +84,9 @@
       prefix="b_bot_"
       joint_limits_parameters_file="$(find ur_description
-				    )/config/ur5/joint_limits.yaml"
+				    )/config/ur5e/joint_limits.yaml"
       physical_parameters_file="$(find ur_description
-				)/config/ur5/physical_parameters.yaml"
+				)/config/ur5e/physical_parameters.yaml"
       visual_parameters_file="$(find ur_description
-			      )/config/ur5/visual_parameters.yaml"
+			      )/config/ur5e/visual_parameters.yaml"
       kinematics_parameters_file="$(find aist_bringup
 				  )/config/b_bot_calibration.yaml"
@@ -99,28 +99,41 @@
     <origin xyz="0 0 0 " rpy="0 0 ${b_bot_theta}"/>
   </joint>
-  <!-- Spawn and attach force sensor -->
-  <xacro:include filename="$(find aist_robotiq)/urdf/ft300.urdf.xacro"/>
-  <xacro:ft300 prefix="b_bot_ftsensor_" parent="b_bot_tool0">
+  <!-- Spawn and attach gripper -->
+  <xacro:include filename="$(find aist_robotiq
+			   )/urdf/robotiq_arg2f_coupling.urdf.xacro"/>
+  <xacro:robotiq_arg2f_coupling prefix="b_bot_gripper_coupling_"
+				parent="b_bot_tool0">
     <origin xyz="0 0 0" rpy="0 ${-pi/2} ${pi/2}"/>
-  </xacro:ft300>
-  <!-- Spawn and attach gripper -->
+  </xacro:robotiq_arg2f_coupling>
+  <xacro:include filename="$(find aist_robotiq
+			   )/urdf/robotiq_85_gripper.urdf.xacro"/>
+  <xacro:robotiq_85_gripper prefix="b_bot_gripper_"
+			    parent="b_bot_gripper_coupling_flange_link">
+    <origin xyz="0 0 0" rpy="0 0 0"/>
+  </xacro:robotiq_85_gripper>
+  <!-- Add USB repeaters -->
   <xacro:include filename="$(find aist_description
-			   )/devices/urdf/single_suction_gripper.urdf.xacro"/>
-  <xacro:single_suction_gripper prefix="b_bot_gripper_"
-  				parent="b_bot_ftsensor_flange_link">
-    <!-- <origin xyz="0 0 0" rpy="0 ${0.2*pi/180} ${-1.2*pi/180}"/> -->
-    <origin xyz="0 0 0" rpy="0 ${0.3*pi/180} ${0.2*pi/180}"/>
-  </xacro:single_suction_gripper>
-  <!-- Add PhoXi 3D scanner -->
+			   )/objects/urdf/usb_repeater.urdf.xacro"/>
+  <xacro:usb_repeater prefix="b_bot_usb_repeater_"
+		      parent="b_bot_wrist_2_link">
+    <origin xyz="0.000 -0.051 0.000" rpy="${pi/2} ${-pi/2} 0"/>
+  </xacro:usb_repeater>
+  <!-- Add Motioncam-3D scanner -->
   <xacro:include filename="$(find aist_description
 			   )/scenes/urdf/load_calibration.urdf.xacro"/>
   <xacro:load_calibration filename="$(find aist_handeye_calibration
-				    )/calib/a_phoxi_m_camera.yaml"/>
+				    )/calib/a_motioncam.yaml"/>
   <xacro:include filename="$(find aist_phoxi_camera
-			   )/urdf/phoxi_m_camera.urdf.xacro"/>
-  <xacro:phoxi_m_camera name="a_phoxi_m_camera" parent="workspace_center">
+			   )/urdf/motioncam_m_camera.urdf.xacro"/>
+  <xacro:motioncam_m_camera name="a_motioncam" parent="workspace_center">
     <origin xyz="${origin[0]} ${origin[1]} ${origin[2]}"
     	    rpy="${origin[3]} ${origin[4]} ${origin[5]}"/>
-  </xacro:phoxi_m_camera>
+  </xacro:motioncam_m_camera>
+  <!-- Add RealSense cameras -->
+  <xacro:include filename="$(find aist_description
+  			   )/devices/urdf/sr305_on_2f85.urdf.xacro" />
+  <xacro:sr305_on_2f85 prefix="b_bot_"
+  		       parent="b_bot_gripper_base_link"
+  		       use_nominal_extrinsics="true"/>
   <!-- Add live camera -->
   <xacro:load_calibration filename="$(find aist_camera_calibration
@@ -147,4 +160,7 @@
     <origin xyz="0 0 0" rpy="0 0 0"/>
   </joint>
+  <!-- Import assembly scene -->
+  <xacro:include filename="$(find aist_description
+			   )/scenes/urdf/assembly.urdf.xacro"/>
   <!-- Include indivisual scene file -->
   <xacro:if value="${'$(arg scene)' != ''}">

File: moveit_config/b_bot_moveit_config/config/gazebo_b_bot_base_scene.urdf (robot description, URDF)
Before this commit: robot b_bot__base_scene, 54 links, 53 joints
Links:
- removed link b_bot_camera_mount
- removed link b_bot_gripper_coupling_base_link
- removed link b_bot_gripper_coupling_flange_link
- removed link b_bot_gripper_left_inner_finger
- removed link b_bot_gripper_left_inner_finger_pad
- removed link b_bot_gripper_left_inner_knuckle
- removed link b_bot_gripper_left_outer_finger
- removed link b_bot_gripper_left_outer_knuckle
- removed link b_bot_gripper_right_inner_finger
- removed link b_bot_gripper_right_inner_finger_pad
- removed link b_bot_gripper_right_inner_knuckle
- removed link b_bot_gripper_right_outer_finger
- removed link b_bot_gripper_right_outer_knuckle
- removed link b_bot_gripper_robotiq_arg2f_base_link
- removed link b_bot_inside_camera_color_frame
- removed link b_bot_inside_camera_color_optical_frame
- removed link b_bot_inside_camera_connector_link
- removed link b_bot_inside_camera_depth_frame
- removed link b_bot_inside_camera_depth_optical_frame
- removed link b_bot_inside_camera_left_ir_frame
- removed link b_bot_inside_camera_left_ir_optical_frame
- removed link b_bot_inside_camera_link
- removed link b_bot_inside_camera_right_ir_frame
- removed link b_bot_inside_camera_right_ir_optical_frame
- removed link b_bot_outside_camera_color_frame
- removed link b_bot_outside_camera_color_optical_frame
- removed link b_bot_outside_camera_connector_link
- removed link b_bot_outside_camera_depth_frame
- removed link b_bot_outside_camera_depth_optical_frame
- removed link b_bot_outside_camera_left_ir_frame
- removed link b_bot_outside_camera_left_ir_optical_frame
- removed link b_bot_outside_camera_link
- removed link b_bot_outside_camera_right_ir_frame
- removed link b_bot_outside_camera_right_ir_optical_frame
- removed link workbox
- added link a_phoxi_m_camera_link, mass 0.1; collision mesh filename=package://aist_phoxi_camera/meshes/collision/PhoXi_M.c.STL scale=0.001 0.001 0.001; visual mesh filename=package://aist_phoxi_camera/meshes/visual/PhoXi_M.f.STL scale=0.001 0.001 0.001
- added link a_phoxi_m_camera_reference
- added link a_phoxi_m_camera_sensor
- added link b_bot_table_base_link, mass 1.0; collision box size=0.05 0.05 0.75; visual box size=0.05 0.05 0.75
- added link b_bot_table_leg1, mass 1.0; collision box size=0.05 0.05 0.75; visual box size=0.05 0.05 0.75
- added link b_bot_table_leg2, mass 1.0; collision box size=0.05 0.05 0.75; visual box size=0.05 0.05 0.75
- added link b_bot_table_leg3, mass 1.0; collision box size=0.05 0.05 0.75; visual box size=0.05 0.05 0.75
- added link b_bot_table_top, mass 1.0; collision box size=0.225 0.225 0.02; visual box size=0.225 0.225 0.02
- added link b_bot_table_top_center
- added link b_bot_table_top_origin
- added link cage_back_left_pillar, mass 1.0; collision box size=0.04 0.04 1.42; visual box size=0.04 0.04 1.42
- added link cage_back_right_pillar, mass 1.0; collision box size=0.04 0.04 1.42; visual box size=0.04 0.04 1.42
- added link cage_front_left_pillar, mass 1.0; collision box size=0.04 0.04 1.42; visual box size=0.04 0.04 1.42
- added link cage_front_right_pillar, mass 1.0; collision box size=0.04 0.04 1.42; visual box size=0.04 0.04 1.42
- added link cage_lower_back_bar, mass 1.0; collision box size=1.1199999999999999 0.04 0.04; visual box size=1.1199999999999999 0.04 0.04
- added link cage_lower_front_bar, mass 1.0; collision box size=1.1199999999999999 0.04 0.04; visual box size=1.1199999999999999 0.04 0.04
- added link cage_lower_left_bar, mass 1.0; collision box size=0.04 1.5 0.04; visual box size=0.04 1.5 0.04
- added link cage_lower_right_bar, mass 1.0; collision box size=0.04 1.5 0.04; visual box size=0.04 1.5 0.04
- added link cage_tool_bar, mass 1.0; collision box size=0.04 1.5 0.04; visual box size=0.04 1.5 0.04
- added link cage_upper_back_bar, mass 1.0; collision box size=1.1199999999999999 0.04 0.04; visual box size=1.1199999999999999 0.04 0.04
- added link cage_upper_front_bar, mass 1.0; collision box size=1.1199999999999999 0.04 0.04; visual box size=1.1199999999999999 0.04 0.04
- added link cage_upper_left_bar, mass 1.0; collision box size=0.04 1.5 0.04; visual box size=0.04 1.5 0.04
- added link cage_upper_right_bar, mass 1.0; collision box size=0.04 1.5 0.04; visual box size=0.04 1.5 0.04
- added link cage_workspace_bar, mass 1.0; collision box size=0.04 1.5 0.04; visual box size=0.04 1.5 0.04
- added link live_camera_optical_frame
- added link screw_tool_m3_holder_base_link, mass 0.1; collision mesh filename=package://aist_description/objects/meshes/screw_tool_holder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 scale=0.001 0.001 0.001; visual mesh filename=package://aist_description/objects/meshes/screw_tool_holder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 scale=0.001 0.001 0.001
- added link screw_tool_m3_holder_link
- added link screw_tool_m4_holder_base_link, mass 0.1; collision mesh filename=package://aist_description/objects/meshes/screw_tool_holder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 scale=0.001 0.001 0.001; visual mesh filename=package://aist_description/objects/meshes/screw_tool_holder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 scale=0.001 0.001 0.001
- added link screw_tool_m4_holder_link
- added link suction_tool_holder_base_link, mass 0.1; collision mesh filename=package://aist_description/objects/meshes/suction_tool_hold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 scale=0.001 0.001 0.001; visual mesh filename=package://aist_description/objects/meshes/suction_tool_hold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 scale=0.001 0.001 0.001
- added link suction_tool_holder_link
- added link virtual_screen
- added link workspace_table_base_link, mass 1.0; collision box size=0.05 0.05 0.75; visual box size=0.05 0.05 0.75
- added link workspace_table_leg1, mass 1.0; collision box size=0.05 0.05 0.75; visual box size=0.05 0.05 0.75
- added link workspace_table_leg2, mass 1.0; collision box size=0.05 0.05 0.75; visual box size=0.05 0.05 0.75
- added link workspace_table_leg3, mass 1.0; collision box size=0.05 0.05 0.75; visual box size=0.05 0.05 0.75
- added link workspace_table_top, mass 1.0; collision box size=0.9 0.75 0.02; visual box size=0.9 0.75 0.02
- added link workspace_table_top_center
- added link workspace_table_top_origin
- link b_bot_forearm_link: mass 2.275 -> 2.33
- link b_bot_gripper_base_link: mass None -> 0.3; geometry collision mesh filename=package://aist_description/devices/meshes/single_suction_gr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 scale=0.001 0.001 0.001; visual mesh filename=package://aist_description/devices/meshes/single_suction_gr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 scale=0.001 0.001 0.001
Joints:
- removed joint b_bot_camera_mount_joint
- removed joint b_bot_gripper_coupling_base_joint
- removed joint b_bot_gripper_coupling_flange_joint
- removed joint b_bot_gripper_finger_joint
- removed joint b_bot_gripper_left_inner_finger_joint
- removed joint b_bot_gripper_left_inner_finger_pad_joint
- removed joint b_bot_gripper_left_inner_knuckle_joint
- removed joint b_bot_gripper_left_outer_finger_joint
- removed joint b_bot_gripper_right_inner_finger_joint
- removed joint b_bot_gripper_right_inner_finger_pad_joint
- removed joint b_bot_gripper_right_inner_knuckle_joint
- removed joint b_bot_gripper_right_outer_finger_joint
- removed joint b_bot_gripper_right_outer_knuckle_joint
- removed joint b_bot_gripper_robotiq_arg2f_base_joint
- removed joint b_bot_gripper_tip_link_joint
- removed joint b_bot_inside_camera_color_joint
- removed joint b_bot_inside_camera_color_optical_joint
- removed joint b_bot_inside_camera_depth_joint
- removed joint b_bot_inside_camera_depth_optical_joint
- removed joint b_bot_inside_camera_joint
- removed joint b_bot_inside_camera_left_ir_joint
- removed joint b_bot_inside_camera_left_ir_optical_joint
- removed joint b_bot_inside_camera_link_joint
- removed joint b_bot_inside_camera_right_ir_joint
- removed joint b_bot_inside_camera_right_ir_optical_joint
- removed joint b_bot_outside_camera_color_joint
- removed joint b_bot_outside_camera_color_optical_joint
- removed joint b_bot_outside_camera_depth_joint
- removed joint b_bot_outside_camera_depth_optical_joint
- removed joint b_bot_outside_camera_joint
- removed joint b_bot_outside_camera_left_ir_joint
- removed joint b_bot_outside_camera_left_ir_optical_joint
- removed joint b_bot_outside_camera_link_joint
- removed joint b_bot_outside_camera_right_ir_joint
- removed joint b_bot_outside_camera_right_ir_optical_joint
- removed joint ground_b_bot_joint
- removed joint ground_to_workspace
- removed joint workbox
- removed joint world_ground_joint
- added joint a_phoxi_m_camera_link_joint: type fixed, parent workspace_center, child a_phoxi_m_camera_link, origin xyz=0.5141294525807852 -0.0391428293642771 0.6227194772673923 rpy=-0.0626579561970891 1.0383878192954172 3.059776671030358
- added joint a_phoxi_m_camera_reference_joint: type fixed, parent a_phoxi_m_camera_link, child a_phoxi_m_camera_reference, origin xyz=0.002164826095 -0.176277236938477 0.0299 rpy=0 0 0.20507618710933373
- added joint a_phoxi_m_camera_sensor_joint: type fixed, parent a_phoxi_m_camera_reference, child a_phoxi_m_camera_sensor, origin xyz=0 0 0 rpy=-1.5707963267948966 0 -1.5707963267948966
- added joint b_bot_base_link_joint: type fixed, parent b_bot_table_top_center, child b_bot_base_link, origin xyz=0 0 0  rpy=0 0 3.141592653589793
- added joint b_bot_gripper_tip_joint: type fixed, parent b_bot_gripper_base_link, child b_bot_gripper_tip_link, origin xyz=0.1855 0 0 rpy=0 -1.5707963267948966 0
- added joint b_bot_table_base_link: type fixed, parent ground, child b_bot_table_base_link, origin xyz=-0.1125 0.375 0 rpy=0 0 0
- added joint b_bot_table_leg1: type fixed, parent b_bot_table_base_link, child b_bot_table_leg1, origin xyz=0.175 0 0 rpy=0 0 0
- added joint b_bot_table_leg2: type fixed, parent b_bot_table_base_link, child b_bot_table_leg2, origin xyz=0 0.175 0 rpy=0 0 0
- added joint b_bot_table_leg3: type fixed, parent b_bot_table_base_link, child b_bot_table_leg3, origin xyz=0.175      0.175      0 rpy=0 0 0
- added joint b_bot_table_top: type fixed, parent b_bot_table_base_link, child b_bot_table_top, origin xyz=0 0 0.75 rpy=0 0 0
- added joint b_bot_table_top_center_joint: type fixed, parent b_bot_table_top_origin, child b_bot_table_top_center, origin xyz=0.1125 0.1125 0 rpy=0 0 0
- added joint b_bot_table_top_origin_joint: type fixed, parent b_bot_table_top, child b_bot_table_top_origin, origin xyz=0 0 0.02 rpy=0 0 0
- added joint cage_back_left_pillar: type fixed, parent cage_front_left_pillar, child cage_back_left_pillar, origin xyz=0 1.54 0 rpy=0 0 0
- added joint cage_back_right_pillar: type fixed, parent cage_front_left_pillar, child cage_back_right_pillar, origin xyz=1.16        1.54        0 rpy=0 0 0
- added joint cage_front_left_pillar: type fixed, parent ground, child cage_front_left_pillar, origin xyz=-0.58    -0.795    0.164 rpy=0 0 0
- added joint cage_front_right_pillar: type fixed, parent cage_front_left_pillar, child cage_front_right_pillar, origin xyz=1.16 0 0 rpy=0 0 0
- added joint cage_lower_back_bar: type fixed, parent cage_front_left_pillar, child cage_lower_back_bar, origin xyz=0.04 1.54 0 rpy=0 0 0
- added joint cage_lower_front_bar: type fixed, parent cage_front_left_pillar, child cage_lower_front_bar, origin xyz=0.04 0 0 rpy=0 0 0
- added joint cage_lower_left_bar: type fixed, parent cage_front_left_pillar, child cage_lower_left_bar, origin xyz=0 0.04 0 rpy=0 0 0
- added joint cage_lower_right_bar: type fixed, parent cage_front_left_pillar, child cage_lower_right_bar, origin xyz=1.16 0.04 0 rpy=0 0 0
- added joint cage_tool_bar: type fixed, parent cage_workspace_bar, child cage_tool_bar, origin xyz=0 0 0.24 rpy=0 0 0
- added joint cage_upper_back_bar: type fixed, parent cage_front_left_pillar, child cage_upper_back_bar, origin xyz=0.04 1.54 1.38 rpy=0 0 0
- added joint cage_upper_front_bar: type fixed, parent cage_front_left_pillar, child cage_upper_front_bar, origin xyz=0.04 0 1.38 rpy=0 0 0
- added joint cage_upper_left_bar: type fixed, parent cage_front_left_pillar, child cage_upper_left_bar, origin xyz=0 0.04 1.38 rpy=0 0 0
- added joint cage_upper_right_bar: type fixed, parent cage_front_left_pillar, child cage_upper_right_bar, origin xyz=1.16 0.04 1.325 rpy=0 0 0
- added joint cage_workspace_bar: type fixed, parent cage_lower_left_bar, child cage_workspace_bar, origin xyz=0 0 0.596 rpy=0 0 0
- added joint ground_joint: type fixed, parent world, child ground, origin xyz=0 0 0 rpy=0 0 0
- added joint live_camera_joint: type fixed, parent workspace_center, child live_camera_optical_frame, origin xyz=0.4176511892059926 -0.07081252327671157 0.7599460149030057 rpy=-2.74696433805391 -0.09019210220491233 1.5692522682584185
- added joint screw_tool_m3_holder_base_joint: type fixed, parent cage_tool_bar, child screw_tool_m3_holder_base_link, origin xyz=0 0.75 0.04 rpy=0 0 0
- added joint screw_tool_m3_holder_joint: type fixed, parent screw_tool_m3_holder_base_link, child screw_tool_m3_holder_link, origin xyz=0.0525 0 0.007 rpy=0 0 0
- added joint screw_tool_m4_holder_base_joint: type fixed, parent cage_tool_bar, child screw_tool_m4_holder_base_link, origin xyz=0 0.85 0.04 rpy=0 0 0
- added joint screw_tool_m4_holder_joint: type fixed, parent screw_tool_m4_holder_base_link, child screw_tool_m4_holder_link, origin xyz=0.0525 0 0.007 rpy=0 0 0
- added joint suction_tool_holder_base_joint: type fixed, parent cage_tool_bar, child suction_tool_holder_base_link, origin xyz=0 0.95 0.04 rpy=0 0 0
- added joint suction_tool_holder_joint: type fixed, parent suction_tool_holder_base_link, child suction_tool_holder_link, origin xyz=0.08732 0.0 -0.002 rpy=0 0.5235987755982988 0
- added joint virtual_screen_joint: type fixed, parent workspace_center, child virtual_screen, origin xyz=0 0 0.048 rpy=0 0 0
- added joint workspace_joint: type fixed, parent ground, child workspace_center, origin xyz=0 0 0.77 rpy=0 0 0
- added joint workspace_table_base_link: type fixed, parent ground, child workspace_table_base_link, origin xyz=-0.5399999999999999 -0.375 0 rpy=0 0 0
- added joint workspace_table_leg1: type fixed, parent workspace_table_base_link, child workspace_table_leg1, origin xyz=0.85 0 0 rpy=0 0 0
- added joint workspace_table_leg2: type fixed, parent workspace_table_base_link, child workspace_table_leg2, origin xyz=0 0.7 0 rpy=0 0 0
- added joint workspace_table_leg3: type fixed, parent workspace_table_base_link, child workspace_table_leg3, origin xyz=0.85      0.7      0 rpy=0 0 0
- added joint workspace_table_top: type fixed, parent workspace_table_base_link, child workspace_table_top, origin xyz=0 0 0.75 rpy=0 0 0
- added joint workspace_table_top_center_joint: type fixed, parent workspace_table_top_origin, child workspace_table_top_center, origin xyz=0.45 0.375 0 rpy=0 0 0
- added joint workspace_table_top_origin_joint: type fixed, parent workspace_table_top, child workspace_table_top_origin, origin xyz=0 0 0.02 rpy=0 0 0
- joint b_bot_elbow_joint: origin xyz=-0.4249927407255726 0 0 rpy=3.141544575566677 3.141258056989769 -3.141547941357519 -> xyz=-0.4254007797241973 0 0 rpy=3.141491900534354 3.139174779924852 3.141584207915057
- joint b_bot_ftsensor_ft300_joint: origin xyz=0 0 0 rpy=3.141592653589793 0 0 -> xyz=0 0 0 rpy=0 -1.5707963267948966 1.5707963267948966; parent b_bot_flange -> b_bot_tool0
- joint b_bot_gripper_base_joint: origin xyz=0 0 0 rpy=0 0 0 -> xyz=0 0 0 rpy=0 0.005235987755982988 0.003490658503988659; parent b_bot_gripper_coupling_flange_link -> b_bot_ftsensor_flange_link
- joint b_bot_shoulder_lift_joint: origin xyz=0.0001298333079647873 0 0 rpy=1.570642973887296 0 1.159216330228952e-05 -> xyz=0.0001547286037767951 0 0 rpy=1.57107250805896 0 3.903724705512494e-06
- joint b_bot_shoulder_pan_joint: origin xyz=0 0 0.0892795739838422 rpy=0 0 -1.372428740606553e-05 -> xyz=0 0 0.162562140016384 rpy=0 0 1.059019818887286e-07
- joint b_bot_wrist_1_joint: origin xyz=-0.3919582400771999 0.001161330843866965 0.1106654674396762 rpy=3.131098971659387 3.138979604311949 3.141566100969229 -> xyz=-0.3921670303947003 -0.0003240755197429875 0.1343741392746988 rpy=0.002411735570303671 0.0008031027282546156 4.878289526670351e-06
- joint b_bot_wrist_2_joint: origin xyz=-0.0002553647085556869 -0.09473296389451868 6.350685479905706e-05 rpy=1.570125949318306 0 1.99895973980563e-05 -> xyz=-4.98866785623302e-05 -0.09969492467843541 2.875493261443601e-05 rpy=1.570507897550281 0 -1.232576915498329e-07
- joint b_bot_wrist_3_joint: origin xyz=0.0002769113618036503 0.08232662392091306 2.876763766918989e-05 rpy=1.571145759762365 3.141592653589793 -3.141518379713017 -> xyz=2.96236030674356e-05 0.09962093212121005 3.771300233813919e-05 rpy=1.571174891818668 3.141592653589793 -3.141592566216859

Commit message: Fix location of tool holders in b_bot configuration

File: aist_description/scenes/urdf/b_bot_base_scene.urdf.xacro (robot description, xacro)
@@ -62,7 +62,7 @@
   </xacro:table>
   <!-- tool holders -->
-  <xacro:property name="screw_tool_m3_holder_y"	value="0.75"/>
-  <xacro:property name="screw_tool_m4_holder_y"	value="0.85"/>
-  <xacro:property name="suction_tool_holder_y"	value="0.95"/>
+  <xacro:property name="screw_tool_m3_holder_y"	value="0.70"/>
+  <xacro:property name="screw_tool_m4_holder_y"	value="0.80"/>
+  <xacro:property name="suction_tool_holder_y"	value="0.90"/>
   <xacro:include filename="$(find aist_description
 			   )/objects/urdf/screw_tool_holder.urdf.xacro"/>
