Commit message: Confirmed that g_bot_camera can be calibrated on simulation

File: aist_description/devices/urdf/conveni_suction_gripper.urdf.xacro (robot description, xacro)
@@ -40,5 +40,5 @@
       <parent link="${prefix}base_link"/>
       <child  link="${prefix}tip_link"/>
-      <origin xyz="0.280 0 0" rpy="0 ${-pi/2} 0"/>
+      <origin xyz="0.280 0 0" rpy="${pi} ${pi/2} 0"/>
     </joint>
   </xacro:macro>

File: aist_description/scenes/urdf/a_bot_calibration.urdf.xacro (robot description, xacro)
@@ -6,7 +6,7 @@
 		   parent="workspace_center"
 		   marker_id="17_26_32_256"
-		   width="0.150" height="0.150" margin="0.005"
+		   width="0.105" height="0.105" margin="0.007"
 		   thickness="0.001">
-    <origin xyz="0.0 0.0 0.0005" rpy="0 0 0"/>
+    <origin xyz="0.0 0.0 0.0001" rpy="0 0 0"/>
   </xacro:ar_marker>
 </robot>

File: aist_description/scenes/urdf/g_bot_base_scene.urdf.xacro (robot description, xacro)
@@ -4,5 +4,5 @@
   <xacro:arg name="scene" default=""/>
   <xacro:property name="g_bot_x"   value="0"/>
-  <xacro:property name="g_bot_y"   value="-0.625"/>
+  <xacro:property name="g_bot_y"   value="-0.9"/>
   <xacro:property name="g_bot_z"   value="0.700"/>
   <xacro:property name="cabinet_w" value="0.900"/>
@@ -74,16 +74,9 @@
   </joint>
   <!-- Attach gripper -->
-  <xacro:include filename="$(find aist_robotiq
-			   )/urdf/robotiq_arg2f_coupling.urdf.xacro"/>
-  <xacro:robotiq_arg2f_coupling prefix="g_bot_gripper_coupling_"
-				parent="g_bot_tool0">
-    <origin xyz="0 0 0" rpy="0 ${-pi/2} ${pi/2}"/>
-  </xacro:robotiq_arg2f_coupling>
-  <xacro:include filename="$(find aist_robotiq
-			   )/urdf/robotiq_140_gripper.urdf.xacro"/>
-  <xacro:robotiq_140_gripper prefix="g_bot_gripper_"
-			     parent="g_bot_gripper_coupling_flange_link">
-    <origin xyz="0 0 0" rpy="0 0 0"/>
-  </xacro:robotiq_140_gripper>
+  <xacro:include filename="$(find aist_description
+			   )/devices/urdf/conveni_suction_gripper.urdf.xacro"/>
+  <xacro:conveni_suction_gripper prefix="g_bot_gripper_" parent="g_bot_tool0">
+    <origin xyz="0 0 0" rpy="0 ${-pi/2} ${-pi/2}"/>
+  </xacro:conveni_suction_gripper>
   <!-- Attach RealSense camera -->
   <xacro:include filename="$(find aist_description
@@ -92,10 +85,10 @@
 				    )/calib/g_bot_camera.yaml"/>
   <xacro:include filename="$(find aist_description
-			   )/devices/urdf/_d415.urdf.xacro"/>
-  <xacro:sensor_d415 name="g_bot_camera" parent="workspace_center"
+			   )/devices/urdf/_d435.urdf.xacro"/>
+  <xacro:sensor_d435 name="g_bot_camera" parent="g_bot_gripper_base_link"
 		     use_nominal_extrinsics="true">
     <origin xyz="${origin[0]} ${origin[1]} ${origin[2]}"
     	    rpy="${origin[3]} ${origin[4]} ${origin[5]}"/>
-  </xacro:sensor_d415>
+  </xacro:sensor_d435>
   <!-- I would like to remove the "world" link definition, but apparently it is necessary for Gazebo -->
   <link name="world"/>

File: aist_description/scenes/urdf/g_bot_calibration.urdf.xacro (robot description, xacro)
@@ -2,10 +2,10 @@
 <robot xmlns:xacro="http://wiki.ros.org/xacro" name="g_bot_calibration">
   <xacro:include filename="$(find aist_aruco_ros)/urdf/ar_marker.urdf.xacro"/>
-  <xacro:ar_marker prefix="g_bot_"
-  		   parent="g_bot_gripper_base_link"
-  		   marker_id="26"
-		   width="0.070" height="0.070" margin="0.005"
-		   thickness="0.005">
-    <origin xyz="0.180 0.0 0.0215" rpy="0 0 ${pi/2}"/>
+  <xacro:ar_marker prefix="workspace_"
+		   parent="workspace_center"
+		   marker_id="100_101_102_103"
+		   width="0.105" height="0.105" margin="0.007"
+		   thickness="0.001">
+    <origin xyz="0 -0.140 0.001" rpy="0 0 0"/>
   </xacro:ar_marker>
 </robot>

File: moveit_config/g_bot_moveit_config/config/gazebo_g_bot_base_scene.urdf (robot description, URDF)
Before this commit: robot g_bot_base_scene, 58 links, 57 joints
Links:
- removed link g_bot_gripper_coupling_base_link
- removed link g_bot_gripper_coupling_flange_link
- removed link g_bot_gripper_left_inner_finger
- removed link g_bot_gripper_left_inner_finger_pad
- removed link g_bot_gripper_left_inner_knuckle
- removed link g_bot_gripper_left_outer_finger
- removed link g_bot_gripper_left_outer_knuckle
- removed link g_bot_gripper_right_inner_finger
- removed link g_bot_gripper_right_inner_finger_pad
- removed link g_bot_gripper_right_inner_knuckle
- removed link g_bot_gripper_right_outer_finger
- removed link g_bot_gripper_right_outer_knuckle
- removed link g_bot_gripper_robotiq_arg2f_base_link
- removed link mounter_table_leg0
- removed link mounter_table_top_origin_center
- added link mounter_table_base_link, mass 1.0; collision box size=0.05 0.05 0.6799999999999999; visual box size=0.05 0.05 0.6799999999999999
- added link mounter_table_top_center
- link g_bot_camera_link: geometry collision box size=0.02505 0.09 0.025; visual mesh filename=package://realsense2_description/meshes/d435.dae
- link g_bot_gripper_base_link: mass None -> 0.3; geometry collision mesh filename=package://aist_description/devices/meshes/collision/conveni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 scale=0.001 0.001 0.001; visual mesh filename=package://aist_description/devices/meshes/conveni_suction_g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 scale=0.001 0.001 0.001
Joints:
- removed joint g_bot_gripper_coupling_base_joint
- removed joint g_bot_gripper_coupling_flange_joint
- removed joint g_bot_gripper_finger_joint
- removed joint g_bot_gripper_left_inner_finger_joint
- removed joint g_bot_gripper_left_inner_finger_pad_joint
- removed joint g_bot_gripper_left_inner_knuckle_joint
- removed joint g_bot_gripper_left_outer_finger_joint
- removed joint g_bot_gripper_right_inner_finger_joint
- removed joint g_bot_gripper_right_inner_finger_pad_joint
- removed joint g_bot_gripper_right_inner_knuckle_joint
- removed joint g_bot_gripper_right_outer_finger_joint
- removed joint g_bot_gripper_right_outer_knuckle_joint
- removed joint g_bot_gripper_robotiq_arg2f_base_joint
- removed joint g_bot_gripper_tip_link_joint
- removed joint mounter_table_leg0
- removed joint mounter_table_top_origin
- removed joint mounter_table_top_origin_center
- added joint g_bot_gripper_tip_joint: type fixed, parent g_bot_gripper_base_link, child g_bot_gripper_tip_link, origin xyz=0.280 0 0 rpy=3.141592653589793 1.5707963267948966 0
- added joint mounter_table_base_link: type fixed, parent ground, child mounter_table_base_link, origin xyz=-0.1 -1.0 0 rpy=0 0 0
- added joint mounter_table_top_center_joint: type fixed, parent mounter_table_top_origin, child mounter_table_top_center, origin xyz=0.1 0.1 0 rpy=0 0 0
- added joint mounter_table_top_origin_joint: type fixed, parent mounter_table_top, child mounter_table_top_origin, origin xyz=0 0 0.02 rpy=0 0 0
- joint g_bot_camera_infra2_joint: origin xyz=0 -0.055 0 rpy=0 0 0 -> xyz=0 -0.05 0 rpy=0 0 0
- joint g_bot_camera_joint: origin xyz=0.0 0.18 0.45 rpy=0.0 1.309 -1.57 -> xyz=0.05 0.032 -0.047 rpy=3.14159 0.0 0.0; parent workspace_center -> g_bot_gripper_base_link
- joint g_bot_camera_link_joint: origin xyz=0 0.02 0.0115 rpy=0 0 0 -> xyz=0.010600000000000002 0.0175 0.0125 rpy=0 0 0
- joint g_bot_gripper_base_joint: origin xyz=0 0 0 rpy=0 0 0 -> xyz=0 0 0 rpy=0 -1.5707963267948966 -1.5707963267948966; parent g_bot_gripper_coupling_flange_link -> g_bot_tool0
- joint ground_g_bot_joint: origin xyz=0 -0.625 0.7 rpy=0 0 0 -> xyz=0 -0.9 0.7 rpy=0 0 0
- joint mounter_table_leg1: parent mounter_table_leg0 -> mounter_table_base_link
- joint mounter_table_leg2: parent mounter_table_leg0 -> mounter_table_base_link
- joint mounter_table_leg3: parent mounter_table_leg0 -> mounter_table_base_link
- joint mounter_table_top: parent mounter_table_leg0 -> mounter_table_base_link
