Commit message: Add collision meshes for sr305_mount

File: aist_description/devices/urdf/sr305_on_2f140.urdf.xacro (robot description, xacro)
@@ -7,7 +7,6 @@
     <xacro:include filename="$(find aist_description
 			     )/devices/urdf/_sr305.urdf.xacro"/>
-    <!-- Add the holder and two SR305 cameras -->
-    <xacro:property name="mount_mesh_file"
-		    value="package://aist_description/devices/meshes/sr305_mount_2f140.stl"/>
+    <xacro:property name="mesh_dir"
+		    value="package://aist_description/devices/meshes"/>
     <link name="${prefix}camera_mount">
       <inertial>
@@ -19,5 +18,6 @@
         <origin rpy="${pi} 0 ${pi/2}" xyz="0 0 0.0"/>
         <geometry>
-          <mesh filename="${mount_mesh_file}" scale=".001 .001 .001"/>
+          <mesh filename="${mesh_dir}/sr305_mount_2f140.stl"
+		scale=".001 .001 .001"/>
         </geometry>
         <material name="white">
@@ -26,7 +26,8 @@
       </visual>
       <collision>
-        <origin rpy="0 0 0" xyz="-.01 0.0 .035"/>
+        <origin rpy="${pi} 0 ${pi/2}" xyz="0 0 0.0"/>
         <geometry>
-          <box size=".03 .12 .08"/>
+          <mesh filename="${mesh_dir}/collision/sr305_mount_2f140.stl"
+		scale=".001 .001 .001"/>
         </geometry>
       </collision>

File: aist_description/devices/urdf/sr305_on_2f85.urdf.xacro (robot description, xacro)
@@ -7,7 +7,6 @@
     <xacro:include filename="$(find aist_description
 			     )/devices/urdf/_sr305.urdf.xacro"/>
-    <!-- Add the holder and two SR305 cameras -->
-    <xacro:property name="mount_mesh_file"
-		    value="package://aist_description/devices/meshes/sr305_mount_2f85.stl"/>
+    <xacro:property name="mesh_dir"
+		    value="package://aist_description/devices/meshes"/>
     <link name="${prefix}camera_mount">
       <inertial>
@@ -19,5 +18,6 @@
         <origin rpy="${pi} 0 ${pi/2}" xyz="0 0 0.0"/>
         <geometry>
-          <mesh filename="${mount_mesh_file}" scale=".001 .001 .001"/>
+          <mesh filename="${mesh_dir}/sr305_mount_2f85.stl"
+		scale=".001 .001 .001"/>
         </geometry>
         <material name="white">
@@ -26,7 +26,8 @@
       </visual>
       <collision>
-        <origin rpy="0 0 0" xyz="-.01 0.0 .035"/>
+        <origin rpy="${pi} 0 ${pi/2}" xyz="0 0 0.0"/>
         <geometry>
-          <box size=".03 .12 .08"/>
+          <mesh filename="${mesh_dir}/collision/sr305_mount_2f85.stl"
+		scale=".001 .001 .001"/>
         </geometry>
       </collision>

File: aist_description/scenes/urdf/a_bot_base_scene.urdf.xacro (robot description, xacro)
@@ -106,25 +106,12 @@
     <origin xyz="0 0 0 " rpy="0 0 0"/>
   </joint>
-  <gazebo reference="a_bot_wrist_2_link">
-    <gravity>true</gravity>
-  </gazebo>
-  <gazebo reference="a_bot_wrist_3_link">
-    <gravity>true</gravity>
-  </gazebo>
-  <gazebo reference="a_bot_wrist_3_joint">
-    <provideFeedback>true</provideFeedback>
-  </gazebo>
-  <gazebo>
-    <plugin name="a_bot_ftsensor" filename="libgazebo_ros_ft_sensor.so">
-      <updateRate>500.0</updateRate>
-      <topicName>/a_bot/wrench</topicName>
-      <jointName>a_bot_wrist_3_joint</jointName>
-      <noise>
-	<type>gaussian</type>
-	<mean>0.0</mean>
-	<stddev>0.003</stddev>
-      </noise>
-    </plugin>
-  </gazebo>
+  <!-- Set gazebo plugin for FT-sensors -->
+  <xacro:include filename="$(find aist_description
+			   )/devices/urdf/gazebo_ftsensor.urdf.xacro"/>
+  <xacro:gazebo_ftsensor name="a_bot_ftsensor"
+			 parent="a_bot_wrist_2_link"
+			 child="a_bot_wrist_3_link"
+			 joint="a_bot_wrist_3_joint"
+			 wrench="/a_bot/wrench"/>
   <!-- Spawn and attach gripper -->
   <xacro:include filename="$(find aist_robotiq

Commit message: Port launch files for displaying parts, fastening tools and precision gripper

File: aist_description/devices/urdf/sr305_on_2f140.urdf.xacro (robot description, xacro)
@@ -40,6 +40,6 @@
     <xacro:include filename="$(find aist_description
 			     )/scenes/urdf/load_calibration.urdf.xacro"/>
-    <xacro:load_calibration filename="$(find aist_handeye_calibration
-				      )/calib/${prefix}camera.yaml"
+    <xacro:load_calibration filename="$(find aist_description
+				      )/scenes/calib/${prefix}camera.yaml"
 			    propname="camera_origin"/>
     <xacro:sensor_sr305 name="${prefix}camera" parent="${parent}"

File: aist_description/devices/urdf/sr305_on_2f85.urdf.xacro (robot description, xacro)
@@ -40,6 +40,6 @@
     <xacro:include filename="$(find aist_description
 			     )/scenes/urdf/load_calibration.urdf.xacro"/>
-    <xacro:load_calibration filename="$(find aist_handeye_calibration
-				      )/calib/${prefix}camera.yaml"
+    <xacro:load_calibration filename="$(find aist_description
+				      )/scenes/calib/${prefix}camera.yaml"
 			    propname="camera_origin"/>
     <xacro:sensor_sr305 name="${prefix}camera" parent="${parent}"

File: aist_description/scenes/urdf/aist_base_scene.urdf.xacro (robot description, xacro)
@@ -96,7 +96,9 @@
   </xacro:suction_tool_holder>
   <!-- robot arms -->
-  <xacro:include filename="$(find ur_gazebo)/urdf/ur_macro.xacro"/>
-  <xacro:ur_robot_gazebo
-      prefix="a_bot_"
+  <xacro:include filename="$(find ur_description)/urdf/ur_macro.xacro"/>
+  <xacro:ur_robot
+      name="a_bot"
+      tf_prefix="a_bot_"
+      parent="a_bot_table_top_center"
       joint_limits_parameters_file="$(find ur_description
 				    )/config/ur5e/joint_limits.yaml"
@@ -105,11 +107,14 @@
       visual_parameters_file="$(find ur_description
 			      )/config/ur5e/visual_parameters.yaml"
-      kinematics_parameters_file="$(find aist_bringup
-				  )/config/a_bot_calibration.yaml"
-      transmission_hw_interface="hardware_interface/PositionJointInterface"
+      kinematics_parameters_file="$(find aist_description
+				  )/scenes/calib/a_bot.yaml"
       safety_limits="true"
-      safety_pos_margin="0.15"/>
-  <xacro:ur_robot_gazebo
-      prefix="b_bot_"
+      safety_pos_margin="0.15">
+    <origin xyz="0 0 0 " rpy="0 0 0"/>
+  </xacro:ur_robot>
+  <xacro:ur_robot
+      name="b_bot"
+      tf_prefix="b_bot_"
+      parent="b_bot_table_top_center"
       joint_limits_parameters_file="$(find ur_description
 				    )/config/ur5e/joint_limits.yaml"
@@ -118,44 +123,10 @@
       visual_parameters_file="$(find ur_description
 			      )/config/ur5e/visual_parameters.yaml"
-      kinematics_parameters_file="$(find aist_bringup
-				  )/config/b_bot_calibration.yaml"
-      transmission_hw_interface="hardware_interface/PositionJointInterface"
+      kinematics_parameters_file="$(find aist_description
+				  )/scenes/calib/b_bot.yaml"
       safety_limits="true"
-      safety_pos_margin="0.15"/>
-  <joint name="a_bot_base_link_joint" type="fixed">
-    <parent link="a_bot_table_top_center"/>
-    <child  link="a_bot_base_link"/>
-    <origin xyz="0 0 0 " rpy="0 0 0"/>
-  </joint>
-  <joint name="b_bot_base_link_joint" type="fixed">
-    <parent link="b_bot_table_top_center"/>
-    <child  link="b_bot_base_link"/>
+      safety_pos_margin="0.15">
     <origin xyz="0 0 0" rpy="0 0 ${b_bot_theta}"/>
-  </joint>
-  <!-- Attach mounter for Zivid2+ camera -->
-  <!-- <xacro:include filename="$(find aist_description)/devices/urdf/zivid_coupling.urdf.xacro"/> -->
-  <!-- <xacro:zivid_coupling prefix="a_bot_zivid_coupling_" parent="a_bot_flange"> -->
-  <!--   <origin xyz="0 0 0" rpy="${pi} 0 0" /> -->
-  <!-- </xacro:zivid_coupling> -->
-  <!-- Spawn and attach Zivid2+ camera -->
-  <!-- <xacro:include filename="$(find aist_description -->
-  <!-- 			   )/scenes/urdf/load_calibration.urdf.xacro"/> -->
-  <!-- <xacro:load_calibration filename="$(find aist_handeye_calibration -->
-  <!-- 				    )/calib/a_bot_zivid.yaml"/> -->
-  <!-- <xacro:include filename="$(find aist_description -->
-  <!-- 			   )/devices/urdf/zivid2plus.urdf.xacro"/> -->
-  <!-- <xacro:zivid2plus name="a_bot_zivid" -->
-  <!-- 		    parent="a_bot_zivid_coupling_flange_link"> -->
-  <!--   <origin xyz="${origin[0]} ${origin[1]} ${origin[2]}" -->
-  <!--   	    rpy="${origin[3]} ${origin[4]} ${origin[5]}"/> -->
-  <!-- </xacro:zivid2plus> -->
-  <!-- Spawn and attach force sensor -->
-  <!-- <xacro:include filename="$(find aist_robotiq)/urdf/ft300.urdf.xacro"/> -->
-  <!-- <xacro:ft300 prefix="a_bot_ftsensor_" parent="a_bot_flange"> -->
-  <!--   <origin xyz="0 0 0" rpy="${pi} 0 0"/> -->
-  <!-- </xacro:ft300> -->
-  <!-- <xacro:ft300 prefix="b_bot_ftsensor_" parent="b_bot_flange"> -->
-  <!--   <origin xyz="0 0 0" rpy="${pi} 0 0"/> -->
-  <!-- </xacro:ft300> -->
+  </xacro:ur_robot>
   <!-- Spawn and attach grippers -->
   <xacro:include filename="$(find aist_robotiq
@@ -196,6 +167,6 @@
   <xacro:include filename="$(find aist_description
 			   )/scenes/urdf/load_calibration.urdf.xacro"/>
-  <xacro:load_calibration filename="$(find aist_handeye_calibration
-				    )/calib/a_motioncam.yaml"/>
+  <xacro:load_calibration filename="$(find aist_description
+				    )/scenes/calib/a_motioncam.yaml"/>
   <xacro:include filename="$(find aist_phoxi_camera
 			   )/urdf/motioncam_m_camera.urdf.xacro"/>
@@ -205,17 +176,17 @@
   </xacro:motioncam_m_camera>
   <!-- Add RealSense cameras -->
-  <xacro:include filename="$(find aist_description
-  			   )/devices/urdf/sr305_on_2f140.urdf.xacro" />
-  <xacro:sr305_on_2f140 prefix="a_bot_"
-  			parent="a_bot_gripper_base_link"
-  			use_nominal_extrinsics="true"/>
-  <xacro:include filename="$(find aist_description
-  			   )/devices/urdf/sr305_on_2f85.urdf.xacro" />
-  <xacro:sr305_on_2f85 prefix="b_bot_"
-  		       parent="b_bot_gripper_base_link"
-  		       use_nominal_extrinsics="true"/>
+  <!-- <xacro:include filename="$(find aist_description -->
+  <!-- 			   )/devices/urdf/sr305_on_2f140.urdf.xacro" /> -->
+  <!-- <xacro:sr305_on_2f140 prefix="a_bot_" -->
+  <!-- 			parent="a_bot_gripper_base_link" -->
+  <!-- 			use_nominal_extrinsics="true"/> -->
+  <!-- <xacro:include filename="$(find aist_description -->
+  <!-- 			   )/devices/urdf/sr305_on_2f85.urdf.xacro" /> -->
+  <!-- <xacro:sr305_on_2f85 prefix="b_bot_" -->
+  <!-- 		       parent="b_bot_gripper_base_link" -->
+  <!-- 		       use_nominal_extrinsics="true"/> -->
   <!-- Add live camera -->
-  <xacro:load_calibration filename="$(find aist_camera_calibration
-				    )/calib/live_camera.yaml"/>
+  <xacro:load_calibration filename="$(find aist_description
+				    )/scenes/calib/live_camera.yaml"/>
   <link name="live_camera_optical_frame"/>
   <joint name="live_camera_joint" type="fixed">
