Commit message: WIP: Use ament_cmake_auto, edit object color

File: aist_description/devices/urdf/_d405.urdf.xacro (robot description, xacro)
@@ -20,52 +20,37 @@
     <!-- Reference should be color_frame because depth is alighed to color -->
     <gazebo reference="${name}_color_frame">
-      <sensor type="depth" name="${name}">
-	<always_on>true</always_on>
-	<visualize>true</visualize>
+      <sensor type="rgbd_camera" name="${name}">
 	<camera>
-	  <!-- Color sensor's FOV(HD): 84 deg. -->
+	  <!-- Color sensor's FOV(VGA): 68 deg. -->
           <horizontal_fov>1.4661</horizontal_fov>
-	  <!-- Color sensor's FOV(VGA): 48.47 deg. -->
-          <!-- <horizontal_fov>0.846</horizontal_fov> -->
           <image>
 	    <!-- HD -->
             <width>1280</width>
             <height>720</height>
-	    <!-- VGA -->
-            <!-- <width>640</width> -->
-            <!-- <height>480</height> -->
             <format>R8G8B8</format>
           </image>
-          <depth_camera>
-          </depth_camera>
           <clip>
             <near>0.1</near>
             <far>100</far>
           </clip>
+	  <gz_frame_id>${name}_color_frame</gz_frame_id>
+	  <optical_frame_id>${name}_color_frame</optical_frame_id>
+	  <noise>
+	    <type>gaussian</type>
+	    <mean>0.0</mean>
+	    <stddev>0.007</stddev>
+	  </noise>
+          <distortion>
+	    <k1>0.0</k1>
+	    <k2>0.0</k2>
+	    <k3>0.0</k3>
+	    <p1>0.0</p1>
+	    <p2>0.0</p2>
+	  </distortion>
 	</camera>
-	<plugin name="${name}_controller"
-		filename="libgazebo_ros_openni_kinect.so">
-          <baseline>0.018</baseline>
-          <alwaysOn>true</alwaysOn>
-          <updateRate>10.0</updateRate>
-          <cameraName>${name}</cameraName>
-          <frameName>${name}_color_optical_frame</frameName>
-          <imageTopicName>color/image_raw</imageTopicName>
-          <cameraInfoTopicName>color/camera_info</cameraInfoTopicName>
-          <depthImageTopicName>aligned_depth_to_color/image_raw</depthImageTopicName>
-          <depthImageCameraInfoTopicName>aligned_depth_to_color/camera_info</depthImageCameraInfoTopicName>
-          <pointCloudTopicName>depth/color/points</pointCloudTopicName>
-          <pointCloudCutoff>0.1</pointCloudCutoff>
-          <!-- <hackBaseline>0.07</hackBaseline> -->
-          <distortionK1>0.0</distortionK1>
-          <distortionK2>0.0</distortionK2>
-          <distortionK3>0.0</distortionK3>
-          <distortionT1>0.0</distortionT1>
-          <distortionT2>0.0</distortionT2>
-          <CxPrime>0.0</CxPrime>
-          <Cx>0.0</Cx>
-          <Cy>0.0</Cy>
-          <focalLength>0.0</focalLength>
-	</plugin>
+	<always_on>true</always_on>
+        <updateRate>10.0</updateRate>
+	<visualize>true</visualize>
+	<topic>${name}</topic>
       </sensor>
     </gazebo>

File: aist_description/devices/urdf/_d415.urdf.xacro (robot description, xacro)
@@ -20,52 +20,37 @@
     <!-- Reference should be color_frame because depth is alighed to color -->
     <gazebo reference="${name}_color_frame">
-      <sensor type="depth" name="${name}">
-	<always_on>true</always_on>
-	<visualize>true</visualize>
+      <sensor type="rgbd_camera" name="${name}">
 	<camera>
-	  <!-- Color sensor's FOV(HD): 69 deg. -->
+	  <!-- Color sensor's FOV(VGA): 68 deg. -->
           <horizontal_fov>1.2043</horizontal_fov>
-	  <!-- Color sensor's FOV(VGA): 42.27 deg. -->
-          <!-- <horizontal_fov>0.9091</horizontal_fov> -->
           <image>
 	    <!-- HD -->
             <width>1280</width>
             <height>720</height>
-	    <!-- VGA -->
-            <!-- <width>640</width> -->
-            <!-- <height>480</height> -->
             <format>R8G8B8</format>
           </image>
-          <depth_camera>
-          </depth_camera>
           <clip>
             <near>0.1</near>
             <far>100</far>
           </clip>
+	  <gz_frame_id>${name}_color_frame</gz_frame_id>
+	  <optical_frame_id>${name}_color_frame</optical_frame_id>
+	  <noise>
+	    <type>gaussian</type>
+	    <mean>0.0</mean>
+	    <stddev>0.007</stddev>
+	  </noise>
+          <distortion>
+	    <k1>0.0</k1>
+	    <k2>0.0</k2>
+	    <k3>0.0</k3>
+	    <p1>0.0</p1>
+	    <p2>0.0</p2>
+	  </distortion>
 	</camera>
-	<plugin name="${name}_controller"
-		filename="libgazebo_ros_openni_kinect.so">
-          <baseline>0.055</baseline>
-          <alwaysOn>true</alwaysOn>
-          <updateRate>10.0</updateRate>
-          <cameraName>${name}</cameraName>
-          <frameName>${name}_color_optical_frame</frameName>
-          <imageTopicName>color/image_raw</imageTopicName>
-          <cameraInfoTopicName>color/camera_info</cameraInfoTopicName>
-          <depthImageTopicName>aligned_depth_to_color/image_raw</depthImageTopicName>
-          <depthImageCameraInfoTopicName>aligned_depth_to_color/camera_info</depthImageCameraInfoTopicName>
-          <pointCloudTopicName>depth/color/points</pointCloudTopicName>
-          <pointCloudCutoff>0.1</pointCloudCutoff>
-          <!-- <hackBaseline>0.07</hackBaseline> -->
-          <distortionK1>0.0</distortionK1>
-          <distortionK2>0.0</distortionK2>
-          <distortionK3>0.0</distortionK3>
-          <distortionT1>0.0</distortionT1>
-          <distortionT2>0.0</distortionT2>
-          <CxPrime>0.0</CxPrime>
-          <Cx>0.0</Cx>
-          <Cy>0.0</Cy>
-          <focalLength>0.0</focalLength>
-	</plugin>
+	<always_on>true</always_on>
+        <updateRate>10.0</updateRate>
+	<visualize>true</visualize>
+	<topic>${name}</topic>
       </sensor>
     </gazebo>

File: aist_description/devices/urdf/_d435.urdf.xacro (robot description, xacro)
@@ -20,52 +20,37 @@
     <!-- Reference should be color_frame because depth is alighed to color -->
     <gazebo reference="${name}_color_frame">
-      <sensor type="depth" name="${name}">
-	<always_on>true</always_on>
-	<visualize>true</visualize>
+      <sensor type="rgbd_camera" name="${name}">
 	<camera>
-	  <!-- Color sensor's FOV(HD): 69 deg. -->
+	  <!-- Color sensor's FOV(VGA): 68 deg. -->
           <horizontal_fov>1.2043</horizontal_fov>
-	  <!-- Color sensor's FOV(VGA): 42.27 deg. -->
-          <!-- <horizontal_fov>0.9091</horizontal_fov> -->
           <image>
 	    <!-- HD -->
             <width>1280</width>
             <height>720</height>
-	    <!-- VGA -->
-            <!-- <width>640</width> -->
-            <!-- <height>480</height> -->
             <format>R8G8B8</format>
           </image>
-          <depth_camera>
-          </depth_camera>
           <clip>
             <near>0.1</near>
             <far>100</far>
           </clip>
+	  <gz_frame_id>${name}_color_frame</gz_frame_id>
+	  <optical_frame_id>${name}_color_frame</optical_frame_id>
+	  <noise>
+	    <type>gaussian</type>
+	    <mean>0.0</mean>
+	    <stddev>0.007</stddev>
+	  </noise>
+          <distortion>
+	    <k1>0.0</k1>
+	    <k2>0.0</k2>
+	    <k3>0.0</k3>
+	    <p1>0.0</p1>
+	    <p2>0.0</p2>
+	  </distortion>
 	</camera>
-	<plugin name="${name}_controller"
-		filename="libgazebo_ros_openni_kinect.so">
-          <baseline>0.050</baseline>
-          <alwaysOn>true</alwaysOn>
-          <updateRate>10.0</updateRate>
-          <cameraName>${name}</cameraName>
-          <frameName>${name}_color_optical_frame</frameName>
-          <imageTopicName>color/image_raw</imageTopicName>
-          <cameraInfoTopicName>color/camera_info</cameraInfoTopicName>
-          <depthImageTopicName>aligned_depth_to_color/image_raw</depthImageTopicName>
-          <depthImageCameraInfoTopicName>aligned_depth_to_color/camera_info</depthImageCameraInfoTopicName>
-          <pointCloudTopicName>depth/color/points</pointCloudTopicName>
-          <pointCloudCutoff>0.1</pointCloudCutoff>
-          <!-- <hackBaseline>0.07</hackBaseline> -->
-          <distortionK1>0.0</distortionK1>
-          <distortionK2>0.0</distortionK2>
-          <distortionK3>0.0</distortionK3>
-          <distortionT1>0.0</distortionT1>
-          <distortionT2>0.0</distortionT2>
-          <CxPrime>0.0</CxPrime>
-          <Cx>0.0</Cx>
-          <Cy>0.0</Cy>
-          <focalLength>0.0</focalLength>
-	</plugin>
+	<always_on>true</always_on>
+        <updateRate>10.0</updateRate>
+	<visualize>true</visualize>
+	<topic>${name}</topic>
       </sensor>
     </gazebo>

File: aist_description/devices/urdf/_sr305.urdf.xacro (robot description, xacro)
@@ -17,7 +17,5 @@
     <!-- Reference should be color_frame because depth is alighed to color -->
     <gazebo reference="${name}_color_frame">
-      <sensor type="depth" name="${name}">
-	<always_on>true</always_on>
-	<visualize>true</visualize>
+      <sensor type="rgbd_camera" name="${name}">
 	<camera>
 	  <!-- Color sensor's FOV(VGA): 68 deg. -->
@@ -29,35 +27,27 @@
             <format>R8G8B8</format>
           </image>
-          <depth_camera>
-          </depth_camera>
           <clip>
             <near>0.1</near>
             <far>100</far>
           </clip>
+	  <gz_frame_id>${name}_color_frame</gz_frame_id>
+	  <optical_frame_id>${name}_color_frame</optical_frame_id>
+	  <noise>
+	    <type>gaussian</type>
+	    <mean>0.0</mean>
+	    <stddev>0.007</stddev>
+	  </noise>
+          <distortion>
+	    <k1>0.0</k1>
+	    <k2>0.0</k2>
+	    <k3>0.0</k3>
+	    <p1>0.0</p1>
+	    <p2>0.0</p2>
+	  </distortion>
 	</camera>
-	<plugin name="${name}_controller"
-		filename="libgazebo_ros_openni_kinect.so">
-          <baseline>0.048</baseline>
-          <alwaysOn>true</alwaysOn>
-          <updateRate>10.0</updateRate>
-          <cameraName>${name}</cameraName>
-          <frameName>${name}_color_optical_frame</frameName>
-          <imageTopicName>color/image_raw</imageTopicName>
-          <cameraInfoTopicName>color/camera_info</cameraInfoTopicName>
-          <depthImageTopicName>aligned_depth_to_color/image_raw</depthImageTopicName>
-          <depthImageCameraInfoTopicName>aligned_depth_to_color/camera_info</depthImageCameraInfoTopicName>
-          <pointCloudTopicName>depth/color/points</pointCloudTopicName>
-          <pointCloudCutoff>0.1</pointCloudCutoff>
-          <!-- <hackBaseline>0.07</hackBaseline> -->
-          <distortionK1>0.0</distortionK1>
-          <distortionK2>0.0</distortionK2>
-          <distortionK3>0.0</distortionK3>
-          <distortionT1>0.0</distortionT1>
-          <distortionT2>0.0</distortionT2>
-          <CxPrime>0.0</CxPrime>
-          <Cx>0.0</Cx>
-          <Cy>0.0</Cy>
-          <focalLength>0.0</focalLength>
-	</plugin>
+	<always_on>true</always_on>
+        <updateRate>10.0</updateRate>
+	<visualize>true</visualize>
+	<topic>${name}</topic>
       </sensor>
     </gazebo>

File: aist_description/devices/urdf/ur_robot_with_ros2_control.urdf.xacro (robot description, xacro)
@@ -5,5 +5,4 @@
 		       ur_type
 		       name
-		       tf_prefix
 		       parent
 		       *origin
@@ -40,5 +39,5 @@
     <xacro:ur_robot
 	name="${name}"
-	tf_prefix="${tf_prefix}"
+	tf_prefix="${name}_"
 	parent="${parent}"
 	joint_limits_parameters_file="$(find ur_description
@@ -62,5 +61,5 @@
       <xacro:ur_ros2_control
 	  name="${name}"
-	  tf_prefix="${tf_prefix}"
+	  tf_prefix="${name}_"
 	  kinematics_parameters_file="$(find aist_description
 				      )/scenes/calib/${name}.yaml"
@@ -97,5 +96,5 @@
       <xacro:ur_ros2_control
 	  name="${name}"
-	  tf_prefix="${tf_prefix}"
+	  tf_prefix="${name}_"
 	  transmission_hw_interface="${transmission_hw_interface}"
 	  initial_positions="${initial_positions}"/>
@@ -104,4 +103,5 @@
 		name="gz_ros2_control::GazeboSimROS2ControlPlugin">
 	  <parameters>${simulation_controllers}</parameters>
+	  <controller_manager_node_name>${name}_controller_manager</controller_manager_node_name>
 	  <ros>
 	    <namepsace>${name}</namepsace>

File: aist_description/objects/urdf/aist_box.urdf.xacro (robot description, xacro)
@@ -3,5 +3,5 @@
   <xacro:macro name="aist_box"
 	       params="name width length height parent
-		       rgba:='0.7 0.7 0.7 1' color_name:=aist_color mass:=1.0
+		       rgba:='0.7 0.7 0.7 1' mass:=1.0
 		       *origin">
     <xacro:include filename="$(find aist_description
@@ -14,5 +14,5 @@
           <box size="${width} ${length} ${height}"/>
         </geometry>
-        <material name="${color_name}">
+        <material name="">
           <color rgba="${rgba}"/>
         </material>
@@ -31,7 +31,4 @@
       </inertial>
     </link>
-    <gazebo reference="${name}">
-      <material>Gazebo/${color_name}</material>
-    </gazebo>
     <joint name="${name}_joint" type="fixed">
       <parent link="${parent}"/>

File: aist_description/objects/urdf/screw_feeder.urdf.xacro (robot description, xacro)
@@ -21,5 +21,5 @@
 		    width="${back_width}" length="${length}"
 		    height="${back_height}"
-		    rgba="0.2 0.2 0.2 1.0" color_name="black">
+		    rgba="0.2 0.2 0.2 1.0">
       <xacro:insert_block name="origin"/>
     </xacro:aist_box>
@@ -28,5 +28,5 @@
 		    width="${front_width}" length="${front_left_length}"
 		    height="${front_height}"
-		    rgba="0.2 0.2 0.2 1.0" color_name="black">
+		    rgba="0.2 0.2 0.2 1.0">
       <origin xyz="${back_width} 0 0" rpy="0 0 0"/>
     </xacro:aist_box>
@@ -35,5 +35,5 @@
 		    width="${front_width}" length="${front_right_length}"
 		    height="${front_height}"
-		    rgba="0.2 0.2 0.2 1.0" color_name="black">
+		    rgba="0.2 0.2 0.2 1.0">
       <origin xyz="${back_width} ${front_left_length + gap_width} 0"
 	      rpy="0 0 0"/>
@@ -43,5 +43,5 @@
 		    width="${front_width}" length="${gap_width}"
 		    height="${gap_height}"
-		    rgba="0.6 0.6 0.6 1.0" color_name="grey">
+		    rgba="0.6 0.6 0.6 1.0">
       <origin xyz="0 ${front_left_length} 0" rpy="0 0 0"/>
     </xacro:aist_box>

File: aist_description/objects/urdf/table.urdf.xacro (robot description, xacro)
@@ -13,5 +13,5 @@
 		    height="${height - table_thickness}"
 		    parent="${parent}"
-		    rgba="${rgba}" color_name="${prefix}table_color">
+		    rgba="${rgba}">
       <xacro:insert_block name="origin"/>
     </xacro:aist_box>
@@ -21,5 +21,5 @@
 		    height="${height - table_thickness}"
 		    parent="${prefix}base_link"
-		    rgba="${rgba}" color_name="${prefix}table_color">
+		    rgba="${rgba}">
       <origin xyz="${width - table_leg_thickness} 0 0" rpy="0 0 0"/>
     </xacro:aist_box>
@@ -29,5 +29,5 @@
 		    height="${height - table_thickness}"
 		    parent="${prefix}base_link"
-		    rgba="${rgba}" color_name="${prefix}table_color">
+		    rgba="${rgba}">
       <origin xyz="0 ${length - table_leg_thickness} 0" rpy="0 0 0"/>
     </xacro:aist_box>
@@ -37,5 +37,5 @@
 		    height="${height - table_thickness}"
 		    parent="${prefix}base_link"
-		    rgba="${rgba}" color_name="${prefix}table_color">
+		    rgba="${rgba}">
       <origin xyz="${width  - table_leg_thickness}
 		   ${length - table_leg_thickness}
@@ -48,5 +48,5 @@
 		    height="${table_thickness}"
 		    parent="${prefix}base_link"
-		    rgba="${rgba}" color_name="${prefix}table_color">
+		    rgba="${rgba}">
       <origin xyz="0 0 ${height - table_thickness}" rpy="0 0 0"/>
     </xacro:aist_box>

File: aist_description/objects/urdf/usb_repeater.urdf.xacro (robot description, xacro)
@@ -23,5 +23,5 @@
             <cylinder radius="${radius}" length="${thickness}"/>
           </geometry>
-          <material name="White">
+          <material name="">
             <color rgba="1.0 1.0 1.0 1.0"/>
           </material>
@@ -39,7 +39,4 @@
 	</inertial>
       </link>
-      <gazebo reference="${name}">
-	<material>Gazebo/White</material>
-      </gazebo>
       <joint name="${name}_joint" type="fixed">
 	<parent link="${parent}"/>
@@ -81,5 +78,5 @@
           <box size="${repeater_width} ${repeater_length} ${repeater_height}"/>
         </geometry>
-        <material name="Black">
+        <material name="">
           <color rgba="0.0 0.0 0.0 1.0"/>
         </material>
@@ -97,7 +94,4 @@
       </inertial>
     </link>
-    <gazebo reference="${prefix}body">
-      <material>Gazebo/Black</material>
-    </gazebo>
     <joint name="${prefix}body_joint" type="fixed">
       <parent link="${prefix}plate"/>

File: aist_description/parts/urdf/object.urdf.xacro (robot description, xacro)
@@ -47,5 +47,5 @@
     	      scale="${scale[0]} ${scale[1]} ${scale[2]}"/>
       </geometry>
-      <material name="${name}/color_${id}">
+      <material name="">
 	<color rgba="${color[0]} ${color[1]} ${color[2]} ${color[3]}"/>
       </material>

File: aist_description/scenes/urdf/a_bot_base_scene.urdf.xacro (robot description, xacro)
@@ -67,5 +67,5 @@
   <xacro:table prefix="a_bot_table_"
 	       width="${bot_table_size}" length="${bot_table_size}"
-	       height="${a_bot_z}" parent="ground">
+	       height="${a_bot_z}" rgba="0.0 0.1 0.3 1" parent="ground">
     <origin xyz="${a_bot_x - bot_table_size/2} ${a_bot_y - bot_table_size/2} 0"
 	    rpy="0 0 0"/>
@@ -106,5 +106,4 @@
       simulation_controllers="$(arg simulation_controllers)"
       ur_type="ur5e"
-      tf_prefix="a_bot_"
       parent="a_bot_table_top_center"
       safety_limits="true"
@@ -122,11 +121,11 @@
   </xacro:ur_robot_with_ros2_control>
   <!-- Set gazebo plugin for FT-sensors -->
-  <xacro:include filename="$(find aist_description
-			   )/devices/urdf/gazebo_ftsensor.urdf.xacro"/>
-  <xacro:gazebo_ftsensor name="a_bot_ftsensor"
-			 parent="a_bot_wrist_2_link"
-			 child="a_bot_wrist_3_link"
-			 joint="a_bot_wrist_3_joint"
-			 wrench="/a_bot/wrench"/>
+  <!-- <xacro:include filename="$(find aist_description -->
+  <!-- 			   )/devices/urdf/gazebo_ftsensor.urdf.xacro"/> -->
+  <!-- <xacro:gazebo_ftsensor name="a_bot_ftsensor" -->
+  <!-- 			 parent="a_bot_wrist_2_link" -->
+  <!-- 			 child="a_bot_wrist_3_link" -->
+  <!-- 			 joint="a_bot_wrist_3_joint" -->
+  <!-- 			 wrench="/a_bot/wrench"/> -->
   <!-- Spawn and attach gripper -->
   <xacro:include filename="$(find aist_robotiq
@@ -150,4 +149,15 @@
     <origin xyz="0.000 -0.051 0.000" rpy="${pi/2} ${-pi/2} 0"/>
   </xacro:usb_repeater>
+  <!-- Add Motioncam-3D scanner -->
+  <xacro:include filename="$(find aist_description
+			   )/scenes/urdf/load_calibration.urdf.xacro"/>
+  <xacro:load_calibration filename="$(find aist_description
+				    )/scenes/calib/a_motioncam.yaml"/>
+  <xacro:include filename="$(find aist_phoxi_camera
+			   )/urdf/motioncam_m_camera.urdf.xacro"/>
+  <xacro:motioncam_m_camera name="a_motioncam" parent="workspace_center">
+    <origin xyz="${origin[0]} ${origin[1]} ${origin[2]}"
+    	    rpy="${origin[3]} ${origin[4]} ${origin[5]}"/>
+  </xacro:motioncam_m_camera>
   <!-- RealSense cameras -->
   <xacro:include filename="$(find aist_description
@@ -171,5 +181,12 @@
 			     scene).urdf.xacro"/>
   </xacro:if>
-  <gazebo reference="world">
-  </gazebo>
+  <xacro:if value="${'$(arg simulation_controllers)' != ''}">
+    <gazebo reference="world">
+    </gazebo>
+    <!-- <gazebo> -->
+    <!--   <plugin filename="gz_ros2_control-system" name="gz::"> -->
+    <!-- 	<render_engine>ogre2</render_engine> -->
+    <!--   </plugin> -->
+    <!-- </gazebo> -->
+  </xacro:if>
 </robot>

File: aist_description/scenes/urdf/aist_base_scene.urdf.xacro (robot description, xacro)
@@ -72,5 +72,5 @@
   <xacro:table prefix="a_bot_table_"
 	       width="${bot_table_size}" length="${bot_table_size}"
-	       height="${a_bot_z}" parent="ground">
+	       height="${a_bot_z}" rgba="0.0 0.1 0.3 1" parent="ground">
     <origin xyz="${a_bot_x - bot_table_size/2} ${a_bot_y - bot_table_size/2} 0"
 	    rpy="0 0 0"/>
@@ -78,5 +78,5 @@
   <xacro:table prefix="b_bot_table_"
 	       width="${bot_table_size}" length="${bot_table_size}"
-	       height="${b_bot_z}" parent="ground">
+	       height="${b_bot_z}" rgba="0.0 0.1 0.3 1" parent="ground">
     <origin xyz="${b_bot_x - bot_table_size/2} ${b_bot_y - bot_table_size/2} 0"
 	    rpy="0 0 0"/>
@@ -117,5 +117,4 @@
       ur_type="ur5e"
       name="a_bot"
-      tf_prefix="a_bot_"
       parent="a_bot_table_top_center"
       safety_limits="true"
@@ -136,5 +135,4 @@
       ur_type="ur5e"
       name="b_bot"
-      tf_prefix="b_bot_"
       parent="b_bot_table_top_center"
       safety_limits="true"

File: aist_description/scenes/urdf/b_bot_base_scene.urdf.xacro (robot description, xacro)
@@ -69,5 +69,5 @@
   <xacro:table prefix="b_bot_table_"
 	       width="${bot_table_size}" length="${bot_table_size}"
-	       height="${b_bot_z}" parent="ground">
+	       height="${b_bot_z}" rgba="0.0 0.1 0.3 1" parent="ground">
     <origin xyz="${b_bot_x - bot_table_size/2} ${b_bot_y - bot_table_size/2} 0"
 	    rpy="0 0 0"/>
@@ -101,5 +101,4 @@
       simulation_controllers="$(arg simulation_controllers)"
       ur_type="ur5e"
-      tf_prefix="b_bot_"
       parent="b_bot_table_top_center"
       safety_limits="true"

File: aist_description/wrc/urdf/base_fixture.urdf.xacro (robot description, xacro)
@@ -13,5 +13,5 @@
         <mesh filename="${top_mesh}" scale=".0001 .0001 .0001"/>
       </geometry>
-      <material name="white">
+      <material name="">
         <color rgba=".9 .9 .9 1"/>
       </material>
@@ -49,5 +49,5 @@
         <box size=".02 ${length} .08"/>
       </geometry>
-      <material name="grey">
+      <material name="">
         <color rgba=".4 .4 .4 1"/>
       </material>
@@ -72,5 +72,5 @@
         <!-- <mesh filename="${long_bar_mesh}" scale=".001 .001 .001"/> -->
       </geometry>
-      <material name="grey">
+      <material name="">
         <color rgba=".4 .4 .4 1"/>
       </material>
@@ -95,5 +95,5 @@
         <!-- <mesh filename="${long_bar_mesh}" scale=".001 .001 .001"/> -->
       </geometry>
-      <material name="grey">
+      <material name="">
         <color rgba=".4 .4 .4 1"/>
       </material>
@@ -118,5 +118,5 @@
         <!-- <mesh filename="${long_bar_mesh}" scale=".001 .001 .001"/> -->
       </geometry>
-      <material name="grey">
+      <material name="">
         <color rgba=".4 .4 .4 1"/>
       </material>

File: aist_description/wrc/urdf/kitting_bins.urdf.xacro (robot description, xacro)
@@ -19,5 +19,5 @@
           <mesh filename="${mesh_file}" scale="0.001 0.001 0.001"/>
         </geometry>
-        <material name="orange">
+        <material name="">
           <color rgba="1 0.5088 0.0468 1"/>
         </material>
@@ -30,7 +30,4 @@
       </collision>
     </link>
-    <gazebo reference="${binname}">
-      <material>Gazebo/Orange</material>
-    </gazebo>
     <joint name="${binname}_joint" type="fixed">
       <parent link="${parent}" />

File: aist_description/wrc/urdf/kitting_trays.urdf.xacro (robot description, xacro)
@@ -24,6 +24,6 @@
           <mesh filename="${mesh_file}" scale="0.001 0.001 0.001"/>
         </geometry>
-        <material name="white">
-          <color rgba="1 1 1 1"/>
+        <material name="">
+          <color rgba="0 0.5 1 1"/>
         </material>
       </visual>
@@ -50,6 +50,6 @@
           <mesh filename="package://aist_description/wrc/meshes/${contents}.stl" scale="0.001 0.001 0.001" />
 	</geometry>
-	<material name="white">
-          <color rgba="1 1 1 1"/>
+	<material name="">
+          <color rgba="0 0 0 1"/>
 	</material>
       </visual>
