Commit message: WIP: Use ament_cmake_auto, edit object color

File: aist_fastening_tools/urdf/base_fixture.urdf.xacro (robot description, xacro)
@@ -46,5 +46,5 @@
 		scale="${body_vscale[0]} ${body_vscale[1]} ${body_vscale[2]}"/>
         </geometry>
-        <material name="Gazebo/Black">
+        <material name="">
           <color rgba="${body_vcolor[0]} ${body_vcolor[1]}
 		       ${body_vcolor[2]} ${body_vcolor[3]}"/>
@@ -106,5 +106,5 @@
 		       ${piston_vscale[2]}"/>
         </geometry>
-        <material name="Gazebo/Grey">
+        <material name="">
           <color rgba="${piston_vcolor[0]} ${piston_vcolor[1]}
       		       ${piston_vcolor[2]} ${piston_vcolor[3]}"/>
@@ -166,10 +166,4 @@
     </joint>
     <link name="${prefix}piston_head"/>
-    <gazebo reference="${prefix}base_link">
-      <material>Gazebo/FlatBlack</material>
-    </gazebo>
-    <gazebo reference="${prefix}piston">
-      <material>Gazebo/Grey</material>
-    </gazebo>
     <!-- Improve grasping physics -->
     <gazebo reference="${prefix}piston">

File: aist_precision_gripper/urdf/precision_gripper.urdf.xacro (robot description, xacro)
@@ -46,5 +46,5 @@
 		scale="${base_vscale[0]} ${base_vscale[1]} ${base_vscale[2]}"/>
         </geometry>
-        <material name="Gazebo/Black">
+        <material name="">
           <color rgba="${base_vcolor[0]} ${base_vcolor[1]}
 		       ${base_vcolor[2]} ${base_vcolor[3]}"/>
@@ -101,5 +101,5 @@
 		       ${left_finger_vscale[2]}"/>
         </geometry>
-        <material name="Gazebo/Grey">
+        <material name="">
           <color rgba="${left_finger_vcolor[0]} ${left_finger_vcolor[1]}
 		       ${left_finger_vcolor[2]} ${left_finger_vcolor[3]}"/>
@@ -159,5 +159,5 @@
 		       ${right_finger_vscale[2]}"/>
         </geometry>
-        <material name="Gazebo/Grey">
+        <material name="">
           <color rgba="${right_finger_vcolor[0]} ${right_finger_vcolor[1]}
 		       ${right_finger_vcolor[2]} ${right_finger_vcolor[3]}"/>
@@ -199,13 +199,4 @@
     </joint>
     <link name="${prefix}tip_link"/>
-    <gazebo reference="${prefix}base_link">
-      <material>Gazebo/FlatBlack</material>
-    </gazebo>
-    <gazebo reference="${prefix}left_finger">
-      <material>Gazebo/Grey</material>
-    </gazebo>
-    <gazebo reference="${prefix}right_finger">
-      <material>Gazebo/Grey</material>
-    </gazebo>
     <!-- Improve grasping physics -->
     <gazebo reference="${prefix}left_finger">
@@ -224,11 +215,26 @@
     </gazebo>
     <!-- Mimic joints -->
+    <ros2_control name="GazeboSystem" type="system">
+      <hardware>
+	<plugin>gz_ros2_control/GazeboSimSystem</plugin>
+      </hardware>
+      <joint name="${prefix}finger_joint">
+	<command_interface name="position"/>
+	<state_interface name="position">
+          <param name="initial_value">0.15</param>
+	</state_interface>
+	<state_interface name="velocity"/>
+	<state_interface name="effort"/>
+      </joint>
+      <joint name="${prefix}right_finger_joint">
+	<state_interface name="position"/>
+	<state_interface name="velocity"/>
+	<state_interface name="effort"/>
+      </joint>
+    </ros2_control>
     <gazebo>
-      <plugin filename="libgazebo_mimic_joint_plugin.so"
-	      name="${prefix}mimic_precision">
-        <joint>${prefix}finger_joint</joint>
-        <mimicJoint>${prefix}right_finger_joint</mimicJoint>
-        <multiplier>1.0</multiplier>
-        <offset>0.0</offset>
+      <plugin filename="gz_ros2_control-system"
+	      name="gz_ros2_control::GazeboSimROS2ControlPlugin">
+	<parameters>$(find gz_ros2_control_demos)/config/gripper_controller_position.yaml</parameters>
       </plugin>
     </gazebo>

File: aist_robotiq/aist_robotiq/urdf/robotiq_140_gripper.urdf.xacro (robot description, xacro)
@@ -24,7 +24,5 @@
         </geometry>
         <material name="">
-          <color rgba="0.792156862745098
-		       0.819607843137255
-		       0.933333333333333 1"/>
+          <color rgba="0.9 0.9 0.9 1"/>
         </material>
       </visual>
@@ -36,7 +34,4 @@
       </collision>
     </link>
-    <gazebo reference="${prefix}${fingerprefix}_outer_knuckle">
-      <material>Gazebo/White</material>
-    </gazebo>
   </xacro:macro>
   <xacro:macro name="outer_finger" params="prefix fingerprefix stroke">
@@ -61,5 +56,5 @@
         </geometry>
         <material name="">
-          <color rgba="0.1 0.1 0.1 1"/>
+          <color rgba="0 0 0 1"/>
         </material>
       </visual>
@@ -71,7 +66,4 @@
       </collision>
     </link>
-    <gazebo reference="${prefix}${fingerprefix}_outer_finger">
-      <material>Gazebo/Black</material>
-    </gazebo>
   </xacro:macro>
   <xacro:macro name="inner_knuckle" params="prefix fingerprefix stroke">
@@ -96,5 +88,5 @@
         </geometry>
         <material name="">
-          <color rgba="0.1 0.1 0.1 1"/>
+          <color rgba="0 0 0 1"/>
         </material>
       </visual>
@@ -106,7 +98,4 @@
       </collision>
     </link>
-    <gazebo reference="${prefix}${fingerprefix}_inner_knuckle">
-      <material>Gazebo/Black</material>
-    </gazebo>
   </xacro:macro>
   <xacro:macro name="inner_finger" params="prefix fingerprefix stroke">
@@ -131,5 +120,5 @@
         </geometry>
         <material name="">
-          <color rgba="0.1 0.1 0.1 1"/>
+          <color rgba="0 0 0 1"/>
         </material>
       </visual>
@@ -141,7 +130,4 @@
       </collision>
     </link>
-    <gazebo reference="${prefix}${fingerprefix}_inner_finger">
-      <material>Gazebo/White</material>
-    </gazebo>
   </xacro:macro>
   <!-- Finger pad link, the default are the "big pads" with rubber-->
@@ -167,7 +153,4 @@
       </collision>
     </link>
-    <gazebo reference="${prefix}${fingerprefix}_inner_finger_pad">
-      <material>Gazebo/Black</material>
-    </gazebo>
   </xacro:macro>
   <xacro:macro name="short_inner_finger_pad" params="prefix fingerprefix">
@@ -289,33 +272,46 @@
     <xacro:robotiq_arg2f_transmission prefix="${prefix}"/>
     <!-- Mimic joints -->
+    <ros2_control name="GazeboSystem" type="system">
+      <hardware>
+	<plugin>gz_ros2_control/GazeboSimSystem</plugin>
+      </hardware>
+      <joint name="${prefix}finger_joint">
+	<command_interface name="position"/>
+	<state_interface name="position">
+          <param name="initial_value">0.15</param>
+	</state_interface>
+	<state_interface name="velocity"/>
+	<state_interface name="effort"/>
+      </joint>
+      <joint name="${prefix}right_outer_knuckle_joint">
+	<state_interface name="position"/>
+	<state_interface name="velocity"/>
+	<state_interface name="effort"/>
+      </joint>
+      <joint name="${prefix}left_inner_knuckle_joint">
+	<state_interface name="position"/>
+	<state_interface name="velocity"/>
+	<state_interface name="effort"/>
+      </joint>
+      <joint name="${prefix}right_inner_knuckle_joint">
+	<state_interface name="position"/>
+	<state_interface name="velocity"/>
+	<state_interface name="effort"/>
+      </joint>
+      <joint name="${prefix}left_inner_finger_joint">
+	<state_interface name="position"/>
+	<state_interface name="velocity"/>
+	<state_interface name="effort"/>
+      </joint>
+      <joint name="${prefix}right_inner_finger_joint">
+	<state_interface name="position"/>
+	<state_interface name="velocity"/>
+	<state_interface name="effort"/>
+      </joint>
+    </ros2_control>
     <gazebo>
-      <plugin filename="libgazebo_mimic_joint_plugin.so"
-	      name="${prefix}mimic_right_outer_knuckle_joint">
-        <joint>${prefix}finger_joint</joint>
-        <mimicJoint>${prefix}right_outer_knuckle_joint</mimicJoint>
-      </plugin>
-      <plugin filename="libgazebo_mimic_joint_plugin.so"
-	      name="${prefix}mimic_left_inner_knuckle_joint">
-        <joint>${prefix}finger_joint</joint>
-        <mimicJoint>${prefix}left_inner_knuckle_joint</mimicJoint>
-      </plugin>
-      <plugin filename="libgazebo_mimic_joint_plugin.so"
-	      name="${prefix}mimic_right_inner_knuckle_joint">
-        <joint>${prefix}finger_joint</joint>
-        <mimicJoint>${prefix}right_inner_knuckle_joint</mimicJoint>
-      </plugin>
-      <plugin filename="libgazebo_mimic_joint_plugin.so"
-	      name="${prefix}mimic_left_inner_finger_joint">
-        <joint>${prefix}finger_joint</joint>
-        <mimicJoint>${prefix}left_inner_finger_joint</mimicJoint>
-        <multiplier>-1.0</multiplier>
-        <offset>0.0</offset>
-      </plugin>
-      <plugin filename="libgazebo_mimic_joint_plugin.so"
-	      name="${prefix}mimic_right_inner_finger_joint">
-        <joint>${prefix}finger_joint</joint>
-        <mimicJoint>${prefix}right_inner_finger_joint</mimicJoint>
-        <multiplier>-1.0</multiplier>
-        <offset>0.0</offset>
+      <plugin filename="gz_ros2_control-system"
+	      name="gz_ros2_control::GazeboSimROS2ControlPlugin">
+	<parameters>$(find gz_ros2_control_demos)/config/gripper_controller_position.yaml</parameters>
       </plugin>
     </gazebo>

File: aist_robotiq/aist_robotiq/urdf/robotiq_85_gripper.urdf.xacro (robot description, xacro)
@@ -25,7 +25,5 @@
         </geometry>
         <material name="">
-          <color rgba="0.792156862745098
-		       0.819607843137255
-		       0.933333333333333 1"/>
+          <color rgba="0.9 0.9 0.9 1"/>
         </material>
       </visual>
@@ -60,5 +58,5 @@
         </geometry>
         <material name="">
-          <color rgba="0.1 0.1 0.1 1"/>
+          <color rgba="0 0 0 1"/>
         </material>
       </visual>
@@ -93,5 +91,5 @@
         </geometry>
         <material name="">
-          <color rgba="0.1 0.1 0.1 1"/>
+          <color rgba="0 0 0 1"/>
         </material>
       </visual>
@@ -127,5 +125,5 @@
         </geometry>
         <material name="">
-          <color rgba="0.1 0.1 0.1 1"/>
+          <color rgba="0 0 0 1"/>
         </material>
       </visual>
@@ -250,33 +248,46 @@
     <xacro:robotiq_arg2f_transmission prefix="${prefix}"/>
     <!-- Mimic joints -->
+    <ros2_control name="GazeboSystem" type="system">
+      <hardware>
+	<plugin>gz_ros2_control/GazeboSimSystem</plugin>
+      </hardware>
+      <joint name="${prefix}finger_joint">
+	<command_interface name="position"/>
+	<state_interface name="position">
+          <param name="initial_value">0.15</param>
+	</state_interface>
+	<state_interface name="velocity"/>
+	<state_interface name="effort"/>
+      </joint>
+      <joint name="${prefix}right_outer_knuckle_joint">
+	<state_interface name="position"/>
+	<state_interface name="velocity"/>
+	<state_interface name="effort"/>
+      </joint>
+      <joint name="${prefix}left_inner_knuckle_joint">
+	<state_interface name="position"/>
+	<state_interface name="velocity"/>
+	<state_interface name="effort"/>
+      </joint>
+      <joint name="${prefix}right_inner_knuckle_joint">
+	<state_interface name="position"/>
+	<state_interface name="velocity"/>
+	<state_interface name="effort"/>
+      </joint>
+      <joint name="${prefix}left_inner_finger_joint">
+	<state_interface name="position"/>
+	<state_interface name="velocity"/>
+	<state_interface name="effort"/>
+      </joint>
+      <joint name="${prefix}right_inner_finger_joint">
+	<state_interface name="position"/>
+	<state_interface name="velocity"/>
+	<state_interface name="effort"/>
+      </joint>
+    </ros2_control>
     <gazebo>
-      <plugin filename="libgazebo_mimic_joint_plugin.so"
-	      name="${prefix}mimic_right_outer_knuckle_joint">
-        <joint>${prefix}finger_joint</joint>
-        <mimicJoint>${prefix}right_outer_knuckle_joint</mimicJoint>
-      </plugin>
-      <plugin filename="libgazebo_mimic_joint_plugin.so"
-	      name="${prefix}mimic_left_inner_knuckle_joint">
-        <joint>${prefix}finger_joint</joint>
-        <mimicJoint>${prefix}left_inner_knuckle_joint</mimicJoint>
-      </plugin>
-      <plugin filename="libgazebo_mimic_joint_plugin.so"
-	      name="${prefix}mimic_right_inner_knuckle_joint">
-        <joint>${prefix}finger_joint</joint>
-        <mimicJoint>${prefix}right_inner_knuckle_joint</mimicJoint>
-      </plugin>
-      <plugin filename="libgazebo_mimic_joint_plugin.so"
-	      name="${prefix}mimic_left_inner_finger_joint">
-        <joint>${prefix}finger_joint</joint>
-        <mimicJoint>${prefix}left_inner_finger_joint</mimicJoint>
-        <multiplier>-1.0</multiplier>
-        <offset>0.0</offset>
-      </plugin>
-      <plugin filename="libgazebo_mimic_joint_plugin.so"
-	      name="${prefix}mimic_right_inner_finger_joint">
-        <joint>${prefix}finger_joint</joint>
-        <mimicJoint>${prefix}right_inner_finger_joint</mimicJoint>
-        <multiplier>-1.0</multiplier>
-        <offset>0.0</offset>
+      <plugin filename="gz_ros2_control-system"
+	      name="gz_ros2_control::GazeboSimROS2ControlPlugin">
+	<parameters>$(find gz_ros2_control_demos)/config/gripper_controller_position.yaml</parameters>
       </plugin>
     </gazebo>
