Commit message: WIP

File: aist_description/devices/urdf/ur_robot_with_ros2_control.urdf.xacro (robot description, xacro)
@@ -2,5 +2,5 @@
 <robot xmlns:xacro="http://wiki.ros.org/xacro">
   <xacro:macro name="ur_robot_with_ros2_control"
-	       params="sim
+	       params="simulation_controllers
 		       ur_type
 		       name
@@ -57,5 +57,5 @@
     </xacro:ur_robot>
     <!-- ros2_control settings for real arms -->
-    <xacro:unless value="$(arg sim)">
+    <xacro:if value="${simulation_controllers == ''}">
       <xacro:include filename="$(find ur_robot_driver
 			       )/urdf/ur.ros2_control.xacro"/>
@@ -90,15 +90,24 @@
 	  non_blocking_read="${non_blocking_read}"
 	  robot_receive_timeout="${robot_receive_timeout}"/>
-    </xacro:unless>
+    </xacro:if>
     <!-- ros2_control settings for gazebo -->
-    <xacro:if value="$(arg sim)">
+    <xacro:unless value="${simulation_controllers == ''}">
       <xacro:include filename="$(find ur_simulation_gz
 			       )/urdf/ur_gz.ros2_control.xacro"/>
-      <xacro:ur_gz_ros2_control
+      <xacro:ur_ros2_control
 	  name="${name}"
 	  tf_prefix="${tf_prefix}"
 	  transmission_hw_interface="${transmission_hw_interface}"
 	  initial_positions="${initial_positions}"/>
-    </xacro:if>
+      <gazebo>
+	<plugin filename="gz_ros2_control-system"
+		name="gz_ros2_control::GazeboSimROS2ControlPlugin">
+	  <parameters>${simulation_controllers}</parameters>
+	  <ros>
+	    <namepsace>${name}</namepsace>
+	  </ros>
+	</plugin>
+      </gazebo>
+    </xacro:unless>
   </xacro:macro>
 </robot>

File: aist_description/objects/urdf/aist_box.urdf.xacro (robot description, xacro)
@@ -34,5 +34,5 @@
       <material>Gazebo/${color_name}</material>
     </gazebo>
-    <joint name="${name}" type="fixed">
+    <joint name="${name}_joint" type="fixed">
       <parent link="${parent}"/>
       <child  link="${name}"/>

File: aist_description/objects/urdf/usb_repeater.urdf.xacro (robot description, xacro)
@@ -42,5 +42,5 @@
 	<material>Gazebo/White</material>
       </gazebo>
-      <joint name="${name}" type="fixed">
+      <joint name="${name}_joint" type="fixed">
 	<parent link="${parent}"/>
 	<child  link="${name}"/>
@@ -49,5 +49,5 @@
     </xacro:macro>
     <link name="${prefix}base_link"/>
-    <joint name="${prefix}base_link" type="fixed">
+    <joint name="${prefix}base_link_joint" type="fixed">
       <parent link="${parent}"/>
       <child  link="${prefix}base_link"/>
@@ -100,5 +100,5 @@
       <material>Gazebo/Black</material>
     </gazebo>
-    <joint name="${prefix}body" type="fixed">
+    <joint name="${prefix}body_joint" type="fixed">
       <parent link="${prefix}plate"/>
       <child  link="${prefix}body"/>

File: aist_description/scenes/urdf/a_bot_base_scene.urdf.xacro (robot description, xacro)
@@ -1,6 +1,6 @@
 <?xml version="1.0"?>
 <robot xmlns:xacro="http://wiki.ros.org/xacro" name="a_bot_base_scene" >
-  <xacro:arg name="scene"	default=""/>
-  <xacro:arg name="sim"		default="false"/>
+  <xacro:arg name="scene"			default=""/>
+  <xacro:arg name="simulation_controllers"	default=""/>
   <!-- ur_robot_driver -->
   <xacro:property name="a_bot_ip"	value="10.66.171.40"/>
@@ -104,5 +104,5 @@
   <xacro:ur_robot_with_ros2_control
       name="a_bot"
-      sim="$(arg sim)"
+      simulation_controllers="$(arg simulation_controllers)"
       ur_type="ur5e"
       tf_prefix="a_bot_"
@@ -150,5 +150,5 @@
     <origin xyz="0.000 -0.051 0.000" rpy="${pi/2} ${-pi/2} 0"/>
   </xacro:usb_repeater>
-  <!-- <!-\- RealSense cameras -\-> -->
+  <!-- RealSense cameras -->
   <xacro:include filename="$(find aist_description
 			   )/devices/urdf/sr305_on_2f140.urdf.xacro" />
@@ -171,3 +171,5 @@
 			     scene).urdf.xacro"/>
   </xacro:if>
+  <gazebo reference="world">
+  </gazebo>
 </robot>

File: aist_description/scenes/urdf/aist_base_scene.urdf.xacro (robot description, xacro)
@@ -1,6 +1,6 @@
 <?xml version="1.0"?>
 <robot xmlns:xacro="http://wiki.ros.org/xacro" name="aist_base_scene" >
-  <xacro:arg name="scene"	default=""/>
-  <xacro:arg name="sim"		default="false"/>
+  <xacro:arg name="scene"			default=""/>
+  <xacro:arg name="simulation_controllers"	default=""/>
   <!-- ur_robot_driver -->
   <xacro:property name="a_bot_ip"	value="10.66.171.40"/>
@@ -114,5 +114,5 @@
 		)/devices/urdf/ur_robot_with_ros2_control.urdf.xacro"/>
   <xacro:ur_robot_with_ros2_control
-      sim="$(arg sim)"
+      simulation_controllers="$(arg simulation_controllers)"
       ur_type="ur5e"
       name="a_bot"
@@ -133,5 +133,5 @@
   </xacro:ur_robot_with_ros2_control>
   <xacro:ur_robot_with_ros2_control
-      sim="$(arg sim)"
+      simulation_controllers="$(arg simulation_controllers)"
       ur_type="ur5e"
       name="b_bot"

File: aist_description/scenes/urdf/b_bot_base_scene.urdf.xacro (robot description, xacro)
@@ -1,6 +1,6 @@
 <?xml version="1.0"?>
 <robot xmlns:xacro="http://wiki.ros.org/xacro" name="b_bot_base_scene" >
-  <xacro:arg name="scene"	default=""/>
-  <xacro:arg name="sim"		default="false"/>
+  <xacro:arg name="scene"			default=""/>
+  <xacro:arg name="simulation_controllers"	default=""/>
   <!-- ur_robot_driver -->
   <xacro:property name="b_bot_ip"	value="10.66.171.41"/>
@@ -99,5 +99,5 @@
   <xacro:ur_robot_with_ros2_control
       name="b_bot"
-      sim="$(arg sim)"
+      simulation_controllers="$(arg simulation_controllers)"
       ur_type="ur5e"
       tf_prefix="b_bot_"
@@ -139,6 +139,6 @@
   <xacro:include filename="$(find aist_description
 			   )/scenes/urdf/load_calibration.urdf.xacro"/>
-  <xacro:load_calibration filename="$(find aist_handeye_calibration
-				    )/calib/a_motioncam.yaml"/>
+  <xacro:load_calibration filename="$(find aist_description
+				    )/scenes/calib/a_motioncam.yaml"/>
   <xacro:include filename="$(find aist_phoxi_camera
 			   )/urdf/motioncam_m_camera.urdf.xacro"/>
@@ -153,7 +153,7 @@
 		       parent="b_bot_gripper_base_link"
 		       use_nominal_extrinsics="true"/>
-  Add live camera
-  <xacro:load_calibration filename="$(find aist_camera_calibration
-				    )/calib/live_camera.yaml"/>
+  <!-- Add live camera -->
+  <xacro:load_calibration filename="$(find aist_description
+				    )/scenes/calib/live_camera.yaml"/>
   <link name="live_camera_optical_frame"/>
   <joint name="live_camera_joint" type="fixed">

File: aist_description/wrc/urdf/kitting_bins.urdf.xacro (robot description, xacro)
@@ -33,5 +33,5 @@
       <material>Gazebo/Orange</material>
     </gazebo>
-    <joint name="${binname}" type="fixed">
+    <joint name="${binname}_joint" type="fixed">
       <parent link="${parent}" />
       <child  link="${binname}" />

File: aist_description/wrc/urdf/kitting_trays.urdf.xacro (robot description, xacro)
@@ -35,5 +35,5 @@
       </collision>
     </link>
-    <joint name="${trayname}" type="fixed">
+    <joint name="${trayname}_joint" type="fixed">
       <parent link="${parent}" />
       <child link = "${trayname}" />
@@ -68,5 +68,5 @@
   <!-- ========== A helper macro for readability in the screw holder definition -->
   <xacro:macro name="auxiliary_frame" params="parent framename *origin">
-    <joint name="${parent}_${framename}" type="fixed">
+    <joint name="${parent}_${framename}_joint" type="fixed">
       <parent link="${parent}" />
       <child link = "${parent}_${framename}"/>

Commit message: WIP

File: aist_description/devices/urdf/ur_robot_with_ros2_control.urdf.xacro (robot description, xacro)
@@ -105,5 +105,5 @@
 	  <parameters>/tmp/${name}_controllers.yaml</parameters>
 	  <ros>
-	    <namepsace>${name}</namepsace>
+	    <namespace>${name}</namespace>
 	    <remapping>robot_description:=/robot_description</remapping>
 	  </ros>

File: aist_description/scenes/urdf/a_bot_base_scene.urdf.xacro (robot description, xacro)
@@ -1,6 +1,6 @@
 <?xml version="1.0"?>
 <robot xmlns:xacro="http://wiki.ros.org/xacro" name="a_bot_base_scene" >
-  <xacro:arg name="scene"			default=""/>
-  <xacro:arg name="simulation_controllers"	default=""/>
+  <xacro:arg name="scene"	default=""/>
+  <xacro:arg name="sim"		default="false"/>
   <!-- ur_robot_driver -->
   <xacro:property name="a_bot_ip"	value="10.66.171.40"/>
@@ -14,4 +14,11 @@
 		  value="$(find ur_robot_driver
 			 )/resources/rtde_input_recipe.txt"/>
+  <xacro:property name="initial_positions"
+		  value="${dict(shoulder_pan_joint=1.5708,
+			        shoulder_lift_joint=-2.1,
+				elbow_joint=1.4,
+				wrist_1_joint=-0.85,
+				wrist_2_joint=-1.5708,
+				wrist_3_joint=0.0)}"/>
   <xacro:arg name="hw_interface"	default="PositionJointInterface"/>
 					<!-- or "VelocityJointInterface" -->
@@ -103,6 +110,6 @@
 		)/devices/urdf/ur_robot_with_ros2_control.urdf.xacro"/>
   <xacro:ur_robot_with_ros2_control
+      sim="$(arg sim)"
       name="a_bot"
-      simulation_controllers="$(arg simulation_controllers)"
       ur_type="ur5e"
       parent="a_bot_table_top_center"
@@ -112,4 +119,5 @@
       input_recipe_filename="${input_recipe_filename}"
       output_recipe_filename="${output_recipe_filename}"
+      initial_positions="${initial_positions}"
       robot_ip="${a_bot_ip}"
       reverse_port="50001"
@@ -182,5 +190,5 @@
   </xacro:if>
   <!-- Import gz plusins -->
-  <xacro:if value="${'$(arg simulation_controllers)' != ''}">
+  <xacro:if value="$(arg sim)">
     <gazebo reference="world">
     </gazebo>
