Commit message: Succesfully connected to a single real robot but two robots

File: aist_description/devices/urdf/ur_robot_ros2_control.urdf.xacro (robot description, xacro)
@@ -1,5 +1,5 @@
 <?xml version="1.0"?>
 <robot xmlns:xacro="http://wiki.ros.org/xacro">
-  <xacro:macro name="ur_robot_with_ros2_control"
+  <xacro:macro name="ur_robot_ros2_control"
 	       params="sim
 		       ur_type

File: aist_description/scenes/urdf/a_bot_base_scene.urdf.xacro (robot description, xacro)
@@ -108,6 +108,6 @@
   <xacro:include
       filename="$(find aist_description
-		)/devices/urdf/ur_robot_with_ros2_control.urdf.xacro"/>
-  <xacro:ur_robot_with_ros2_control
+		)/devices/urdf/ur_robot_ros2_control.urdf.xacro"/>
+  <xacro:ur_robot_ros2_control
       sim="$(arg sim)"
       name="a_bot"
@@ -127,5 +127,5 @@
       trajectory_port="50003">
     <origin xyz="0 0 0 " rpy="0 0 0"/>
-  </xacro:ur_robot_with_ros2_control>
+  </xacro:ur_robot_ros2_control>
   <!-- Set gazebo plugin for FT-sensors -->
   <!-- <xacro:include filename="$(find aist_description -->
@@ -143,11 +143,12 @@
     <origin xyz="0 0 0" rpy="0 ${-pi/2} ${pi/2}"/>
   </xacro:robotiq_arg2f_coupling>
-  <xacro:include filename="$(find aist_robotiq
-			   )/urdf/robotiq_140_gripper.urdf.xacro"/>
-  <xacro:robotiq_140_gripper prefix="a_bot_gripper_"
-			     parent="a_bot_gripper_coupling_flange_link"
-			     short_finger="true">
+  <xacro:include
+      filename="$(find aist_description
+		)/devices/urdf/robotiq_gripper_ros2_control.urdf.xacro"/>
+  <xacro:robotiq_gripper_ros2_control
+      sim="$(arg sim)" type="robotiq_140" name="a_bot_gripper"
+      parent="a_bot_gripper_coupling_flange_link" short_finger="true">
     <origin xyz="0 0 0" rpy="0 0 0"/>
-  </xacro:robotiq_140_gripper>
+  </xacro:robotiq_gripper_ros2_control>
   <!-- Add USB repeater -->
   <xacro:include filename="$(find aist_description
@@ -169,9 +170,9 @@
   </xacro:motioncam_m_camera>
   <!-- RealSense cameras -->
-  <xacro:include filename="$(find aist_description
-			   )/devices/urdf/sr305_on_2f140.urdf.xacro" />
-  <xacro:sr305_on_2f140 prefix="a_bot_"
-			parent="a_bot_gripper_base_link"
-			use_nominal_extrinsics="true"/>
+  <!-- <xacro:include filename="$(find aist_description -->
+  <!-- 			   )/devices/urdf/sr305_on_2f140.urdf.xacro" /> -->
+  <!-- <xacro:sr305_on_2f140 prefix="a_bot_" -->
+  <!-- 			parent="a_bot_gripper_base_link" -->
+  <!-- 			use_nominal_extrinsics="true"/> -->
   <!-- I would like to remove the "world" link definition, but apparently it is necessary for Gazebo -->
   <link name="world"/>

File: aist_description/scenes/urdf/aist_base_scene.urdf.xacro (robot description, xacro)
@@ -119,6 +119,6 @@
   <xacro:include
       filename="$(find aist_description
-		)/devices/urdf/ur_robot_with_ros2_control.urdf.xacro"/>
-  <xacro:ur_robot_with_ros2_control
+		)/devices/urdf/ur_robot_ros2_control.urdf.xacro"/>
+  <xacro:ur_robot_ros2_control
       sim="$(arg sim)"
       name="a_bot"
@@ -138,6 +138,6 @@
       trajectory_port="50003">
     <origin xyz="0 0 0 " rpy="0 0 0"/>
-  </xacro:ur_robot_with_ros2_control>
-  <xacro:ur_robot_with_ros2_control
+  </xacro:ur_robot_ros2_control>
+  <xacro:ur_robot_ros2_control
       sim="$(arg sim)"
       name="b_bot"
@@ -146,7 +146,7 @@
       safety_limits="true"
       safety_pos_margin="0.15"
-      script_filename=""
-      input_recipe_filename=""
-      output_recipe_filename=""
+      script_filename="${script_filename}"
+      input_recipe_filename="${input_recipe_filename}"
+      output_recipe_filename="${output_recipe_filename}"
       initial_positions="${initial_positions}"
       robot_ip="${b_bot_ip}"
@@ -157,5 +157,5 @@
       trajectory_port="50007">
     <origin xyz="0 0 0" rpy="0 0 ${b_bot_theta}"/>
-  </xacro:ur_robot_with_ros2_control>
+  </xacro:ur_robot_ros2_control>
   <!-- Spawn and attach grippers -->
   <xacro:include filename="$(find aist_robotiq
@@ -165,21 +165,20 @@
     <origin xyz="0 0 0" rpy="0 ${-pi/2} ${pi/2}"/>
   </xacro:robotiq_arg2f_coupling>
-  <xacro:include filename="$(find aist_robotiq
-			   )/urdf/robotiq_140_gripper.urdf.xacro"/>
-  <xacro:robotiq_140_gripper prefix="a_bot_gripper_"
-			     parent="a_bot_gripper_coupling_flange_link"
-			     short_finger="true">
+  <xacro:include filename="$(find aist_description
+			   )/devices/urdf/robotiq_gripper_ros2_control.urdf.xacro"/>
+  <xacro:robotiq_gripper_ros2_control
+      sim="$(arg sim)" type="robotiq_140" name="a_bot_gripper"
+      parent="a_bot_gripper_coupling_flange_link" short_finger="true">
     <origin xyz="0 0 0" rpy="0 0 0"/>
-  </xacro:robotiq_140_gripper>
+  </xacro:robotiq_gripper_ros2_control>
   <xacro:robotiq_arg2f_coupling prefix="b_bot_gripper_coupling_"
 				parent="b_bot_tool0">
     <origin xyz="0 0 0" rpy="0 ${-pi/2} ${pi/2}"/>
   </xacro:robotiq_arg2f_coupling>
-  <xacro:include filename="$(find aist_robotiq
-			   )/urdf/robotiq_85_gripper.urdf.xacro"/>
-  <xacro:robotiq_85_gripper prefix="b_bot_gripper_"
-			    parent="b_bot_gripper_coupling_flange_link">
+  <xacro:robotiq_gripper_ros2_control
+      sim="$(arg sim)" type="robotiq_85" name="b_bot_gripper"
+      parent="b_bot_gripper_coupling_flange_link" short_finger="true">
     <origin xyz="0 0 0" rpy="0 0 0"/>
-  </xacro:robotiq_85_gripper>
+  </xacro:robotiq_gripper_ros2_control>
   <!-- Add USB repeaters -->
   <xacro:include filename="$(find aist_description
@@ -252,10 +251,4 @@
     </gazebo>
     <gazebo>
-      <!-- <plugin filename="gz-sim-physics-system" -->
-      <!-- 	      name="gz::sim::systems::Physics"> -->
-      <!-- 	<engine> -->
-      <!-- 	  <filename>libgz-physics-bullet-featherstone-plugin.so</filename> -->
-      <!-- 	</engine> -->
-      <!-- </plugin> -->
       <plugin filename="gz-sim-sensors-system"
 	      name="gz::sim::systems::Sensors">

File: aist_description/scenes/urdf/b_bot_base_scene.urdf.xacro (robot description, xacro)
@@ -14,4 +14,11 @@
 		  value="$(find ur_robot_driver
 			 )/resources/rtde_input_recipe.txt"/>
+  <xacro:property name="initial_positions"
+		  value="${dict(shoulder_pan_joint=1.5708,
+			        shoulder_lift_joint=-2.1,
+				elbow_joint=1.4,
+				wrist_1_joint=-0.85,
+				wrist_2_joint=-1.5708,
+				wrist_3_joint=0.0)}"/>
   <xacro:arg name="hw_interface"	default="PositionJointInterface"/>
 					<!-- or "VelocityJointInterface" -->
@@ -96,15 +103,16 @@
   <xacro:include
       filename="$(find aist_description
-		)/devices/urdf/ur_robot_with_ros2_control.urdf.xacro"/>
-  <xacro:ur_robot_with_ros2_control
+		)/devices/urdf/ur_robot_ros2_control.urdf.xacro"/>
+  <xacro:ur_robot_ros2_control
+      sim="$(arg sim)"
       name="b_bot"
-      simulation_controllers="$(arg simulation_controllers)"
       ur_type="ur5e"
       parent="b_bot_table_top_center"
       safety_limits="true"
       safety_pos_margin="0.15"
-      script_filename=""
-      input_recipe_filename=""
-      output_recipe_filename=""
+      script_filename="${script_filename}"
+      input_recipe_filename="${input_recipe_filename}"
+      output_recipe_filename="${output_recipe_filename}"
+      initial_positions="${initial_positions}"
       robot_ip="${b_bot_ip}"
       reverse_port="50005"
@@ -114,5 +122,5 @@
       trajectory_port="50007">
     <origin xyz="0 0 0" rpy="0 0 ${b_bot_theta}"/>
-  </xacro:ur_robot_with_ros2_control>
+  </xacro:ur_robot_ros2_control>
   <!-- Spawn and attach gripper -->
   <xacro:include filename="$(find aist_robotiq
@@ -122,10 +130,12 @@
     <origin xyz="0 0 0" rpy="0 ${-pi/2} ${pi/2}"/>
   </xacro:robotiq_arg2f_coupling>
-  <xacro:include filename="$(find aist_robotiq
-			   )/urdf/robotiq_85_gripper.urdf.xacro"/>
-  <xacro:robotiq_85_gripper prefix="b_bot_gripper_"
-			    parent="b_bot_gripper_coupling_flange_link">
+  <xacro:include
+      filename="$(find aist_description
+		)/devices/urdf/robotiq_gripper_ros2_control.urdf.xacro"/>
+  <xacro:robotiq_gripper_ros2_control
+      sim="$(arg sim)" type="robotiq_85" name="b_bot_gripper"
+      parent="b_bot_gripper_coupling_flange_link">
     <origin xyz="0 0 0" rpy="0 0 0"/>
-  </xacro:robotiq_85_gripper>
+  </xacro:robotiq_gripper_ros2_control>
   <!-- Add USB repeaters -->
   <xacro:include filename="$(find aist_description

File: aist_robotiq/aist_robotiq/urdf/robotiq_140_gripper.urdf.xacro (robot description, xacro)
@@ -271,53 +271,4 @@
     <xacro:right_outer_knuckle_joint prefix="${prefix}"/>
     <xacro:robotiq_arg2f_transmission prefix="${prefix}"/>
-    <!-- Mimic joints -->
-    <ros2_control name="GazeboSystem" type="system">
-      <hardware>
-	<plugin>gz_ros2_control/GazeboSimSystem</plugin>
-      </hardware>
-      <joint name="${prefix}finger_joint">
-	<command_interface name="position"/>
-	<state_interface name="position">
-          <param name="initial_value">0.15</param>
-	</state_interface>
-	<state_interface name="velocity"/>
-	<state_interface name="effort"/>
-      </joint>
-      <joint name="${prefix}right_outer_knuckle_joint">
-	<state_interface name="position"/>
-	<state_interface name="velocity"/>
-	<state_interface name="effort"/>
-      </joint>
-      <joint name="${prefix}left_inner_knuckle_joint">
-	<state_interface name="position"/>
-	<state_interface name="velocity"/>
-	<state_interface name="effort"/>
-      </joint>
-      <joint name="${prefix}right_inner_knuckle_joint">
-	<state_interface name="position"/>
-	<state_interface name="velocity"/>
-	<state_interface name="effort"/>
-      </joint>
-      <joint name="${prefix}left_inner_finger_joint">
-	<state_interface name="position"/>
-	<state_interface name="velocity"/>
-	<state_interface name="effort"/>
-      </joint>
-      <joint name="${prefix}right_inner_finger_joint">
-	<state_interface name="position"/>
-	<state_interface name="velocity"/>
-	<state_interface name="effort"/>
-      </joint>
-    </ros2_control>
-    <gazebo>
-      <plugin filename="gz_ros2_control-system"
-	      name="gz_ros2_control::GazeboSimROS2ControlPlugin">
-	<parameters>/tmp/${prefix}controllers.yaml</parameters>
-	<ros>
-	  <namespace>${prefix[0:-1]}</namespace>
-	  <remapping>robot_description:=/robot_description</remapping>
-	</ros>
-      </plugin>
-    </gazebo>
   </xacro:macro>
 </robot>

File: aist_robotiq/aist_robotiq/urdf/robotiq_85_gripper.urdf.xacro (robot description, xacro)
@@ -247,53 +247,4 @@
     <xacro:right_outer_knuckle_joint prefix="${prefix}"/>
     <xacro:robotiq_arg2f_transmission prefix="${prefix}"/>
-    <!-- Mimic joints -->
-    <ros2_control name="GazeboSystem" type="system">
-      <hardware>
-	<plugin>gz_ros2_control/GazeboSimSystem</plugin>
-      </hardware>
-      <joint name="${prefix}finger_joint">
-	<command_interface name="position"/>
-	<state_interface name="position">
-          <param name="initial_value">0.15</param>
-	</state_interface>
-	<state_interface name="velocity"/>
-	<state_interface name="effort"/>
-      </joint>
-      <joint name="${prefix}right_outer_knuckle_joint">
-	<state_interface name="position"/>
-	<state_interface name="velocity"/>
-	<state_interface name="effort"/>
-      </joint>
-      <joint name="${prefix}left_inner_knuckle_joint">
-	<state_interface name="position"/>
-	<state_interface name="velocity"/>
-	<state_interface name="effort"/>
-      </joint>
-      <joint name="${prefix}right_inner_knuckle_joint">
-	<state_interface name="position"/>
-	<state_interface name="velocity"/>
-	<state_interface name="effort"/>
-      </joint>
-      <joint name="${prefix}left_inner_finger_joint">
-	<state_interface name="position"/>
-	<state_interface name="velocity"/>
-	<state_interface name="effort"/>
-      </joint>
-      <joint name="${prefix}right_inner_finger_joint">
-	<state_interface name="position"/>
-	<state_interface name="velocity"/>
-	<state_interface name="effort"/>
-      </joint>
-    </ros2_control>
-    <gazebo>
-      <plugin filename="gz_ros2_control-system"
-	      name="gz_ros2_control::GazeboSimROS2ControlPlugin">
-	<parameters>/tmp/${prefix}controllers.yaml</parameters>
-	<ros>
-	  <namespace>${prefix[0:-1]}</namespace>
-	  <remapping>robot_description:=/robot_description</remapping>
-	</ros>
-      </plugin>
-    </gazebo>
   </xacro:macro>
 </robot>

File: aist_robotiq/aist_robotiq/urdf/robotiq_hande_gripper.urdf.xacro (robot description, xacro)
@@ -125,33 +125,4 @@
       <minDepth>0.001</minDepth>
     </gazebo>
-    <!-- Mimic joints -->
-    <ros2_control name="GazeboSystem" type="system">
-      <hardware>
-	<plugin>gz_ros2_control/GazeboSimSystem</plugin>
-      </hardware>
-      <joint name="${prefix}finger_joint">
-	<command_interface name="position"/>
-	<state_interface name="position">
-          <param name="initial_value">0.15</param>
-	</state_interface>
-	<state_interface name="velocity"/>
-	<state_interface name="effort"/>
-      </joint>
-      <joint name="${prefix}right_finger_joint">
-	<state_interface name="position"/>
-	<state_interface name="velocity"/>
-	<state_interface name="effort"/>
-      </joint>
-    </ros2_control>
-    <gazebo>
-      <plugin filename="gz_ros2_control-system"
-	      name="gz_ros2_control::GazeboSimROS2ControlPlugin">
-	<parameters>/tmp/${prefix}controllers.yaml</parameters>
-	<ros>
-	  <namespace>${prefix[0:-1]}</namespace>
-	  <remapping>robot_description:=/robot_description</remapping>
-	</ros>
-      </plugin>
-    </gazebo>
   </xacro:macro>
 </robot>
