Commit message: Confirmed controllers of two arms and two grippers activated succesfully

File: aist_description/devices/urdf/robotiq_gripper.urdf.xacro (robot description, xacro)
@@ -1,5 +1,5 @@
 <?xml version="1.0"?>
 <robot xmlns:xacro="http://wiki.ros.org/xacro">
-  <xacro:macro name="robotiq_gripper_ros2_control"
+  <xacro:macro name="robotiq_gripper"
 	       params="sim type name parent short_finger:=false *origin">
     <xacro:include filename="$(find aist_robotiq
@@ -23,5 +23,5 @@
     <!-- ros2_control settings for gazebo -->
     <xacro:if value="${sim}">
-      <ros2_control name="GazeboSystem" type="system">
+      <ros2_control name="${name}" type="system">
 	<hardware>
           <plugin>gz_ros2_control/GazeboSimSystem</plugin>
@@ -78,14 +78,4 @@
 	</xacro:if>
       </ros2_control>.
-      <gazebo>
-	<plugin filename="gz_ros2_control-system"
-		name="gz_ros2_control::GazeboSimROS2ControlPlugin">
-	  <parameters>/tmp/${name}_controllers.yaml</parameters>
-	  <!-- <ros> -->
-	  <!--   <namespace>${name}</namespace> -->
-	  <!--   <remapping>robot_description:=/robot_description</remapping> -->
-	  <!-- </ros> -->
-	</plugin>
-      </gazebo>
     </xacro:if>
   </xacro:macro>

File: aist_description/devices/urdf/ur_robot.urdf.xacro (robot description, xacro)
@@ -1,5 +1,5 @@
 <?xml version="1.0"?>
 <robot xmlns:xacro="http://wiki.ros.org/xacro">
-  <xacro:macro name="ur_robot_ros2_control"
+  <xacro:macro name="ur_robot"
 	       params="sim
 		       ur_type
@@ -7,4 +7,6 @@
 		       parent
 		       *origin
+		       transmission_hw_interface:=hardware_interface/PositionJointInterface
+		       initial_positions:=${dict(shoulder_pan_joint=0.0,shoulder_lift_joint=-1.57,elbow_joint=0.0,wrist_1_joint=-1.57,wrist_2_joint=0.0,wrist_3_joint=0.0)}
 		       safety_limits:=false
 		       safety_pos_margin:=0.15
@@ -15,9 +17,7 @@
 		       input_recipe_filename
 		       output_recipe_filename
-		       transmission_hw_interface:=hardware_interface/PositionJointInterface
 		       use_mock_hardware:=false
 		       mock_sensor_commands:=false
 		       headless_mode:=false
-		       initial_positions:=${dict(shoulder_pan_joint=0.0,shoulder_lift_joint=-1.57,elbow_joint=0.0,wrist_1_joint=-1.57,wrist_2_joint=0.0,wrist_3_joint=0.0)}
 		       use_tool_communication:=false
 		       tool_voltage:=0
@@ -62,4 +62,6 @@
 	  name="${name}"
 	  tf_prefix="${name}_"
+	  transmission_hw_interface="${transmission_hw_interface}"
+	  initial_positions="${initial_positions}"
 	  kinematics_parameters_file="$(find aist_description
 				      )/scenes/calib/${name}.yaml"
@@ -68,9 +70,7 @@
 	  input_recipe_filename="${input_recipe_filename}"
 	  output_recipe_filename="${output_recipe_filename}"
-	  transmission_hw_interface="${transmission_hw_interface}"
 	  use_mock_hardware="${use_mock_hardware}"
 	  mock_sensor_commands="${mock_sensor_commands}"
 	  headless_mode="${headless_mode}"
-	  initial_positions="${initial_positions}"
 	  use_tool_communication="{use_tool_communications}"
 	  tool_voltage="${tool_voltage}"
@@ -100,14 +100,4 @@
 	  initial_positions="${initial_positions}">
       </xacro:ur_ros2_control>
-      <gazebo>
-	<plugin filename="gz_ros2_control-system"
-		name="gz_ros2_control::GazeboSimROS2ControlPlugin">
-	  <parameters>/tmp/${name}_controllers.yaml</parameters>
-	  <!-- <ros> -->
-	  <!--   <namespace>${name}</namespace> -->
-	  <!--   <remapping>robot_description:=/robot_description</remapping> -->
-	  <!-- </ros> -->
-	</plugin>
-      </gazebo>
     </xacro:if>
   </xacro:macro>

File: aist_description/scenes/urdf/a_bot_base_scene.urdf.xacro (robot description, xacro)
@@ -3,4 +3,7 @@
   <xacro:arg name="scene"	default=""/>
   <xacro:arg name="sim"		default="false"/>
+  <xacro:arg name="transmission_hw_interface"
+	     default="hw_interface/PositionJointInterface"/>
+  <!-- or "hw_intercae/VelocityJointInterface" -->
   <!-- ur_robot_driver -->
   <xacro:property name="a_bot_ip"	value="10.66.171.40"/>
@@ -21,6 +24,4 @@
 				wrist_2_joint=-1.5708,
 				wrist_3_joint=0.0)}"/>
-  <xacro:arg name="hw_interface"	default="PositionJointInterface"/>
-					<!-- or "VelocityJointInterface" -->
   <xacro:property name="a_bot_x"	value="0"/>
   <xacro:property name="a_bot_y"	value="-0.4875"/>
@@ -106,26 +107,25 @@
   </xacro:suction_tool_holder>
   <!-- robot arms -->
-  <xacro:include
-      filename="$(find aist_description
-		)/devices/urdf/ur_robot_ros2_control.urdf.xacro"/>
-  <xacro:ur_robot_ros2_control
-      sim="$(arg sim)"
-      name="a_bot"
-      ur_type="ur5e"
-      parent="a_bot_table_top_center"
-      safety_limits="true"
-      safety_pos_margin="0.15"
-      script_filename="${script_filename}"
-      input_recipe_filename="${input_recipe_filename}"
-      output_recipe_filename="${output_recipe_filename}"
-      initial_positions="${initial_positions}"
-      robot_ip="${a_bot_ip}"
-      reverse_port="50001"
-      script_sender_port="50002"
-      reverse_ip="0.0.0.0"
-      script_command_port="50004"
-      trajectory_port="50003">
+  <xacro:include filename="$(find aist_description
+			   )/devices/urdf/ur_robot.urdf.xacro"/>
+  <xacro:ur_robot sim="$(arg sim)"
+		  name="a_bot"
+		  ur_type="ur5e"
+		  parent="a_bot_table_top_center"
+		  transmission_hw_interface="$(arg transmission_hw_interface)"
+		  initial_positions="${initial_positions}"
+		  safety_limits="true"
+		  safety_pos_margin="0.15"
+		  script_filename="${script_filename}"
+		  input_recipe_filename="${input_recipe_filename}"
+		  output_recipe_filename="${output_recipe_filename}"
+		  robot_ip="${a_bot_ip}"
+		  reverse_port="50001"
+		  script_sender_port="50002"
+		  reverse_ip="0.0.0.0"
+		  script_command_port="50004"
+		  trajectory_port="50003">
     <origin xyz="0 0 0 " rpy="0 0 0"/>
-  </xacro:ur_robot_ros2_control>
+  </xacro:ur_robot>
   <!-- Set gazebo plugin for FT-sensors -->
   <!-- <xacro:include filename="$(find aist_description -->
@@ -143,12 +143,13 @@
     <origin xyz="0 0 0" rpy="0 ${-pi/2} ${pi/2}"/>
   </xacro:robotiq_arg2f_coupling>
-  <xacro:include
-      filename="$(find aist_description
-		)/devices/urdf/robotiq_gripper_ros2_control.urdf.xacro"/>
-  <xacro:robotiq_gripper_ros2_control
-      sim="$(arg sim)" type="robotiq_140" name="a_bot_gripper"
-      parent="a_bot_gripper_coupling_flange_link" short_finger="true">
+  <xacro:include filename="$(find aist_description
+			   )/devices/urdf/robotiq_gripper.urdf.xacro"/>
+  <xacro:robotiq_gripper sim="$(arg sim)"
+			 type="robotiq_140"
+			 name="a_bot_gripper"
+			 parent="a_bot_gripper_coupling_flange_link"
+			 short_finger="true">
     <origin xyz="0 0 0" rpy="0 0 0"/>
-  </xacro:robotiq_gripper_ros2_control>
+  </xacro:robotiq_gripper>
   <!-- Add USB repeater -->
   <xacro:include filename="$(find aist_description
@@ -170,9 +171,9 @@
   </xacro:motioncam_m_camera>
   <!-- RealSense cameras -->
-  <!-- <xacro:include filename="$(find aist_description -->
-  <!-- 			   )/devices/urdf/sr305_on_2f140.urdf.xacro" /> -->
-  <!-- <xacro:sr305_on_2f140 prefix="a_bot_" -->
-  <!-- 			parent="a_bot_gripper_base_link" -->
-  <!-- 			use_nominal_extrinsics="true"/> -->
+  <xacro:include filename="$(find aist_description
+			   )/devices/urdf/sr305_on_2f140.urdf.xacro" />
+  <xacro:sr305_on_2f140 prefix="a_bot_"
+			parent="a_bot_gripper_base_link"
+			use_nominal_extrinsics="true"/>
   <!-- I would like to remove the "world" link definition, but apparently it is necessary for Gazebo -->
   <link name="world"/>
@@ -190,9 +191,16 @@
 			     scene).urdf.xacro"/>
   </xacro:if>
-  <!-- Import gz plusins -->
+  <!-- Import gz plugins -->
   <xacro:if value="$(arg sim)">
     <gazebo reference="world">
     </gazebo>
     <gazebo>
+      <!-- Simulate arms and grippers -->
+      <plugin filename="gz_ros2_control-system"
+	      name="gz_ros2_control::GazeboSimROS2ControlPlugin">
+	<parameters>/tmp/a_bot_controllers.yaml</parameters>
+	<parameters>/tmp/a_bot_gripper_controllers.yaml</parameters>
+      </plugin>
+      <!-- Simulate cameras -->
       <plugin filename="gz-sim-sensors-system"
 	      name="gz::sim::systems::Sensors">

File: aist_description/scenes/urdf/aist_base_scene.urdf.xacro (robot description, xacro)
@@ -3,4 +3,7 @@
   <xacro:arg name="scene"	default=""/>
   <xacro:arg name="sim"		default="false"/>
+  <xacro:arg name="transmission_hw_interface"
+	     default="hw_interface/PositionJointInterface"/>
+  <!-- or "hw_intercae/VelocityJointInterface" -->
   <!-- ur_robot_driver -->
   <xacro:property name="a_bot_ip"	value="10.66.171.40"/>
@@ -117,45 +120,44 @@
   </xacro:suction_tool_holder>
   <!-- robot arms -->
-  <xacro:include
-      filename="$(find aist_description
-		)/devices/urdf/ur_robot_ros2_control.urdf.xacro"/>
-  <xacro:ur_robot_ros2_control
-      sim="$(arg sim)"
-      name="a_bot"
-      ur_type="ur5e"
-      parent="a_bot_table_top_center"
-      safety_limits="true"
-      safety_pos_margin="0.15"
-      script_filename="${script_filename}"
-      input_recipe_filename="${input_recipe_filename}"
-      output_recipe_filename="${output_recipe_filename}"
-      initial_positions="${initial_positions}"
-      robot_ip="${a_bot_ip}"
-      reverse_port="50001"
-      script_sender_port="50002"
-      reverse_ip="0.0.0.0"
-      script_command_port="50004"
-      trajectory_port="50003">
+  <xacro:include filename="$(find aist_description
+			   )/devices/urdf/ur_robot.urdf.xacro"/>
+  <xacro:ur_robot sim="$(arg sim)"
+		  name="a_bot"
+		  ur_type="ur5e"
+		  parent="a_bot_table_top_center"
+		  transmission_hw_interface="$(arg transmission_hw_interface)"
+		  initial_positions="${initial_positions}"
+		  safety_limits="true"
+		  safety_pos_margin="0.15"
+		  script_filename="${script_filename}"
+		  input_recipe_filename="${input_recipe_filename}"
+		  output_recipe_filename="${output_recipe_filename}"
+		  robot_ip="${a_bot_ip}"
+		  reverse_port="50001"
+		  script_sender_port="50002"
+		  reverse_ip="0.0.0.0"
+		  script_command_port="50004"
+		  trajectory_port="50003">
     <origin xyz="0 0 0 " rpy="0 0 0"/>
-  </xacro:ur_robot_ros2_control>
-  <xacro:ur_robot_ros2_control
-      sim="$(arg sim)"
-      name="b_bot"
-      ur_type="ur5e"
-      parent="b_bot_table_top_center"
-      safety_limits="true"
-      safety_pos_margin="0.15"
-      script_filename="${script_filename}"
-      input_recipe_filename="${input_recipe_filename}"
-      output_recipe_filename="${output_recipe_filename}"
-      initial_positions="${initial_positions}"
-      robot_ip="${b_bot_ip}"
-      reverse_port="50005"
-      script_sender_port="50006"
-      reverse_ip="0.0.0.0"
-      script_command_port="50008"
-      trajectory_port="50007">
+  </xacro:ur_robot>
+  <xacro:ur_robot sim="$(arg sim)"
+		  name="b_bot"
+		  ur_type="ur5e"
+		  parent="b_bot_table_top_center"
+		  transmission_hw_interface="$(arg transmission_hw_interface)"
+		  initial_positions="${initial_positions}"
+		  safety_limits="true"
+		  safety_pos_margin="0.15"
+		  script_filename="${script_filename}"
+		  input_recipe_filename="${input_recipe_filename}"
+		  output_recipe_filename="${output_recipe_filename}"
+		  robot_ip="${b_bot_ip}"
+		  reverse_port="50005"
+		  script_sender_port="50006"
+		  reverse_ip="0.0.0.0"
+		  script_command_port="50008"
+		  trajectory_port="50007">
     <origin xyz="0 0 0" rpy="0 0 ${b_bot_theta}"/>
-  </xacro:ur_robot_ros2_control>
+  </xacro:ur_robot>
   <!-- Spawn and attach grippers -->
   <xacro:include filename="$(find aist_robotiq
@@ -166,19 +168,23 @@
   </xacro:robotiq_arg2f_coupling>
   <xacro:include filename="$(find aist_description
-			   )/devices/urdf/robotiq_gripper_ros2_control.urdf.xacro"/>
-  <xacro:robotiq_gripper_ros2_control
-      sim="$(arg sim)" type="robotiq_140" name="a_bot_gripper"
-      parent="a_bot_gripper_coupling_flange_link" short_finger="true">
+			   )/devices/urdf/robotiq_gripper.urdf.xacro"/>
+  <xacro:robotiq_gripper sim="$(arg sim)"
+			 type="robotiq_140"
+			 name="a_bot_gripper"
+			 parent="a_bot_gripper_coupling_flange_link"
+			 short_finger="true">
     <origin xyz="0 0 0" rpy="0 0 0"/>
-  </xacro:robotiq_gripper_ros2_control>
+  </xacro:robotiq_gripper>
   <xacro:robotiq_arg2f_coupling prefix="b_bot_gripper_coupling_"
 				parent="b_bot_tool0">
     <origin xyz="0 0 0" rpy="0 ${-pi/2} ${pi/2}"/>
   </xacro:robotiq_arg2f_coupling>
-  <xacro:robotiq_gripper_ros2_control
-      sim="$(arg sim)" type="robotiq_85" name="b_bot_gripper"
-      parent="b_bot_gripper_coupling_flange_link" short_finger="true">
+  <xacro:robotiq_gripper sim="$(arg sim)"
+			 type="robotiq_85"
+			 name="b_bot_gripper"
+			 parent="b_bot_gripper_coupling_flange_link"
+			 short_finger="true">
     <origin xyz="0 0 0" rpy="0 0 0"/>
-  </xacro:robotiq_gripper_ros2_control>
+  </xacro:robotiq_gripper>
   <!-- Add USB repeaters -->
   <xacro:include filename="$(find aist_description
@@ -207,10 +213,10 @@
 			   )/devices/urdf/sr305_on_2f140.urdf.xacro" />
   <xacro:sr305_on_2f140 prefix="a_bot_"
-			parent="a_bot_gripper_base_link"
+			parent="a_bot_gripper_coupling_flange_link"
 			use_nominal_extrinsics="true"/>
   <xacro:include filename="$(find aist_description
 			   )/devices/urdf/sr305_on_2f85.urdf.xacro" />
   <xacro:sr305_on_2f85 prefix="b_bot_"
-		       parent="b_bot_gripper_base_link"
+		       parent="b_bot_gripper_coupling_flange_link"
 		       use_nominal_extrinsics="true"/>
   <!-- Add live camera -->
@@ -246,13 +252,22 @@
 			     scene).urdf.xacro"/>
   </xacro:if>
-  <!-- Import gz plusins -->
+  <!-- Import gz plugins -->
   <xacro:if value="$(arg sim)">
-    <gazebo reference="world">
-    </gazebo>
+    <!-- <gazebo reference="world"> -->
+    <!-- </gazebo> -->
     <gazebo>
-      <plugin filename="gz-sim-sensors-system"
-	      name="gz::sim::systems::Sensors">
-	<render_engine>ogre2</render_engine>
+      <!-- Simulate arms and grippers -->
+      <plugin filename="gz_ros2_control-system"
+	      name="gz_ros2_control::GazeboSimROS2ControlPlugin">
+	<parameters>/tmp/a_bot_controllers.yaml</parameters>
+	<parameters>/tmp/a_bot_gripper_controllers.yaml</parameters>
+	<parameters>/tmp/b_bot_controllers.yaml</parameters>
+	<parameters>/tmp/b_bot_gripper_controllers.yaml</parameters>
       </plugin>
+      <!-- Simulate cameras -->
+      <!-- <plugin filename="gz-sim-sensors-system" -->
+      <!-- 	      name="gz::sim::systems::Sensors"> -->
+      <!-- 	<render_engine>ogre2</render_engine> -->
+      <!-- </plugin> -->
     </gazebo>
   </xacro:if>

File: aist_description/scenes/urdf/b_bot_base_scene.urdf.xacro (robot description, xacro)
@@ -1,6 +1,9 @@
 <?xml version="1.0"?>
 <robot xmlns:xacro="http://wiki.ros.org/xacro" name="b_bot_base_scene" >
-  <xacro:arg name="scene"			default=""/>
-  <xacro:arg name="simulation_controllers"	default=""/>
+  <xacro:arg name="scene"	default=""/>
+  <xacro:arg name="sim"		default="false"/>
+  <xacro:arg name="transmission_hw_interface"
+	     default="hw_interface/PositionJointInterface"/>
+  <!-- or "hw_intercae/VelocityJointInterface" -->
   <!-- ur_robot_driver -->
   <xacro:property name="b_bot_ip"	value="10.66.171.41"/>
@@ -101,26 +104,25 @@
   </xacro:suction_tool_holder>
   <!-- robot arms -->
-  <xacro:include
-      filename="$(find aist_description
-		)/devices/urdf/ur_robot_ros2_control.urdf.xacro"/>
-  <xacro:ur_robot_ros2_control
-      sim="$(arg sim)"
-      name="b_bot"
-      ur_type="ur5e"
-      parent="b_bot_table_top_center"
-      safety_limits="true"
-      safety_pos_margin="0.15"
-      script_filename="${script_filename}"
-      input_recipe_filename="${input_recipe_filename}"
-      output_recipe_filename="${output_recipe_filename}"
-      initial_positions="${initial_positions}"
-      robot_ip="${b_bot_ip}"
-      reverse_port="50005"
-      script_sender_port="50006"
-      reverse_ip="0.0.0.0"
-      script_command_port="50008"
-      trajectory_port="50007">
+  <xacro:include filename="$(find aist_description
+			   )/devices/urdf/ur_robot.urdf.xacro"/>
+  <xacro:ur_robot sim="$(arg sim)"
+		  name="b_bot"
+		  ur_type="ur5e"
+		  parent="b_bot_table_top_center"
+		  transmission_hw_interface="$(arg transmission_hw_interface)"
+		  initial_positions="${initial_positions}"
+		  safety_limits="true"
+		  safety_pos_margin="0.15"
+		  script_filename="${script_filename}"
+		  input_recipe_filename="${input_recipe_filename}"
+		  output_recipe_filename="${output_recipe_filename}"
+		  robot_ip="${b_bot_ip}"
+		  reverse_port="50005"
+		  script_sender_port="50006"
+		  reverse_ip="0.0.0.0"
+		  script_command_port="50008"
+		  trajectory_port="50007">
     <origin xyz="0 0 0" rpy="0 0 ${b_bot_theta}"/>
-  </xacro:ur_robot_ros2_control>
+  </xacro:ur_robot>
   <!-- Spawn and attach gripper -->
   <xacro:include filename="$(find aist_robotiq
@@ -130,12 +132,12 @@
     <origin xyz="0 0 0" rpy="0 ${-pi/2} ${pi/2}"/>
   </xacro:robotiq_arg2f_coupling>
-  <xacro:include
-      filename="$(find aist_description
-		)/devices/urdf/robotiq_gripper_ros2_control.urdf.xacro"/>
-  <xacro:robotiq_gripper_ros2_control
-      sim="$(arg sim)" type="robotiq_85" name="b_bot_gripper"
-      parent="b_bot_gripper_coupling_flange_link">
+  <xacro:include filename="$(find aist_description
+			   )/devices/urdf/robotiq_gripper.urdf.xacro"/>
+  <xacro:robotiq_gripper sim="$(arg sim)"
+			 type="robotiq_85"
+			 name="b_bot_gripper"
+			 parent="b_bot_gripper_coupling_flange_link">
     <origin xyz="0 0 0" rpy="0 0 0"/>
-  </xacro:robotiq_gripper_ros2_control>
+  </xacro:robotiq_gripper>
   <!-- Add USB repeaters -->
   <xacro:include filename="$(find aist_description
@@ -194,9 +196,16 @@
 			     scene).urdf.xacro"/>
   </xacro:if>
-  <!-- Import gz plusins -->
-  <xacro:if value="${'$(arg simulation_controllers)' != ''}">
+  <!-- Import gz plugins -->
+  <xacro:if value="$(arg sim)">
     <gazebo reference="world">
     </gazebo>
     <gazebo>
+      <!-- Simulate arms and grippers -->
+      <plugin filename="gz_ros2_control-system"
+	      name="gz_ros2_control::GazeboSimROS2ControlPlugin">
+	<parameters>/tmp/b_bot_controllers.yaml</parameters>
+	<parameters>/tmp/b_bot_gripper_controllers.yaml</parameters>
+      </plugin>
+      <!-- Simulate cameras -->
       <plugin filename="gz-sim-sensors-system"
 	      name="gz::sim::systems::Sensors">
