Commit message: Change position of short finger

File: aist_robotiq/urdf/robotiq_140_gripper.urdf.xacro (robot description, xacro)
@@ -174,7 +174,7 @@
     <link name="${prefix}${fingerprefix}_inner_finger_pad">
       <visual>
-        <origin xyz="0 -0.00275 0" rpy="0 0 0"/>
-        <geometry>
-          <box size="0.027 0.0375 0.0075"/>
+        <origin xyz="0 -0.01375 0" rpy="0 0 0"/>
+        <geometry>
+          <box size="0.022 0.0375 0.0075"/>
         </geometry>
         <material name="">
@@ -183,7 +183,7 @@
       </visual>
       <collision>
-        <origin xyz="0 -0.00275 0" rpy="0 0 0"/>
-        <geometry>
-          <box size="0.027 0.0375 0.0075"/>
+        <origin xyz="0 -0.01375 0" rpy="0 0 0"/>
+        <geometry>
+          <box size="0.022 0.0375 0.0075"/>
         </geometry>
         <material name="">
@@ -273,5 +273,5 @@
       <child link="${prefix}tip_link"/>
       <xacro:if value="${short_finger}">
-	<origin rpy="0.0 ${-pi/2} 0.0" xyz=".2168 0.0 0.0"/>
+	<origin rpy="0.0 ${-pi/2} 0.0" xyz=".2053 0.0 0.0"/>
       </xacro:if>
       <xacro:unless value="${short_finger}">
