Commit message: Confirmed both detector_3d and multi_detector work

File: aist_aruco_ros/aist_aruco_ros/urdf/ar_marker.urdf.xacro (robot description, xacro)
@@ -33,5 +33,14 @@
          gazebo_media_path in package.xml. -->
     <gazebo reference="${prefix}ar_marker">
-      <material>Aruco/${marker_name}</material>
+      <material>
+	<pbr>
+	  <diffuse>1.0 1.0 1.0</diffuse>
+	  <specular>1.0 1.0 1.0</specular>
+	  <metal>
+	    <albedo_map>model://aist_aruco_ros/media/materials/textures/${marker_name}.png</albedo_map>
+	    <normal_map>model://aist_aruco_ros/media/materials/textures/${marker_name}.png</normal_map>
+	  </metal>
+	</pbr>
+      </material>
     </gazebo>
   </xacro:macro>
