Commit message: Integrate aist_precision_gripper into aist_fastening_tools

File: aist_fastening_tools/urdf/precision_coupling.urdf.xacro (robot description, xacro)
@@ -10,5 +10,5 @@
         <origin xyz="-0.0045 0 0" rpy="${pi/2} 0 ${pi/2}" />
         <geometry>
-          <mesh filename="package://aist_precision_gripper/meshes/visual/precision_coupling.stl"
+          <mesh filename="package://aist_fastening_tools/meshes/visual/precision_coupling.stl"
 		scale="0.001 0.001 0.001"/>
         </geometry>

File: aist_fastening_tools/urdf/precision_gripper.urdf.xacro (robot description, xacro)
@@ -15,8 +15,8 @@
 		      scope="parent"/>
     </xacro:macro>
-    <xacro:include filename="$(find aist_precision_gripper
-			     )/urdf/precision_transmission.xacro"/>
-    <xacro:precision_transmission prefix="${prefix}"/>
-    <xacro:load_properties filename="$(find aist_precision_gripper
+    <xacro:include filename="$(find aist_fastening_tools
+			     )/urdf/precision_gripper_transmission.xacro"/>
+    <xacro:precision_gripper_transmission prefix="${prefix}"/>
+    <xacro:load_properties filename="$(find aist_fastening_tools
 				     )/config/precision_tool_properties.yaml"/>
     <xacro:property name="max_gap"	value="0.010"/>
@@ -214,6 +214,6 @@
       <minDepth>0.001</minDepth>
     </gazebo>
-    <!-- Mimic joints -->
-    <ros2_control name="GazeboSystem" type="system">
+    <!-- ros2_control settings for gazebo -->
+    <ros2_control name="${prefix[0:-1]}" type="system">
       <hardware>
 	<plugin>gz_ros2_control/GazeboSimSystem</plugin>
@@ -233,10 +233,4 @@
       </joint>
     </ros2_control>
-    <gazebo>
-      <plugin filename="gz_ros2_control-system"
-	      name="gz_ros2_control::GazeboSimROS2ControlPlugin">
-	<parameters>$(find gz_ros2_control_demos)/config/gripper_controller_position.yaml</parameters>
-      </plugin>
-    </gazebo>
   </xacro:macro>
 </robot>

File: aist_fastening_tools/urdf/precision_gripper_transmission.xacro (robot description, xacro)
@@ -1,5 +1,5 @@
 <?xml version="1.0"?>
 <robot xmlns:xacro="http://ros.org/wiki/xacro">
-  <xacro:macro name="precision_transmission" params="prefix">
+  <xacro:macro name="precision_gripper_transmission" params="prefix">
     <transmission name="${prefix}finger_joint_trans">
       <type>transmission_interface/SimpleTransmission</type>
