Commit message: Make URDF of UR robots constructable from YAML config file

File: aist_bringup/urdf/ur.urdf.xacro (robot description, xacro)
@@ -10,20 +10,20 @@
 			   )/urdf/inc/ur_transmissions.xacro" />
   <!-- Load hardware configuration parameters from YAML -->
+  <xacro:property name ="name"
+		  value="$(arg name)"/>
   <xacro:property name ="config_file"
-		  value="$(find aist_bringup
-			 )/config/hardware/$(arg name).yaml"/>
+		  value="$(find aist_bringup)/config/devices/arms.yaml"/>
   <xacro:property name ="config"
-		  value="${xacro.load_yaml(config_file)}"/>
+		  value="${xacro.load_yaml(config_file)[name]}"/>
   <!-- parameters -->
   <xacro:property name ="ur_type"
 		  value="${config.get('ur_type', 'ur5e')}"/>
   <xacro:property name ="tf_prefix"
-		  value="$(arg name)_"/>
+		  value="${name}_"/>
   <xacro:property name="joint_limit_params"
 		  value="$(find ur_description
 			 )/config/${ur_type}/joint_limits.yaml"/>
   <xacro:property name ="kinematics_params"
-		  value="$(find aist_description
-			 )/scenes/calib/$(arg name).yaml"/>
+		  value="$(find aist_description)/scenes/calib/${name}.yaml"/>
   <xacro:property name ="physical_params"
 		  value="$(find ur_description
@@ -38,4 +38,6 @@
   <xacro:property name ="safety_k_position"
 		  value="${str(config.get('safety_k_position', 20))}"/>
+  <xacro:property name ="force_abs_paths"
+		  value="${config.get('force_abs_paths', 'false')}"/>
   <xacro:property name ="transmission_hw_interface"
 		  value="${config.get('transmission_hw_interface',
@@ -106,5 +108,5 @@
   <link name="world" />
   <xacro:ur_robot
-    name="$(arg name)"
+    name="${name}"
     tf_prefix="${tf_prefix}"
     parent="world"
@@ -115,11 +117,10 @@
     safety_limits="${safety_limits}"
     safety_pos_margin="${safety_pos_margin}"
-    safety_k_position="${safety_k_position}"
-    >
-     <origin xyz="0 0 0" rpy="0 0 0" />          <!-- position robot in the world -->
+    safety_k_position="${safety_k_position}">
+    <origin xyz="0 0 0" rpy="0 0 0" />	<!-- position robot in the world -->
   </xacro:ur_robot>
   <!-- ros2 control instance -->
- <xacro:ur_ros2_control
-    name="$(arg name)"
+  <xacro:ur_ros2_control
+    name="${name}"
     tf_prefix="${tf_prefix}"
     kinematics_parameters_file="${kinematics_params}"

File: aist_description/devices/urdf/ur_robot.urdf.xacro (robot description, xacro)
@@ -2,38 +2,50 @@
 <robot xmlns:xacro="http://wiki.ros.org/xacro">
   <xacro:macro name="ur_robot"
-	       params="sim
-		       ur_type
-		       name
-		       parent
-		       *origin
-		       transmission_hw_interface:=hardware_interface/PositionJointInterface
-		       initial_positions:=${dict(shoulder_pan_joint=0.0,shoulder_lift_joint=-1.57,elbow_joint=0.0,wrist_1_joint=-1.57,wrist_2_joint=0.0,wrist_3_joint=0.0)}
-		       safety_limits:=false
-		       safety_pos_margin:=0.15
-		       safety_k_position:=20
-		       force_abs_paths:=false
-		       robot_ip
-		       script_filename
-		       input_recipe_filename
-		       output_recipe_filename
-		       use_mock_hardware:=false
-		       mock_sensor_commands:=false
-		       headless_mode:=false
-		       use_tool_communication:=false
-		       tool_voltage:=0
-		       tool_parity:=0
-		       tool_baud_rate:=115200
-		       tool_stop_bits:=1
-		       tool_rx_idle_chars:=1.5
-		       tool_tx_idle_chars:=3.5
-		       tool_device_name:=/tmp/ttyUR
-		       tool_tcp_port:=54321
-		       reverse_port:=50001
-		       script_sender_port:=50002
-		       reverse_ip:=0.0.0.0
-		       script_command_port:=50004
-		       trajectory_port:=50003
-		       non_blocking_read:=true
-		       robot_receive_timeout:=0.04">
+	       params="sim name parent *origin">
+    <!-- Load hardware configuration parameters from YAML -->
+    <xacro:property name ="config_file"
+		    value="$(find aist_bringup)/config/devices/arms.yaml"/>
+    <xacro:property name ="config"
+		    value="${xacro.load_yaml(config_file)[name]}"/>
+    <!-- parameters -->
+    <xacro:property name ="ur_type"
+		    value="${config.get('ur_type', 'ur5e')}"/>
+    <xacro:property name ="tf_prefix"
+		    value="${name}_"/>
+    <xacro:property name="joint_limit_params"
+		    value="$(find ur_description
+			   )/config/${ur_type}/joint_limits.yaml"/>
+    <xacro:property name ="kinematics_params"
+		    value="$(find aist_description
+			   )/scenes/calib/${name}.yaml"/>
+    <xacro:property name ="physical_params"
+		    value="$(find ur_description
+			   )/config/${ur_type}/physical_parameters.yaml"/>
+    <xacro:property name ="visual_params"
+		    value="$(find ur_description
+			   )/config/${ur_type}/visual_parameters.yaml"/>
+    <xacro:property name ="safety_limits"
+		    value="${config.get('safety_limits', 'false')}"/>
+    <xacro:property name ="safety_pos_margin"
+		    value="${str(config.get('safety_limits', 0.15))}"/>
+    <xacro:property name ="safety_k_position"
+		    value="${str(config.get('safety_k_position', 20))}"/>
+    <xacro:property name ="force_abs_paths"
+		    value="${config.get('force_abs_paths', 'false')}"/>
+    <xacro:property name ="transmission_hw_interface"
+		    value="${config.get('transmission_hw_interface',
+			   'hw_interface/PositionJointInterface')}"/>
+    <!-- initial position for simulations (Mock Hardware, Gazebo, Ignition) -->
+    <xacro:property name ="initial_positions_array"
+		    value="${config.get('initial_positions',
+			   [0.0, 0.0, 0.0, 0.0, 0.0, 0.0])}"/>
+    <xacro:property name ="initial_positions"
+		    value="${dict(
+			   shoulder_pan_joint=initial_positions_array[0],
+			   shoulder_lift_joint=initial_positions_array[1],
+			   elbow_joint=initial_positions_array[2],
+			   wrist_1_joint=initial_positions_array[3],
+			   wrist_2_joint=initial_positions_array[4],
+			   wrist_3_joint=initial_positions_array[5])}"/>
     <xacro:include filename="$(find ur_description)/urdf/ur_macro.xacro"/>
     <xacro:ur_robot
@@ -55,39 +67,4 @@
       <xacro:insert_block name="origin"/>
     </xacro:ur_robot>
-    <!-- ros2_control settings for real arms -->
-    <xacro:unless value="${sim}">
-      <xacro:include filename="$(find ur_robot_driver
-			       )/urdf/ur.ros2_control.xacro"/>
-      <xacro:ur_ros2_control
-	  name="${name}"
-	  tf_prefix="${name}_"
-	  transmission_hw_interface="${transmission_hw_interface}"
-	  initial_positions="${initial_positions}"
-	  kinematics_parameters_file="$(find aist_description
-				      )/scenes/calib/${name}.yaml"
-	  robot_ip="${robot_ip}"
-	  script_filename="${script_filename}"
-	  input_recipe_filename="${input_recipe_filename}"
-	  output_recipe_filename="${output_recipe_filename}"
-	  use_mock_hardware="${use_mock_hardware}"
-	  mock_sensor_commands="${mock_sensor_commands}"
-	  headless_mode="${headless_mode}"
-	  use_tool_communication="{use_tool_communications}"
-	  tool_voltage="${tool_voltage}"
-	  tool_parity="${tool_parity}"
-	  tool_baud_rate="${tool_baud_rate}"
-	  tool_stop_bits="${tool_stop_bits}"
-	  tool_rx_idle_chars="${tool_rx_idle_chars}"
-	  tool_tx_idle_chars="${tool_tx_idle_chars}"
-	  tool_device_name="${tool_device_name}"
-	  tool_tcp_port="${tool_tcp_port}"
-	  reverse_port="${reverse_port}"
-	  script_sender_port="${script_sender_port}"
-	  reverse_ip="${reverse_ip}"
-	  script_command_port="${script_command_port}"
-	  trajectory_port="${trajectory_port}"
-	  non_blocking_read="${non_blocking_read}"
-	  robot_receive_timeout="${robot_receive_timeout}"/>
-    </xacro:unless>
     <!-- ros2_control settings for gazebo -->
     <xacro:if value="${sim}">

File: aist_description/scenes/urdf/a_bot_base_scene.urdf.xacro (robot description, xacro)
@@ -3,25 +3,5 @@
   <xacro:arg name="scene"	default=""/>
   <xacro:arg name="sim"		default="false"/>
-  <xacro:arg name="transmission_hw_interface"
-	     default="hw_interface/PositionJointInterface"/>
-  <!-- or "hw_intercae/VelocityJointInterface" -->
-  <!-- ur_robot_driver -->
-  <xacro:property name="a_bot_ip"	value="10.66.171.40"/>
-  <xacro:property name="script_filename"
-		  value="$(find ur_client_library
-			 )/resources/external_control.urscript"/>
-  <xacro:property name="output_recipe_filename"
-		  value="$(find ur_robot_driver
-			 )/resources/rtde_output_recipe.txt"/>
-  <xacro:property name="input_recipe_filename"
-		  value="$(find ur_robot_driver
-			 )/resources/rtde_input_recipe.txt"/>
-  <xacro:property name="initial_positions"
-		  value="${dict(shoulder_pan_joint=1.5708,
-			        shoulder_lift_joint=-2.1,
-				elbow_joint=1.4,
-				wrist_1_joint=-0.85,
-				wrist_2_joint=-1.5708,
-				wrist_3_joint=0.0)}"/>
+  <!-- location of robot arms -->
   <xacro:property name="a_bot_x"	value="0"/>
   <xacro:property name="a_bot_y"	value="-0.4875"/>
@@ -106,24 +86,10 @@
     <origin xyz="0 ${suction_tool_holder_y} ${cage_t}" rpy="0 0 0"/>
   </xacro:suction_tool_holder>
-  <!-- robot arms -->
+  <!-- Spawn robot arms -->
   <xacro:include filename="$(find aist_description
 			   )/devices/urdf/ur_robot.urdf.xacro"/>
   <xacro:ur_robot sim="$(arg sim)"
 		  name="a_bot"
-		  ur_type="ur5e"
-		  parent="a_bot_table_top_center"
-		  transmission_hw_interface="$(arg transmission_hw_interface)"
-		  initial_positions="${initial_positions}"
-		  safety_limits="true"
-		  safety_pos_margin="0.15"
-		  script_filename="${script_filename}"
-		  input_recipe_filename="${input_recipe_filename}"
-		  output_recipe_filename="${output_recipe_filename}"
-		  robot_ip="${a_bot_ip}"
-		  reverse_port="50001"
-		  script_sender_port="50002"
-		  reverse_ip="0.0.0.0"
-		  script_command_port="50004"
-		  trajectory_port="50003">
+		  parent="a_bot_table_top_center">
     <origin xyz="0 0 0 " rpy="0 0 0"/>
   </xacro:ur_robot>
@@ -201,8 +167,8 @@
 			     scene).urdf.xacro"/>
   </xacro:if>
-  <!-- Import gz plugins -->
+  <!-- Settings for gazebo simulation -->
   <xacro:if value="$(arg sim)">
     <gazebo>
-      <!-- Simulate arms -->
+      <!-- Launch controller managers for arms -->
       <plugin filename="gz_ros2_control-system"
 	      name="gz_ros2_control::GazeboSimROS2ControlPlugin">
@@ -213,5 +179,5 @@
 	</ros>
       </plugin>
-      <!-- Simulate grippers -->
+      <!-- Launch controller manager for grippers -->
       <!-- <plugin filename="gz_ros2_control-system" -->
       <!-- 	      name="gz_ros2_control::GazeboSimROS2ControlPlugin"> -->

File: aist_description/scenes/urdf/aist_base_scene.urdf.xacro (robot description, xacro)
@@ -3,26 +3,4 @@
   <xacro:arg name="scene"	default=""/>
   <xacro:arg name="sim"		default="false"/>
-  <xacro:arg name="transmission_hw_interface"
-	     default="hw_interface/PositionJointInterface"/>
-  <!-- or "hw_intercae/VelocityJointInterface" -->
-  <!-- ur_robot_driver -->
-  <xacro:property name="a_bot_ip"	value="10.66.171.40"/>
-  <xacro:property name="b_bot_ip"	value="10.66.171.41"/>
-  <xacro:property name="script_filename"
-		  value="$(find ur_client_library
-			 )/resources/external_control.urscript"/>
-  <xacro:property name="output_recipe_filename"
-		  value="$(find ur_robot_driver
-			 )/resources/rtde_output_recipe.txt"/>
-  <xacro:property name="input_recipe_filename"
-		  value="$(find ur_robot_driver
-			 )/resources/rtde_input_recipe.txt"/>
-  <xacro:property name="initial_positions"
-		  value="${dict(shoulder_pan_joint=1.5708,
-			        shoulder_lift_joint=-2.1,
-				elbow_joint=1.4,
-				wrist_1_joint=-0.85,
-				wrist_2_joint=-1.5708,
-				wrist_3_joint=0.0)}"/>
   <!-- location of robot arms -->
   <xacro:property name="a_bot_x"	value="0"/>
@@ -124,39 +102,11 @@
   <xacro:ur_robot sim="$(arg sim)"
 		  name="a_bot"
-		  ur_type="ur5e"
-		  parent="a_bot_table_top_center"
-		  transmission_hw_interface="$(arg transmission_hw_interface)"
-		  initial_positions="${initial_positions}"
-		  safety_limits="true"
-		  safety_pos_margin="0.15"
-		  script_filename="${script_filename}"
-		  input_recipe_filename="${input_recipe_filename}"
-		  output_recipe_filename="${output_recipe_filename}"
-		  robot_ip="${a_bot_ip}"
-		  reverse_port="50001"
-		  script_sender_port="50002"
-		  reverse_ip="0.0.0.0"
-		  script_command_port="50004"
-		  trajectory_port="50003">
+		  parent="a_bot_table_top_center">
     <origin xyz="0 0 0 " rpy="0 0 0"/>
   </xacro:ur_robot>
   <xacro:ur_robot sim="$(arg sim)"
 		  name="b_bot"
-		  ur_type="ur5e"
-		  parent="b_bot_table_top_center"
-		  transmission_hw_interface="$(arg transmission_hw_interface)"
-		  initial_positions="${initial_positions}"
-		  safety_limits="true"
-		  safety_pos_margin="0.15"
-		  script_filename="${script_filename}"
-		  input_recipe_filename="${input_recipe_filename}"
-		  output_recipe_filename="${output_recipe_filename}"
-		  robot_ip="${b_bot_ip}"
-		  reverse_port="50005"
-		  script_sender_port="50006"
-		  reverse_ip="0.0.0.0"
-		  script_command_port="50008"
-		  trajectory_port="50007">
-    <origin xyz="0 0 0" rpy="0 0 ${b_bot_theta}"/>
+		  parent="b_bot_table_top_center">
+    <origin xyz="0 0 0 " rpy="0 0 ${b_bot_theta}"/>
   </xacro:ur_robot>
   <!-- Spawn and attach grippers -->
@@ -259,10 +209,8 @@
 			     scene).urdf.xacro"/>
   </xacro:if>
-  <!-- Import gz plugins -->
+  <!-- Settings for gazebo simulation -->
   <xacro:if value="$(arg sim)">
-    <!-- <gazebo reference="world"> -->
-    <!-- </gazebo> -->
     <gazebo>
-      <!-- Simulate arms -->
+      <!-- Launch controller managers for arms -->
       <plugin filename="gz_ros2_control-system"
 	      name="gz_ros2_control::GazeboSimROS2ControlPlugin">
@@ -281,10 +229,10 @@
 	</ros>
       </plugin>
-      <!-- Simulate grippers -->
-      <!-- <plugin filename="gz_ros2_control-system" -->
-      <!-- 	      name="gz_ros2_control::GazeboSimROS2ControlPlugin"> -->
-      <!-- 	<parameters>/tmp/a_bot_gripper_controllers.yaml</parameters> -->
-      <!-- 	<parameters>/tmp/b_bot_gripper_controllers.yaml</parameters> -->
-      <!-- </plugin> -->
+      <!-- Launch controller manager for grippers -->
+      <plugin filename="gz_ros2_control-system"
+	      name="gz_ros2_control::GazeboSimROS2ControlPlugin">
+	<parameters>/tmp/a_bot_gripper_controllers.yaml</parameters>
+	<parameters>/tmp/b_bot_gripper_controllers.yaml</parameters>
+      </plugin>
       <!-- simulate cameras -->
       <!-- <plugin filename="gz-sim-sensors-system" -->

File: aist_description/scenes/urdf/b_bot_base_scene.urdf.xacro (robot description, xacro)
@@ -3,27 +3,5 @@
   <xacro:arg name="scene"	default=""/>
   <xacro:arg name="sim"		default="false"/>
-  <xacro:arg name="transmission_hw_interface"
-	     default="hw_interface/PositionJointInterface"/>
-  <!-- or "hw_intercae/VelocityJointInterface" -->
-  <!-- ur_robot_driver -->
-  <xacro:property name="b_bot_ip"	value="10.66.171.41"/>
-  <xacro:property name="script_filename"
-		  value="$(find ur_client_library
-			 )/resources/external_control.urscript"/>
-  <xacro:property name="output_recipe_filename"
-		  value="$(find ur_robot_driver
-			 )/resources/rtde_output_recipe.txt"/>
-  <xacro:property name="input_recipe_filename"
-		  value="$(find ur_robot_driver
-			 )/resources/rtde_input_recipe.txt"/>
-  <xacro:property name="initial_positions"
-		  value="${dict(shoulder_pan_joint=1.5708,
-			        shoulder_lift_joint=-2.1,
-				elbow_joint=1.4,
-				wrist_1_joint=-0.85,
-				wrist_2_joint=-1.5708,
-				wrist_3_joint=0.0)}"/>
-  <xacro:arg name="hw_interface"	default="PositionJointInterface"/>
-					<!-- or "VelocityJointInterface" -->
+  <!-- location of robot arms -->
   <xacro:property name="b_bot_x"	value="0"/>
   <xacro:property name="b_bot_y"	value="0.4875"/>
@@ -108,19 +86,5 @@
   <xacro:ur_robot sim="$(arg sim)"
 		  name="b_bot"
-		  ur_type="ur5e"
-		  parent="b_bot_table_top_center"
-		  transmission_hw_interface="$(arg transmission_hw_interface)"
-		  initial_positions="${initial_positions}"
-		  safety_limits="true"
-		  safety_pos_margin="0.15"
-		  script_filename="${script_filename}"
-		  input_recipe_filename="${input_recipe_filename}"
-		  output_recipe_filename="${output_recipe_filename}"
-		  robot_ip="${b_bot_ip}"
-		  reverse_port="50005"
-		  script_sender_port="50006"
-		  reverse_ip="0.0.0.0"
-		  script_command_port="50008"
-		  trajectory_port="50007">
+		  parent="b_bot_table_top_center">
     <origin xyz="0 0 0" rpy="0 0 ${b_bot_theta}"/>
   </xacro:ur_robot>
@@ -198,10 +162,8 @@
 			     scene).urdf.xacro"/>
   </xacro:if>
-  <!-- Import gz plugins -->
+  <!-- Settings for gazebo simulation -->
   <xacro:if value="$(arg sim)">
-    <gazebo reference="world">
-    </gazebo>
     <gazebo>
-      <!-- Simulate arms -->
+      <!-- Launch controller managers for arms -->
       <plugin filename="gz_ros2_control-system"
 	      name="gz_ros2_control::GazeboSimROS2ControlPlugin">
@@ -212,5 +174,5 @@
 	</ros>
       </plugin>
-      <!-- Simulate grippers -->
+      <!-- Launch controller manager for grippers -->
       <!-- <plugin filename="gz_ros2_control-system" -->
       <!-- 	      name="gz_ros2_control::GazeboSimROS2ControlPlugin"> -->
