Commit message: Include parent link and arm pose w.r.t it in the configuration YAML file

File: aist_bringup/urdf/ur.urdf.xacro (robot description, xacro)
@@ -3,45 +3,25 @@
   <!-- robot name parameter -->
   <xacro:arg name="name" default="ur"/>
-  <xacro:include filename="$(find ur_description)/urdf/ur_macro.xacro"/>
-  <!-- ros2 control include -->
-  <xacro:include filename="$(find ur_robot_driver
-			   )/urdf/ur.ros2_control.xacro" />
-  <xacro:include filename="$(find ur_description
-			   )/urdf/inc/ur_transmissions.xacro" />
-  <!-- Load hardware configuration parameters from YAML -->
   <xacro:property name ="name"
 		  value="$(arg name)"/>
+  <!-- Load hardware configuration parameters from YAML -->
   <xacro:property name ="config_file"
 		  value="$(find aist_bringup)/config/devices/arms.yaml"/>
   <xacro:property name ="config"
 		  value="${xacro.load_yaml(config_file)[name]}"/>
-  <!-- parameters -->
-  <xacro:property name ="ur_type"
-		  value="${config.get('ur_type', 'ur5e')}"/>
-  <xacro:property name ="tf_prefix"
-		  value="${name}_"/>
-  <xacro:property name="joint_limit_params"
-		  value="$(find ur_description
-			 )/config/${ur_type}/joint_limits.yaml"/>
+  <!-- geometry of the arm -->
+  <xacro:property name ="parent"
+		  value="${config.get('parent', 'world')}"/>
+  <link name="${parent}"/>
+  <xacro:include filename="$(find aist_description
+			   )/devices/urdf/ur_robot.urdf.xacro"/>
+  <xacro:ur_robot sim="false" name="${name}"/>
+  <!-- ros2_control related parameters -->
   <xacro:property name ="kinematics_params"
-		  value="$(find aist_description)/scenes/calib/${name}.yaml"/>
-  <xacro:property name ="physical_params"
-		  value="$(find ur_description
-			 )/config/${ur_type}/physical_parameters.yaml"/>
-  <xacro:property name ="visual_params"
-		  value="$(find ur_description
-			 )/config/${ur_type}/visual_parameters.yaml"/>
-  <xacro:property name ="safety_limits"
-		  value="${config.get('safety_limits', 'false')}"/>
-  <xacro:property name ="safety_pos_margin"
-		  value="${str(config.get('safety_limits', 0.15))}"/>
-  <xacro:property name ="safety_k_position"
-		  value="${str(config.get('safety_k_position', 20))}"/>
-  <xacro:property name ="force_abs_paths"
-		  value="${config.get('force_abs_paths', 'false')}"/>
+		  value="$(find aist_description
+			 )/scenes/calib/${name}.yaml"/>
   <xacro:property name ="transmission_hw_interface"
 		  value="${config.get('transmission_hw_interface',
 			 'hw_interface/PositionJointInterface')}"/>
-  <!-- ros2_control related parameters -->
   <xacro:property name ="headless_mode"
 		  value="${config.get('headless_mode', 'false')}" />
@@ -67,5 +47,5 @@
   <xacro:property name ="trajectory_port"
 		  value="${str(config.get('trajectory_port', 50003))}"/>
-  <!--   tool communication related parameters-->
+  <!-- tool communication related parameters -->
   <xacro:property name ="use_tool_communication"
 		  value="${config.get('use_tool_communication', 'false')}"/>
@@ -86,42 +66,29 @@
   <xacro:property name ="tool_tcp_port"
 		  value="${str(config.get('tool_tcp_port', 54321))}"/>
-  <!-- Simulation parameters -->
+  <!-- simulation parameters -->
   <xacro:property name ="use_mock_hardware"
 		  value="${config.get('use_mock_hardware', 'false')}"/>
   <xacro:property name ="mock_sensor_commands"
 		  value="${config.get('mock_sensor_commands', 'false')}"/>
-  <xacro:property name ="simulation_controllers"
-		  value="${config.get('simulation_controllers', '')}"/>
-  <!-- initial position for simulations (Mock Hardware, Gazebo, Ignition) -->
-  <xacro:property name ="initial_positions_array"
+  <!-- initial positions -->
+  <xacro:property name ="initial_position_coordinates"
 		  value="${config.get('initial_positions',
 			 [0.0, 0.0, 0.0, 0.0, 0.0, 0.0])}"/>
   <xacro:property name ="initial_positions"
 		  value="${dict(
-			 shoulder_pan_joint=initial_positions_array[0],
-			 shoulder_lift_joint=initial_positions_array[1],
-			 elbow_joint=initial_positions_array[2],
-			 wrist_1_joint=initial_positions_array[3],
-			 wrist_2_joint=initial_positions_array[4],
-			 wrist_3_joint=initial_positions_array[5])}"/>
-  <!-- create link fixed to the "world" -->
-  <link name="world" />
-  <xacro:ur_robot
-    name="${name}"
-    tf_prefix="${tf_prefix}"
-    parent="world"
-    joint_limits_parameters_file="${joint_limit_params}"
-    kinematics_parameters_file="${kinematics_params}"
-    physical_parameters_file="${physical_params}"
-    visual_parameters_file="${visual_params}"
-    safety_limits="${safety_limits}"
-    safety_pos_margin="${safety_pos_margin}"
-    safety_k_position="${safety_k_position}">
-    <origin xyz="0 0 0" rpy="0 0 0" />	<!-- position robot in the world -->
-  </xacro:ur_robot>
+			 shoulder_pan_joint=initial_position_coordinates[0],
+			 shoulder_lift_joint=initial_position_coordinates[1],
+			 elbow_joint=initial_position_coordinates[2],
+			 wrist_1_joint=initial_position_coordinates[3],
+			 wrist_2_joint=initial_position_coordinates[4],
+			 wrist_3_joint=initial_position_coordinates[5])}"/>
   <!-- ros2 control instance -->
+  <xacro:include filename="$(find ur_robot_driver
+			   )/urdf/ur.ros2_control.xacro" />
+  <!-- <xacro:include filename="$(find ur_description -->
+  <!-- 			   )/urdf/inc/ur_transmissions.xacro" /> -->
   <xacro:ur_ros2_control
     name="${name}"
-    tf_prefix="${tf_prefix}"
+    tf_prefix="${name}_"
     kinematics_parameters_file="${kinematics_params}"
     transmission_hw_interface="${transmission_hw_interface}"

File: aist_description/devices/urdf/ur_robot.urdf.xacro (robot description, xacro)
@@ -1,6 +1,5 @@
 <?xml version="1.0"?>
 <robot xmlns:xacro="http://wiki.ros.org/xacro">
-  <xacro:macro name="ur_robot"
-	       params="sim name parent *origin">
+  <xacro:macro name="ur_robot" params="sim name">
     <!-- Load hardware configuration parameters from YAML -->
     <xacro:property name ="config_file"
@@ -37,15 +36,21 @@
 			   'hw_interface/PositionJointInterface')}"/>
     <!-- initial position for simulations (Mock Hardware, Gazebo, Ignition) -->
-    <xacro:property name ="initial_positions_array"
+    <xacro:property name ="initial_position_coordinates"
 		    value="${config.get('initial_positions',
 			   [0.0, 0.0, 0.0, 0.0, 0.0, 0.0])}"/>
     <xacro:property name ="initial_positions"
 		    value="${dict(
-			   shoulder_pan_joint=initial_positions_array[0],
-			   shoulder_lift_joint=initial_positions_array[1],
-			   elbow_joint=initial_positions_array[2],
-			   wrist_1_joint=initial_positions_array[3],
-			   wrist_2_joint=initial_positions_array[4],
-			   wrist_3_joint=initial_positions_array[5])}"/>
+			   shoulder_pan_joint=initial_position_coordinates[0],
+			   shoulder_lift_joint=initial_position_coordinates[1],
+			   elbow_joint=initial_position_coordinates[2],
+			   wrist_1_joint=initial_position_coordinates[3],
+			   wrist_2_joint=initial_position_coordinates[4],
+			   wrist_3_joint=initial_position_coordinates[5])}"/>
+    <!-- Pose of robots -->
+    <xacro:property name ="parent"
+		    value="${config.get('parent', 'world')}"/>
+    <xacro:property name ="origin"
+		    value="${config.get('origin',
+			   [0.0, 0.0, 0.0, 0.0, 0.0, 0.0])}"/>
     <xacro:include filename="$(find ur_description)/urdf/ur_macro.xacro"/>
     <xacro:ur_robot
@@ -65,5 +70,8 @@
 	safety_k_position="${safety_k_position}"
 	force_abs_paths="${force_abs_paths}">
-      <xacro:insert_block name="origin"/>
+      <origin xyz="${origin[0]} ${origin[1]} ${origin[2]}"
+	      rpy="${radians(origin[3])}
+		   ${radians(origin[4])}
+		   ${radians(origin[5])}"/>
     </xacro:ur_robot>
     <!-- ros2_control settings for gazebo -->

File: aist_description/scenes/urdf/a_bot_base_scene.urdf.xacro (robot description, xacro)
@@ -89,9 +89,5 @@
   <xacro:include filename="$(find aist_description
 			   )/devices/urdf/ur_robot.urdf.xacro"/>
-  <xacro:ur_robot sim="$(arg sim)"
-		  name="a_bot"
-		  parent="a_bot_table_top_center">
-    <origin xyz="0 0 0 " rpy="0 0 0"/>
-  </xacro:ur_robot>
+  <xacro:ur_robot sim="$(arg sim)" name="a_bot"/>
   <!-- Set gazebo plugin for FT-sensors -->
   <!-- <xacro:include filename="$(find aist_description -->

File: aist_description/scenes/urdf/aist_base_scene.urdf.xacro (robot description, xacro)
@@ -100,14 +100,6 @@
   <xacro:include filename="$(find aist_description
 			   )/devices/urdf/ur_robot.urdf.xacro"/>
-  <xacro:ur_robot sim="$(arg sim)"
-		  name="a_bot"
-		  parent="a_bot_table_top_center">
-    <origin xyz="0 0 0 " rpy="0 0 0"/>
-  </xacro:ur_robot>
-  <xacro:ur_robot sim="$(arg sim)"
-		  name="b_bot"
-		  parent="b_bot_table_top_center">
-    <origin xyz="0 0 0 " rpy="0 0 ${b_bot_theta}"/>
-  </xacro:ur_robot>
+  <xacro:ur_robot sim="$(arg sim)" name="a_bot"/>
+  <xacro:ur_robot sim="$(arg sim)" name="b_bot"/>
   <!-- Spawn and attach grippers -->
   <xacro:include filename="$(find aist_robotiq

File: aist_description/scenes/urdf/b_bot_base_scene.urdf.xacro (robot description, xacro)
@@ -84,9 +84,5 @@
   <xacro:include filename="$(find aist_description
 			   )/devices/urdf/ur_robot.urdf.xacro"/>
-  <xacro:ur_robot sim="$(arg sim)"
-		  name="b_bot"
-		  parent="b_bot_table_top_center">
-    <origin xyz="0 0 0" rpy="0 0 ${b_bot_theta}"/>
-  </xacro:ur_robot>
+  <xacro:ur_robot sim="$(arg sim)" name="b_bot"/>
   <!-- Spawn and attach gripper -->
   <xacro:include filename="$(find aist_robotiq
