Commit message: Confirmed that both arms and grippers work in gazebo simulation

File: aist_bringup/urdf/ur.ros2_control.urdf.xacro (robot description, xacro)
@@ -1,6 +1,6 @@
 <?xml version="1.0"?>
-<robot xmlns:xacro="http://wiki.ros.org/xacro" name="$(arg name)">
+<robot xmlns:xacro="http://wiki.ros.org/xacro" name="ur_ros2_control">
   <!-- robot name parameter -->
-  <xacro:arg name="name" default="ur"/>
+  <xacro:arg name="name" default="a_bot"/>
   <xacro:property name ="name"
 		  value="$(arg name)"/>
@@ -79,6 +79,4 @@
   <xacro:include filename="$(find ur_robot_driver
 			   )/urdf/ur.ros2_control.xacro" />
-  <!-- <xacro:include filename="$(find ur_description -->
-  <!-- 			   )/urdf/inc/ur_transmissions.xacro" /> -->
   <xacro:ur_ros2_control
     name="${name}"

File: aist_description/devices/urdf/ur_robot.urdf.xacro (robot description, xacro)
@@ -1,5 +1,5 @@
 <?xml version="1.0"?>
 <robot xmlns:xacro="http://wiki.ros.org/xacro">
-  <xacro:macro name="ur_robot" params="sim name">
+  <xacro:macro name="ur_robot" params="name parent *origin">
     <!-- Load hardware configuration parameters from YAML -->
     <xacro:property name ="config_file"
@@ -15,7 +15,4 @@
 		    value="$(find ur_description
 			   )/config/${ur_type}/joint_limits.yaml"/>
-    <xacro:property name ="kinematics_params"
-		    value="$(find aist_description
-			   )/scenes/calib/${name}.yaml"/>
     <xacro:property name ="physical_params"
 		    value="$(find ur_description
@@ -24,4 +21,7 @@
 		    value="$(find ur_description
 			   )/config/${ur_type}/visual_parameters.yaml"/>
+    <xacro:property name ="kinematics_params"
+		    value="$(find aist_description
+			   )/scenes/calib/${name}.yaml"/>
     <xacro:property name ="safety_limits"
 		    value="${config.get('safety_limits', 'false')}"/>
@@ -32,25 +32,5 @@
     <xacro:property name ="force_abs_paths"
 		    value="${config.get('force_abs_paths', 'false')}"/>
-    <xacro:property name ="transmission_hw_interface"
-		    value="${config.get('transmission_hw_interface',
-			   'hw_interface/PositionJointInterface')}"/>
-    <!-- initial position for simulations (Mock Hardware, Gazebo, Ignition) -->
-    <xacro:property name ="initial_position_coordinates"
-		    value="${config.get('initial_positions',
-			   [0.0, 0.0, 0.0, 0.0, 0.0, 0.0])}"/>
-    <xacro:property name ="initial_positions"
-		    value="${dict(
-			   shoulder_pan_joint=initial_position_coordinates[0],
-			   shoulder_lift_joint=initial_position_coordinates[1],
-			   elbow_joint=initial_position_coordinates[2],
-			   wrist_1_joint=initial_position_coordinates[3],
-			   wrist_2_joint=initial_position_coordinates[4],
-			   wrist_3_joint=initial_position_coordinates[5])}"/>
-    <!-- Pose of robots -->
-    <xacro:property name ="parent"
-		    value="${config.get('parent', 'world')}"/>
-    <xacro:property name ="origin"
-		    value="${config.get('origin',
-			   [0.0, 0.0, 0.0, 0.0, 0.0, 0.0])}"/>
+    <!-- UR arm -->
     <xacro:include filename="$(find ur_description)/urdf/ur_macro.xacro"/>
     <xacro:ur_robot
@@ -70,20 +50,6 @@
 	safety_k_position="${safety_k_position}"
 	force_abs_paths="${force_abs_paths}">
-      <origin xyz="${origin[0]} ${origin[1]} ${origin[2]}"
-	      rpy="${radians(origin[3])}
-		   ${radians(origin[4])}
-		   ${radians(origin[5])}"/>
+      <xacro:insert_block name="origin"/>
     </xacro:ur_robot>
-    <!-- ros2_control settings for gazebo -->
-    <xacro:if value="${sim}">
-      <xacro:include filename="$(find ur_simulation_gz
-			       )/urdf/ur_gz.ros2_control.xacro"/>
-      <xacro:ur_ros2_control
-	  name="${name}"
-	  tf_prefix="${name}_"
-	  transmission_hw_interface="${transmission_hw_interface}"
-	  initial_positions="${initial_positions}">
-      </xacro:ur_ros2_control>
-    </xacro:if>
   </xacro:macro>
 </robot>

File: aist_description/scenes/urdf/a_bot_base_scene.urdf.xacro (robot description, xacro)
@@ -89,5 +89,7 @@
   <xacro:include filename="$(find aist_description
 			   )/devices/urdf/ur_robot.urdf.xacro"/>
-  <xacro:ur_robot sim="$(arg sim)" name="a_bot"/>
+  <xacro:ur_robot name="a_bot" parent="a_bot_table_top_center">
+    <origin xyz="0 0 0" rpy="0 0 0"/>
+  </xacro:ur_robot>
   <!-- Set gazebo plugin for FT-sensors -->
   <!-- <xacro:include filename="$(find aist_description -->
@@ -172,5 +174,5 @@
 	<ros>
 	  <namespace>a_bot</namespace>
-	  <remapping>robot_description:=/robot_description</remapping>
+	  <!-- <remapping>robot_description:=/robot_description</remapping> -->
 	</ros>
       </plugin>

File: aist_description/scenes/urdf/aist_base_scene.urdf.xacro (robot description, xacro)
@@ -100,6 +100,10 @@
   <xacro:include filename="$(find aist_description
 			   )/devices/urdf/ur_robot.urdf.xacro"/>
-  <xacro:ur_robot sim="$(arg sim)" name="a_bot"/>
-  <xacro:ur_robot sim="$(arg sim)" name="b_bot"/>
+  <xacro:ur_robot name="a_bot" parent="a_bot_table_top_center">
+    <origin xyz="0 0 0" rpy="0 0 0"/>
+  </xacro:ur_robot>
+  <xacro:ur_robot name="b_bot" parent="b_bot_table_top_center">
+    <origin xyz="0 0 0" rpy="0 0 ${b_bot_theta}"/>
+  </xacro:ur_robot>
   <!-- Spawn and attach grippers -->
   <xacro:include filename="$(find aist_robotiq
@@ -210,5 +214,5 @@
 	<ros>
 	  <namespace>a_bot</namespace>
-	  <remapping>robot_description:=/robot_description</remapping>
+	  <!-- <remapping>robot_description:=/robot_description</remapping> -->
 	</ros>
       </plugin>
@@ -218,5 +222,5 @@
 	<ros>
 	  <namespace>b_bot</namespace>
-	  <remapping>robot_description:=/robot_description</remapping>
+	  <!-- <remapping>robot_description:=/robot_description</remapping> -->
 	</ros>
       </plugin>

File: aist_description/scenes/urdf/b_bot_base_scene.urdf.xacro (robot description, xacro)
@@ -84,5 +84,7 @@
   <xacro:include filename="$(find aist_description
 			   )/devices/urdf/ur_robot.urdf.xacro"/>
-  <xacro:ur_robot sim="$(arg sim)" name="b_bot"/>
+  <xacro:ur_robot name="b_bot" parent="b_bot_table_top_center">
+    <origin xyz="0 0 0" rpy="0 0 ${b_bot_theta}"/>
+  </xacro:ur_robot>
   <!-- Spawn and attach gripper -->
   <xacro:include filename="$(find aist_robotiq
@@ -167,5 +169,5 @@
 	<ros>
 	  <namespace>b_bot</namespace>
-	  <remapping>robot_description:=/robot_description</remapping>
+	  <!-- <remapping>robot_description:=/robot_description</remapping> -->
 	</ros>
       </plugin>
