Commit message: WIP

File: aist_bringup/urdf/robotiq.ros2_control.urdf.xacro (robot description, xacro)
@@ -4,5 +4,6 @@
   <xacro:arg name="name" default="a_bot_gripper"/>
   <xacro:arg name="sim"  default="false"/>
-  <xacro:property name ="controller_name" value="$(arg name)_controller"/>
+  <xacro:property name ="controller_name"
+		  value="$(arg name)/gripper_controller"/>
   <!-- Load hardware configuration parameters from YAML -->
   <xacro:property name ="config_file"

File: aist_description/scenes/urdf/a_bot_base_scene.urdf.xacro (robot description, xacro)
@@ -107,9 +107,8 @@
     <origin xyz="0 0 0" rpy="0 ${-pi/2} ${pi/2}"/>
   </xacro:robotiq_arg2f_coupling>
-  <xacro:include filename="$(find aist_description
-			   )/devices/urdf/robotiq_gripper.urdf.xacro"/>
-  <xacro:robotiq_gripper sim="$(arg sim)"
-			 type="robotiq_140"
-			 name="a_bot_gripper"
+  <xacro:include filename="$(find aist_robotiq
+			   )/urdf/robotiq_gripper.urdf.xacro"/>
+  <xacro:robotiq_gripper type="robotiq_140"
+			 prefix="a_bot_gripper_"
 			 parent="a_bot_gripper_coupling_flange_link"
 			 short_finger="true">
@@ -174,12 +173,14 @@
 	<ros>
 	  <namespace>a_bot</namespace>
-	  <!-- <remapping>robot_description:=/robot_description</remapping> -->
 	</ros>
       </plugin>
       <!-- Launch controller manager for grippers -->
-      <!-- <plugin filename="gz_ros2_control-system" -->
-      <!-- 	      name="gz_ros2_control::GazeboSimROS2ControlPlugin"> -->
-      <!-- 	<parameters>/tmp/a_bot_gripper_controllers.yaml</parameters> -->
-      <!-- </plugin> -->
+      <plugin filename="gz_ros2_control-system"
+	      name="gz_ros2_control::GazeboSimROS2ControlPlugin">
+	<parameters>/tmp/a_bot_gripper_controllers.yaml</parameters>
+	<ros>
+	  <namespace>a_bot_gripper</namespace>
+	</ros>
+      </plugin>
       <!-- Simulate cameras -->
       <!-- <plugin filename="gz-sim-sensors-system" -->

File: aist_description/scenes/urdf/aist_base_scene.urdf.xacro (robot description, xacro)
@@ -113,9 +113,8 @@
     <origin xyz="0 0 0" rpy="0 ${-pi/2} ${pi/2}"/>
   </xacro:robotiq_arg2f_coupling>
-  <xacro:include filename="$(find aist_description
-			   )/devices/urdf/robotiq_gripper.urdf.xacro"/>
-  <xacro:robotiq_gripper sim="$(arg sim)"
-			 type="robotiq_140"
-			 name="a_bot_gripper"
+  <xacro:include filename="$(find aist_robotiq
+			   )/urdf/robotiq_gripper.urdf.xacro"/>
+  <xacro:robotiq_gripper type="robotiq_140"
+			 prefix="a_bot_gripper_"
 			 parent="a_bot_gripper_coupling_flange_link"
 			 short_finger="true">
@@ -126,7 +125,6 @@
     <origin xyz="0 0 0" rpy="0 ${-pi/2} ${pi/2}"/>
   </xacro:robotiq_arg2f_coupling>
-  <xacro:robotiq_gripper sim="$(arg sim)"
-			 type="robotiq_85"
-			 name="b_bot_gripper"
+  <xacro:robotiq_gripper type="robotiq_85"
+			 prefix="b_bot_gripper_"
 			 parent="b_bot_gripper_coupling_flange_link"
 			 short_finger="true">
@@ -214,5 +212,4 @@
 	<ros>
 	  <namespace>a_bot</namespace>
-	  <!-- <remapping>robot_description:=/robot_description</remapping> -->
 	</ros>
       </plugin>
@@ -222,5 +219,4 @@
 	<ros>
 	  <namespace>b_bot</namespace>
-	  <!-- <remapping>robot_description:=/robot_description</remapping> -->
 	</ros>
       </plugin>

File: aist_description/scenes/urdf/b_bot_base_scene.urdf.xacro (robot description, xacro)
@@ -94,9 +94,8 @@
     <origin xyz="0 0 0" rpy="0 ${-pi/2} ${pi/2}"/>
   </xacro:robotiq_arg2f_coupling>
-  <xacro:include filename="$(find aist_description
-			   )/devices/urdf/robotiq_gripper.urdf.xacro"/>
-  <xacro:robotiq_gripper sim="$(arg sim)"
-			 type="robotiq_85"
-			 name="b_bot_gripper"
+  <xacro:include filename="$(find aist_robotiq
+			   )/urdf/robotiq_gripper.urdf.xacro"/>
+  <xacro:robotiq_gripper type="robotiq_85"
+			 prefix="b_bot_gripper_"
 			 parent="b_bot_gripper_coupling_flange_link">
     <origin xyz="0 0 0" rpy="0 0 0"/>
@@ -169,12 +168,11 @@
 	<ros>
 	  <namespace>b_bot</namespace>
-	  <!-- <remapping>robot_description:=/robot_description</remapping> -->
 	</ros>
       </plugin>
       <!-- Launch controller manager for grippers -->
-      <!-- <plugin filename="gz_ros2_control-system" -->
-      <!-- 	      name="gz_ros2_control::GazeboSimROS2ControlPlugin"> -->
-      <!-- 	<parameters>/tmp/b_bot_gripper_controllers.yaml</parameters> -->
-      <!-- </plugin> -->
+      <plugin filename="gz_ros2_control-system"
+	      name="gz_ros2_control::GazeboSimROS2ControlPlugin">
+	<parameters>/tmp/b_bot_gripper_controllers.yaml</parameters>
+      </plugin>
       <!-- Simulate cameras -->
       <!-- <plugin filename="gz-sim-sensors-system" -->
