Commit message: Refactor URDF of Robotiq-3F gripper

File: aist_robotiq/aist_robotiq/urdf/robotiq_3f_gripper.urdf (robot description, URDF)
Before this commit: robot robotiq_3f_gripper, 1 links, 0 joints
Links:
- removed link base_link
- added link world

File: aist_robotiq/aist_robotiq/urdf/robotiq_3f_gripper.urdf.xacro (robot description, xacro)
@@ -3,355 +3,150 @@
        xmlns:xacro="http://ros.org/wiki/xacro">
   <xacro:macro name="robotiq_3f_gripper" params="prefix parent *origin">
+    <xacro:property name="tip_height"	value="0.204"/>
+    <xacro:macro name="set_frame" params="name parent *origin">
+      <joint name="${name}_joint" type="fixed">
+	<parent link="${parent}"/>
+	<child  link="${name}"/>
+	<xacro:insert_block name="origin"/>
+      </joint>
+      <link name="${name}"/>
+    </xacro:macro>
+    <xacro:macro name="robotiq_3f_finger" params="prefix fingerprefix">
+      <link name="${prefix}${fingerprefix}link_0">
+	<visual>
+	  <origin rpy="0 0 0" xyz="0.020 0 0"/>
+	  <geometry>
+            <mesh filename="package://aist_robotiq/meshes/visual/robotiq_3f_link_0.dae"/>
+	  </geometry>
+	  <material name="green">
+            <color rgba="0 1 0 1"/>
+	  </material>
+	</visual>
+	<collision>
+	  <origin rpy="0 0 0" xyz="0.020 0 0"/>
+	  <geometry>
+            <mesh filename="package://aist_robotiq/meshes/collision/robotiq_3f_link_0.stl"/>
+	  </geometry>
+	  <material name="yellow">
+            <color rgba="0 1 1 1"/>
+	  </material>
+	</collision>
+	<inertial>
+	  <origin rpy="0 0 0" xyz="0 0 0"/>
+	  <mass value="0.05"/>
+	  <inertia ixx="0.01" ixy="-0.00002" ixz="0.00001"
+		   iyy="0.0008" iyz="0" izz="0.001"/>
+	</inertial>
+      </link>
+      <joint name="${prefix}${fingerprefix}joint" type="revolute">
+	<parent link="${prefix}${fingerprefix}link_0"/>
+	<child link="${prefix}${fingerprefix}link_1"/>
+	<axis xyz="0 0 1"/>
+	<origin xyz="0.020 0 0" rpy="0 0 0"/>
+	<limit effort="100" lower="0" upper="${radians(180)}" velocity="100"/>
+      </joint>
+      <link name="${prefix}${fingerprefix}link_1">
+	<visual>
+	  <origin xyz="0.050 -.028 0" rpy="0 0 -0.52"/>
+	  <geometry>
+            <mesh filename="package://aist_robotiq/meshes/visual/robotiq_3f_link_1.dae"/>
+	  </geometry>
+	  <material name="green"/>
+	</visual>
+	<collision>
+	  <origin xyz="0.050 -.028 0" rpy="0 0 -0.52"/>
+	  <geometry>
+            <mesh filename="package://aist_robotiq/meshes/collision/robotiq_3f_link_1.stl"/>
+	  </geometry>
+	  <material name="yellow"/>
+	</collision>
+	<inertial>
+	  <origin xyz="0 0 0" rpy="0 0 0"/>
+	  <mass value="0.15"/>
+	  <inertia ixx="0.001859" ixy="-0.000376" ixz="0.000028"
+		   iyy="0.012756" iyz="0" izz="0.0024"/>
+	</inertial>
+      </link>
+      <joint name="${prefix}${fingerprefix}joint_2" type="revolute">
+	<parent link="${prefix}${fingerprefix}link_1"/>
+	<child link="${prefix}${fingerprefix}link_2"/>
+	<axis xyz="0 0 1"/>
+	<origin xyz="0.050 -.028 0" rpy="0 0 -0.52"/>
+	<limit effort="100" lower="0" upper="${radians(180)}" velocity="100"/>
+	<mimic joint="${prefix}${fingerprefix}joint"
+	       multiplier="1" offset="0"/>
+      </joint>
+      <link name="${prefix}${fingerprefix}link_2">
+	<!--
+	    NOTE: This link has an offset in the z-direction based on the models that were
+	    used to generate grap-it poses.  With the offset below the model appears visually
+	    correct, but it is suspect.
+	-->
+	<visual>
+	  <origin xyz="0.039 0 0.0075" rpy="0 0 0"/>
+	  <geometry>
+            <mesh filename="package://aist_robotiq/meshes/visual/robotiq_3f_link_2.dae"/>
+	  </geometry>
+	  <material name="green"/>
+	</visual>
+	<collision>
+	  <origin xyz="0.039 0 0.0075" rpy="0 0 0"/>
+	  <geometry>
+            <mesh filename="package://aist_robotiq/meshes/collision/robotiq_3f_link_2.stl"/>
+	  </geometry>
+	  <material name="yellow"/>
+	</collision>
+	<inertial>
+	  <origin xyz="0 0 0" rpy="0 0 0"/>
+	  <mass value="0.15"/>
+	  <inertia ixx="0.001859" ixy="-0.000376" ixz="0.000028"
+		   iyy="0.012756" iyz="0" izz="0.0024"/>
+	</inertial>
+      </link>
+      <joint name="${prefix}${fingerprefix}joint_3" type="revolute">
+	<parent link="${prefix}${fingerprefix}link_2"/>
+	<child link="${prefix}${fingerprefix}link_3"/>
+	<axis xyz="0 0 1"/>
+	<origin xyz="0.039 0 0" rpy="0 0 0"/>
+	<limit effort="100" lower="0" upper="${radians(180)}" velocity="100"/>
+	<mimic joint="${prefix}${fingerprefix}joint"
+	       multiplier="1" offset="0"/>
+      </joint>
+      <link name="${prefix}${fingerprefix}link_3">
+	<visual>
+	  <origin xyz="0 0 0" rpy="0 0 0.52"/>
+	  <geometry>
+            <mesh filename="package://aist_robotiq/meshes/visual/robotiq_3f_link_3.dae"/>
+	  </geometry>
+	  <material name="green"/>
+	</visual>
+	<collision>
+	  <origin xyz="0 0 0" rpy="0 0 0.52"/>
+	  <geometry>
+            <mesh filename="package://aist_robotiq/meshes/collision/robotiq_3f_link_3.stl"/>
+	  </geometry>
+	  <material name="yellow"/>
+	</collision>
+	<inertial>
+	  <origin xyz="0 0 0" rpy="0 0 0"/>
+	  <mass value="0.05"/>
+	  <inertia ixx="0.001239" ixy="-0.000251" ixz="0.000019"
+		   iyy="0.00085" iyz="0" izz="0.001632"/>
+	</inertial>
+      </link>
+    </xacro:macro>
+    <!-- Base -->
+    <link name="${prefix}base_link"/>
     <joint name="${prefix}base_joint" type="fixed">
       <parent link="${parent}"/>
+      <child  link="${prefix}base_link"/>
+      <xacro:insert_block name="origin"/>
+    </joint>
+    <!-- Palm -->
+    <joint name="${prefix}palm_joint" type="fixed">
+      <parent link="${prefix}base_link"/>
       <child  link="${prefix}palm"/>
-      <xacro:insert_block name="origin"/>
-    </joint>
-    <!-- Finger 1-->
-    <link name="${prefix}finger_1_link_0">
-      <visual>
-	<origin rpy="0 0 0" xyz="0.020 0 0"/>
-	<geometry>
-          <mesh filename="package://aist_robotiq/meshes/visual/robotiq_3f_link_0.dae"/>
-	</geometry>
-	<material name="green">
-          <color rgba="0 1 0 1"/>
-	</material>
-      </visual>
-      <collision>
-	<origin rpy="0 3.1416 -1.57" xyz="-0.0455 0.0414 0.036"/>
-	<geometry>
-          <mesh filename="package://aist_robotiq/meshes/collision/robotiq_3f_link_0.stl"/>
-	</geometry>
-	<material name="yellow">
-          <color rgba="0 1 1 1"/>
-	</material>
-      </collision>
-      <inertial>
-	<origin rpy="0 0 0" xyz="0 0 0"/>
-	<mass value="0.05"/>
-	<inertia ixx="0.01" ixy="-0.00002" ixz="0.00001" iyy="0.0008" iyz="0" izz="0.001"/>
-      </inertial>
-    </link>
-    <link name="${prefix}finger_1_link_1">
-      <visual>
-	<origin rpy="0 0 -0.52" xyz="0.050 -.028 0"/>
-	<geometry>
-          <mesh filename="package://aist_robotiq/meshes/visual/robotiq_3f_link_1.dae"/>
-	</geometry>
-	<material name="green"/>
-      </visual>
-      <collision>
-	<origin rpy="0 0 -0.52" xyz="0.050 -.028 0"/>
-	<geometry>
-          <mesh filename="package://aist_robotiq/meshes/collision/robotiq_3f_link_1.stl"/>
-	</geometry>
-	<material name="yellow"/>
-      </collision>
-      <inertial>
-	<origin rpy="0 0 0" xyz="0 0 0"/>
-	<mass value="0.15"/>
-	<inertia ixx="0.001859" ixy="-0.000376" ixz="0.000028" iyy="0.012756" iyz="0" izz="0.0024"/>
-      </inertial>
-    </link>
-    <link name="${prefix}finger_1_link_2">
-      <!--
-	  NOTE: This link has an offset in the z-direction based on the models that were
-	  used to generate grap-it poses.  With the offset below the model appears visually
-	  correct, but it is suspect.
-      -->
-      <visual>
-	<origin rpy="0 0 0" xyz="0.039 0 0.0075"/>
-	<geometry>
-          <mesh filename="package://aist_robotiq/meshes/visual/robotiq_3f_link_2.dae"/>
-	</geometry>
-	<material name="green"/>
-      </visual>
-      <collision>
-	<origin rpy="0 0 0" xyz="0.039 0 0.0075"/>
-	<geometry>
-          <mesh filename="package://aist_robotiq/meshes/collision/robotiq_3f_link_2.stl"/>
-	</geometry>
-	<material name="yellow"/>
-      </collision>
-      <inertial>
-	<origin rpy="0 0 0" xyz="0 0 0"/>
-	<mass value="0.15"/>
-	<inertia ixx="0.001859" ixy="-0.000376" ixz="0.000028" iyy="0.012756" iyz="0" izz="0.0024"/>
-      </inertial>
-    </link>
-    <link name="${prefix}finger_1_link_3">
-      <visual>
-	<origin rpy="0 0 0.52" xyz="0 0 0"/>
-	<geometry>
-          <mesh filename="package://aist_robotiq/meshes/visual/robotiq_3f_link_3.dae"/>
-	</geometry>
-	<material name="green"/>
-      </visual>
-      <collision>
-	<origin rpy="0 0 0.52" xyz="0 0 0"/>
-	<geometry>
-          <mesh filename="package://aist_robotiq/meshes/collision/robotiq_3f_link_3.stl"/>
-	</geometry>
-	<material name="yellow"/>
-      </collision>
-      <inertial>
-	<origin rpy="0 0 0" xyz="0 0 0"/>
-	<mass value="0.05"/>
-	<inertia ixx="0.001239" ixy="-0.000251" ixz="0.000019" iyy="0.00085" iyz="0" izz="0.001632"/>
-      </inertial>
-    </link>
-    <joint name="${prefix}finger_1_joint_1" type="revolute">
-      <parent link="${prefix}finger_1_link_0"/>
-      <child link="${prefix}finger_1_link_1"/>
-      <axis xyz="0 0 1"/>
-      <origin rpy="0 0 0" xyz="0.020 0 0"/>
-      <limit effort="100" lower="0" upper="3.1416" velocity="100"/>
-    </joint>
-    <joint name="${prefix}finger_1_joint_2" type="revolute">
-      <parent link="${prefix}finger_1_link_1"/>
-      <child link="${prefix}finger_1_link_2"/>
-      <axis xyz="0 0 1"/>
-      <origin rpy="0 0 -0.52" xyz="0.050 -.028 0"/>
-      <limit effort="100" lower="0" upper="3.1416" velocity="100"/>
-    </joint>
-    <joint name="${prefix}finger_1_joint_3" type="revolute">
-      <parent link="${prefix}finger_1_link_2"/>
-      <child link="${prefix}finger_1_link_3"/>
-      <axis xyz="0 0 1"/>
-      <origin rpy="0 0 0" xyz="0.039 0 0"/>
-      <limit effort="100" lower="0" upper="3.1416" velocity="100"/>
-    </joint>
-    <!-- Finger 2-->
-    <link name="${prefix}finger_2_link_0">
-      <visual>
-	<origin rpy="0 0 0" xyz="0.020 0 0"/>
-	<geometry>
-          <mesh filename="package://aist_robotiq/meshes/visual/robotiq_3f_link_0.dae"/>
-	</geometry>
-	<material name="green">
-          <color rgba="0 1 0 1"/>
-	</material>
-      </visual>
-      <collision>
-	<origin rpy="0 3.1416 -1.57" xyz="-0.0455 0.0414 0.036"/>
-	<geometry>
-          <mesh filename="package://aist_robotiq/meshes/collision/robotiq_3f_link_0.stl"/>
-	</geometry>
-	<material name="yellow">
-          <color rgba="0 1 1 1"/>
-	</material>
-      </collision>
-      <inertial>
-	<origin rpy="0 0 0" xyz="0 0 0"/>
-	<mass value="0.05"/>
-	<inertia ixx="0.01" ixy="-0.00002" ixz="0.00001" iyy="0.0008" iyz="0" izz="0.001"/>
-      </inertial>
-    </link>
-    <link name="${prefix}finger_2_link_1">
-      <visual>
-	<origin rpy="0 0 -0.52" xyz="0.050 -.028 0"/>
-	<geometry>
-          <mesh filename="package://aist_robotiq/meshes/visual/robotiq_3f_link_1.dae"/>
-	</geometry>
-	<material name="green"/>
-      </visual>
-      <collision>
-	<origin rpy="0 0 -0.52" xyz="0.050 -.028 0"/>
-	<geometry>
-          <mesh filename="package://aist_robotiq/meshes/collision/robotiq_3f_link_1.stl"/>
-	</geometry>
-	<material name="yellow"/>
-      </collision>
-      <inertial>
-	<origin rpy="0 0 0" xyz="0 0 0"/>
-	<mass value="0.15"/>
-	<inertia ixx="0.001859" ixy="-0.000376" ixz="0.000028" iyy="0.012756" iyz="0" izz="0.0024"/>
-      </inertial>
-    </link>
-    <link name="${prefix}finger_2_link_2">
-      <!--
-	  NOTE: This link has an offset in the z-direction based on the models that were
-	  used to generate grap-it poses.  With the offset below the model appears visually
-	  correct, but it is suspect.
-      -->
-      <visual>
-	<origin rpy="0 0 0" xyz="0.039 0 0.0075"/>
-	<geometry>
-          <mesh filename="package://aist_robotiq/meshes/visual/robotiq_3f_link_2.dae"/>
-	</geometry>
-	<material name="green"/>
-      </visual>
-      <collision>
-	<origin rpy="0 0 0" xyz="0.039 0 0.0075"/>
-	<geometry>
-          <mesh filename="package://aist_robotiq/meshes/collision/robotiq_3f_link_2.stl"/>
-	</geometry>
-	<material name="yellow"/>
-      </collision>
-      <inertial>
-	<origin rpy="0 0 0" xyz="0 0 0"/>
-	<mass value="0.15"/>
-	<inertia ixx="0.001859" ixy="-0.000376" ixz="0.000028" iyy="0.012756" iyz="0" izz="0.0024"/>
-      </inertial>
-    </link>
-    <link name="${prefix}finger_2_link_3">
-      <visual>
-	<origin rpy="0 0 0.52" xyz="0 0 0"/>
-	<geometry>
-          <mesh filename="package://aist_robotiq/meshes/visual/robotiq_3f_link_3.dae"/>
-	</geometry>
-	<material name="green"/>
-      </visual>
-      <collision>
-	<origin rpy="0 0 0.52" xyz="0 0 0"/>
-	<geometry>
-          <mesh filename="package://aist_robotiq/meshes/collision/robotiq_3f_link_3.stl"/>
-	</geometry>
-	<material name="yellow"/>
-      </collision>
-      <inertial>
-	<origin rpy="0 0 0" xyz="0 0 0"/>
-	<mass value="0.05"/>
-	<inertia ixx="0.001239" ixy="-0.000251" ixz="0.000019" iyy="0.00085" iyz="0" izz="0.001632"/>
-      </inertial>
-    </link>
-    <joint name="${prefix}finger_2_joint_1" type="revolute">
-      <parent link="${prefix}finger_2_link_0"/>
-      <child link="${prefix}finger_2_link_1"/>
-      <axis xyz="0 0 1"/>
-      <origin rpy="0 0 0" xyz="0.020 0 0"/>
-      <limit effort="100" lower="0" upper="3.1416" velocity="100"/>
-    </joint>
-    <joint name="${prefix}finger_2_joint_2" type="revolute">
-      <parent link="${prefix}finger_2_link_1"/>
-      <child link="${prefix}finger_2_link_2"/>
-      <axis xyz="0 0 1"/>
-      <origin rpy="0 0 -0.52" xyz="0.050 -.028 0"/>
-      <limit effort="100" lower="0" upper="3.1416" velocity="100"/>
-    </joint>
-    <joint name="${prefix}finger_2_joint_3" type="revolute">
-      <parent link="${prefix}finger_2_link_2"/>
-      <child link="${prefix}finger_2_link_3"/>
-      <axis xyz="0 0 1"/>
-      <origin rpy="0 0 0" xyz="0.039 0 0"/>
-      <limit effort="100" lower="0" upper="3.1416" velocity="100"/>
-    </joint>
-    <!-- Finger middle -->
-    <link name="${prefix}finger_middle_link_0">
-      <visual>
-	<origin rpy="0 0 0" xyz="0.020 0 0"/>
-	<geometry>
-          <mesh filename="package://aist_robotiq/meshes/visual/robotiq_3f_link_0.dae"/>
-	</geometry>
-	<material name="green">
-          <color rgba="0 1 0 1"/>
-	</material>
-      </visual>
-      <collision>
-	<origin rpy="0 3.1416 -1.57" xyz="-0.0455 0.0414 0.036"/>
-	<geometry>
-          <mesh filename="package://aist_robotiq/meshes/collision/robotiq_3f_link_0.stl"/>
-	</geometry>
-	<material name="yellow">
-          <color rgba="0 1 1 1"/>
-	</material>
-      </collision>
-      <inertial>
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