Commit message: Add URDF model of Robotiq 3F gripper

File: aist_robotiq/aist_robotiq/urdf/robotiq_3f_gripper.urdf.xacro (robot description, xacro)
@@ -1,48 +1,386 @@
-<!--
-robotiq-3f-gripper_articulated_macro(prefix)
-Creates an articulated robotiq-3f-gripper hand with the passed in prefix.  If there
-is only one hand in the urdf then an empty prefix can be used "".  If
-there are multiple hands then a prefix followed by an "_" is needed.
--->
-<robot xmlns:xacro="http://ros.org/wiki/xacro">
-  <xacro:include filename="$(find aist_robotiq)/urdf/robotiq-3f-gripper_finger_articulated_macro.xacro" />
-  <xacro:macro name="robotiq-3f-gripper_articulated" params="prefix">
-    <xacro:robotiq-3f-gripper_finger_articulated prefix="${prefix}finger_1_"/>
-    <xacro:robotiq-3f-gripper_finger_articulated prefix="${prefix}finger_2_"/>
-    <xacro:robotiq-3f-gripper_finger_articulated prefix="${prefix}finger_middle_"/>
-    <!-- link list -->
+<?xml version="1.0" ?>
+<robot name="robotiq-3f-gripper_articulated"
+       xmlns:xacro="http://ros.org/wiki/xacro">
+  <xacro:macro name="robotiq_3f_gripper" params="prefix parent *origin">
+    <joint name="${prefix}base_joint" type="fixed">
+      <parent link="${parent}"/>
+      <child  link="${prefix}palm"/>
+      <xacro:insert_block name="origin"/>
+    </joint>
+    <!-- Finger 1-->
+    <link name="${prefix}finger_1_link_0">
+      <visual>
+	<origin rpy="0 0 0" xyz="0.020 0 0"/>
+	<geometry>
+          <mesh filename="package://aist_robotiq/meshes/visual/robotiq_3f_link_0.dae"/>
+	</geometry>
+	<material name="green">
+          <color rgba="0 1 0 1"/>
+	</material>
+      </visual>
+      <collision>
+	<origin rpy="0 3.1416 -1.57" xyz="-0.0455 0.0414 0.036"/>
+	<geometry>
+          <mesh filename="package://aist_robotiq/meshes/collision/robotiq_3f_link_0.stl"/>
+	</geometry>
+	<material name="yellow">
+          <color rgba="0 1 1 1"/>
+	</material>
+      </collision>
+      <inertial>
+	<origin rpy="0 0 0" xyz="0 0 0"/>
+	<mass value="0.05"/>
+	<inertia ixx="0.01" ixy="-0.00002" ixz="0.00001" iyy="0.0008" iyz="0" izz="0.001"/>
+      </inertial>
+    </link>
+    <link name="${prefix}finger_1_link_1">
+      <visual>
+	<origin rpy="0 0 -0.52" xyz="0.050 -.028 0"/>
+	<geometry>
+          <mesh filename="package://aist_robotiq/meshes/visual/robotiq_3f_link_1.dae"/>
+	</geometry>
+	<material name="green"/>
+      </visual>
+      <collision>
+	<origin rpy="0 0 -0.52" xyz="0.050 -.028 0"/>
+	<geometry>
+          <mesh filename="package://aist_robotiq/meshes/collision/robotiq_3f_link_1.stl"/>
+	</geometry>
+	<material name="yellow"/>
+      </collision>
+      <inertial>
+	<origin rpy="0 0 0" xyz="0 0 0"/>
+	<mass value="0.15"/>
+	<inertia ixx="0.001859" ixy="-0.000376" ixz="0.000028" iyy="0.012756" iyz="0" izz="0.0024"/>
+      </inertial>
+    </link>
+    <link name="${prefix}finger_1_link_2">
+      <!--
+	  NOTE: This link has an offset in the z-direction based on the models that were
+	  used to generate grap-it poses.  With the offset below the model appears visually
+	  correct, but it is suspect.
+      -->
+      <visual>
+	<origin rpy="0 0 0" xyz="0.039 0 0.0075"/>
+	<geometry>
+          <mesh filename="package://aist_robotiq/meshes/visual/robotiq_3f_link_2.dae"/>
+	</geometry>
+	<material name="green"/>
+      </visual>
+      <collision>
+	<origin rpy="0 0 0" xyz="0.039 0 0.0075"/>
+	<geometry>
+          <mesh filename="package://aist_robotiq/meshes/collision/robotiq_3f_link_2.stl"/>
+	</geometry>
+	<material name="yellow"/>
+      </collision>
+      <inertial>
+	<origin rpy="0 0 0" xyz="0 0 0"/>
+	<mass value="0.15"/>
+	<inertia ixx="0.001859" ixy="-0.000376" ixz="0.000028" iyy="0.012756" iyz="0" izz="0.0024"/>
+      </inertial>
+    </link>
+    <link name="${prefix}finger_1_link_3">
+      <visual>
+	<origin rpy="0 0 0.52" xyz="0 0 0"/>
+	<geometry>
+          <mesh filename="package://aist_robotiq/meshes/visual/robotiq_3f_link_3.dae"/>
+	</geometry>
+	<material name="green"/>
+      </visual>
+      <collision>
+	<origin rpy="0 0 0.52" xyz="0 0 0"/>
+	<geometry>
+          <mesh filename="package://aist_robotiq/meshes/collision/robotiq_3f_link_3.stl"/>
+	</geometry>
+	<material name="yellow"/>
+      </collision>
+      <inertial>
+	<origin rpy="0 0 0" xyz="0 0 0"/>
+	<mass value="0.05"/>
+	<inertia ixx="0.001239" ixy="-0.000251" ixz="0.000019" iyy="0.00085" iyz="0" izz="0.001632"/>
+      </inertial>
+    </link>
+    <joint name="${prefix}finger_1_joint_1" type="revolute">
+      <parent link="${prefix}finger_1_link_0"/>
+      <child link="${prefix}finger_1_link_1"/>
+      <axis xyz="0 0 1"/>
+      <origin rpy="0 0 0" xyz="0.020 0 0"/>
+      <limit effort="100" lower="0" upper="3.1416" velocity="100"/>
+    </joint>
+    <joint name="${prefix}finger_1_joint_2" type="revolute">
+      <parent link="${prefix}finger_1_link_1"/>
+      <child link="${prefix}finger_1_link_2"/>
+      <axis xyz="0 0 1"/>
+      <origin rpy="0 0 -0.52" xyz="0.050 -.028 0"/>
+      <limit effort="100" lower="0" upper="3.1416" velocity="100"/>
+    </joint>
+    <joint name="${prefix}finger_1_joint_3" type="revolute">
+      <parent link="${prefix}finger_1_link_2"/>
+      <child link="${prefix}finger_1_link_3"/>
+      <axis xyz="0 0 1"/>
+      <origin rpy="0 0 0" xyz="0.039 0 0"/>
+      <limit effort="100" lower="0" upper="3.1416" velocity="100"/>
+    </joint>
+    <!-- Finger 2-->
+    <link name="${prefix}finger_2_link_0">
+      <visual>
+	<origin rpy="0 0 0" xyz="0.020 0 0"/>
+	<geometry>
+          <mesh filename="package://aist_robotiq/meshes/visual/robotiq_3f_link_0.dae"/>
+	</geometry>
+	<material name="green">
+          <color rgba="0 1 0 1"/>
+	</material>
+      </visual>
+      <collision>
+	<origin rpy="0 3.1416 -1.57" xyz="-0.0455 0.0414 0.036"/>
+	<geometry>
+          <mesh filename="package://aist_robotiq/meshes/collision/robotiq_3f_link_0.stl"/>
+	</geometry>
+	<material name="yellow">
+          <color rgba="0 1 1 1"/>
+	</material>
+      </collision>
+      <inertial>
+	<origin rpy="0 0 0" xyz="0 0 0"/>
+	<mass value="0.05"/>
+	<inertia ixx="0.01" ixy="-0.00002" ixz="0.00001" iyy="0.0008" iyz="0" izz="0.001"/>
+      </inertial>
+    </link>
+    <link name="${prefix}finger_2_link_1">
+      <visual>
+	<origin rpy="0 0 -0.52" xyz="0.050 -.028 0"/>
+	<geometry>
+          <mesh filename="package://aist_robotiq/meshes/visual/robotiq_3f_link_1.dae"/>
+	</geometry>
+	<material name="green"/>
+      </visual>
+      <collision>
+	<origin rpy="0 0 -0.52" xyz="0.050 -.028 0"/>
+	<geometry>
+          <mesh filename="package://aist_robotiq/meshes/collision/robotiq_3f_link_1.stl"/>
+	</geometry>
+	<material name="yellow"/>
+      </collision>
+      <inertial>
+	<origin rpy="0 0 0" xyz="0 0 0"/>
+	<mass value="0.15"/>
+	<inertia ixx="0.001859" ixy="-0.000376" ixz="0.000028" iyy="0.012756" iyz="0" izz="0.0024"/>
+      </inertial>
+    </link>
+    <link name="${prefix}finger_2_link_2">
+      <!--
+	  NOTE: This link has an offset in the z-direction based on the models that were
+	  used to generate grap-it poses.  With the offset below the model appears visually
+	  correct, but it is suspect.
+      -->
+      <visual>
+	<origin rpy="0 0 0" xyz="0.039 0 0.0075"/>
+	<geometry>
+          <mesh filename="package://aist_robotiq/meshes/visual/robotiq_3f_link_2.dae"/>
+	</geometry>
+	<material name="green"/>
+      </visual>
+      <collision>
+	<origin rpy="0 0 0" xyz="0.039 0 0.0075"/>
+	<geometry>
+          <mesh filename="package://aist_robotiq/meshes/collision/robotiq_3f_link_2.stl"/>
+	</geometry>
+	<material name="yellow"/>
+      </collision>
+      <inertial>
+	<origin rpy="0 0 0" xyz="0 0 0"/>
+	<mass value="0.15"/>
+	<inertia ixx="0.001859" ixy="-0.000376" ixz="0.000028" iyy="0.012756" iyz="0" izz="0.0024"/>
+      </inertial>
+    </link>
+    <link name="${prefix}finger_2_link_3">
+      <visual>
+	<origin rpy="0 0 0.52" xyz="0 0 0"/>
+	<geometry>
+          <mesh filename="package://aist_robotiq/meshes/visual/robotiq_3f_link_3.dae"/>
+	</geometry>
+	<material name="green"/>
+      </visual>
+      <collision>
+	<origin rpy="0 0 0.52" xyz="0 0 0"/>
+	<geometry>
+          <mesh filename="package://aist_robotiq/meshes/collision/robotiq_3f_link_3.stl"/>
+	</geometry>
+	<material name="yellow"/>
+      </collision>
+      <inertial>
+	<origin rpy="0 0 0" xyz="0 0 0"/>
+	<mass value="0.05"/>
+	<inertia ixx="0.001239" ixy="-0.000251" ixz="0.000019" iyy="0.00085" iyz="0" izz="0.001632"/>
+      </inertial>
+    </link>
+    <joint name="${prefix}finger_2_joint_1" type="revolute">
+      <parent link="${prefix}finger_2_link_0"/>
+      <child link="${prefix}finger_2_link_1"/>
+      <axis xyz="0 0 1"/>
+      <origin rpy="0 0 0" xyz="0.020 0 0"/>
+      <limit effort="100" lower="0" upper="3.1416" velocity="100"/>
+    </joint>
+    <joint name="${prefix}finger_2_joint_2" type="revolute">
+      <parent link="${prefix}finger_2_link_1"/>
+      <child link="${prefix}finger_2_link_2"/>
+      <axis xyz="0 0 1"/>
+      <origin rpy="0 0 -0.52" xyz="0.050 -.028 0"/>
+      <limit effort="100" lower="0" upper="3.1416" velocity="100"/>
+    </joint>
+    <joint name="${prefix}finger_2_joint_3" type="revolute">
+      <parent link="${prefix}finger_2_link_2"/>
+      <child link="${prefix}finger_2_link_3"/>
+      <axis xyz="0 0 1"/>
+      <origin rpy="0 0 0" xyz="0.039 0 0"/>
+      <limit effort="100" lower="0" upper="3.1416" velocity="100"/>
+    </joint>
+    <!-- Finger middle -->
+    <link name="${prefix}finger_middle_link_0">
+      <visual>
+	<origin rpy="0 0 0" xyz="0.020 0 0"/>
+	<geometry>
+          <mesh filename="package://aist_robotiq/meshes/visual/robotiq_3f_link_0.dae"/>
+	</geometry>
+	<material name="green">
+          <color rgba="0 1 0 1"/>
+	</material>
+      </visual>
+      <collision>
+	<origin rpy="0 3.1416 -1.57" xyz="-0.0455 0.0414 0.036"/>
+	<geometry>
+          <mesh filename="package://aist_robotiq/meshes/collision/robotiq_3f_link_0.stl"/>
+	</geometry>
+	<material name="yellow">
+          <color rgba="0 1 1 1"/>
+	</material>
+      </collision>
+      <inertial>
+	<origin rpy="0 0 0" xyz="0 0 0"/>
+	<mass value="0.05"/>
+	<inertia ixx="0.01" ixy="-0.00002" ixz="0.00001" iyy="0.0008" iyz="0" izz="0.001"/>
+      </inertial>
+    </link>
+    <link name="${prefix}finger_middle_link_1">
+      <visual>
+	<origin rpy="0 0 -0.52" xyz="0.050 -.028 0"/>
+	<geometry>
+          <mesh filename="package://aist_robotiq/meshes/visual/robotiq_3f_link_1.dae"/>
+	</geometry>
+	<material name="green"/>
+      </visual>
+      <collision>
+	<origin rpy="0 0 -0.52" xyz="0.050 -.028 0"/>
+	<geometry>
+          <mesh filename="package://aist_robotiq/meshes/collision/robotiq_3f_link_1.stl"/>
+	</geometry>
+	<material name="yellow"/>
+      </collision>
+      <inertial>
+	<origin rpy="0 0 0" xyz="0 0 0"/>
+	<mass value="0.15"/>
+	<inertia ixx="0.001859" ixy="-0.000376" ixz="0.000028" iyy="0.012756" iyz="0" izz="0.0024"/>
+      </inertial>
+    </link>
+    <link name="${prefix}finger_middle_link_2">
+      <!--
+	  NOTE: This link has an offset in the z-direction based on the models that were
+	  used to generate grap-it poses.  With the offset below the model appears visually
+	  correct, but it is suspect.
+      -->
+      <visual>
+	<origin rpy="0 0 0" xyz="0.039 0 0.0075"/>
+	<geometry>
+          <mesh filename="package://aist_robotiq/meshes/visual/robotiq_3f_link_2.dae"/>
+	</geometry>
+	<material name="green"/>
+      </visual>
+      <collision>
+	<origin rpy="0 0 0" xyz="0.039 0 0.0075"/>
+	<geometry>
+          <mesh filename="package://aist_robotiq/meshes/collision/robotiq_3f_link_2.stl"/>
+	</geometry>
+	<material name="yellow"/>
+      </collision>
+      <inertial>
+	<origin rpy="0 0 0" xyz="0 0 0"/>
+	<mass value="0.15"/>
+	<inertia ixx="0.001859" ixy="-0.000376" ixz="0.000028" iyy="0.012756" iyz="0" izz="0.0024"/>
+      </inertial>
+    </link>
+    <link name="${prefix}finger_middle_link_3">
+      <visual>
+	<origin rpy="0 0 0.52" xyz="0 0 0"/>
+	<geometry>
+          <mesh filename="package://aist_robotiq/meshes/visual/robotiq_3f_link_3.dae"/>
+	</geometry>
+	<material name="green"/>
+      </visual>
+      <collision>
+	<origin rpy="0 0 0.52" xyz="0 0 0"/>
+	<geometry>
+          <mesh filename="package://aist_robotiq/meshes/collision/robotiq_3f_link_3.stl"/>
+	</geometry>
+	<material name="yellow"/>
+      </collision>
+      <inertial>
+	<origin rpy="0 0 0" xyz="0 0 0"/>
+	<mass value="0.05"/>
+	<inertia ixx="0.001239" ixy="-0.000251" ixz="0.000019" iyy="0.00085" iyz="0" izz="0.001632"/>
+      </inertial>
+    </link>
+    <joint name="${prefix}finger_middle_joint_1" type="revolute">
+      <parent link="${prefix}finger_middle_link_0"/>
+      <child link="${prefix}finger_middle_link_1"/>
+      <axis xyz="0 0 1"/>
+      <origin rpy="0 0 0" xyz="0.020 0 0"/>
+      <limit effort="100" lower="0" upper="3.1416" velocity="100"/>
+    </joint>
+    <joint name="${prefix}finger_middle_joint_2" type="revolute">
+      <parent link="${prefix}finger_middle_link_1"/>
+      <child link="${prefix}finger_middle_link_2"/>
+      <axis xyz="0 0 1"/>
+      <origin rpy="0 0 -0.52" xyz="0.050 -.028 0"/>
+      <limit effort="100" lower="0" upper="3.1416" velocity="100"/>
+    </joint>
+    <joint name="${prefix}finger_middle_joint_3" type="revolute">
+      <parent link="${prefix}finger_middle_link_2"/>
+      <child link="${prefix}finger_middle_link_3"/>
+      <axis xyz="0 0 1"/>
+      <origin rpy="0 0 0" xyz="0.039 0 0"/>
+      <limit effort="100" lower="0" upper="3.1416" velocity="100"/>
+    </joint>
+    <!-- Palm -->
     <link name="${prefix}palm">
       <visual>
 	<geometry>
-          <mesh filename="package://aist_robotiq/meshes/robotiq-3f-gripper_articulated/visual/palm.dae" />
-	</geometry>
-	<material name="gray">
-	  <color rgba="0.2 0.2 0.2 1"/>
-	</material>
-      </visual>
-      <collision>
-	<geometry>
-          <mesh
-	      filename="package://aist_robotiq/meshes/robotiq-3f-gripper_articulated/collision/palm.stl" />
+          <mesh filename="package://aist_robotiq/meshes/visual/robotiq_3f_palm.dae"/>
+	</geometry>
+	<material name="green">
+          <color rgba="0 1 0 1"/>
+	</material>
+      </visual>
+      <collision>
+	<geometry>
+          <mesh filename="package://aist_robotiq/meshes/collision/robotiq_3f_palm.stl"/>
 	</geometry>
 	<material name="yellow">
-	  <color rgba="0 1 1 1"/>
-	</material>
-      </collision>
-    </link>
-    <link name="${prefix}tool0"/>
+          <color rgba="0 1 1 1"/>
+	</material>
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
Commit message: Confirmed that robotiq_3f works with ModbusTCP driver

File: aist_robotiq/aist_robotiq/urdf/robotiq_3f_gripper.urdf.xacro (robot description, xacro)
@@ -12,6 +12,6 @@
       <link name="${name}"/>
     </xacro:macro>
-    <xacro:macro name="robotiq_3f_finger" params="prefix fingerprefix">
-      <link name="${prefix}${fingerprefix}link_0">
+    <xacro:macro name="robotiq_3f_finger" params="fingerprefix">
+      <link name="${fingerprefix}link_0">
 	<visual>
 	  <origin rpy="0 0 0" xyz="0.020 0 0"/>
@@ -39,12 +39,12 @@
 	</inertial>
       </link>
-      <joint name="${prefix}${fingerprefix}joint" type="revolute">
-	<parent link="${prefix}${fingerprefix}link_0"/>
-	<child link="${prefix}${fingerprefix}link_1"/>
+      <joint name="${fingerprefix}joint" type="revolute">
+	<parent link="${fingerprefix}link_0"/>
+	<child link="${fingerprefix}link_1"/>
 	<axis xyz="0 0 1"/>
 	<origin xyz="0.020 0 0" rpy="0 0 0"/>
 	<limit effort="100" lower="0" upper="${radians(180)}" velocity="100"/>
       </joint>
-      <link name="${prefix}${fingerprefix}link_1">
+      <link name="${fingerprefix}link_1">
 	<visual>
 	  <origin xyz="0.050 -.028 0" rpy="0 0 -0.52"/>
@@ -68,14 +68,14 @@
 	</inertial>
       </link>
-      <joint name="${prefix}${fingerprefix}joint_2" type="revolute">
-	<parent link="${prefix}${fingerprefix}link_1"/>
-	<child link="${prefix}${fingerprefix}link_2"/>
+      <joint name="${fingerprefix}joint_2" type="revolute">
+	<parent link="${fingerprefix}link_1"/>
+	<child link="${fingerprefix}link_2"/>
 	<axis xyz="0 0 1"/>
 	<origin xyz="0.050 -.028 0" rpy="0 0 -0.52"/>
 	<limit effort="100" lower="0" upper="${radians(180)}" velocity="100"/>
-	<mimic joint="${prefix}${fingerprefix}joint"
+	<mimic joint="${fingerprefix}joint"
 	       multiplier="1" offset="0"/>
       </joint>
-      <link name="${prefix}${fingerprefix}link_2">
+      <link name="${fingerprefix}link_2">
 	<!--
 	    NOTE: This link has an offset in the z-direction based on the models that were
@@ -104,14 +104,14 @@
 	</inertial>
       </link>
-      <joint name="${prefix}${fingerprefix}joint_3" type="revolute">
-	<parent link="${prefix}${fingerprefix}link_2"/>
-	<child link="${prefix}${fingerprefix}link_3"/>
+      <joint name="${fingerprefix}joint_3" type="revolute">
+	<parent link="${fingerprefix}link_2"/>
+	<child link="${fingerprefix}link_3"/>
 	<axis xyz="0 0 1"/>
 	<origin xyz="0.039 0 0" rpy="0 0 0"/>
 	<limit effort="100" lower="0" upper="${radians(180)}" velocity="100"/>
-	<mimic joint="${prefix}${fingerprefix}joint"
+	<mimic joint="${fingerprefix}joint"
 	       multiplier="1" offset="0"/>
       </joint>
-      <link name="${prefix}${fingerprefix}link_3">
+      <link name="${fingerprefix}link_3">
 	<visual>
 	  <origin xyz="0 0 0" rpy="0 0 0.52"/>
@@ -187,5 +187,5 @@
       <limit effort="100" lower="-0.16" upper="0.25" velocity="100"/>
     </joint>
-    <xacro:robotiq_3f_finger prefix="${prefix}" fingerprefix="finger_1_"/>
+    <xacro:robotiq_3f_finger fingerprefix="${prefix}finger_1_"/>
     <!-- Finger 2 -->
     <joint name="${prefix}palm_finger_2_joint" type="revolute">
@@ -198,5 +198,5 @@
       <mimic joint="${prefix}scissor_joint" multiplier="-1" offset="0"/>
     </joint>
-    <xacro:robotiq_3f_finger prefix="${prefix}" fingerprefix="finger_2_"/>
+    <xacro:robotiq_3f_finger fingerprefix="${prefix}finger_2_"/>
     <!-- Finger middle -->
     <joint name="${prefix}palm_finger_middle_joint" type="fixed">
@@ -206,5 +206,5 @@
       <origin xyz="0.0455 0.0214 0" rpy="0 0 ${radians(90)}"/>
     </joint>
-    <xacro:robotiq_3f_finger prefix="${prefix}" fingerprefix="finger_middle_"/>
+    <xacro:robotiq_3f_finger fingerprefix="${prefix}finger_middle_"/>
     <!--
         <include filename="$(find aist_robotiq)/cfg/robotiq-3f-gripper_finger_articulated_macro.xacro" />
